File: kicad_osm_env01/OSM_env01.sch (KiCad schematic (older format))
At the start: 172 parts, among them J1 USB_B_Micro, J2 Conn_01x08, J3 Conn_01x08, Q1 SI2301BDS-T1-E3, Q4 IRF7319TRPBF, Q6 FK3503010L, Q7 SSM3J328R, SW1 SW_SPST, SW2 SW_SPST, SW3 SW_Push, U1 MCP73833(MSOP10), U10 NL3S22S_DPDT_anlogue_switch, U2 NCP1117-3.3_SOT223, U3 ESP-WROOM-32, U4 ISL83485, U6 ERIC-LORA, U7 TSL2561, U8 M74VHC1GT14DFT2G, U9 MIC2288YD5-TR

Commit message: audio circuit updated
Parts:
- removed R25: 10K, Resistor_SMD:R_0603_1608Metric, symbol OSM_env01-rescue:R-device-ESP32-EVB_Rev_D-rescue
- removed TP20, TP21, TP23, TP24: Test_Point, TestPoint:TestPoint_THTPad_D1.0mm_Drill0.5mm, symbol OSM_env01-rescue:Test_Point-Connector-ESP32-EVB_Rev_D-rescue
- removed U10: NL3S22S_DPDT_anlogue_switch, Package_DFN_QFN:UQFN-10_1.4x1.8mm_P0.4mm, symbol OSM_env01-rescue:NL3S22S_DPDT_anlogue_switch-Devtank-ESP32-EVB_Rev_D-rescue
- added C?: DNF, Capacitor_SMD:C_0603_1608Metric, symbol OSM_env01-rescue:C-device-ESP32-EVB_Rev_D-rescue
- added C? (x2): 100nF, symbol device:C
- added C? (x2): 10uF, symbol device:C
- added J?: Conn_01x12, symbol Connector:Conn_01x12
- added TP? (x4): Test_Point, symbol Connector:Test_Point
- added U?: RAK4270, symbol Devtank:RAK4270
- C9: value 100nF -> DNF
Connections:
- net labels added: CS, MISO, MOSI, RX, SCK, TX
- net labels removed: SW_EN
- wire segments 422 -> 460
- no-connect marks 17 -> 30
Other:
- note added: "Parts to add:\n-Fiducial\n-Gpio support\n-add second footprint for lora chip\n-add new microcontroller"
- note removed: "Audio Circuit\n"
- note removed: "D+/D- Function\nNC\nAUDP/AUDN\nHDP/HDN"
- note removed: "DPDT Analogue Switch"
- note removed: "EN\n0\n1\n1"
- note removed: "SEL\nX\n0\n1"
- note removed: "Shunt Status\nON\nOFF\nON"
- note removed: "test batt\ndo we need cts and dtr of usb cct\nconnect USB gpio lines to esp\nFSUSB30MUX new anlogue switch"
- moved on the sheet: C11, C22, C23, C24, C25, C26, C6, C7, D7, D8, JP2, L2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

Commit message: pushed latest schematics got started with micro into schematic
Parts:
- removed 400MA_E1: Closed, Connector_PinHeader_1.27mm:PinHeader_1x02_P1.27mm_Vertical, symbol OSM_env01-rescue:SJ_Closed-ESP32-EVB_Rev_D
- removed BAT1: 18650, Battery:BatteryHolder_Keystone_1042_1x18650, symbol OSM_env01-rescue:BAT_CON-ESP32-EVB_Rev_D
- removed C1, C2, C4, C5: 47uF, Capacitor_SMD:C_0805_2012Metric, symbol OSM_env01-rescue:C-ESP32-EVB_Rev_D
- removed C11, C7: 10uF, Capacitor_SMD:C_Elec_4x5.4, symbol OSM_env01-rescue:CP-device-ESP32-EVB_Rev_D-rescue
- removed C14, C42, C8, C?: 100nF, Capacitor_SMD:C_0402_1005Metric, symbol OSM_env01-rescue:C-device-ESP32-EVB_Rev_D-rescue
- removed C22, C33: 1uF, Capacitor_SMD:C_0603_1608Metric, symbol OSM_env01-rescue:C-device-ESP32-EVB_Rev_D-rescue
- removed C23: 0.1uF, Capacitor_SMD:C_0603_1608Metric, symbol OSM_env01-rescue:C-device-ESP32-EVB_Rev_D-rescue
- removed C24: 10uF, Capacitor_SMD:C_0603_1608Metric, symbol OSM_env01-rescue:C-device-ESP32-EVB_Rev_D-rescue
- removed C25: 2.2uF, Capacitor_SMD:C_0805_2012Metric, symbol OSM_env01-rescue:C-device-ESP32-EVB_Rev_D-rescue
- removed C26: 10uF, Capacitor_SMD:C_1206_3216Metric, symbol OSM_env01-rescue:C-device-ESP32-EVB_Rev_D-rescue
- removed C38: 10uF, Capacitor_SMD:C_0805_2012Metric, symbol OSM_env01-rescue:C-device-ESP32-EVB_Rev_D-rescue
- removed C39: DNF, Capacitor_SMD:C_0603_1608Metric, symbol OSM_env01-rescue:C-device-ESP32-EVB_Rev_D-rescue
- removed C40, C41: 100nF, Capacitor_SMD:C_0603_1608Metric, symbol OSM_env01-rescue:C-device-ESP32-EVB_Rev_D-rescue
- removed C6: DNF, Capacitor_SMD:C_1206_3216Metric, symbol OSM_env01-rescue:C-device-ESP32-EVB_Rev_D-rescue
- removed C9: DNF, Capacitor_SMD:C_0402_1005Metric, symbol OSM_env01-rescue:C-device-ESP32-EVB_Rev_D-rescue
- removed C? (x2): 100nF, symbol device:C
- removed C? (x2): 10uF, symbol device:C
- removed CHARGING1: YLW, Devtank_PCB_lib:LED_Rectangular_W4.5mm_H7.3mm_Horizontal_2.54mm_Z5.0mm, symbol OSM_env01-rescue:LED-ESP32-EVB_Rev_D
- removed COMPLETE1: GRN, Devtank_PCB_lib:LED_Rectangular_W4.5mm_H7.3mm_Horizontal_2.54mm_Z5.0mm, symbol OSM_env01-rescue:LED-ESP32-EVB_Rev_D
- removed D1: SP0503BAHT, Package_TO_SOT_SMD:SOT-143, symbol OSM_env01-rescue:SP0503BAHT-ESD_Protection-ESP32-EVB_Rev_D-rescue
- removed D2: SMBJ6.0A, Diode_SMD:D_SMB, symbol OSM_env01-rescue:SMBJ6.0A-ESP32-EVB_Rev_D
- removed D3: SS34, Diode_SMD:D_SMA, symbol OSM_env01-rescue:D_Schottky-ESP32-EVB_Rev_D
- removed D7, D8: SK24A, Diode_SMD:D_SMA, symbol OSM_env01-rescue:D_Schottky-device-ESP32-EVB_Rev_D-rescue
- removed J1: USB_B_Micro, Devtank_PCB_lib:MOLEX_105017-0001_USB_B, symbol Connector:USB_B_Micro
- removed J3: Conn_01x08, Connector_Molex:Molex_PicoBlade_53047-0810_1x08_P1.25mm_Vertical, symbol OSM_env01-rescue:Conn_01x08-Connector-ESP32-EVB_Rev_D-rescue
- removed JP2: Jumper_NC_Dual, Connector_PinHeader_1.27mm:PinHeader_1x03_P1.27mm_Vertical, symbol OSM_env01-rescue:Jumper_NC_Dual-device-ESP32-EVB_Rev_D-rescue
- removed L2: 10uH, Inductor_SMD:L_1812_4532Metric, symbol OSM_env01-rescue:L-device-ESP32-EVB_Rev_D-rescue
- removed PWRLED1, PWR_GOOD1: RED, LED_SMD:LED_0603_1608Metric, symbol OSM_env01-rescue:LED-ESP32-EVB_Rev_D
- removed Q1: SI2301BDS-T1-E3, Package_TO_SOT_SMD:SOT-23, symbol OSM_env01-rescue:SI2301BDS-T1-E3-Devtank-ESP32-EVB_Rev_D-rescue
- removed Q4: IRF7319TRPBF, Package_SO:SO-8_3.9x4.9mm_P1.27mm, symbol OSM_env01-rescue:IRF7319TRPBF-Devtank-ESP32-EVB_Rev_D-rescue
- removed Q6: FK3503010L, Devtank_PCB_lib:SMini3-F2-B, symbol OSM_env01-rescue:2N7002-Transistor-ESP32-EVB_Rev_D-rescue
- removed Q7: SSM3J328R, Package_TO_SOT_SMD:SOT-23, symbol OSM_env01-rescue:NTR2101P-Transistor-ESP32-EVB_Rev_D-rescue
- removed R1, R9: 2.2K, Resistor_SMD:R_0603_1608Metric, symbol OSM_env01-rescue:R-ESP32-EVB_Rev_D
- removed R10: DNF, Resistor_SMD:R_0603_1608Metric, symbol OSM_env01-rescue:R-ESP32-EVB_Rev_D
- removed R13, R14, R22, R78, R83: 10K, Resistor_SMD:R_0603_1608Metric, symbol OSM_env01-rescue:R-device-ESP32-EVB_Rev_D-rescue
- removed R16, R18: 470R, Resistor_SMD:R_0603_1608Metric, symbol OSM_env01-rescue:R-device-ESP32-EVB_Rev_D-rescue
- removed R17: 120R, Resistor_SMD:R_0603_1608Metric, symbol OSM_env01-rescue:R-device-ESP32-EVB_Rev_D-rescue
- removed R2, R4: 330R, Resistor_SMD:R_0603_1608Metric, symbol OSM_env01-rescue:R-ESP32-EVB_Rev_D
- removed R27: 15K, Resistor_SMD:R_0603_1608Metric, symbol OSM_env01-rescue:R-device-ESP32-EVB_Rev_D-rescue
- removed R28: 4.87K, Resistor_SMD:R_0603_1608Metric, symbol OSM_env01-rescue:R-device-ESP32-EVB_Rev_D-rescue
- removed R3, R5: 4.99K, Resistor_SMD:R_0603_1608Metric, symbol OSM_env01-rescue:R-ESP32-EVB_Rev_D
- removed R7: 0R, Resistor_SMD:R_0603_1608Metric, symbol OSM_env01-rescue:R-ESP32-EVB_Rev_D
- removed R72, R79, R80, R?: DNF, Resistor_SMD:R_0603_1608Metric, symbol OSM_env01-rescue:R-device-ESP32-EVB_Rev_D-rescue
- removed R73, R?: 0R, Resistor_SMD:R_0603_1608Metric, symbol OSM_env01-rescue:R-device-ESP32-EVB_Rev_D-rescue
- removed R74, R84, R86, R91, R92: 100K, Resistor_SMD:R_0603_1608Metric, symbol OSM_env01-rescue:R-device-ESP32-EVB_Rev_D-rescue
- removed R75: 47K, Resistor_SMD:R_0603_1608Metric, symbol OSM_env01-rescue:R-device-ESP32-EVB_Rev_D-rescue
- removed R85: 300K, Resistor_SMD:R_0603_1608Metric, symbol OSM_env01-rescue:R-device-ESP32-EVB_Rev_D-rescue
- removed R?: 100K, symbol OSM_env01-rescue:R-device-ESP32-EVB_Rev_D-rescue
- removed SW3: SW_Push, Devtank_PCB_lib:SW_Tactile_SPST_Angled_PTS645Vx58-2LFS, symbol Switch:SW_Push
- removed TH1: DNF, Resistor_THT:R_Axial_DIN0204_L3.6mm_D1.6mm_P2.54mm_Vertical, symbol OSM_env01-rescue:Thermistor_NTC-device-ESP32-EVB_Rev_D-rescue
- removed TH2: 10K, Resistor_SMD:R_1206_3216Metric, symbol OSM_env01-rescue:Thermistor_NTC-device-ESP32-EVB_Rev_D-rescue
- removed TP10, TP17, TP18, TP19, TP22, TP25, TP26, TP27, TP28, TP29, TP30, TP31, TP32, TP33, TP34, TP35, TP36, TP4, TP45, TP47, TP49, TP5, TP50, TP51, TP52, TP54, TP55, TP6, TP7, TP9, TP? (x2): Test_Point, TestPoint:TestPoint_THTPad_D1.0mm_Drill0.5mm, symbol OSM_env01-rescue:Test_Point-Connector-ESP32-EVB_Rev_D-rescue
- removed U1: MCP73833(MSOP10), Devtank_PCB_lib:MCP8833-AMI_UN, symbol OSM_env01-rescue:MCP73833(MSOP10)-ESP32-EVB_Rev_D
- removed U2: NCP1117-3.3_SOT223, Package_TO_SOT_SMD:SOT-223, symbol OSM_env01-rescue:NCP1117-3.3_SOT223-regul-ESP32-EVB_Rev_D-rescue
- removed U4: ISL83485, Package_SO:SOIC-8_3.9x4.9mm_P1.27mm, symbol OSM_env01-rescue:ISL83485-Devtank-ESP32-EVB_Rev_D-rescue
- removed U6: ERIC-LORA, Devtank_PCB_lib:eRIC-LoRa_RF_Module, symbol OSM_env01-rescue:ERIC-LORA-Devtank-ESP32-EVB_Rev_D-rescue
- removed U7: TSL2561, Devtank_PCB_lib:TSL2561T, symbol OSM_env01-rescue:TSL2561-Devtank-ESP32-EVB_Rev_D-rescue
- removed U8: M74VHC1GT14DFT2G, Package_TO_SOT_SMD:SOT-353_SC-70-5, symbol OSM_env01-rescue:NL17SZ14-Devtank-ESP32-EVB_Rev_D-rescue
- removed U9: MIC2288YD5-TR, Package_TO_SOT_SMD:SOT-23-5, symbol OSM_env01-rescue:MIC2288YD5-TR_BOOST-Devtank-ESP32-EVB_Rev_D-rescue
- removed U?: HDC2080, Devtank_PCB_lib:HDC2080DMBR, symbol OSM_env01-rescue:HDC2080-Devtank-ESP32-EVB_Rev_D-rescue
- removed U?: RAK4270, symbol Devtank:RAK4270
- added U?: STM32L412K8U6, QFN32_5X5_STM, symbol Devtank:STM32L412K8U6
Connections:
- no-connect marks 30 -> 11
Other:
- note added: "Auto Programming"
- note added: "Easy access gnd\npins for debug\n"
- note added: "Optional module"
- note added: "Parts to add:\n-Fiducial\n-Gpio support\n-add second footprint for lora chip\n-add new microcontroller\n-Fix particulate in rush issue"
- note removed: "Battery voltage monitor"
- note removed: "Electricty Meter"
- note removed: "Ich = 1000/Rp\n200mA->4.99k\n400mA->4.99k || 4.99k"
- note removed: "LORA"
- note removed: "Light Sensor\n"
- note removed: "Particulate Sensor\n"
- note removed: "Parts to add:\n-Fiducial\n-Gpio support\n-add second footprint for lora chip\n-add new microcontroller"
- note removed: "Powerdown circuit\n"
- note removed: "Pulse 2\n\n"
- note removed: "Rp"
- note removed: "Sound Level Meter\n"
- note removed: "Temp and Humidity\n"
- note removed: "Vout=Vrefx(R1/R2 + 1)\nVref=1.24V\nR2 not to exceed 5K\n"
- note removed: "Water Pump\n"
- note removed: "auto-off top position (default)\nauto-on bottom position"
- note removed: "black wire"
- note removed: "divider ratio=47/147=31.97\n5/1024=1adc=4.88mm\n(4.2/4.88m)*0.3197=275.15adc=fully charged and above\n\n"
- note removed: "red wire"
- moved on the sheet: C12, C13, C18, C19, C20, C21, C27, C28, C29, C30, C?, ESP_STATUS1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

Commit message: stm32 added to kicad
Parts:
- removed R56, R57, R58, R64, R67, R69: 0R, Resistor_SMD:R_0603_1608Metric, symbol OSM_env01-rescue:R-device-ESP32-EVB_Rev_D-rescue
- removed U?: STM32L412K8U6, QFN32_5X5_STM, symbol Devtank:STM32L412K8U6
- added R? (x15): 0R, Resistor_SMD:R_0603_1608Metric, symbol OSM_env01-rescue:R-device-ESP32-EVB_Rev_D-rescue
- added R? (x2): 4.7K, Resistor_SMD:R_0603_1608Metric, symbol OSM_env01-rescue:R-device-ESP32-EVB_Rev_D-rescue
- added TP? (x4): Test_Point, TestPoint:TestPoint_THTPad_D1.0mm_Drill0.5mm, symbol OSM_env01-rescue:Test_Point-Connector-ESP32-EVB_Rev_D-rescue
Connections:
- net +3V3: now also J2.8 (Pin_8), R?.1, R?.1
- net CS: now also R?.2
- net ESP_EN: now also TP?.1
- net GND: no longer J?.11 (Pin_11)
- net LIGHT_INT: now also R?.2
- net at U3.11 (GPIO26/DAC_2/ADC2_CH9/RTC_GPIO7/EMAC_RXD1): no longer R68.1
- net at U3.13 (GPIO14/ADC2_CH6/TOUCH6/RTC_GPIO16/MTMS/HSPICLK/HS2_CLK/SD_CLK/EMAC_TXD2): no longer R82.1
- net at U3.16 (GPIO13/ADC2_CH4/TOUCH4/RTC_GPIO14/MTCK/HSPID/HS2_DATA3/SD_DATA3/EMAC_RX_ER): no longer R81.1
- net STM_WAKEUP: now reaches U3.5 (GPI39/SENSOR_VN/ADC1_CH3/ADC_H/RTC_GPIO3)
- net STM_WAKEUP: now also R?.2
- net at U3.6 (GPI34/ADC1_CH6/RTC_GPIO4): no longer R66.1
- net at U3.7 (GPI35/ADC1_CH7/RTC_GPIO5): no longer R65.1
- net at U3.8 (GPIO32/XTAL_32K_P/ADC1_CH4/TOUCH9/RTC_GPIO9): no longer R24.1
- net MISO renamed STM_MISO
- net STM_MISO: now also R?.2
- net MOSI renamed STM_MOSI
- net STM_MOSI: now also R?.2
- net RX renamed STM2_TX
- net STM2_TX: now also R?.2
- net SCK renamed STM_SCK
- net STM_SCK: now also R?.2
- net SCL renamed ESP_SCL
- net ESP_SCL: now also R?.2; no longer J?.3 (Pin_3)
- net SDA renamed ESP_SDA
- net ESP_SDA: now also R?.2; no longer J?.4 (Pin_4)
- net TX renamed STM2_RX
- net STM2_RX: now also R?.2
- new net STM1_RX: R?.2
- new net STM1_TX: R?.2
- new net STM32L4/PA0: R?.1
- new net STM32L4/PA1: R?.1
- new net STM32L4/PA10: R?.1
- new net STM32L4/PA13: R68.1
- new net STM32L4/PA14: R65.1
- new net STM32L4/PA15: R?.1
- new net STM32L4/PA2: R?.1
- new net STM32L4/PA3: R?.1
- new net STM32L4/PA5: R66.1
- new net STM32L4/PA6: R?.1
- new net STM32L4/PA7: R?.1
- new net STM32L4/PA8: R?.1
- new net STM32L4/PA9: R?.1
- new net STM32L4/PB0: R24.1
- new net STM32L4/PB1: R82.1
- new net STM32L4/PB3: R?.1
- new net STM32L4/PB4: R?.1
- new net STM32L4/PB5: R?.1
- new net STM32L4/PB6: R?.1
- new net STM32L4/PB7: R?.1
- new net STM_BOOT0: TP?.1
- new net STM_SCL: J?.3 (Pin_3), R?.2
- new net STM_SDA: J?.4 (Pin_4), R?.2, R?.2
- new net USB_debug/ESP_RES1: TP?.1
- new net USB_debug/ESP_RES2: TP?.1
- new net extra_gpio: J?.11 (Pin_11), R?.2
- no-connect marks 11 -> 21
Other:
- note added: "add status led"
- moved on the sheet: R24, R65, R66, R68, R81, R82

Commit message: kicad review sch initial
Parts:
- removed R?: 0R, Resistor_SMD:R_0603_1608Metric, symbol OSM_env01-rescue:R-device-ESP32-EVB_Rev_D-rescue
- added R? (x2): 0R, Resistor_SMD:R_0603_1608Metric, symbol OSM_env01-rescue:R-device-ESP32-EVB_Rev_D-rescue
Connections:
- net CS: no longer R?.2
- net STM2_RX: no longer J?.6 (Pin_6)
- net STM2_TX: no longer J?.5 (Pin_5)
- net STM_SCL: now also R?.2
- net STM_WAKEUP: no longer U3.5 (GPI39/SENSOR_VN/ADC1_CH3/ADC_H/RTC_GPIO3)
- net at U3.27 (GPIO16/HS1_DATA4/U2RXD/EMAC_CLK_OUT): now also R?.1
- net at U3.28 (GPIO17/HS1_DATA5/U2TXD/EMAC_CLK_OUT_180): now also R?.1
- net USB_debug/ESP_RES1 renamed LORA_NRST
- new net HPM_EN: R?.2
- new net RS485_RX: R?.2
- new net RS485_TX: R?.2
- new net extra_RX: J?.6 (Pin_6)
- new net extra_TX: J?.5 (Pin_5)
- no-connect marks 21 -> 19
Other:
- note added: "7 gpio\n3 gpi\n"
Changed lines of the file:
@@
 Text Label 3800 13425 0    50   ~ 0
 PULSE2_EXT
-Text Notes 8725 3100 0    50   ~ 0
+Text Notes 17975 2900 0    50   ~ 0
 \n
 $Comp
@@
 	1425 13975 1275 13975
 $Sheet
-S 1050 975  1675 1175
+S 1050 975  925  575
 U 60688D25
 F0 "PowerSupply" 50
 F1 "PowerSupply.sch" 50
+F2 "5Vin" I L 1050 1250 50
+F3 "5Vout" I R 1975 1125 50
+F4 "3.3Vout" I R 1975 1250 50
+F5 "BatMon" I R 1975 1375 50
 $EndSheet
 $Sheet
-S 3850 1000 1300 1400
+S 3825 900  1125 950
 U 60880AD8
 F0 "LORA" 50
 F1 "LORA.sch" 50
-$EndSheet
-$Sheet
-S 6250 1025 2600 2050
-U 608F4675
-F0 "Sensors_AND_IO" 50
-F1 "Sensors_AND_IO.sch" 50
+F2 "LORA_RX" I L 3825 1450 50
+F3 "LORA_TX" I L 3825 1575 50
+F4 "LORA_CTS" I R 4950 1125 50
+F5 "LORA_NRST" I L 3825 1125 50
 $EndSheet
 Text Notes 750  14525 0    118  ~ 0
 Optional module
 $Sheet
-S 10275 1250 1700 1550
+S 6575 1075 1150 675
 U 609D4B87
 F0 "RS485_Comms" 50
 F1 "RS485_Comms.sch" 50
+F2 "RS485-" I L 6575 1350 50
+F3 "RS485+" I L 6575 1225 50
+F4 "DE_485" I L 6575 1600 50
+F5 "RS485_TX" I R 7725 1350 50
+F6 "RS485_RX" I R 7725 1475 50
 $EndSheet
 Text Notes 5850 14000 0    118  ~ 0
@@
 F16 "PB4" I R 15150 5075 50
 F17 "PB3" I R 15150 4950 50
-F18 "PA15" I L 14000 6350 50
-F19 "PA14" I L 14000 6225 50
-F20 "PA9" I L 14000 5850 50
-F21 "PA8" I L 14000 5725 50
-F22 "PA10" I L 14000 5975 50
-F23 "PA13" I L 14000 6100 50
+F18 "PA14" I L 14000 6225 50
+F19 "PA9" I L 14000 5850 50
+F20 "PA8" I L 14000 5725 50
+F21 "PA10" I L 14000 5975 50
+F22 "PA13" I L 14000 6100 50
 $EndSheet
 Text Label 7475 5825 2    50   ~ 0
@@
 NoConn ~ 6725 6325
 NoConn ~ 6725 6225
-NoConn ~ 6725 5525
-NoConn ~ 6725 5425
 NoConn ~ 6725 5225
 NoConn ~ 6725 5125
@@
 Text Label 1050 13175 0    50   ~ 0
 STM_SDA
-Text Label 13050 5725 0    50   ~ 0
+Text Label 7650 7125 0    50   ~ 0
 CS
-Text Label 13050 6350 0    50   ~ 0
+Text Label 7475 7300 0    50   ~ 0
 extra_gpio
-Wire Wire Line
-	14000 6350 13950 6350
-$Comp
-L OSM_env01-rescue:R-device-ESP32-EVB_Rev_D-rescue R?
-U 1 1 611289C8
-P 13800 6350
-F 0 "R?" V 13775 5275 50  0000 C CNN
-F 1 "0R" V 13775 5525 50  0000 C CNN
-F 2 "Resistor_SMD:R_0603_1608Metric" V 13730 6350 50  0001 C CNN
-F 3 "" H 13800 6350 50  0001 C CNN
-	1    13800 6350
-	0    1    1    0
-$EndComp
-Wire Wire Line
-	13650 6350 13050 6350
 Wire Wire Line
 	14000 5725 13950 5725
@@
 STM2_RX
 Text Label 1050 13275 0    50   ~ 0
-STM2_TX
+extra_TX
 Text Label 1050 13375 0    50   ~ 0
-STM2_RX
+extra_RX
 Wire Wire Line
 	4400 13625 4400 13725
@@
 NoConn ~ 6725 6825
 Wire Wire Line
-	6725 6925 7325 6925
-Text Label 7325 6925 2    50   ~ 0
+	7275 7500 7875 7500
+Text Label 7875 7500 2    50   ~ 0
 STM_WAKEUP
 Text Label 3375 9350 2    60   ~ 0
@@
 Text Notes 15950 5950 0    50   ~ 0
 add status led
+Text Label 7125 10025 2    50   ~ 0
+STM_SCL
+Text Label 15150 2325 0    50   ~ 0
+STM2_TX
+Text Label 15150 2175 0    50   ~ 0
+STM2_RX
+Wire Wire Line
+	3825 1575 3425 1575
+Text Label 3425 1575 0    50   ~ 0
+LORA_TX
+Text Label 3425 1450 0    50   ~ 0
+LORA_RX
+Wire Wire Line
+	3825 1450 3425 1450
+Text Label 3425 1125 0    50   ~ 0
+LORA_NRST
+Wire Wire Line
+	3825 1125 3425 1125
+Text Label 5350 1125 2    50   ~ 0
+LORA_CTS
+Wire Wire Line
+	4950 1125 5350 1125
+Text Label 3425 9650 2    50   ~ 0
+LORA_NRST
+Wire Wire Line
+	1050 1250 725  1250
+Text Label 725  1250 0    50   ~ 0
+5V_IN
+$Comp
+L power:+3V3 #PWR?
+U 1 1 607B31BD
+P 2525 925
+F 0 "#PWR?" H 2525 775 50  0001 C CNN
+F 1 "+3V3" H 2540 1098 50  0000 C CNN
+F 2 "" H 2525 925 50  0001 C CNN
+F 3 "" H 2525 925 50  0001 C CNN
+	1    2525 925
+	1    0    0    -1
+$EndComp
+$Comp
+L power:+5V #PWR?
+U 1 1 607B37D8
+P 2250 925
+F 0 "#PWR?" H 2250 775 50  0001 C CNN
+F 1 "+5V" H 2265 1098 50  0000 C CNN
+F 2 "" H 2250 925 50  0001 C CNN
+F 3 "" H 2250 925 50  0001 C CNN
+	1    2250 925
+	1    0    0    -1
+$EndComp
+Wire Wire Line
+	1975 1375 2575 1375
+Text Label 2575 1375 2    50   ~ 0
+BAT_MON
+Wire Wire Line
+	1975 1125 2250 1125
+Wire Wire Line
+	2250 1125 2250 925
+Wire Wire Line
+	1975 1250 2525 1250
+Wire Wire Line
+	2525 1250 2525 925
+Text Label 5975 1225 0    50   ~ 0
+RS485+
+Wire Wire Line
+	5975 1225 6575 1225
+Text Label 5975 1350 0    50   ~ 0
+RS485-
+Wire Wire Line
+	5975 1350 6575 1350
+Wire Wire Line
+	5975 1600 6575 1600
+Text Label 5975 1600 0    50   ~ 0
+DE_485
+Wire Wire Line
+	6725 5525 6775 5525
+$Comp
+L OSM_env01-rescue:R-device-ESP32-EVB_Rev_D-rescue R?
+U 1 1 6089B2FF
+P 6925 5525
+F 0 "R?" V 6900 4825 50  0000 C CNN
+F 1 "0R" V 6900 4650 50  0000 C CNN
+F 2 "Resistor_SMD:R_0603_1608Metric" V 6855 5525 50  0001 C CNN
+F 3 "" H 6925 5525 50  0001 C CNN
+	1    6925 5525
+	0    -1   1    0
+$EndComp
+Wire Wire Line
+	6725 5425 6775 5425
+$Comp
+L OSM_env01-rescue:R-device-ESP32-EVB_Rev_D-rescue R?
+U 1 1 6089B306
+P 6925 5425
+F 0 "R?" V 6900 4725 50  0000 C CNN
+F 1 "0R" V 6900 4550 50  0000 C CNN
+F 2 "Resistor_SMD:R_0603_1608Metric" V 6855 5425 50  0001 C CNN
+F 3 "" H 6925 5425 50  0001 C CNN
+	1    6925 5425
+	0    -1   1    0
+$EndComp
+Wire Wire Line
+	7075 5425 7475 5425
+Text Label 7475 5425 2    50   ~ 0
+RS485_TX
+Wire Wire Line
+	7075 5525 7475 5525
+Text Label 7475 5525 2    50   ~ 0
+RS485_RX
+Wire Wire Line
+	7725 1350 8125 1350
+Text Label 8125 1350 2    50   ~ 0
+RS485_TX
+Wire Wire Line
+	7725 1475 8125 1475
+Text Label 8125 1475 2    50   ~ 0
+RS485_RX
+Text Label 13050 5725 0    60   ~ 0
+HPM_EN
+Text Notes 8050 7375 0    50   ~ 0
+7 gpio\n3 gpi\n
+$Sheet
+S 15500 825  1525 1650
+U 608F4675
+F0 "Sensors_AND_IO" 50
+F1 "Sensors_AND_IO.sch" 50
+F2 "HPM_RX" I L 15500 2175 50
+F3 "HPM_TX" I L 15500 2325 50
+F4 "HPM_EN" I L 15500 1000 50
+F5 "TEMP_INT" I R 17025 1000 50
+F6 "SCL" I L 15500 1800 50
+F7 "SDA" I L 15500 1650 50
+F8 "LIGHT_INT" I R 17025 1150 50
+F9 "AUDIO_OP" I R 17025 1650 50
+F10 "PULSE1_EXT" I L 15500 1150 50
+F11 "PULSE2_EXT" I L 15500 1300 50
+F12 "PULSE_IN1" I R 17025 1800 50
+F13 "PULSE_IN2" I R 17025 1950 50
+$EndSheet
+Wire Wire Line
+	15500 2175 15150 2175
+Wire Wire Line
+	15500 2325 15150 2325
+Wire Wire Line
+	15500 1650 14900 1650
+Wire Wire Line
+	15500 1800 14900 1800
+Text Label 14900 1800 0    50   ~ 0
+STM_SCL
+Text Label 14900 1650 0    50   ~ 0
+STM_SDA
+Wire Wire Line
+	15500 1150 14900 1150
+Text Label 14900 1150 0    50   ~ 0
+PULSE1_EXT
+Text Label 14900 1300 0    50   ~ 0
+PULSE2_EXT
+Wire Wire Line
+	14900 1300 15500 1300
+Wire Wire Line
+	15500 1000 14900 1000
+Text Label 14900 1000 0    50   ~ 0
+HPM_EN
+Wire Wire Line
+	17025 1150 17625 1150
+Text Label 17625 1150 2    50   ~ 0
+LIGHT_INT
+Wire Wire Line
+	17025 1000 17625 1000
+Text Label 17625 1000 2    50   ~ 0
+TEMP_INT
+Text Label 17625 1650 2    50   ~ 0
+AUDIO_OP
+Wire Wire Line
+	17625 1650 17025 1650
+Wire Wire Line
+	17025 1950 17625 1950
+Text Label 17625 1950 2    50   ~ 0
+PULSE_IN2
+Text Label 17600 1800 2    50   ~ 0
+PULSE_IN1
+Wire Wire Line
+	17025 1800 17600 1800
 $EndSCHEMATC

Commit message: updated schematics
Parts:
- removed R68, R82, R?: 0R, Resistor_SMD:R_0603_1608Metric, symbol OSM_env01-rescue:R-device-ESP32-EVB_Rev_D-rescue
- added R10, R13, R14, R17, R18, R3, R33, R36, R4, R9: 0R, Resistor_SMD:R_0603_1608Metric, symbol OSM_env01-rescue:R-device-ESP32-EVB_Rev_D-rescue
- added R122: DNF, Resistor_SMD:R_0603_1608Metric, symbol OSM_env01-rescue:R-device-ESP32-EVB_Rev_D-rescue
- added TP19, TP20, TP21, TP22: Test_Point, symbol Connector:Test_Point
- gave numbers to parts that had none: 28
Connections:
- net extra_RX is gone; now on net STM1_RX: J1.6 (Pin_6)
- net extra_TX is gone; now on net STM1_TX: J1.5 (Pin_5)
- net CS: now also R33.2
- net LORA_NRST: no longer TP6.1
- net STM32L4/PA1: now also R22.1
- net STM32L4/PA4: now also R81.1
- net STM32L4/PA8: now also R122.1; no longer R22.1
- net STM32L4/PB1: now also R36.1
- net STM_BOOT0: now also U3.13 (GPIO14/ADC2_CH6/TOUCH6/RTC_GPIO16/MTMS/HSPICLK/HS2_CLK/SD_CLK/EMAC_TXD2), R18.2; no longer TP5.1
- net STM_WAKEUP: now also U3.26 (GPIO4/ADC2_CH0/TOUCH0/RTC_GPIO10/HSPIHD/HS2_DATA1/SD_DATA1/EMAC_TX_ER)
- net at U3.11 (GPIO26/DAC_2/ADC2_CH9/RTC_GPIO7/EMAC_RXD1): now also R9.1
- net at U3.12 (GPIO27/ADC2_CH7/TOUCH7/RTC_GPIO17/EMAC_RX_DV): now also R10.1
- net extra_gpio2: now reaches U3.14 (GPIO12/ADC2_CH5/TOUCH5/RTC_GPIO15/MTDI/HSPIQ/HS2_DATA2/SD_DATA2/EMAC_TXD3)
- net extra_gpio2: now also TP19.1
- net STM_NRST: now reaches U3.16 (GPIO13/ADC2_CH4/TOUCH4/RTC_GPIO14/MTCK/HSPID/HS2_DATA3/SD_DATA3/EMAC_RX_ER)
- net STM_NRST: now also R17.2
- net at U3.23 (GPIO15/ADC2_CH3/TOUCH3/MTDO/HSPICS0/RTC_GPIO13/HS2_CMD/SD_CMD/EMAC_RXD3): now also R4.1
- net at U3.29 (GPIO5/VSPICS0/HS1_DATA6/EMAC_RX_CLK): now also R3.1
- net extra_gpi4: now reaches U3.4 (GPI36/SENSOR_VP/ADC_H/ADC1_CH0/RTC_GPIO0)
- net extra_gpi4: now also TP21.1
- net extra_gpi5: now reaches U3.5 (GPI39/SENSOR_VN/ADC1_CH3/ADC_H/RTC_GPIO3)
- net extra_gpi5: now also TP22.1
- net extra_gpi3: now reaches U3.6 (GPI34/ADC1_CH6/RTC_GPIO4)
- net extra_gpi3: now also TP20.1
- net at U3.7 (GPI35/ADC1_CH7/RTC_GPIO5): now also R14.1
- net at U3.8 (GPIO32/XTAL_32K_P/ADC1_CH4/TOUCH9/RTC_GPIO9): now also R13.1
- net STM32L4/PA14 renamed STM32L4/PA11
- net USB_debug/ESP_RES2 renamed extra_gpio8
- net extra_gpio renamed extra_gpio1
- net extra_gpio1: now also R36.2
- new net CAN_RX: R14.2
- new net CAN_TX: R3.2
- new net MIC_LR: R9.2
- new net MIC_SCK: R10.2
- new net MIC_SD: R4.2
- new net MIC_WS: R13.2
- new net STM32L4/PA12: R33.1
- new net STM32L4/STM_BOOT0: R18.1
- new net STM32L4/STM_NRST: R17.1
- new net extra_gpio6: TP5.1
- new net extra_gpio7: TP6.1
- no-connect marks 19 -> 6
Other:
- note removed: "7 gpio\n3 gpi\n"
- moved on the sheet: R22, R24, R34, R35, R37, R38, R39, R40, R65, R81
