File: kicad_osm_env01/OSM_env01.sch (KiCad schematic (older format))
At the start: 105 parts, among them J1 Conn_01x12, J2 Conn_02x10_Counter_Clockwise, J6 Conn_01x06, SW1 SW_SPST, SW2 SW_SPST, U3 ESP-WROOM-32

Commit message: Throwdown of parts
Parts:
- added C75, C76, C77, C78: 100pF, Capacitor_SMD:C_0402_1005Metric, symbol OSM_env01-rescue:C-device-ESP32-EVB_Rev_D-rescue
- J2: footprint Connector_PinHeader_2.00mm:PinHeader_2x10_P2.00mm_Vertical -> Devtank_PCB_lib:molex_milligrid_87831-2019
- TP10, TP17, TP18, TP3, TP9: footprint TestPoint:TestPoint_THTPad_D1.0mm_Drill0.5mm -> TestPoint:TestPoint_THTPad_4.0x4.0mm_Drill2.0mm
Connections:
- wire segments 256 -> 265
Other:
- moved on the sheet: TP10, TP17, TP18, TP9
Changed lines of the file:
@@
 L Connector:Test_Point TP9
 U 1 1 608677C1
-P 9275 10000
-F 0 "TP9" H 9200 10200 50  0000 L CNN
-F 1 "Test_Point" H 9333 10027 50  0001 L CNN
-F 2 "TestPoint:TestPoint_THTPad_D1.0mm_Drill0.5mm" H 9475 10000 50  0001 C CNN
-F 3 "~" H 9475 10000 50  0001 C CNN
-	1    9275 10000
+P 13550 9225
+F 0 "TP9" H 13475 9425 50  0000 L CNN
+F 1 "Test_Point" H 13608 9252 50  0001 L CNN
+F 2 "TestPoint:TestPoint_THTPad_4.0x4.0mm_Drill2.0mm" H 13750 9225 50  0001 C CNN
+F 3 "~" H 13750 9225 50  0001 C CNN
+	1    13550 9225
 	1    0    0    -1
 $EndComp
@@
 L Connector:Test_Point TP10
 U 1 1 6086F915
-P 9550 10000
-F 0 "TP10" H 9450 10200 50  0000 L CNN
-F 1 "Test_Point" H 9608 10027 50  0001 L CNN
-F 2 "TestPoint:TestPoint_THTPad_D1.0mm_Drill0.5mm" H 9750 10000 50  0001 C CNN
-F 3 "~" H 9750 10000 50  0001 C CNN
-	1    9550 10000
+P 13825 9225
+F 0 "TP10" H 13725 9425 50  0000 L CNN
+F 1 "Test_Point" H 13883 9252 50  0001 L CNN
+F 2 "TestPoint:TestPoint_THTPad_4.0x4.0mm_Drill2.0mm" H 14025 9225 50  0001 C CNN
+F 3 "~" H 14025 9225 50  0001 C CNN
+	1    13825 9225
 	1    0    0    -1
 $EndComp
@@
 L Connector:Test_Point TP17
 U 1 1 608A0166
-P 9825 10000
-F 0 "TP17" H 9725 10200 50  0000 L CNN
-F 1 "Test_Point" H 9883 10027 50  0001 L CNN
-F 2 "TestPoint:TestPoint_THTPad_D1.0mm_Drill0.5mm" H 10025 10000 50  0001 C CNN
-F 3 "~" H 10025 10000 50  0001 C CNN
-	1    9825 10000
+P 14100 9225
+F 0 "TP17" H 14000 9425 50  0000 L CNN
+F 1 "Test_Point" H 14158 9252 50  0001 L CNN
+F 2 "TestPoint:TestPoint_THTPad_4.0x4.0mm_Drill2.0mm" H 14300 9225 50  0001 C CNN
+F 3 "~" H 14300 9225 50  0001 C CNN
+	1    14100 9225
 	1    0    0    -1
 $EndComp
@@
 L Connector:Test_Point TP18
 U 1 1 608D0934
-P 10100 10000
-F 0 "TP18" H 10000 10200 50  0000 L CNN
-F 1 "Test_Point" H 10158 10027 50  0001 L CNN
-F 2 "TestPoint:TestPoint_THTPad_D1.0mm_Drill0.5mm" H 10300 10000 50  0001 C CNN
-F 3 "~" H 10300 10000 50  0001 C CNN
-	1    10100 10000
+P 14375 9225
+F 0 "TP18" H 14275 9425 50  0000 L CNN
+F 1 "Test_Point" H 14433 9252 50  0001 L CNN
+F 2 "TestPoint:TestPoint_THTPad_4.0x4.0mm_Drill2.0mm" H 14575 9225 50  0001 C CNN
+F 3 "~" H 14575 9225 50  0001 C CNN
+	1    14375 9225
 	1    0    0    -1
 $EndComp
@@
 L OSM_env01:GND #PWR013
 U 1 1 609012E4
-P 9275 10150
-F 0 "#PWR013" H 9275 9900 50  0001 C CNN
-F 1 "GND" H 9280 9977 50  0000 C CNN
-F 2 "" H 9275 10150 60  0000 C CNN
-F 3 "" H 9275 10150 60  0000 C CNN
-	1    9275 10150
-	1    0    0    -1
-$EndComp
-Wire Wire Line
-	9275 10150 9275 10075
-Wire Wire Line
-	9275 10075 9550 10075
-Wire Wire Line
-	9550 10075 9550 10000
-Connection ~ 9275 10075
-Wire Wire Line
-	9275 10075 9275 10000
-Wire Wire Line
-	9550 10075 9825 10075
-Wire Wire Line
-	9825 10075 9825 10000
-Connection ~ 9550 10075
-Wire Wire Line
-	9825 10075 10100 10075
-Wire Wire Line
-	10100 10075 10100 10000
-Connection ~ 9825 10075
+P 13550 9375
+F 0 "#PWR013" H 13550 9125 50  0001 C CNN
+F 1 "GND" H 13555 9202 50  0000 C CNN
+F 2 "" H 13550 9375 60  0000 C CNN
+F 3 "" H 13550 9375 60  0000 C CNN
+	1    13550 9375
+	1    0    0    -1
+$EndComp
+Wire Wire Line
+	13550 9375 13550 9300
+Wire Wire Line
+	13550 9300 13825 9300
+Wire Wire Line
+	13825 9300 13825 9225
+Connection ~ 13550 9300
+Wire Wire Line
+	13550 9300 13550 9225
+Wire Wire Line
+	13825 9300 14100 9300
+Wire Wire Line
+	14100 9300 14100 9225
+Connection ~ 13825 9300
+Wire Wire Line
+	14100 9300 14375 9300
+Wire Wire Line
+	14375 9300 14375 9225
+Connection ~ 14100 9300
 $Comp
 L power:+3V3 #PWR06
@@
 F6 "RS485_RX" I R 8125 7475 50
 $EndSheet
-Text Notes 9100 9225 0    118  ~ 24
+Text Notes 13375 8450 0    118  ~ 24
 Easy access gnd\npins for debug\n
 Text Notes 1375 8350 0    79   ~ 0
@@
 F 0 "TP3" H 2700 1000 50  0000 C CNN
 F 1 "Test_Point" H 2950 800 50  0001 C CNN
-F 2 "TestPoint:TestPoint_THTPad_D1.0mm_Drill0.5mm" H 2900 775 50  0001 C CNN
+F 2 "TestPoint:TestPoint_THTPad_4.0x4.0mm_Drill2.0mm" H 2900 775 50  0001 C CNN
 F 3 "~" H 2900 775 50  0001 C CNN
 	1    2700 775
@@
 HPM_EN
 $Sheet
-S 7075 9175 1025 725
+S 9525 9400 1025 725
 U 6064BC1D
 F0 "CanTransciever" 50
 F1 "CanTransciever.sch" 50
-F2 "CAN_RX" I R 8100 9425 50
-F3 "CAN_TX" I R 8100 9650 50
-F4 "CAN_L" I L 7075 9425 50
-F5 "CAN_H" I L 7075 9650 50
+F2 "CAN_RX" I R 10550 9650 50
+F3 "CAN_TX" I R 10550 9875 50
+F4 "CAN_L" I L 9525 9650 50
+F5 "CAN_H" I L 9525 9875 50
 $EndSheet
 Wire Wire Line
-	7075 9425 6675 9425
-Text Label 6675 9425 0    50   ~ 0
+	9525 9650 9125 9650
+Text Label 9125 9650 0    50   ~ 0
 CAN_L
 Wire Wire Line
-	7075 9650 6675 9650
-Text Label 6675 9650 0    50   ~ 0
+	9525 9875 9125 9875
+Text Label 9125 9875 0    50   ~ 0
 CAN_H
 Wire Wire Line
-	8100 9425 8500 9425
-Text Label 8500 9425 2    50   ~ 0
+	10550 9650 10950 9650
+Text Label 10950 9650 2    50   ~ 0
 CAN_RX
 Wire Wire Line
-	8100 9650 8500 9650
-Text Label 8500 9650 2    50   ~ 0
+	10550 9875 10950 9875
+Text Label 10950 9875 2    50   ~ 0
 CAN_TX
 Wire Wire Line
@@
 Text Notes 6675 6850 0    118  ~ 24
 RS485 Transciever\n
-Text Notes 6875 8975 0    118  ~ 24
+Text Notes 9325 9200 0    118  ~ 24
 CAN Transciever\n
 Text Notes 13475 5125 0    118  ~ 24
@@
 Text Label 5750 9500 2    50   ~ 0
 CT-
-Wire Wire Line
-	5750 9500 5425 9500
 Text Label 5750 9400 2    50   ~ 0
 CT+
-Wire Wire Line
-	5750 9400 5425 9400
 $Comp
 L OSM_env01:GND #PWR?
@@
 F 0 "J2" H 5175 10417 50  0000 C CNN
 F 1 "Conn_02x10_Counter_Clockwise" H 5175 10326 50  0000 C CNN
-F 2 "Connector_PinHeader_2.00mm:PinHeader_2x10_P2.00mm_Vertical" H 5125 9800 50  0001 C CNN
+F 2 "Devtank_PCB_lib:molex_milligrid_87831-2019" H 5125 9800 50  0001 C CNN
 F 3 "~" H 5125 9800 50  0001 C CNN
 	1    5125 9800
@@
 Wire Wire Line
 	4825 10300 4825 10000
-Wire Wire Line
-	5425 9700 5825 9700
 Text Label 5825 9700 2    50   ~ 0
 CAN_L
-Wire Wire Line
-	5425 9800 5825 9800
 Text Label 5825 9800 2    50   ~ 0
 CAN_H
@@
 NoConn ~ 5425 10200
 NoConn ~ 5425 10300
+$Comp
+L OSM_env01-rescue:C-device-ESP32-EVB_Rev_D-rescue C75
+U 1 1 60B52D72
+P 6150 9400
+F 0 "C75" H 6265 9446 50  0000 L CNN
+F 1 "100pF" H 6265 9355 50  0000 L CNN
+F 2 "Capacitor_SMD:C_0402_1005Metric" H 6188 9250 50  0001 C CNN
+F 3 "" H 6150 9400 50  0001 C CNN
+	1    6150 9400
+	0    -1   -1   0
+$EndComp
+$Comp
+L OSM_env01-rescue:C-device-ESP32-EVB_Rev_D-rescue C77
+U 1 1 60BA4214
+P 6550 9500
+F 0 "C77" H 6665 9546 50  0000 L CNN
+F 1 "100pF" H 6665 9455 50  0000 L CNN
+F 2 "Capacitor_SMD:C_0402_1005Metric" H 6588 9350 50  0001 C CNN
+F 3 "" H 6550 9500 50  0001 C CNN
+	1    6550 9500
+	0    -1   -1   0
+$EndComp
+$Comp
+L OSM_env01-rescue:C-device-ESP32-EVB_Rev_D-rescue C76
+U 1 1 60BBBEED
+P 6150 9700
+F 0 "C76" H 6265 9746 50  0000 L CNN
+F 1 "100pF" H 6265 9655 50  0000 L CNN
+F 2 "Capacitor_SMD:C_0402_1005Metric" H 6188 9550 50  0001 C CNN
+F 3 "" H 6150 9700 50  0001 C CNN
+	1    6150 9700
+	0    -1   -1   0
+$EndComp
+$Comp
+L OSM_env01-rescue:C-device-ESP32-EVB_Rev_D-rescue C78
+U 1 1 60BD379E
+P 6550 9800
+F 0 "C78" H 6665 9846 50  0000 L CNN
+F 1 "100pF" H 6665 9755 50  0000 L CNN
+F 2 "Capacitor_SMD:C_0402_1005Metric" H 6588 9650 50  0001 C CNN
+F 3 "" H 6550 9800 50  0001 C CNN
+	1    6550 9800
+	0    -1   -1   0
+$EndComp
+$Comp
+L OSM_env01-rescue:GND-ESP32-EVB_Rev_D #PWR082
+U 1 1 60BEC5E6
+P 7075 9875
+F 0 "#PWR082" H 7075 9625 50  0001 C CNN
+F 1 "GND" H 7080 9702 50  0000 C CNN
+F 2 "" H 7075 9875 60  0000 C CNN
+F 3 "" H 7075 9875 60  0000 C CNN
+	1    7075 9875
+	-1   0    0    -1
+$EndComp
+Wire Wire Line
+	7075 9875 7075 9800
+Wire Wire Line
+	6700 9800 6825 9800
+Connection ~ 6825 9800
+Wire Wire Line
+	6825 9800 7075 9800
+Wire Wire Line
+	6825 9500 6700 9500
+Wire Wire Line
+	6300 9700 6825 9700
+Connection ~ 6825 9500
+Wire Wire Line
+	5425 9500 6400 9500
+Connection ~ 6825 9700
+Wire Wire Line
+	6825 9700 6825 9800
+Wire Wire Line
+	6825 9500 6825 9700
+Wire Wire Line
+	5425 9700 6000 9700
+Wire Wire Line
+	5425 9800 6400 9800
+Wire Wire Line
+	6825 9400 6825 9500
+Wire Wire Line
+	5425 9400 6000 9400
+Wire Wire Line
+	6300 9400 6825 9400
 $EndSCHEMATC

Commit message: added stm to schematic
Parts:
- removed C1: DNF, Capacitor_SMD:C_0603_1608Metric, symbol OSM_env01-rescue:C-device-ESP32-EVB_Rev_D-rescue
- removed C12, C13: DNF, Capacitor_SMD:C_0805_2012Metric, symbol OSM_env01-rescue:C-device-ESP32-EVB_Rev_D-rescue
- removed C27, C30: 1nF, Capacitor_SMD:C_0603_1608Metric, symbol OSM_env01-rescue:C-device-ESP32-EVB_Rev_D-rescue
- removed C28: 100nF, Capacitor_SMD:C_0402_1005Metric, symbol OSM_env01-rescue:C-device-ESP32-EVB_Rev_D-rescue
- removed C29: 1uF, Capacitor_SMD:C_0603_1608Metric, symbol OSM_env01-rescue:C-device-ESP32-EVB_Rev_D-rescue
- removed ESP_STATUS1: LED, Devtank_PCB_lib:LED_Rectangular_W4.5mm_H7.3mm_Horizontal_2.54mm_Z5.0mm, symbol OSM_env01-rescue:LED-device-ESP32-EVB_Rev_D-rescue
- removed J6: Conn_01x06, Connector_PinHeader_2.54mm:PinHeader_1x06_P2.54mm_Vertical, symbol Connector:Conn_01x06
- removed R15, R19: 4.7K, Resistor_SMD:R_0603_1608Metric, symbol OSM_env01-rescue:R-device-ESP32-EVB_Rev_D-rescue
- removed R16: 0R, Resistor_SMD:R_0603_1608Metric, symbol OSM_env01-rescue:R-device-ESP32-EVB_Rev_D-rescue
- removed R26: 330R, Resistor_SMD:R_0603_1608Metric, symbol OSM_env01-rescue:R-device-ESP32-EVB_Rev_D-rescue
- removed R6: 12K, Resistor_SMD:R_0603_1608Metric, symbol OSM_env01-rescue:R-ESP32-EVB_Rev_D
- removed R71: 470R, Resistor_SMD:R_0603_1608Metric, symbol OSM_env01-rescue:R-device-ESP32-EVB_Rev_D-rescue
- removed SW1: SW_SPST, Button_Switch_SMD:SW_SPST_B3U-1000P, symbol Switch:SW_SPST
- removed TP1, TP2, TP65, TP66: Test_Point, TestPoint:TestPoint_THTPad_D1.0mm_Drill0.5mm, symbol OSM_env01-rescue:Test_Point-Connector-ESP32-EVB_Rev_D-rescue
- removed TP3: Test_Point, TestPoint:TestPoint_THTPad_4.0x4.0mm_Drill2.0mm, symbol OSM_env01-rescue:Test_Point-Connector-ESP32-EVB_Rev_D-rescue
- removed U3: ESP-WROOM-32, Devtank_PCB_lib:ESP32-WROOM-32U, symbol OSM_env01-rescue:ESP-WROOM-32-ESP32-EVB_Rev_D
Connections:
- wire segments 265 -> 208
Other:
- note removed: "Boot"
- note removed: "ESP"
- note removed: "ESP I2C Pullup"
- note removed: "ESP Programming \nheader\n"
- note removed: "Reset\n"
- note removed: "gpio6-11 used for spi"

Commit message: schematics awaiting review
Parts:
- removed C75, C77: 100pF, Capacitor_SMD:C_0402_1005Metric, symbol OSM_env01-rescue:C-device-ESP32-EVB_Rev_D-rescue
- removed J2: Conn_02x10_Counter_Clockwise, Devtank_PCB_lib:molex_milligrid_87831-2019, symbol Connector:Conn_02x10_Counter_Clockwise
- removed R10, R122, R13, R14, R17, R18, R22, R24, R25, R27, R28, R3, R30, R31, R32, R33, R34, R35, R36, R37, R38, R39, R4, R40, R5, R55, R59, R60, R61, R62, R63, R65, R66, R7, R8, R81, R9: 0R, Resistor_SMD:R_0603_1608Metric, symbol OSM_env01-rescue:R-device-ESP32-EVB_Rev_D-rescue
- removed SW2: SW_SPST, Button_Switch_SMD:SW_SPST_B3U-1000P, symbol Switch:SW_SPST
- removed TP10, TP17, TP18: Test_Point, TestPoint:TestPoint_THTPad_4.0x4.0mm_Drill2.0mm, symbol Connector:Test_Point
- removed TP13, TP14, TP20, TP21, TP22, TP69, TP71, TP73: Test_Point, TestPoint:TestPoint_THTPad_D1.0mm_Drill0.5mm, symbol OSM_env01-rescue:Test_Point-Connector-ESP32-EVB_Rev_D-rescue
- added C52, C53: 100nF, Capacitor_SMD:C_0402_1005Metric, symbol OSM_env01-rescue:C-device-ESP32-EVB_Rev_D-rescue
- added F1, F2, F3, F4: Fiducial, symbol Devtank:Fiducial
- added J2: Conn_02x07_Counter_Clockwise, symbol Connector:Conn_02x07_Counter_Clockwise
- added R10, R11, R12, R13, R14, R17, R3, R4, R5, R7, R8, R9: 0R, symbol device:R
- added TP10, TP17, TP2, TP3: Test_Point, TestPoint:TestPoint_THTPad_D1.0mm_Drill0.5mm, symbol OSM_env01-rescue:Test_Point-Connector-ESP32-EVB_Rev_D-rescue
Connections:
- net labels added: 3V3_RAIL_MONITOR, 5V_RAIL_MONITOR, ADC+GPIO, CAN_RS, GPIO_7, GPIO_8, HPM_RX, HPM_TX, PULSE1_OUT, PULSE2_OUT
- net labels removed: CT-, ESP_EN, ESP_IO0, ESP_SCL, ESP_SDA, MIC_LR, PULSE_IN1, PULSE_IN2, STM2_RX, STM2_TX, extra_gpi3, extra_gpi4, extra_gpi5, extra_gpio1, extra_gpio6, extra_gpio7, extra_gpio8
- wire segments 208 -> 164
- no-connect marks 10 -> 1
Other:
- note added: "Analogue Voltage Reference\n\n"
- note added: "Communication\n\n"
- note added: "Fiducials\n"
- note added: "Note: Low power mode selected through DE along with RE\n\n"
- note added: "Note: Low power mode selected through RS\n"
- note removed: "Auto Programming"
- note removed: "DTR\n1\n0\n1\n0"
- note removed: "EN\n1\n1\n0\n1"
- note removed: "IO0\n1\n1\n1\n0"
- note removed: "Precision Voltage Reference\n\n"
- note removed: "RTS-->\n1\n0\n0\n1"
- moved on the sheet: C18, C19, C20, C21, C76, C78, J1, R1, R2, TP11, TP12, TP19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

Commit message: rough layout with throwdown of parts
Parts:
- removed R14, R17, R5, R7: 0R, symbol device:R
- removed TP19, TP24, TP59, TP60, TP61, TP62, TP63, TP74, TP75, TP76, TP77, TP78: Test_Point, TestPoint:TestPoint_THTPad_D1.0mm_Drill0.5mm, symbol OSM_env01-rescue:Test_Point-Connector-ESP32-EVB_Rev_D-rescue
- added TP21, TP52, TP53: Test_Point, TestPoint:TestPoint_Pad_D1.0mm, symbol OSM_env01-rescue:Test_Point-Connector-ESP32-EVB_Rev_D-rescue
- F1, F2, F3, F4: footprint (none) -> Fiducial:Fiducial_1mm_Mask2mm
- J1: footprint Connector_PinHeader_2.54mm:PinHeader_2x06_P2.54mm_Vertical -> Devtank_PCB_lib:Milligrid_878311220_12way
- J2: footprint (none) -> Devtank_PCB_lib:Milligrid_878311420_14way
- R1, R2: footprint Resistor_SMD:R_0603_1608Metric -> Resistor_SMD:R_0402_1005Metric
- R10, R11, R12, R13, R3, R4, R8, R9: footprint (none) -> Resistor_SMD:R_0603_1608Metric
- TP10, TP15, TP16, TP17, TP2, TP3, TP64, TP67, TP70: footprint TestPoint:TestPoint_THTPad_D1.0mm_Drill0.5mm -> TestPoint:TestPoint_Pad_D1.0mm
- TP11, TP12, TP4, TP5, TP6, TP7, TP72, TP8: footprint TestPoint:TestPoint_THTPad_D1.0mm_Drill0.5mm -> TestPoint:TestPoint_Pad_D1.5mm
Connections:
- net labels removed: +3V3_A, +5VA, AUDIO_OP, MIC_GND
- wire segments 164 -> 155
Other:
- note removed: "Analogue Voltage Reference\n\n"
- note removed: "\n"
- moved on the sheet: TP16, TP17, TP2, TP3

Commit message: updated schematics
Parts:
- removed J1: Conn_01x12, Devtank_PCB_lib:Milligrid_878311220_12way, symbol Connector:Conn_01x12
- removed TP16: Test_Point, TestPoint:TestPoint_Pad_D1.0mm, symbol OSM_env01-rescue:Test_Point-Connector-ESP32-EVB_Rev_D-rescue
- added J?: Conn_02x07_Counter_Clockwise, symbol Connector:Conn_02x07_Odd_Even
- J2: symbol Connector:Conn_02x07_Counter_Clockwise -> Connector:Conn_02x07_Odd_Even
Connections:
- net +3V3: now also J2.4 (Pin_4), J?.1 (Pin_1); no longer J2.13 (Pin_13)
- net +5V: now also J2.2 (Pin_2), J?.3 (Pin_3); no longer J2.14 (Pin_14)
- net ADC+GPIO: now also J?.8 (Pin_8)
- net CAN_L: now also J2.8 (Pin_8); no longer J2.11 (Pin_11)
- net CS: now also J?.6 (Pin_6)
- net GND: now also J2.12 (Pin_12), J2.13 (Pin_13), J2.14 (Pin_14), J?.10 (Pin_10), J?.12 (Pin_12), J?.14 (Pin_14); no longer J2.3 (Pin_3), J2.7 (Pin_7), J2.8 (Pin_8)
- net PULSE1_EXT: now also J2.7 (Pin_7); no longer J2.4 (Pin_4)
- net PULSE2_EXT: now also J2.11 (Pin_11); no longer J2.6 (Pin_6)
- net RS485-: now also J2.3 (Pin_3); no longer J2.2 (Pin_2)
- net STM1_RX: now also J?.11 (Pin_11)
- net STM1_TX: now also J?.9 (Pin_9)
- net STM_MISO: now also J?.13 (Pin_13)
- net STM_MOSI: now also J?.2 (Pin_2)
- net STM_SCK: now also J?.4 (Pin_4)
- net STM_SCL: now also J?.5 (Pin_5)
- net STM_SDA: now also J?.7 (Pin_7)
Changed lines of the file:
@@
 	7250 9825 6875 9825
 Wire Wire Line
-	7250 9925 6875 9925
-$Comp
-L Connector:Conn_01x12 J1
-U 1 1 60CBF5A8
-P 7450 9725
-F 0 "J1" H 7400 10425 50  0000 L CNN
-F 1 "Conn_01x12" H 7530 9626 50  0001 L CNN
-F 2 "Devtank_PCB_lib:Milligrid_878311220_12way" H 7450 9725 50  0001 C CNN
-F 3 "~" H 7450 9725 50  0001 C CNN
-	1    7450 9725
-	1    0    0    -1
-$EndComp
-Wire Wire Line
-	7250 10025 6875 10025
-Wire Wire Line
-	7250 10125 6875 10125
-Text Label 6875 10125 0    50   ~ 0
+	7750 9225 8125 9225
+Wire Wire Line
+	7750 9325 8125 9325
+Wire Wire Line
+	7750 9425 8125 9425
+Text Label 8125 9425 2    50   ~ 0
 CS
 $Comp
 L OSM_env01:GND #PWR08
 U 1 1 60DF2DDC
-P 7100 10425
-F 0 "#PWR08" H 7100 10175 50  0001 C CNN
-F 1 "GND" H 7105 10252 50  0000 C CNN
-F 2 "" H 7100 10425 60  0000 C CNN
-F 3 "" H 7100 10425 60  0000 C CNN
-	1    7100 10425
-	1    0    0    -1
-$EndComp
-Wire Wire Line
-	7100 10425 7100 10325
-Wire Wire Line
-	7250 10325 7100 10325
+P 7900 9925
+F 0 "#PWR08" H 7900 9675 50  0001 C CNN
+F 1 "GND" H 7905 9752 50  0000 C CNN
+F 2 "" H 7900 9925 60  0000 C CNN
+F 3 "" H 7900 9925 60  0000 C CNN
+	1    7900 9925
+	-1   0    0    -1
+$EndComp
+Wire Wire Line
+	7900 9925 7900 9825
+Wire Wire Line
+	7750 9825 7900 9825
 $Sheet
 S 13275 5600 925  1025
@@
 F0 "LORA" 50
 F1 "LORA.sch" 50
-F2 "LORA_RX" I L 14100 1950 50
-F3 "LORA_TX" I L 14100 2075 50
-F4 "LORA_CTS" I R 15225 1625 50
-F5 "LORA_NRST" I L 14100 1625 50
+F2 "LORA_CTS" I R 15225 1625 50
+F3 "LORA_NRST" I L 14100 1625 50
 $EndSheet
 Text Notes 6200 8325 0    118  ~ 24
 Optional module
 $Sheet
-S 14050 3150 1150 675
+S 14050 3150 1150 825
 U 609D4B87
 F0 "RS485_Comms" 50
@@
 F5 "RS485_TX" I R 15200 3425 50
 F6 "RS485_RX" I R 15200 3550 50
+F7 "RS485_RE" I L 14050 3800 50
 $EndSheet
 Text Notes 9725 4800 0    118  ~ 24
 Easy access gnd\npins for debug\n
 Wire Wire Line
-	7250 10225 6875 10225
-Text Label 6875 10225 0    50   ~ 0
+	7750 9525 8125 9525
+Text Label 8125 9525 2    50   ~ 0
 ADC+GPIO
 Text Label 1275 4650 0    50   ~ 0
@@
 Text Label 6875 9425 0    50   ~ 0
 STM_SCL
-Text Label 6875 9925 0    50   ~ 0
+Text Label 8125 9225 2    50   ~ 0
 STM_MOSI
-Text Label 6875 10025 0    50   ~ 0
+Text Label 8125 9325 2    50   ~ 0
 STM_SCK
 Text Label 6875 9825 0    50   ~ 0
@@
 Text Label 6550 2675 0    50   ~ 0
 HPM_RX
-Wire Wire Line
-	14100 2075 13700 2075
-Text Label 13700 2075 0    50   ~ 0
-LORA_TX
-Text Label 13700 1950 0    50   ~ 0
-LORA_RX
-Wire Wire Line
-	14100 1950 13700 1950
 Text Label 13700 1625 0    50   ~ 0
 LORA_NRST
@@
 	1    0    0    -1
 $EndComp
-Text Label 3200 9700 2    50   ~ 0
+Text Label 3250 9700 2    50   ~ 0
 CAN_L
-Text Label 3200 9800 2    50   ~ 0
+Text Label 3250 9800 2    50   ~ 0
 CAN_H
 Wire Wire Line
@@
 Wire Wire Line
 	3850 2000 4425 2000
-Text Label 4425 2000 2    50   ~ 0
-LORA_TX
-Text Label 4425 2150 2    50   ~ 0
-LORA_RX
 Wire Wire Line
 	3850 2150 4425 2150
 $Comp
-L Connector:Conn_02x07_Counter_Clockwise J2
+L Connector:Conn_02x07_Odd_Even J2
 U 1 1 61BD7603
 P 2500 9700
@@
 Wire Wire Line
 	3725 9500 3775 9500
-NoConn ~ 2800 9600
 Text Label 7975 6600 2    50   ~ 0
 STM_WAKEUP
@@
 $Comp
 L OSM_env01-rescue:Test_Point-Connector-ESP32-EVB_Rev_D-rescue TP?
-U 1 1 61CAC829
-P 1275 4350
-AR Path="/60688D25/61CAC829" Ref="TP?"  Part="1"
-AR Path="/61CAC829" Ref="TP16"  Part="1"
-F 0 "TP16" V 1275 4625 50  0000 C CNN
-F 1 "Test_Point" V 1379 4422 50  0001 C CNN
-F 2 "TestPoint:TestPoint_Pad_D1.0mm" H 1475 4350 50  0001 C CNN
-F 3 "~" H 1475 4350 50  0001 C CNN
-	1    1275 4350
-	0    -1   1    0
-$EndComp
-$Comp
-L OSM_env01-rescue:Test_Point-Connector-ESP32-EVB_Rev_D-rescue TP?
 U 1 1 61CAC82F
 P 1275 3450
@@
 	0    -1   1    0
 $EndComp
+Text GLabel 4425 2000 2    50   Input ~ 0
+LORA_TX
+Text GLabel 4425 2150 2    50   Input ~ 0
+LORA_RX
+$Comp
+L Connector:Conn_02x07_Odd_Even J?
+U 1 1 619137D5
+P 7450 9525
+F 0 "J?" H 7500 9950 50  0000 C CNN
+F 1 "Conn_02x07_Counter_Clockwise" H 7500 9951 50  0001 C CNN
+F 2 "" H 7450 9525 50  0001 C CNN
+F 3 "~" H 7450 9525 50  0001 C CNN
+	1    7450 9525
+	1    0    0    -1
+$EndComp
+Wire Wire Line
+	7750 9625 7900 9625
+Connection ~ 7900 9825
+Wire Wire Line
+	7900 9625 7900 9725
+Wire Wire Line
+	7750 9725 7900 9725
+Connection ~ 7900 9725
+Wire Wire Line
+	7900 9725 7900 9825
+NoConn ~ 2800 9600
+Wire Wire Line
+	13450 3800 14050 3800
+Text Label 13450 3800 0    50   ~ 0
+RE_485
+Text Label 1275 4350 0    50   ~ 0
+RE_485
 $EndSCHEMATC
