File: kicad_osm_env01/OSM_env01.sch (KiCad schematic (older format))
At the start: 44 parts, among them J2 Conn_02x07_Counter_Clockwise

Commit message: updated schematics
Parts:
- added TP16: Test_Point, TestPoint:TestPoint_Pad_D1.0mm, symbol OSM_env01-rescue:Test_Point-Connector-ESP32-EVB_Rev_D-rescue
- gave numbers to parts that had none: 1
Connections:
- net RS485_RX: now also R10.1; no longer R11.1
- net RS485_TX: now also R11.1; no longer R10.1
- new net STM32L4/GPIO11: TP16.1
Other:
- note removed: "Parts to add:\n-Fiducial\n-Fix particulate in rush issue\n-lora rst not routed and rst through hardware rc"
Changed lines of the file:
@@
 F0 "LORA" 50
 F1 "LORA.sch" 50
-F2 "LORA_CTS" I R 15225 1625 50
-F3 "LORA_NRST" I L 14100 1625 50
+F2 "LORA_NRST" I L 14100 1850 50
+F3 "LORA_RX" I R 15225 1725 50
+F4 "LORA_TX" I R 15225 2000 50
 $EndSheet
 Text Notes 6200 8325 0    118  ~ 24
@@
 Text Label 8125 9525 2    50   ~ 0
 ADC+GPIO
-Text Label 1275 4650 0    50   ~ 0
-LORA_CTS
 Text Label 4425 1600 2    50   ~ 0
 RS232_TX
@@
 Text Label 6550 2675 0    50   ~ 0
 HPM_RX
-Text Label 13700 1625 0    50   ~ 0
+Text Label 13700 1850 0    50   ~ 0
 LORA_NRST
 Wire Wire Line
-	14100 1625 13700 1625
-Text Label 15625 1625 2    50   ~ 0
-LORA_CTS
-Wire Wire Line
-	15225 1625 15625 1625
+	14100 1850 13700 1850
 Wire Wire Line
 	13275 5875 12950 5875
@@
 Wire Wire Line
 	7150 3475 6575 3475
-$Sheet
-S 7150 1325 1550 2500
-U 608F4675
-F0 "Sensors_AND_IO" 50
-F1 "Sensors_AND_IO.sch" 50
-F2 "HPM_RX" I L 7150 2675 50
-F3 "HPM_TX" I L 7150 2825 50
-F4 "HPM_EN" I L 7150 1500 50
-F5 "SCL" I L 7150 2300 50
-F6 "SDA" I L 7150 2150 50
-F7 "PULSE1_EXT" I L 7150 1650 50
-F8 "PULSE2_EXT" I L 7150 1800 50
-F9 "MIC_SD" I R 8700 3325 50
-F10 "MIC_SCK" I L 7150 3325 50
-F11 "MIC_WS" I L 7150 3475 50
-F12 "CT+" I R 8700 2675 50
-F13 "PULSE_IN1" I R 8700 1650 50
-F14 "PULSE_IN2" I R 8700 1800 50
-$EndSheet
 Text Label 1275 3300 0    60   ~ 0
 HPM_EN
@@
 Text Label 6875 9725 0    50   ~ 0
 STM1_RX
-Text Notes 14700 10250 0    50   ~ 0
-Parts to add:\n-Fiducial\n-Fix particulate in rush issue\n-lora rst not routed and rst through hardware rc
 $Comp
 L OSM_env01-rescue:Test_Point-Connector-ESP32-EVB_Rev_D-rescue TP?
@@
 Wire Wire Line
 	3850 1200 4425 1200
+Text Label 4425 2550 2    50   ~ 0
+RS485_TX
+Wire Wire Line
+	3850 1350 4425 1350
 Text Label 4425 2400 2    50   ~ 0
-RS485_TX
-Wire Wire Line
-	3850 1350 4425 1350
-Text Label 4425 2550 2    50   ~ 0
 RS485_RX
 Wire Wire Line
@@
 	0    -1   1    0
 $EndComp
-Text GLabel 4425 2000 2    50   Input ~ 0
-LORA_TX
-Text GLabel 4425 2150 2    50   Input ~ 0
-LORA_RX
-$Comp
-L Connector:Conn_02x07_Odd_Even J?
+$Comp
+L Connector:Conn_02x07_Odd_Even J1
 U 1 1 619137D5
 P 7450 9525
-F 0 "J?" H 7500 9950 50  0000 C CNN
+F 0 "J1" H 7500 9950 50  0000 C CNN
 F 1 "Conn_02x07_Counter_Clockwise" H 7500 9951 50  0001 C CNN
 F 2 "" H 7450 9525 50  0001 C CNN
@@
 Text Label 1275 4350 0    50   ~ 0
 RE_485
+$Comp
+L OSM_env01-rescue:Test_Point-Connector-ESP32-EVB_Rev_D-rescue TP?
+U 1 1 614D8D9C
+P 1275 4650
+AR Path="/60688D25/614D8D9C" Ref="TP?"  Part="1"
+AR Path="/614D8D9C" Ref="TP16"  Part="1"
+F 0 "TP16" V 1275 4925 50  0000 C CNN
+F 1 "Test_Point" V 1379 4722 50  0001 C CNN
+F 2 "TestPoint:TestPoint_Pad_D1.0mm" H 1475 4650 50  0001 C CNN
+F 3 "~" H 1475 4650 50  0001 C CNN
+	1    1275 4650
+	0    -1   1    0
+$EndComp
+$Sheet
+S 7150 1325 1550 2500
+U 608F4675
+F0 "Sensors_AND_IO" 50
+F1 "Sensors_AND_IO.sch" 50
+F2 "HPM_RX" I L 7150 2675 50
+F3 "HPM_TX" I L 7150 2825 50
+F4 "HPM_EN" I L 7150 1500 50
+F5 "SCL" I L 7150 2300 50
+F6 "SDA" I L 7150 2150 50
+F7 "PULSE1_EXT" I L 7150 1650 50
+F8 "PULSE2_EXT" I L 7150 1800 50
+F9 "MIC_SD" I R 8700 3325 50
+F10 "MIC_SCK" I L 7150 3325 50
+F11 "MIC_WS" I L 7150 3475 50
+F12 "CT+" I R 8700 2675 50
+F13 "PULSE_IN1" I R 8700 1650 50
+F14 "PULSE_IN2" I R 8700 1800 50
+$EndSheet
+Text Label 4425 2000 2    50   ~ 0
+LORA_TX
+Text Label 4425 2150 2    50   ~ 0
+LORA_RX
+Wire Wire Line
+	15225 2000 15800 2000
+Wire Wire Line
+	15225 1725 15800 1725
+Text Label 15800 2000 2    50   ~ 0
+LORA_TX
+Text Label 15800 1725 2    50   ~ 0
+LORA_RX
 $EndSCHEMATC

Commit message: Updated schematics
Parts:
- removed C52, C53: 100nF, Capacitor_SMD:C_0402_1005Metric, symbol OSM_env01-rescue:C-device-ESP32-EVB_Rev_D-rescue
- J1: symbol Connector:Conn_02x07_Odd_Even -> Connector:Conn_02x07_Counter_Clockwise
Connections:
- net +3V3: now also C18.1, C19.2, C20.1, C21.1, C76.2, C78.2, J1.10 (Pin_10), J1.2 (Pin_2), J1.8 (Pin_8), J1.9 (Pin_9), J2.12 (Pin_12), J2.13 (Pin_13), J2.14 (Pin_14), J2.2 (Pin_2), J2.5 (Pin_5), J2.9 (Pin_9), TP9.1
- net ADC+GPIO: now also J1.11 (Pin_11); no longer J1.8 (Pin_8)
- net CS: now also J1.12 (Pin_12); no longer J1.6 (Pin_6)
- net STM1_RX: now also J1.6 (Pin_6); no longer J1.11 (Pin_11)
- net STM1_TX: now also J1.5 (Pin_5); no longer J1.9 (Pin_9)
- net STM_MISO: now also J1.7 (Pin_7); no longer J1.13 (Pin_13)
- net STM_MOSI: now also J1.14 (Pin_14); no longer J1.2 (Pin_2)
- net STM_SCK: now also J1.13 (Pin_13); no longer J1.4 (Pin_4)
- net STM_SCL: now also J1.3 (Pin_3); no longer J1.5 (Pin_5)
- net STM_SDA: now also J1.4 (Pin_4); no longer J1.7 (Pin_7)
- removed net +5V: J1.3 (Pin_3), J2.2 (Pin_2)
- removed net GND: C18.1, C19.2, C20.1, C21.1, C76.2, C78.2, J1.10 (Pin_10), J1.12 (Pin_12), J1.14 (Pin_14), J2.12 (Pin_12), J2.13 (Pin_13), J2.14 (Pin_14), J2.5 (Pin_5), J2.9 (Pin_9), TP9.1
Changed lines of the file:
@@
 Sheet 1 9
 Title "Open Smart Monitor"
-Date ""
-Rev "A"
-Comp "Devtank Ltd"
-Comment1 "www.devtank.co.uk"
+Date "2021-09-22"
+Rev "B"
+Comp "Devtank LTD"
+Comment1 "AB"
 Comment2 ""
 Comment3 ""
@@
 F0 "LORA" 50
 F1 "LORA.sch" 50
-F2 "LORA_NRST" I L 14100 1850 50
-F3 "LORA_RX" I R 15225 1725 50
-F4 "LORA_TX" I R 15225 2000 50
+F2 "LORA_RX" I R 15225 1725 50
+F3 "LORA_TX" I R 15225 2000 50
 $EndSheet
 Text Notes 6200 8325 0    118  ~ 24
@@
 Text Label 6550 2675 0    50   ~ 0
 HPM_RX
-Text Label 13700 1850 0    50   ~ 0
-LORA_NRST
-Wire Wire Line
-	14100 1850 13700 1850
 Wire Wire Line
 	13275 5875 12950 5875
@@
 Text Label 6550 1500 0    50   ~ 0
 HPM_EN
-Text Label 11000 1700 0    50   ~ 0
+Text Label 11000 1800 0    50   ~ 0
 CAN_L
-Text Label 11000 1925 0    50   ~ 0
+Text Label 11000 2025 0    50   ~ 0
 CAN_H
 Text Label 6550 3325 0    50   ~ 0
@@
 	2200 10000 2200 10425
 $Comp
-L OSM_env01-rescue:C-device-ESP32-EVB_Rev_D-rescue C52
-U 1 1 61C1510C
-P 3525 9400
-F 0 "C52" H 3640 9446 50  0000 L CNN
-F 1 "100nF" H 3640 9355 50  0000 L CNN
-F 2 "Capacitor_SMD:C_0402_1005Metric" H 3563 9250 50  0001 C CNN
-F 3 "" H 3525 9400 50  0001 C CNN
-	1    3525 9400
-	0    -1   -1   0
-$EndComp
-$Comp
-L OSM_env01-rescue:C-device-ESP32-EVB_Rev_D-rescue C53
-U 1 1 61C15112
-P 3925 9500
-F 0 "C53" H 4040 9546 50  0000 L CNN
-F 1 "100nF" H 4040 9455 50  0000 L CNN
-F 2 "Capacitor_SMD:C_0402_1005Metric" H 3963 9350 50  0001 C CNN
-F 3 "" H 3925 9500 50  0001 C CNN
-	1    3925 9500
-	0    -1   -1   0
-$EndComp
-$Comp
 L OSM_env01-rescue:GND-ESP32-EVB_Rev_D #PWR0104
 U 1 1 61C15118
@@
 Wire Wire Line
 	4450 9575 4450 9500
-Wire Wire Line
-	4075 9500 4200 9500
 Connection ~ 4200 9500
 Wire Wire Line
 	4200 9500 4450 9500
-Wire Wire Line
-	3675 9400 4200 9400
 Wire Wire Line
 	4200 9400 4200 9500
@@
 Connection ~ 3275 9400
 Wire Wire Line
-	3275 9400 3375 9400
-Wire Wire Line
 	3725 9500 3725 9100
 Connection ~ 3725 9500
-Wire Wire Line
-	3725 9500 3775 9500
 Text Label 7975 6600 2    50   ~ 0
 STM_WAKEUP
@@
 Wire Wire Line
 	3350 2950 3550 2950
-Text Label 11000 1525 0    50   ~ 0
+Text Label 11000 1575 0    50   ~ 0
 CAN_RS
 Text Label 1275 5100 0    50   ~ 0
@@
 Note: Low power mode selected through RS\n
 Wire Wire Line
-	11400 1525 11000 1525
+	11400 1575 11000 1575
 Text Label 12825 1925 2    50   ~ 0
 CAN_TX
@@
 	12425 1700 12825 1700
 Wire Wire Line
-	11400 1925 11000 1925
-Wire Wire Line
-	11400 1700 11000 1700
+	11400 2025 11000 2025
+Wire Wire Line
+	11400 1800 11000 1800
 $Sheet
 S 11400 1450 1025 725
@@
 F2 "CAN_RX" I R 12425 1700 50
 F3 "CAN_TX" I R 12425 1925 50
-F4 "CAN_L" I L 11400 1700 50
-F5 "CAN_H" I L 11400 1925 50
-F6 "CAN_RS" I L 11400 1525 50
+F4 "CAN_L" I L 11400 1800 50
+F5 "CAN_H" I L 11400 2025 50
+F6 "CAN_RS" I L 11400 1575 50
 $EndSheet
 Wire Notes Line
@@
 $EndComp
 $Comp
-L Connector:Conn_02x07_Odd_Even J1
+L Connector:Conn_02x07_Counter_Clockwise J1
 U 1 1 619137D5
 P 7450 9525
@@
 Text Label 15800 1725 2    50   ~ 0
 LORA_RX
+Wire Wire Line
+	3275 9400 4200 9400
+Wire Wire Line
+	3725 9500 4200 9500
 $EndSCHEMATC
