File: kicad_osm_env01/OSM_env01.sch (KiCad schematic (older format))
At the start: 43 parts, among them J1 Conn_02x07_Counter_Clockwise, J2 Conn_02x07_Counter_Clockwise

Commit message: rough throwdown of all parts
Parts:
- removed J2: Conn_02x07_Counter_Clockwise, Devtank_PCB_lib:Milligrid_878311420_14way, symbol Connector:Conn_02x07_Odd_Even
- added J2: DB9_Female_MountingHoles, Connector_Dsub:DSUB-9_Female_Horizontal_P2.77x2.84mm_EdgePinOffset7.70mm_Housed_MountingHolesOffset9.12mm, symbol Connector:DB9_Female_MountingHoles
- added R49: 0R, Resistor_SMD:R_0603_1608Metric, symbol device:R
- added R55: DNF, Resistor_SMD:R_0603_1608Metric, symbol device:R
- added TP31, TP32: Test_Point, TestPoint:TestPoint_Pad_D1.5mm, symbol OSM_env01-rescue:Test_Point-Connector-ESP32-EVB_Rev_D-rescue
- J1: footprint (none) -> Connector_PinSocket_2.54mm:PinSocket_2x07_P2.54mm_Vertical
- R1, R2: value 4.7K -> 4.7k; footprint Resistor_SMD:R_0402_1005Metric -> Resistor_SMD:R_0603_1608Metric
Connections:
- wire segments 156 -> 159
- no-connect marks 1 -> 0
Other:
- moved on the sheet: C18, C19, C20, C21, C76, C78

Commit message: schematics and layout submitted for review
Parts:
- TP31, TP32, TP72, TP8: footprint TestPoint:TestPoint_Pad_D1.5mm -> TestPoint:TestPoint_THTPad_D1.0mm_Drill0.5mm
Connections:
- net ADC+GPIO: now also J1.12 (Pin_12); no longer J1.11 (Pin_11)
- net CAN_H: now also C18.2, J2.9; no longer C20.2, J2.7
- net CAN_L: now also C19.1, J2.5; no longer C21.2, J2.3
- net CS: now also J1.4 (Pin_4); no longer J1.12 (Pin_12)
- net GND: now also J1.3 (Pin_3), J1.5 (Pin_5), J1.7 (Pin_7), J2.2, J2.8; no longer J1.10 (Pin_10), J1.8 (Pin_8), J1.9 (Pin_9), J2.5, J2.9
- net PULSE1_EXT: now also C21.2, J2.4; no longer C18.2, J2.8
- net PULSE2_EXT: now also C20.2, J2.3; no longer C19.1, J2.4
- net RS485+: now also C78.2, J2.7; no longer C76.2, J2.6
- net RS485-: now also C76.2, J2.6; no longer C78.2, J2.2
- net STM1_RX: now also J1.14 (Pin_14); no longer J1.6 (Pin_6)
- net STM1_TX: now also J1.13 (Pin_13); no longer J1.5 (Pin_5)
- net STM32L4/GPIO12: now also TP15.1; no longer TP10.1
- net STM32L4/GPIO13: now also TP10.1; no longer TP15.1
- net STM_MISO: now also J1.8 (Pin_8); no longer J1.7 (Pin_7)
- net STM_MOSI: now also J1.10 (Pin_10); no longer J1.14 (Pin_14)
- net STM_SCK: now also J1.6 (Pin_6); no longer J1.13 (Pin_13)
- net STM_SCL: now also J1.9 (Pin_9); no longer J1.3 (Pin_3)
- net STM_SDA: now also J1.11 (Pin_11); no longer J1.4 (Pin_4)
- net STM32L4/GPIO3 renamed STM32L4/GPIO2
- net STM32L4/GPIO5 renamed STM32L4/ADC8
Other:
- moved on the sheet: J2, TP10, TP15, TP17

Commit message: osm env-01 revB finished
Connections:
- net STM32L4/ADC1 renamed STM32L4/GPIO16
Other:
- moved on the sheet: TP3, TP53
Changed lines of the file:
@@
 Sheet 1 9
 Title "Open Smart Monitor"
-Date "2021-09-22"
+Date "2021-09-29"
 Rev "B"
 Comp "Devtank LTD"
-Comment1 "AB"
+Comment1 "Part No: 304-010"
 Comment2 ""
 Comment3 ""
@@
 F20 "GPIO4" I L 1875 3600 50
 F21 "GPIO6" I L 1875 3900 50
-F22 "ADC1" I L 1875 1850 50
-F23 "ADC2" I L 1875 2000 50
-F24 "ADC3" I L 1875 2150 50
-F25 "ADC4" I L 1875 2300 50
-F26 "ADC5" I L 1875 2450 50
-F27 "ADC6" I L 1875 2600 50
-F28 "LPUART1_RX" I R 3350 2800 50
-F29 "LPUART1_TX" I R 3350 2950 50
-F30 "UART4_RX" I R 3350 2400 50
-F31 "UART4_TX" I R 3350 2550 50
-F32 "WKUP2" I L 1875 1500 50
-F33 "SAI1_SCK_A" I R 3350 4700 50
-F34 "SAI1_FS_A" I R 3350 5000 50
-F35 "SAI1_SD_A" I R 3350 4850 50
-F36 "GPIO7" I L 1875 4050 50
-F37 "GPIO8" I L 1875 4200 50
-F38 "GPIO9" I L 1875 4350 50
-F39 "GPIO10" I L 1875 4500 50
-F40 "GPIO11" I L 1875 4650 50
-F41 "GPIO12" I L 1875 4800 50
-F42 "GPIO13" I L 1875 4950 50
-F43 "GPIO14" I L 1875 5100 50
-F44 "GPIO15" I L 1875 5250 50
-F45 "BOOT0" I L 1875 1350 50
-F46 "ADC7" I L 1875 2750 50
-F47 "ADC8" I L 1875 3750 50
+F22 "ADC2" I L 1875 2000 50
+F23 "ADC3" I L 1875 2150 50
+F24 "ADC4" I L 1875 2300 50
+F25 "ADC5" I L 1875 2450 50
+F26 "ADC6" I L 1875 2600 50
+F27 "LPUART1_RX" I R 3350 2800 50
+F28 "LPUART1_TX" I R 3350 2950 50
+F29 "UART4_RX" I R 3350 2400 50
+F30 "UART4_TX" I R 3350 2550 50
+F31 "WKUP2" I L 1875 1500 50
+F32 "SAI1_SCK_A" I R 3350 4700 50
+F33 "SAI1_FS_A" I R 3350 5000 50
+F34 "SAI1_SD_A" I R 3350 4850 50
+F35 "GPIO7" I L 1875 4050 50
+F36 "GPIO8" I L 1875 4200 50
+F37 "GPIO9" I L 1875 4350 50
+F38 "GPIO10" I L 1875 4500 50
+F39 "GPIO11" I L 1875 4650 50
+F40 "GPIO12" I L 1875 4800 50
+F41 "GPIO13" I L 1875 4950 50
+F42 "GPIO14" I L 1875 5100 50
+F43 "GPIO15" I L 1875 5250 50
+F44 "BOOT0" I L 1875 1350 50
+F45 "ADC7" I L 1875 2750 50
+F46 "ADC8" I L 1875 2900 50
+F47 "GPIO16" I L 1875 5400 50
 $EndSheet
 Wire Wire Line
@@
 	1275 3600 1875 3600
 Wire Wire Line
-	1275 3750 1875 3750
+	1275 2900 1875 2900
 Wire Wire Line
 	1275 4800 1875 4800
@@
 L OSM_env01-rescue:Test_Point-Connector-ESP32-EVB_Rev_D-rescue TP?
 U 1 1 61CAC847
-P 1275 3750
+P 1275 2900
 AR Path="/60688D25/61CAC847" Ref="TP?"  Part="1"
 AR Path="/61CAC847" Ref="TP3"  Part="1"
-F 0 "TP3" V 1275 4025 50  0000 C CNN
-F 1 "Test_Point" V 1379 3822 50  0001 C CNN
-F 2 "TestPoint:TestPoint_Pad_D1.0mm" H 1475 3750 50  0001 C CNN
-F 3 "~" H 1475 3750 50  0001 C CNN
-	1    1275 3750
+F 0 "TP3" V 1275 3175 50  0000 C CNN
+F 1 "Test_Point" V 1379 2972 50  0001 C CNN
+F 2 "TestPoint:TestPoint_Pad_D1.0mm" H 1475 2900 50  0001 C CNN
+F 3 "~" H 1475 2900 50  0001 C CNN
+	1    1275 2900
 	0    -1   1    0
 $EndComp
@@
 $EndComp
 Wire Wire Line
-	1275 1850 1875 1850
+	1275 5400 1875 5400
 $Comp
 L OSM_env01-rescue:Test_Point-Connector-ESP32-EVB_Rev_D-rescue TP?
 U 1 1 6178280E
-P 1275 1850
+P 1275 5400
 AR Path="/60688D25/6178280E" Ref="TP?"  Part="1"
 AR Path="/6178280E" Ref="TP53"  Part="1"
-F 0 "TP53" V 1275 2125 50  0000 C CNN
-F 1 "Test_Point" V 1379 1922 50  0001 C CNN
-F 2 "TestPoint:TestPoint_Pad_D1.0mm" H 1475 1850 50  0001 C CNN
-F 3 "~" H 1475 1850 50  0001 C CNN
-	1    1275 1850
+F 0 "TP53" V 1275 5675 50  0000 C CNN
+F 1 "Test_Point" V 1379 5472 50  0001 C CNN
+F 2 "TestPoint:TestPoint_Pad_D1.0mm" H 1475 5400 50  0001 C CNN
+F 3 "~" H 1475 5400 50  0001 C CNN
+	1    1275 5400
 	0    -1   1    0
 $EndComp

Commit message: updated folder
Parts:
- added D16: BAV99, Package_TO_SOT_SMD:SOT-23, symbol Diode:BAV99
Connections:
- net +3V3: now also D16.2 (K)
- net CT+: now also D16.3 (A), D16.3 (K)
- net GND: now also D16.1 (A)
Changed lines of the file:
@@
 Wire Wire Line
 	1875 2000 1125 2000
-Wire Wire Line
-	8700 2675 9300 2675
 Text Label 9300 2675 2    50   ~ 0
 CT+
@@
 Wire Wire Line
 	3175 10375 3525 10375
+$Comp
+L Diode:BAV99 D16
+U 1 1 615D7584
+P 9925 2900
+F 0 "D16" H 9925 3115 50  0000 C CNN
+F 1 "BAV99" H 9925 3024 50  0000 C CNN
+F 2 "Package_TO_SOT_SMD:SOT-23" H 9925 2750 50  0001 C CNN
+F 3 "www.nxp.com/documents/data_sheet/BAV99_SER.pdf" H 9925 3000 50  0001 C CNN
+	1    9925 2900
+	0    1    1    0
+$EndComp
+$Comp
+L Diode:BAV99 D16
+U 2 1 615D798D
+P 9925 2450
+F 0 "D16" H 9925 2665 50  0000 C CNN
+F 1 "BAV99" H 9925 2574 50  0000 C CNN
+F 2 "Package_TO_SOT_SMD:SOT-23" H 9925 2300 50  0001 C CNN
+F 3 "www.nxp.com/documents/data_sheet/BAV99_SER.pdf" H 9925 2550 50  0001 C CNN
+	2    9925 2450
+	0    1    1    0
+$EndComp
+$Comp
+L power:+3V3 #PWR0104
+U 1 1 615FB753
+P 9925 2200
+F 0 "#PWR0104" H 9925 2050 50  0001 C CNN
+F 1 "+3V3" H 9940 2373 50  0000 C CNN
+F 2 "" H 9925 2200 50  0001 C CNN
+F 3 "" H 9925 2200 50  0001 C CNN
+	1    9925 2200
+	1    0    0    -1
+$EndComp
+$Comp
+L OSM_env01:GND #PWR0154
+U 1 1 615FBE5E
+P 9925 3125
+F 0 "#PWR0154" H 9925 2875 50  0001 C CNN
+F 1 "GND" H 9930 2952 50  0000 C CNN
+F 2 "" H 9925 3125 60  0000 C CNN
+F 3 "" H 9925 3125 60  0000 C CNN
+	1    9925 3125
+	1    0    0    -1
+$EndComp
+Wire Wire Line
+	9925 2675 9925 2600
+Wire Wire Line
+	8700 2675 9925 2675
+Wire Wire Line
+	9925 2675 9925 2750
+Connection ~ 9925 2675
+Wire Wire Line
+	9925 2300 9925 2200
+Wire Wire Line
+	9925 3125 9925 3050
 $EndSCHEMATC
