File: kicad_osm_env01/Sound.sch (KiCad schematic (older format))
At the start: 39 parts, among them U11 LMV324

Commit message: audio circuit updated
Parts:
- removed C35, C37: 1.0uF, Capacitor_SMD:C_0603_1608Metric, symbol OSM_env01-rescue:C-device-ESP32-EVB_Rev_D-rescue
- removed C36: 10uF, Capacitor_SMD:C_0603_1608Metric, symbol OSM_env01-rescue:C-device-ESP32-EVB_Rev_D-rescue
- removed D4, D5: RB751, Diode_SMD:D_SOD-523, symbol OSM_env01-rescue:D_Zener-device-ESP32-EVB_Rev_D-rescue
- removed D6: LED, LED_SMD:LED_0603_1608Metric, symbol OSM_env01-rescue:LED-device-ESP32-EVB_Rev_D-rescue
- removed JP1: Jumper_NC_Small, Connector_PinHeader_1.27mm:PinHeader_1x02_P1.27mm_Vertical, symbol OSM_env01-rescue:Jumper_NC_Small-device-ESP32-EVB_Rev_D-rescue
- removed R37, R40: 10K, Resistor_SMD:R_0603_1608Metric, symbol OSM_env01-rescue:R-device-ESP32-EVB_Rev_D-rescue
- removed R38: 22K, Resistor_SMD:R_0603_1608Metric, symbol OSM_env01-rescue:R-device-ESP32-EVB_Rev_D-rescue
- removed R39, R42, R54: 100R, Resistor_SMD:R_0603_1608Metric, symbol OSM_env01-rescue:R-device-ESP32-EVB_Rev_D-rescue
- removed R41, R43: 1K, Resistor_SMD:R_0603_1608Metric, symbol OSM_env01-rescue:R-device-ESP32-EVB_Rev_D-rescue
- removed R44, R46: 100K, Resistor_SMD:R_0603_1608Metric, symbol OSM_env01-rescue:R-device-ESP32-EVB_Rev_D-rescue
- removed R45: 3.3K, Resistor_SMD:R_0603_1608Metric, symbol OSM_env01-rescue:R-device-ESP32-EVB_Rev_D-rescue
- removed R47: 2.2K, Resistor_SMD:R_0603_1608Metric, symbol OSM_env01-rescue:R-device-ESP32-EVB_Rev_D-rescue
- removed TP39, TP40, TP41, TP42, TP43, TP44: Test_Point, TestPoint:TestPoint_THTPad_D1.0mm_Drill0.5mm, symbol OSM_env01-rescue:Test_Point-Connector-ESP32-EVB_Rev_D-rescue
- removed unit 4 of U11
- removed unit 3 of U11
- added C? (x2): 100nF, symbol device:C
- added C?: DNF, symbol device:C
- added C? (x2): 10nF, symbol OSM_env01-rescue:C-device-ESP32-EVB_Rev_D-rescue
- added D?: LM4040DEX3-3.3+T, TO_SOT_Packages_SMD:SOT-23, symbol references:LM4040DBZ-3
- added L?: Ferrite_Bead, symbol device:Ferrite_Bead
- added R?: 820R, symbol device:R
- added R?: 18k, Resistor_SMD:R_0603_1608Metric, symbol OSM_env01-rescue:R-device-ESP32-EVB_Rev_D-rescue
- added R?: 1k, Resistor_SMD:R_0603_1608Metric, symbol OSM_env01-rescue:R-device-ESP32-EVB_Rev_D-rescue
- added R?: DNF, Resistor_SMD:R_0603_1608Metric, symbol OSM_env01-rescue:R-device-ESP32-EVB_Rev_D-rescue
- added SW?: SW_SPST, symbol Switch:SW_SPST
- added TP?: Test_Point, symbol Connector:Test_Point
- C? (x2): value 20nF -> 10nF
- R35: value 39K -> 20k
Connections:
- net labels added: +5V, 3V3_AN, 3V3_ref
- net labels removed: Envelope, Gate
- wire segments 99 -> 75
Other:
- note added: "R=Vs/I\n5-3.3/2mA=850mA\nR=820R"
- note added: "amp1gain=rf/rin=20\namp2gain=1+rf/rin= 19-1=18k/1k ampgain2=19\nTotalgain=39"
- moved on the sheet: C34, C?, Mic1, R30, R31, R32, R33, R34, R35, R36, TP37, TP38

Commit message: pushed latest schematics got started with micro into schematic
Parts:
- renumbered C34 to C?, Mic1 to Mic?, R34 to R?, R36 to R?, R31 to R?, R35 to R?, R33 to R?, R32 to R?, R30 to R?, U11 to U?
Changed lines of the file:
@@
 $Descr A4 11693 8268
 encoding utf-8
-Sheet 4 4
+Sheet 4 8
 Title "Open Smart Monitor"
 Date ""
@@
 	5425 3900 5750 3900
 $Comp
-L OSM_env01-rescue:R-device-ESP32-EVB_Rev_D-rescue R34
+L OSM_env01-rescue:R-device-ESP32-EVB_Rev_D-rescue R?
 U 1 1 5E1A0EBB
 P 5275 3900
-F 0 "R34" V 5125 3900 50  0000 C CNN
+F 0 "R?" V 5125 3900 50  0000 C CNN
 F 1 "DNF" V 5200 3900 50  0000 C CNN
 F 2 "Resistor_SMD:R_0603_1608Metric" V 5205 3900 50  0001 C CNN
@@
 	7050 4950 7025 4950
 $Comp
-L OSM_env01-rescue:R-device-ESP32-EVB_Rev_D-rescue R36
+L OSM_env01-rescue:R-device-ESP32-EVB_Rev_D-rescue R?
 U 1 1 5E1A0EFD
 P 7200 4950
-F 0 "R36" V 7050 4925 50  0000 C CNN
+F 0 "R?" V 7050 4925 50  0000 C CNN
 F 1 "100R" V 7125 4950 50  0000 C CNN
 F 2 "Resistor_SMD:R_0603_1608Metric" V 7130 4950 50  0001 C CNN
@@
 	5125 4150 4850 4150
 $Comp
-L OSM_env01-rescue:R-device-ESP32-EVB_Rev_D-rescue R31
+L OSM_env01-rescue:R-device-ESP32-EVB_Rev_D-rescue R?
 U 1 1 5E1A0F57
 P 3375 4750
-F 0 "R31" V 3168 4750 50  0000 C CNN
+F 0 "R?" V 3168 4750 50  0000 C CNN
 F 1 "1K" V 3259 4750 50  0000 C CNN
 F 2 "Resistor_SMD:R_0603_1608Metric" V 3305 4750 50  0001 C CNN
@@
 $EndComp
 $Comp
-L OSM_env01-rescue:R-device-ESP32-EVB_Rev_D-rescue R35
+L OSM_env01-rescue:R-device-ESP32-EVB_Rev_D-rescue R?
 U 1 1 5E1A0F5D
 P 5275 4150
-F 0 "R35" V 5125 4150 50  0000 C CNN
+F 0 "R?" V 5125 4150 50  0000 C CNN
 F 1 "20k" V 5200 4150 50  0000 C CNN
 F 2 "Resistor_SMD:R_0603_1608Metric" V 5205 4150 50  0001 C CNN
@@
 	5150 5325 5150 5150
 $Comp
-L power:GND #PWR0149
+L power:GND #PWR?
 U 1 1 5E1A0F6C
 P 5150 5325
-F 0 "#PWR0149" H 5150 5075 50  0001 C CNN
+F 0 "#PWR?" H 5150 5075 50  0001 C CNN
 F 1 "GND" H 5155 5152 50  0000 C CNN
 F 2 "" H 5150 5325 50  0001 C CNN
@@
 	3600 5350 3600 5325
 $Comp
-L power:GND #PWR0150
+L power:GND #PWR?
 U 1 1 5E1A0F76
 P 3600 5350
-F 0 "#PWR0150" H 3600 5100 50  0001 C CNN
+F 0 "#PWR?" H 3600 5100 50  0001 C CNN
 F 1 "GND" H 3605 5177 50  0000 C CNN
 F 2 "" H 3600 5350 50  0001 C CNN
@@
 	3600 4725 3600 4950
 $Comp
-L OSM_env01-rescue:R-device-ESP32-EVB_Rev_D-rescue R33
+L OSM_env01-rescue:R-device-ESP32-EVB_Rev_D-rescue R?
 U 1 1 5E1A0F7D
 P 3600 5175
-F 0 "R33" H 3530 5129 50  0000 R CNN
+F 0 "R?" H 3530 5129 50  0000 R CNN
 F 1 "10K" H 3530 5220 50  0000 R CNN
 F 2 "Resistor_SMD:R_0603_1608Metric" V 3530 5175 50  0001 C CNN
@@
 $EndComp
 $Comp
-L OSM_env01-rescue:R-device-ESP32-EVB_Rev_D-rescue R32
+L OSM_env01-rescue:R-device-ESP32-EVB_Rev_D-rescue R?
 U 1 1 5E1A0F83
 P 3600 4575
-F 0 "R32" H 3530 4529 50  0000 R CNN
+F 0 "R?" H 3530 4529 50  0000 R CNN
 F 1 "10K" H 3530 4620 50  0000 R CNN
 F 2 "Resistor_SMD:R_0603_1608Metric" V 3530 4575 50  0001 C CNN
@@
 $EndComp
 $Comp
-L power:GND #PWR0151
+L power:GND #PWR?
 U 1 1 5E1A0F89
 P 2575 5375
-F 0 "#PWR0151" H 2575 5125 50  0001 C CNN
+F 0 "#PWR?" H 2575 5125 50  0001 C CNN
 F 1 "GND" H 2580 5202 50  0000 C CNN
 F 2 "" H 2575 5375 50  0001 C CNN
@@
 	3150 4750 3225 4750
 $Comp
-L OSM_env01-rescue:C-device-ESP32-EVB_Rev_D-rescue C34
+L OSM_env01-rescue:C-device-ESP32-EVB_Rev_D-rescue C?
 U 1 1 5E1A0F91
 P 3000 4750
-F 0 "C34" V 2748 4750 50  0000 C CNN
+F 0 "C?" V 2748 4750 50  0000 C CNN
 F 1 "10uF" V 2839 4750 50  0000 C CNN
 F 2 "Capacitor_SMD:C_0603_1608Metric" H 3038 4600 50  0001 C CNN
@@
 	2575 4400 2575 4275
 $Comp
-L OSM_env01-rescue:R-device-ESP32-EVB_Rev_D-rescue R30
+L OSM_env01-rescue:R-device-ESP32-EVB_Rev_D-rescue R?
 U 1 1 5E1A0F9B
 P 2575 4550
-F 0 "R30" H 2645 4596 50  0000 L CNN
+F 0 "R?" H 2645 4596 50  0000 L CNN
 F 1 "2.2K" H 2645 4505 50  0000 L CNN
 F 2 "Resistor_SMD:R_0603_1608Metric" V 2505 4550 50  0001 C CNN
@@
 	2575 4800 2575 4750
 $Comp
-L OSM_env01-rescue:Microphone_Condenser-device-ESP32-EVB_Rev_D-rescue Mic1
+L OSM_env01-rescue:Microphone_Condenser-device-ESP32-EVB_Rev_D-rescue Mic?
 U 1 1 5E1A0FA3
 P 2575 5000
-F 0 "Mic1" V 2325 5000 50  0000 L CNN
+F 0 "Mic?" V 2325 5000 50  0000 L CNN
 F 1 "DNF" V 2400 4650 50  0000 L CNN
 F 2 "Capacitor_SMD:C_1210_3225Metric" V 2575 5100 50  0001 C CNN
@@
 $EndComp
 $Comp
-L OSM_env01-rescue:LMV324-linear-ESP32-EVB_Rev_D-rescue U11
+L OSM_env01-rescue:LMV324-linear-ESP32-EVB_Rev_D-rescue U?
 U 1 1 5E1A9DFD
 P 5250 4850
-F 0 "U11" H 5250 5025 50  0000 L CNN
+F 0 "U?" H 5250 5025 50  0000 L CNN
 F 1 "LMV324" H 5250 5100 50  0000 L CNN
 F 2 "Package_SO:SOIC-14_3.9x8.7mm_P1.27mm" H 5200 4950 50  0001 C CNN
@@
 $EndComp
 $Comp
-L OSM_env01-rescue:LMV324-linear-ESP32-EVB_Rev_D-rescue U11
+L OSM_env01-rescue:LMV324-linear-ESP32-EVB_Rev_D-rescue U?
 U 2 1 5E1BC702
 P 6500 4950
-F 0 "U11" H 6450 5125 50  0000 L CNN
+F 0 "U?" H 6450 5125 50  0000 L CNN
 F 1 "LMV324" H 6450 5200 50  0000 L CNN
 F 2 "Package_SO:SOIC-14_3.9x8.7mm_P1.27mm" H 6450 5050 50  0001 C CNN
@@
 Audio
 $Comp
-L power:+3V3 #PWR09
+L power:+3V3 #PWR?
 U 1 1 5E1E12E8
 P 6425 1400
-F 0 "#PWR09" H 6425 1250 50  0001 C CNN
+F 0 "#PWR?" H 6425 1250 50  0001 C CNN
 F 1 "+3V3" H 6275 1475 50  0000 C CNN
 F 2 "" H 6425 1400 50  0001 C CNN
@@
 AR Path="/5E3B4FEF" Ref="TP?"  Part="1"
 AR Path="/5E19E083/5E3B4FEF" Ref="TP37"  Part="1"
-F 0 "TP37" H 4750 3875 50  0000 C CNN
+F 0 "TP?" H 4750 3875 50  0000 C CNN
 F 1 "Test_Point" H 4850 3775 50  0000 C CNN
 F 2 "TestPoint:TestPoint_THTPad_D1.0mm_Drill0.5mm" H 5050 3550 50  0001 C CNN
@@
 AR Path="/5E3B7A56" Ref="TP?"  Part="1"
 AR Path="/5E19E083/5E3B7A56" Ref="TP38"  Part="1"
-F 0 "TP38" V 5945 3622 50  0000 C CNN
+F 0 "TP?" V 5945 3622 50  0000 C CNN
 F 1 "Test_Point" V 5854 3622 50  0000 C CNN
 F 2 "TestPoint:TestPoint_THTPad_D1.0mm_Drill0.5mm" H 5950 3550 50  0001 C CNN

Commit message: updated schematics
Parts:
- removed C? (x2): 100nF, symbol device:C
- removed D?: LM4040DEX3-3.3+T, TO_SOT_Packages_SMD:SOT-23, symbol references:LM4040DBZ-3
- removed L?: Ferrite_Bead, symbol device:Ferrite_Bead
- removed R?: 820R, symbol device:R
- removed TP?: Test_Point, symbol Connector:Test_Point
- removed U? (x2): LMV324, Package_SO:SOIC-14_3.9x8.7mm_P1.27mm, symbol OSM_env01-rescue:LMV324-linear-ESP32-EVB_Rev_D-rescue
- added C52, C53, C54, C55: 10nF, symbol OSM_env01-rescue:C-device-ESP32-EVB_Rev_D-rescue
- added C56: DNF, symbol device:C
- added C57: C, symbol device:C
- added R116: R, symbol device:R
- added TP56, TP57: Test_Point, symbol Connector:Test_Point
- added U14: OPA1678IDG, symbol linear:OP249
- gave numbers to parts that had none: 18
Connections:
- net labels added: +3V3_A, +5VA, 5V_A, GNDA, GND_A
- net labels removed: +3V3, +5V, 3V3_AN, 3V3_ref, GND
- wire segments 75 -> 86
Other:
- note added: "Fc=1/2xpiXRXC"
- note added: "low pass filter"
- note removed: "R=Vs/I\n5-3.3/2mA=850mA\nR=820R"
- moved on the sheet: C46, C47, C48, C49, C50, C51, Mic1, R106, R107, R108, R109, R110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

Commit message: schematics awaiting review
Parts:
- added TP83, TP84, TP87: Test_Point, symbol Connector:Test_Point
Connections:
- net +5VA is gone; now on net +3V3_A: U14.8 (V+), U14.8 (V+)
- net +3V3_A: now also TP83.1, TP87.1
- net GNDA: now also TP84.1
- net MIC_IN: now reaches C46.2, Mic1.2 (+), R106.2, SW4.2 (B)
Changed lines of the file:
@@
 AR Path="/5E19E083/5E3B4FEF" Ref="TP37"  Part="1"
 AR Path="/608F4675/60959880/5E3B4FEF" Ref="TP54"  Part="1"
-F 0 "TP54" H 4825 2575 50  0000 C CNN
-F 1 "Test_Point" H 4925 2475 50  0000 C CNN
+F 0 "TP54" H 4925 2475 50  0000 C CNN
+F 1 "Test_Point" H 4925 2475 50  0001 C CNN
 F 2 "TestPoint:TestPoint_THTPad_D1.0mm_Drill0.5mm" H 5125 2250 50  0001 C CNN
 F 3 "~" H 5125 2250 50  0001 C CNN
@@
 AR Path="/5E19E083/5E3B7A56" Ref="TP38"  Part="1"
 AR Path="/608F4675/60959880/5E3B7A56" Ref="TP55"  Part="1"
-F 0 "TP55" V 6020 2322 50  0000 C CNN
-F 1 "Test_Point" V 5929 2322 50  0000 C CNN
+F 0 "TP55" H 5825 2475 50  0000 C CNN
+F 1 "Test_Point" V 5929 2322 50  0001 C CNN
 F 2 "TestPoint:TestPoint_THTPad_D1.0mm_Drill0.5mm" H 6025 2250 50  0001 C CNN
 F 3 "~" H 6025 2250 50  0001 C CNN
@@
 U 1 1 612E07DC
 P 9150 3275
-F 0 "TP57" H 9208 3393 50  0000 L CNN
-F 1 "Test_Point" H 9208 3302 50  0000 L CNN
+F 0 "TP57" H 9075 3500 50  0000 L CNN
+F 1 "Test_Point" H 9208 3302 50  0001 L CNN
 F 2 "" H 9350 3275 50  0001 C CNN
 F 3 "~" H 9350 3275 50  0001 C CNN
@@
 U 1 1 612E198E
 P 8175 3300
-F 0 "TP56" H 8233 3418 50  0000 L CNN
-F 1 "Test_Point" H 8233 3327 50  0000 L CNN
+F 0 "TP56" H 8075 3525 50  0000 L CNN
+F 1 "Test_Point" H 8233 3327 50  0001 L CNN
 F 2 "" H 8375 3300 50  0001 C CNN
 F 3 "~" H 8375 3300 50  0001 C CNN
@@
 Text Notes 8850 4925 0    50   ~ 0
 Fc=1/2xpiXRXC
-$Comp
-L power:PWR_FLAG #FLG0102
-U 1 1 614DA96A
-P 725 825
-F 0 "#FLG0102" H 725 900 50  0001 C CNN
-F 1 "PWR_FLAG" H 725 998 50  0000 C CNN
-F 2 "" H 725 825 50  0001 C CNN
-F 3 "" H 725 825 50  0001 C CNN
-	1    725  825
-	1    0    0    -1
-$EndComp
 $Comp
 L power:PWR_FLAG #FLG0103
@@
 $EndComp
 Wire Wire Line
-	725  825  725  975
-Wire Wire Line
-	725  975  1125 975
-Connection ~ 1125 975
-Wire Wire Line
 	1850 825  2075 825
 Connection ~ 2075 825
+$Comp
+L Connector:Test_Point TP83
+U 1 1 60785772
+P 1375 975
+F 0 "TP83" V 1375 1150 50  0000 L CNN
+F 1 "Test_Point" H 1433 1002 50  0001 L CNN
+F 2 "" H 1575 975 50  0001 C CNN
+F 3 "~" H 1575 975 50  0001 C CNN
+	1    1375 975
+	0    1    1    0
+$EndComp
+$Comp
+L Connector:Test_Point TP84
+U 1 1 607878CE
+P 2300 825
+F 0 "TP84" V 2300 1025 50  0000 L CNN
+F 1 "Test_Point" H 2358 852 50  0001 L CNN
+F 2 "" H 2500 825 50  0001 C CNN
+F 3 "~" H 2500 825 50  0001 C CNN
+	1    2300 825
+	0    1    1    0
+$EndComp
+Text HLabel 1625 3450 0    50   Input ~ 0
+MIC_IN
+Wire Wire Line
+	1875 3450 1625 3450
+Connection ~ 1875 3450
+$Comp
+L Devtank:+3V3_A #PWR0133
+U 1 1 60D990F9
+P 1275 1775
+F 0 "#PWR0133" H 1275 1625 50  0001 C CNN
+F 1 "+3V3_A" H 1290 1948 50  0000 C CNN
+F 2 "" H 1275 1775 50  0000 C CNN
+F 3 "" H 1275 1775 50  0000 C CNN
+	1    1275 1775
+	1    0    0    -1
+$EndComp
+Wire Wire Line
+	1275 1925 1275 1775
+Wire Wire Line
+	1275 1925 1525 1925
+Text Label 1525 1925 2    50   ~ 0
+5V_A
+$Comp
+L Connector:Test_Point TP87
+U 1 1 60D9B3F1
+P 1525 1925
+F 0 "TP87" V 1525 2100 50  0000 L CNN
+F 1 "Test_Point" H 1583 1952 50  0001 L CNN
+F 2 "" H 1725 1925 50  0001 C CNN
+F 3 "~" H 1725 1925 50  0001 C CNN
+	1    1525 1925
+	0    1    1    0
+$EndComp
+Wire Wire Line
+	725  975  1125 975
+Wire Wire Line
+	725  825  725  975
+$Comp
+L power:PWR_FLAG #FLG02
+U 1 1 60D9B3E8
+P 725 825
+F 0 "#FLG02" H 725 900 50  0001 C CNN
+F 1 "PWR_FLAG" H 725 998 50  0000 C CNN
+F 2 "" H 725 825 50  0001 C CNN
+F 3 "" H 725 825 50  0001 C CNN
+	1    725  825
+	1    0    0    -1
+$EndComp
+Connection ~ 1125 975
 $EndSCHEMATC

Commit message: updated schematics
Parts:
- C47, C48, C49, C50, C51, C52, C53, C54, C55, C56: footprint (none) -> Capacitor_SMD:C_0603_1608Metric
- C57: footprint (none) -> Capacitor_SMD:C_0805_2012Metric
- R116: footprint (none) -> Resistor_SMD:R_0805_2012Metric
- TP56, TP57, TP83, TP84, TP87: footprint (none) -> TestPoint:TestPoint_THTPad_D1.0mm_Drill0.5mm
- U14: footprint (none) -> Package_SO:VSSOP-8_3.0x3.0mm_P0.65mm
Changed lines of the file:
@@
 $Descr A4 11693 8268
 encoding utf-8
-Sheet 9 11
+Sheet 9 12
 Title "Open Smart Monitor"
 Date ""
@@
 F 0 "C49" H 4640 3321 50  0000 L CNN
 F 1 "10nF" H 4640 3230 50  0000 L CNN
-F 2 "" H 4563 3125 50  0001 C CNN
+F 2 "Capacitor_SMD:C_0603_1608Metric" H 4563 3125 50  0001 C CNN
 F 3 "" H 4525 3275 50  0001 C CNN
 	1    4525 3275
@@
 F 0 "C50" H 4640 3846 50  0000 L CNN
 F 1 "10nF" H 4640 3755 50  0000 L CNN
-F 2 "" H 4563 3650 50  0001 C CNN
+F 2 "Capacitor_SMD:C_0603_1608Metric" H 4563 3650 50  0001 C CNN
 F 3 "" H 4525 3800 50  0001 C CNN
 	1    4525 3800
@@
 F 0 "C47" H 4215 3321 50  0000 L CNN
 F 1 "10nF" H 4215 3230 50  0000 L CNN
-F 2 "" H 4138 3125 50  0001 C CNN
+F 2 "Capacitor_SMD:C_0603_1608Metric" H 4138 3125 50  0001 C CNN
 F 3 "" H 4100 3275 50  0001 C CNN
 	1    4100 3275
@@
 F 0 "C48" H 4215 3846 50  0000 L CNN
 F 1 "10nF" H 4215 3755 50  0000 L CNN
-F 2 "" H 4138 3650 50  0001 C CNN
+F 2 "Capacitor_SMD:C_0603_1608Metric" H 4138 3650 50  0001 C CNN
 F 3 "" H 4100 3800 50  0001 C CNN
 	1    4100 3800
@@
 F 0 "C51" V 5098 2250 50  0000 C CNN
 F 1 "DNF" V 5189 2250 50  0000 C CNN
-F 2 "" H 5388 2100 50  0001 C CNN
+F 2 "Capacitor_SMD:C_0603_1608Metric" H 5388 2100 50  0001 C CNN
 F 3 "" H 5350 2250 50  0001 C CNN
 	1    5350 2250
@@
 F 0 "U14" H 5150 3975 50  0000 C CNN
 F 1 "OPA1678IDG" H 5300 4075 50  0000 C CNN
-F 2 "" H 5325 3550 50  0001 C CNN
+F 2 "Package_SO:VSSOP-8_3.0x3.0mm_P0.65mm" H 5325 3550 50  0001 C CNN
 F 3 "http://www.analog.com/media/en/technical-documentation/data-sheets/OP249.pdf" H 5325 3550 50  0001 C CNN
 	1    5325 3550
@@
 F 0 "U14" H 7450 4250 50  0000 L CNN
 F 1 "OPA1678IDG" H 7450 4150 50  0000 L CNN
-F 2 "" H 7700 3650 50  0001 C CNN
+F 2 "Package_SO:VSSOP-8_3.0x3.0mm_P0.65mm" H 7700 3650 50  0001 C CNN
 F 3 "http://www.analog.com/media/en/technical-documentation/data-sheets/OP249.pdf" H 7700 3650 50  0001 C CNN
 	2    7700 3650
@@
 F 0 "R116" H 8920 3696 50  0000 L CNN
 F 1 "R" H 8920 3605 50  0000 L CNN
-F 2 "" V 8780 3650 50  0001 C CNN
+F 2 "Resistor_SMD:R_0805_2012Metric" V 8780 3650 50  0001 C CNN
 F 3 "" H 8850 3650 50  0001 C CNN
 	1    8850 3650
@@
 F 0 "C57" H 9265 3921 50  0000 L CNN
 F 1 "C" H 9265 3830 50  0000 L CNN
-F 2 "" H 9188 3725 50  0001 C CNN
+F 2 "Capacitor_SMD:C_0805_2012Metric" H 9188 3725 50  0001 C CNN
 F 3 "" H 9150 3875 50  0001 C CNN
 	1    9150 3875
@@
 F 0 "C54" H 6865 3421 50  0000 L CNN
 F 1 "10nF" H 6865 3330 50  0000 L CNN
-F 2 "" H 6788 3225 50  0001 C CNN
+F 2 "Capacitor_SMD:C_0603_1608Metric" H 6788 3225 50  0001 C CNN
 F 3 "" H 6750 3375 50  0001 C CNN
 	1    6750 3375
@@
 F 0 "C55" H 6865 3946 50  0000 L CNN
 F 1 "10nF" H 6865 3855 50  0000 L CNN
-F 2 "" H 6788 3750 50  0001 C CNN
+F 2 "Capacitor_SMD:C_0603_1608Metric" H 6788 3750 50  0001 C CNN
 F 3 "" H 6750 3900 50  0001 C CNN
 	1    6750 3900
@@
 F 0 "C52" H 6440 3421 50  0000 L CNN
 F 1 "10nF" H 6440 3330 50  0000 L CNN
-F 2 "" H 6363 3225 50  0001 C CNN
+F 2 "Capacitor_SMD:C_0603_1608Metric" H 6363 3225 50  0001 C CNN
 F 3 "" H 6325 3375 50  0001 C CNN
 	1    6325 3375
@@
 F 0 "C53" H 6440 3946 50  0000 L CNN
 F 1 "10nF" H 6440 3855 50  0000 L CNN
-F 2 "" H 6363 3750 50  0001 C CNN
+F 2 "Capacitor_SMD:C_0603_1608Metric" H 6363 3750 50  0001 C CNN
 F 3 "" H 6325 3900 50  0001 C CNN
 	1    6325 3900
@@
 F 0 "C56" V 7423 4900 50  0000 C CNN
 F 1 "DNF" V 7514 4900 50  0000 C CNN
-F 2 "" H 7713 4750 50  0001 C CNN
+F 2 "Capacitor_SMD:C_0603_1608Metric" H 7713 4750 50  0001 C CNN
 F 3 "" H 7675 4900 50  0001 C CNN
 	1    7675 4900
@@
 F 0 "TP57" H 9075 3500 50  0000 L CNN
 F 1 "Test_Point" H 9208 3302 50  0001 L CNN
-F 2 "" H 9350 3275 50  0001 C CNN
+F 2 "TestPoint:TestPoint_THTPad_D1.0mm_Drill0.5mm" H 9350 3275 50  0001 C CNN
 F 3 "~" H 9350 3275 50  0001 C CNN
 	1    9150 3275
@@
 F 0 "TP56" H 8075 3525 50  0000 L CNN
 F 1 "Test_Point" H 8233 3327 50  0001 L CNN
-F 2 "" H 8375 3300 50  0001 C CNN
+F 2 "TestPoint:TestPoint_THTPad_D1.0mm_Drill0.5mm" H 8375 3300 50  0001 C CNN
 F 3 "~" H 8375 3300 50  0001 C CNN
 	1    8175 3300
@@
 F 0 "TP83" V 1375 1150 50  0000 L CNN
 F 1 "Test_Point" H 1433 1002 50  0001 L CNN
-F 2 "" H 1575 975 50  0001 C CNN
+F 2 "TestPoint:TestPoint_THTPad_D1.0mm_Drill0.5mm" H 1575 975 50  0001 C CNN
 F 3 "~" H 1575 975 50  0001 C CNN
 	1    1375 975
@@
 F 0 "TP84" V 2300 1025 50  0000 L CNN
 F 1 "Test_Point" H 2358 852 50  0001 L CNN
-F 2 "" H 2500 825 50  0001 C CNN
+F 2 "TestPoint:TestPoint_THTPad_D1.0mm_Drill0.5mm" H 2500 825 50  0001 C CNN
 F 3 "~" H 2500 825 50  0001 C CNN
 	1    2300 825
@@
 F 0 "TP87" V 1525 2100 50  0000 L CNN
 F 1 "Test_Point" H 1583 1952 50  0001 L CNN
-F 2 "" H 1725 1925 50  0001 C CNN
+F 2 "TestPoint:TestPoint_THTPad_D1.0mm_Drill0.5mm" H 1725 1925 50  0001 C CNN
 F 3 "~" H 1725 1925 50  0001 C CNN
 	1    1525 1925

Commit message: started layout
Parts:
- added C74: 100nF, Capacitor_SMD:C_0603_1608Metric, symbol OSM_env01-rescue:C-device-ESP32-EVB_Rev_D-rescue
- SW4: footprint (none) -> Button_Switch_SMD:SW_DIP_SPSTx01_Slide_6.7x4.1mm_W6.73mm_P2.54mm_LowProfile_JPin
- U14: footprint Package_SO:VSSOP-8_3.0x3.0mm_P0.65mm -> Package_SO:SOIC-8_3.9x4.9mm_P1.27mm
Connections:
- net +3V3_A: no longer TP83.1, U14.8 (V+), U14.8 (V+)
- net GNDA: now also C74.1
- new net +5VA: C74.2, TP83.1, U14.8 (V+), U14.8 (V+)
Other:
- moved on the sheet: TP87
Changed lines of the file:
@@
 $Descr A4 11693 8268
 encoding utf-8
-Sheet 9 12
+Sheet 9 11
 Title "Open Smart Monitor"
 Date ""
@@
 F 0 "SW4" V 1921 3612 50  0000 R CNN
 F 1 "SW_SPST" V 1830 3612 50  0000 R CNN
-F 2 "" H 1875 3700 50  0001 C CNN
+F 2 "Button_Switch_SMD:SW_DIP_SPSTx01_Slide_6.7x4.1mm_W6.73mm_P2.54mm_LowProfile_JPin" H 1875 3700 50  0001 C CNN
 F 3 "" H 1875 3700 50  0001 C CNN
 	1    1875 3700
@@
 F 0 "U14" H 5150 3975 50  0000 C CNN
 F 1 "OPA1678IDG" H 5300 4075 50  0000 C CNN
-F 2 "Package_SO:VSSOP-8_3.0x3.0mm_P0.65mm" H 5325 3550 50  0001 C CNN
+F 2 "Package_SO:SOIC-8_3.9x4.9mm_P1.27mm" H 5325 3550 50  0001 C CNN
 F 3 "http://www.analog.com/media/en/technical-documentation/data-sheets/OP249.pdf" H 5325 3550 50  0001 C CNN
 	1    5325 3550
@@
 F 0 "U14" H 7450 4250 50  0000 L CNN
 F 1 "OPA1678IDG" H 7450 4150 50  0000 L CNN
-F 2 "Package_SO:VSSOP-8_3.0x3.0mm_P0.65mm" H 7700 3650 50  0001 C CNN
+F 2 "Package_SO:SOIC-8_3.9x4.9mm_P1.27mm" H 7700 3650 50  0001 C CNN
 F 3 "http://www.analog.com/media/en/technical-documentation/data-sheets/OP249.pdf" H 7700 3650 50  0001 C CNN
 	2    7700 3650
@@
 Connection ~ 5825 3550
 Wire Wire Line
-	1125 975  1375 975
-Wire Wire Line
 	2075 825  2300 825
 Text Label 1375 975  2    50   ~ 0
@@
 L Devtank:+3V3_A #PWR0133
 U 1 1 60D990F9
-P 1275 1775
-F 0 "#PWR0133" H 1275 1625 50  0001 C CNN
-F 1 "+3V3_A" H 1290 1948 50  0000 C CNN
-F 2 "" H 1275 1775 50  0000 C CNN
-F 3 "" H 1275 1775 50  0000 C CNN
-	1    1275 1775
-	1    0    0    -1
-$EndComp
-Wire Wire Line
-	1275 1925 1275 1775
-Wire Wire Line
-	1275 1925 1525 1925
-Text Label 1525 1925 2    50   ~ 0
-5V_A
+P 1375 1975
+F 0 "#PWR0133" H 1375 1825 50  0001 C CNN
+F 1 "+3V3_A" H 1390 2148 50  0000 C CNN
+F 2 "" H 1375 1975 50  0000 C CNN
+F 3 "" H 1375 1975 50  0000 C CNN
+	1    1375 1975
+	1    0    0    -1
+$EndComp
+Wire Wire Line
+	1375 2125 1375 1975
 $Comp
 L Connector:Test_Point TP87
 U 1 1 60D9B3F1
-P 1525 1925
-F 0 "TP87" V 1525 2100 50  0000 L CNN
-F 1 "Test_Point" H 1583 1952 50  0001 L CNN
-F 2 "TestPoint:TestPoint_THTPad_D1.0mm_Drill0.5mm" H 1725 1925 50  0001 C CNN
-F 3 "~" H 1725 1925 50  0001 C CNN
-	1    1525 1925
+P 1625 2125
+F 0 "TP87" V 1625 2300 50  0000 L CNN
+F 1 "Test_Point" H 1683 2152 50  0001 L CNN
+F 2 "TestPoint:TestPoint_THTPad_D1.0mm_Drill0.5mm" H 1825 2125 50  0001 C CNN
+F 3 "~" H 1825 2125 50  0001 C CNN
+	1    1625 2125
 	0    1    1    0
 $EndComp
@@
 $EndComp
 Connection ~ 1125 975
+$Comp
+L OSM_env01-rescue:C-device-ESP32-EVB_Rev_D-rescue C74
+U 1 1 60B32488
+P 725 1125
+F 0 "C74" H 840 1171 50  0000 L CNN
+F 1 "100nF" H 840 1080 50  0000 L CNN
+F 2 "Capacitor_SMD:C_0603_1608Metric" H 763 975 50  0001 C CNN
+F 3 "" H 725 1125 50  0001 C CNN
+	1    725  1125
+	1    0    0    1
+$EndComp
+Wire Wire Line
+	725  1275 725  1375
+$Comp
+L power:GNDA #PWR0144
+U 1 1 60B3248F
+P 725 1375
+F 0 "#PWR0144" H 725 1125 50  0001 C CNN
+F 1 "GNDA" H 730 1202 50  0000 C CNN
+F 2 "" H 725 1375 50  0001 C CNN
+F 3 "" H 725 1375 50  0001 C CNN
+	1    725  1375
+	1    0    0    -1
+$EndComp
+Connection ~ 725  975
+Wire Wire Line
+	1125 975  1375 975
+Wire Wire Line
+	975  1975 975  2125
+$Comp
+L power:PWR_FLAG #FLG03
+U 1 1 60BB7AEA
+P 975 1975
+F 0 "#FLG03" H 975 2050 50  0001 C CNN
+F 1 "PWR_FLAG" H 975 2148 50  0000 C CNN
+F 2 "" H 975 1975 50  0001 C CNN
+F 3 "" H 975 1975 50  0001 C CNN
+	1    975  1975
+	1    0    0    -1
+$EndComp
+Connection ~ 1375 2125
+Wire Wire Line
+	1375 2125 1625 2125
+Wire Wire Line
+	975  2125 1375 2125
 $EndSCHEMATC
