File: kicad_osm_env01/LORA.sch (KiCad schematic (older format))
At the start: 15 parts, among them U5 ERIC-LORA, U6 RAK4270

Commit message: updated schematics
Parts:
- C26, C33, C70: footprint (none) -> Capacitor_SMD:C_0603_1608Metric
- C34, C35: footprint (none) -> Capacitor_SMD:C_0805_2012Metric
- R123: footprint (none) -> Resistor_SMD:R_0603_1608Metric
Changed lines of the file:
@@
 $Descr A4 11693 8268
 encoding utf-8
-Sheet 3 11
+Sheet 3 12
 Title ""
 Date ""
@@
 F 0 "C26" H 7965 2596 50  0000 L CNN
 F 1 "100nF" H 7965 2505 50  0000 L CNN
-F 2 "" H 7888 2400 50  0001 C CNN
+F 2 "Capacitor_SMD:C_0603_1608Metric" H 7888 2400 50  0001 C CNN
 F 3 "" H 7850 2550 50  0001 C CNN
 	1    7850 2550
@@
 F 0 "C33" H 7515 2596 50  0000 L CNN
 F 1 "100nF" H 7515 2505 50  0000 L CNN
-F 2 "" H 7438 2400 50  0001 C CNN
+F 2 "Capacitor_SMD:C_0603_1608Metric" H 7438 2400 50  0001 C CNN
 F 3 "" H 7400 2550 50  0001 C CNN
 	1    7400 2550
@@
 F 0 "C34" H 7065 2596 50  0000 L CNN
 F 1 "10uF" H 7065 2505 50  0000 L CNN
-F 2 "" H 6988 2400 50  0001 C CNN
+F 2 "Capacitor_SMD:C_0805_2012Metric" H 6988 2400 50  0001 C CNN
 F 3 "" H 6950 2550 50  0001 C CNN
 	1    6950 2550
@@
 F 0 "C35" H 6590 2596 50  0000 L CNN
 F 1 "10uF" H 6590 2505 50  0000 L CNN
-F 2 "" H 6513 2400 50  0001 C CNN
+F 2 "Capacitor_SMD:C_0805_2012Metric" H 6513 2400 50  0001 C CNN
 F 3 "" H 6475 2550 50  0001 C CNN
 	1    6475 2550
@@
 F 0 "R123" H 9645 3146 50  0000 L CNN
 F 1 "10k" H 9645 3055 50  0000 L CNN
-F 2 "" V 9505 3100 50  0001 C CNN
+F 2 "Resistor_SMD:R_0603_1608Metric" V 9505 3100 50  0001 C CNN
 F 3 "" H 9575 3100 50  0001 C CNN
 	1    9575 3100
@@
 F 0 "C70" H 9690 3571 50  0000 L CNN
 F 1 "100nF" H 9690 3480 50  0000 L CNN
-F 2 "" H 9613 3375 50  0001 C CNN
+F 2 "Capacitor_SMD:C_0603_1608Metric" H 9613 3375 50  0001 C CNN
 F 3 "" H 9575 3525 50  0001 C CNN
 	1    9575 3525

Commit message: started layout
Parts:
- U6: footprint (none) -> Devtank_PCB_lib:RAK4270
Changed lines of the file:
@@
 $Descr A4 11693 8268
 encoding utf-8
-Sheet 3 12
+Sheet 3 11
 Title ""
 Date ""
@@
 F 0 "U6" H 8625 4750 50  0000 C CNN
 F 1 "RAK4270" H 8750 4650 50  0000 C CNN
-F 2 "" H 7900 4175 50  0001 C CNN
+F 2 "Devtank_PCB_lib:RAK4270" H 7900 4175 50  0001 C CNN
 F 3 "" H 7900 4175 50  0001 C CNN
 	1    8150 3800

Commit message: Throwdown of parts
Parts:
- C26, C33: footprint Capacitor_SMD:C_0603_1608Metric -> Capacitor_SMD:C_0402_1005Metric
Connections:
- net LORA_RX: now also U6.5 (UART1_RX); no longer U6.4 (UART1_TX)
- net LORA_TX: now also U6.4 (UART1_TX); no longer U6.5 (UART1_RX)
Changed lines of the file:
@@
 F 0 "C26" H 7965 2596 50  0000 L CNN
 F 1 "100nF" H 7965 2505 50  0000 L CNN
-F 2 "Capacitor_SMD:C_0603_1608Metric" H 7888 2400 50  0001 C CNN
+F 2 "Capacitor_SMD:C_0402_1005Metric" H 7888 2400 50  0001 C CNN
 F 3 "" H 7850 2550 50  0001 C CNN
 	1    7850 2550
@@
 F 0 "C33" H 7515 2596 50  0000 L CNN
 F 1 "100nF" H 7515 2505 50  0000 L CNN
-F 2 "Capacitor_SMD:C_0603_1608Metric" H 7438 2400 50  0001 C CNN
+F 2 "Capacitor_SMD:C_0402_1005Metric" H 7438 2400 50  0001 C CNN
 F 3 "" H 7400 2550 50  0001 C CNN
 	1    7400 2550
@@
 NoConn ~ 9025 3425
 NoConn ~ 7275 3550
-$Comp
-L Devtank:RAK4270 U?
-U 1 1 608CFA5C
-P 8150 3800
-AR Path="/608CFA5C" Ref="U?"  Part="1"
-AR Path="/60880AD8/608CFA5C" Ref="U6"  Part="1"
-F 0 "U6" H 8625 4750 50  0000 C CNN
-F 1 "RAK4270" H 8750 4650 50  0000 C CNN
-F 2 "Devtank_PCB_lib:RAK4270" H 7900 4175 50  0001 C CNN
-F 3 "" H 7900 4175 50  0001 C CNN
-	1    8150 3800
-	1    0    0    -1
-$EndComp
 NoConn ~ 7275 4425
 NoConn ~ 7275 4300
@@
 Wire Wire Line
 	7275 3800 6900 3800
+Text HLabel 6900 3800 0    50   Input ~ 0
+LORA_RX
 Text HLabel 6900 3675 0    50   Input ~ 0
-LORA_RX
-Text HLabel 6900 3800 0    50   Input ~ 0
 LORA_TX
 Text HLabel 3175 3350 0    50   Input ~ 0
@@
 	0    1    1    0
 $EndComp
+$Comp
+L Devtank:RAK4270 U6
+U 1 1 6075834F
+P 8150 3800
+F 0 "U6" H 8150 4881 50  0000 C CNN
+F 1 "RAK4270" H 8150 4790 50  0000 C CNN
+F 2 "Devtank_PCB_lib:RAK4270" H 7900 4175 50  0001 C CNN
+F 3 "" H 7900 4175 50  0001 C CNN
+	1    8150 3800
+	1    0    0    -1
+$EndComp
 $EndSCHEMATC

Commit message: updated 3d step file
Parts:
- U6: symbol Devtank:RAK4270 -> OSM_env01-rescue:RAK4270-Devtank
Changed lines of the file:
@@
 $EndComp
 $Comp
-L Devtank:RAK4270 U6
+L OSM_env01-rescue:RAK4270-Devtank U6
 U 1 1 6075834F
 P 8150 3800
