File: kicad_osm_env01/Sensors_AND_IO.sch (KiCad schematic (older format))
At the start: 36 parts

Commit message: kicad review sch initial
Parts:
- removed TP? (x2): Test_Point, TestPoint:TestPoint_THTPad_D1.0mm_Drill0.5mm, symbol OSM_env01-rescue:Test_Point-Connector-ESP32-EVB_Rev_D-rescue
- added C?: C, symbol device:C
- added R?: R, symbol device:R
- added R?: DNF, symbol device:R
- added R?: 0R, symbol device:R
Connections:
- net GND: now also C?.2
- net HMP_RX renamed HPM_RX
- net HMP_TX renamed HPM_TX
- net SW_SEL renamed HPM_EN
- new net: C?.1, R?.1, R?.2
Other:
- moved on the sheet: C?, R?, TP?, U?

Commit message: updated schematics
Parts:
- added R96, R97: DNF, symbol device:R
- added R99: 100k, symbol device:R
- added U10: ICS-43432, MIC_ICS-43432, symbol Devtank:ICS-43432
- gave numbers to parts that had none: 38
Connections:
- net +3V3: now also R96.1
- net GND: now also R97.2, R99.2
- new net +3V3_A: U10.5 (VDD)
- new net GNDA: U10.3 (GND)
- new net MIC_LR: R96.2, R97.1, U10.2 (LR)
- new net MIC_SCK: U10.4 (SCK)
- new net MIC_SD: R99.1, U10.6 (SD)
- new net MIC_WS: U10.1 (WS)
Other:
- note added: "Microphone module\n"

Commit message: schematics awaiting review
Parts:
- added C71: 10uF, symbol device:CP
- added J7: Conn_01x04, symbol Connector:Conn_01x04
- added R124: Shunt, symbol device:R
- added R125, R126: 470k, symbol device:R
- added TP68, TP82, TP88: Test_Point, TestPoint:TestPoint_THTPad_D1.0mm_Drill0.5mm, symbol OSM_env01-rescue:Test_Point-Connector-ESP32-EVB_Rev_D-rescue
Connections:
- net labels added: CT+, CT-, MIC_GND
- net labels removed: LIGHT_INT, TEMP_INT
- wire segments 108 -> 131
- no-connect marks 4 -> 5
Other:
- note added: "CT Clamp\n\n"
- note added: "Inrush potential fixes\n-mosfet control timing\n-RC filter\n-resistors to limit current\n-Thermistor\n-super caps"
- note added: "bypass capacitor few hundred ohms\nhttps://learn.openenergymonitor.org/electricity-monitoring/ct-sensors/interface-with-arduino"
- moved on the sheet: R91, R92, R93, R94, R96, R97, R99, TP51, U10

Commit message: updated schematics
Parts:
- removed C39: C, symbol device:C
- removed R88: R, symbol device:R
- removed R89: DNF, symbol device:R
- removed R90: 0R, symbol device:R
- added C73: DNF, symbol device:C
- added D11: D, symbol device:D
- added R129: 0R, Resistor_SMD:R_0603_1608Metric, symbol OSM_env01-rescue:R-device-ESP32-EVB_Rev_D-rescue
- added TH3: Thermistor_NTC, symbol device:Thermistor_NTC
- C71: footprint (none) -> Capacitor_SMD:CP_Elec_6.3x7.7
- J7: footprint (none) -> Connector_JST:JST_EH_B4B-EH-A_1x04_P2.50mm_Vertical
- R125, R126, R96, R97, R99: footprint (none) -> Resistor_SMD:R_0603_1608Metric
- U10: footprint MIC_ICS-43432 -> (none)
Connections:
- wire segments 131 -> 138
Other:
- moved on the sheet: C43, Q6, R95, R98, TP48, U9

Commit message: started layout
Parts:
- removed J7: Conn_01x04, Connector_JST:JST_EH_B4B-EH-A_1x04_P2.50mm_Vertical, symbol Connector:Conn_01x04
- added C39: 100nF, Capacitor_SMD:C_0603_1608Metric, symbol OSM_env01-rescue:C-device-ESP32-EVB_Rev_D-rescue
- added R88: Shunt, Resistor_SMD:R_0805_2012Metric, symbol device:R
- C71: footprint Capacitor_SMD:CP_Elec_6.3x7.7 -> Capacitor_SMD:CP_Elec_4x5.4
- C73: footprint (none) -> Capacitor_SMD:C_0603_1608Metric
- D11: footprint (none) -> Diode_SMD:D_SOD-123
- R124: footprint (none) -> Resistor_SMD:R_1206_3216Metric
- TH3: footprint (none) -> Resistor_THT:R_Axial_DIN0204_L3.6mm_D1.6mm_P5.08mm_Horizontal
- U10: value ICS-43432 -> ICS-43434; footprint (none) -> Devtank_PCB_lib:MIC_ICS-43434
- U11: footprint Devtank_PCB_lib:HDC2080DMBR -> Devtank_PCB_lib:HDC2080
- U12: footprint Devtank_PCB_lib:TSL2561T -> Devtank_PCB_lib:TSL2561T_ALS
Connections:
- wire segments 138 -> 141
- no-connect marks 5 -> 4
Other:
- moved on the sheet: TP68, TP88
Changed lines of the file:
@@
 $Descr A4 11693 8268
 encoding utf-8
-Sheet 7 12
+Sheet 7 11
 Title ""
 Date ""
@@
 F 0 "U12" H 9487 3740 50  0000 C CNN
 F 1 "TSL2561" H 9487 3649 50  0000 C CNN
-F 2 "Devtank_PCB_lib:TSL2561T" H 9500 2950 50  0001 C CNN
+F 2 "Devtank_PCB_lib:TSL2561T_ALS" H 9500 2950 50  0001 C CNN
 F 3 "http://www.ti.com/lit/ds/symlink/hdc1080.pdf" H 9275 3625 50  0001 C CNN
 	1    9475 3300
@@
 F 0 "U11" H 8962 1640 50  0000 C CNN
 F 1 "HDC2080" H 8962 1549 50  0000 C CNN
-F 2 "Devtank_PCB_lib:HDC2080DMBR" H 8975 850 50  0001 C CNN
+F 2 "Devtank_PCB_lib:HDC2080" H 8975 850 50  0001 C CNN
 F 3 "http://www.ti.com/lit/ds/symlink/hdc1080.pdf" H 8750 1525 50  0001 C CNN
 	1    8950 1200
@@
 Microphone module\n
 Wire Wire Line
-	5850 1175 5850 1050
+	5850 1175 5850 1125
 $Comp
 L device:R R99
@@
 P 5850 1975
 F 0 "U10" H 5325 2750 50  0000 C CNN
-F 1 "ICS-43432" H 5500 2650 50  0000 C CNN
-F 2 "" H 5850 1975 50  0001 L BNN
+F 1 "ICS-43434" H 5500 2650 50  0000 C CNN
+F 2 "Devtank_PCB_lib:MIC_ICS-43434" H 5850 1975 50  0001 L BNN
 F 3 "" H 5850 1975 50  0001 L BNN
 	1    5850 1975
@@
 F 0 "C71" H 6043 4571 50  0000 L CNN
 F 1 "10uF" H 6043 4480 50  0000 L CNN
-F 2 "Capacitor_SMD:CP_Elec_6.3x7.7" H 5963 4375 50  0001 C CNN
+F 2 "Capacitor_SMD:CP_Elec_4x5.4" H 5963 4375 50  0001 C CNN
 F 3 "" H 5925 4525 50  0001 C CNN
 	1    5925 4525
@@
 Wire Wire Line
 	6325 4225 6325 4325
-Connection ~ 5750 4325
-Wire Wire Line
-	5750 4325 5575 4325
-Wire Wire Line
-	5750 3900 5575 3900
+Wire Wire Line
+	5400 3900 5225 3900
 Wire Wire Line
 	5750 3950 5750 3900
@@
 F 0 "R124" H 5820 4146 50  0000 L CNN
 F 1 "Shunt" H 5820 4055 50  0000 L CNN
-F 2 "" V 5680 4100 50  0001 C CNN
+F 2 "Resistor_SMD:R_1206_3216Metric" V 5680 4100 50  0001 C CNN
 F 3 "" H 5750 4100 50  0001 C CNN
 	1    5750 4100
@@
 Wire Wire Line
 	6325 4700 6325 4675
-Text HLabel 5450 3900 0    50   Input ~ 0
+Text HLabel 5100 3900 0    50   Input ~ 0
 CT+
 Wire Wire Line
@@
 	1450 3325 1225 3325
 Connection ~ 1225 3325
-Text Notes 5175 3650 0    118  ~ 0
+Text Notes 4825 3650 0    118  ~ 0
 CT Clamp\n\n
 $Comp
 L OSM_env01-rescue:Test_Point-Connector-ESP32-EVB_Rev_D-rescue TP?
 U 1 1 612C306D
-P 5400 3750
+P 5050 3750
 AR Path="/5F6F7717/612C306D" Ref="TP?"  Part="1"
 AR Path="/612C306D" Ref="TP?"  Part="1"
 AR Path="/608F4675/612C306D" Ref="TP68"  Part="1"
-F 0 "TP68" V 5400 4025 50  0000 C CNN
-F 1 "Test_Point" V 5475 3975 50  0001 C CNN
-F 2 "TestPoint:TestPoint_THTPad_D1.0mm_Drill0.5mm" H 5600 3750 50  0001 C CNN
-F 3 "~" H 5600 3750 50  0001 C CNN
-	1    5400 3750
+F 0 "TP68" V 5050 4025 50  0000 C CNN
+F 1 "Test_Point" V 5125 3975 50  0001 C CNN
+F 2 "TestPoint:TestPoint_THTPad_D1.0mm_Drill0.5mm" H 5250 3750 50  0001 C CNN
+F 3 "~" H 5250 3750 50  0001 C CNN
+	1    5050 3750
 	0    -1   1    0
 $EndComp
@@
 L OSM_env01-rescue:Test_Point-Connector-ESP32-EVB_Rev_D-rescue TP?
 U 1 1 612C3073
-P 5400 4475
+P 5050 4475
 AR Path="/5F6F7717/612C3073" Ref="TP?"  Part="1"
 AR Path="/612C3073" Ref="TP?"  Part="1"
 AR Path="/608F4675/612C3073" Ref="TP88"  Part="1"
-F 0 "TP88" V 5400 4750 50  0000 C CNN
-F 1 "Test_Point" V 5475 4700 50  0001 C CNN
-F 2 "TestPoint:TestPoint_THTPad_D1.0mm_Drill0.5mm" H 5600 4475 50  0001 C CNN
-F 3 "~" H 5600 4475 50  0001 C CNN
-	1    5400 4475
+F 0 "TP88" V 5050 4750 50  0000 C CNN
+F 1 "Test_Point" V 5125 4700 50  0001 C CNN
+F 2 "TestPoint:TestPoint_THTPad_D1.0mm_Drill0.5mm" H 5250 4475 50  0001 C CNN
+F 3 "~" H 5250 4475 50  0001 C CNN
+	1    5050 4475
 	0    -1   1    0
 $EndComp
 Wire Wire Line
-	5400 4475 5575 4475
-Wire Wire Line
-	5575 4475 5575 4325
-Connection ~ 5575 4325
-Wire Wire Line
-	5575 3900 5575 3750
-Wire Wire Line
-	5575 3750 5400 3750
-Connection ~ 5575 3900
-Wire Wire Line
-	5575 3900 5450 3900
-Text Label 5250 4325 0    50   ~ 0
-CT-
-Wire Wire Line
-	5250 4325 5575 4325
-Text Label 4575 4075 2    50   ~ 0
-CT-
-Wire Wire Line
-	4575 4075 4250 4075
-$Comp
-L Connector:Conn_01x04 J7
-U 1 1 612F7D00
-P 4050 4075
-F 0 "J7" H 3968 4392 50  0000 C CNN
-F 1 "Conn_01x04" H 3968 4301 50  0000 C CNN
-F 2 "Connector_JST:JST_EH_B4B-EH-A_1x04_P2.50mm_Vertical" H 4050 4075 50  0001 C CNN
-F 3 "~" H 4050 4075 50  0001 C CNN
-	1    4050 4075
-	-1   0    0    -1
-$EndComp
-Text Label 4575 3975 2    50   ~ 0
-CT+
-Wire Wire Line
-	4575 3975 4250 3975
-NoConn ~ 4250 4275
-$Comp
-L OSM_env01:GND #PWR?
-U 1 1 6130D84E
-P 4450 4350
-AR Path="/611AF79D/6130D84E" Ref="#PWR?"  Part="1"
-AR Path="/608F4675/6130D84E" Ref="#PWR0142"  Part="1"
-F 0 "#PWR0142" H 4450 4100 50  0001 C CNN
-F 1 "GND" H 4455 4177 50  0000 C CNN
-F 2 "" H 4450 4350 60  0000 C CNN
-F 3 "" H 4450 4350 60  0000 C CNN
-	1    4450 4350
-	1    0    0    -1
-$EndComp
-Wire Wire Line
-	4250 4175 4450 4175
-Wire Wire Line
-	4450 4175 4450 4350
+	5050 4475 5225 4475
+Wire Wire Line
+	5225 4475 5225 4325
+Wire Wire Line
+	5225 3900 5225 3750
+Wire Wire Line
+	5225 3750 5050 3750
+Connection ~ 5225 3900
+Wire Wire Line
+	5225 3900 5100 3900
 Text Notes 3575 5100 0    50   ~ 0
 bypass capacitor few hundred ohms\nhttps://learn.openenergymonitor.org/electricity-monitoring/ct-sensors/interface-with-arduino
@@
 F 0 "C73" H 5790 6071 50  0000 L CNN
 F 1 "DNF" H 5790 5980 50  0000 L CNN
-F 2 "" H 5713 5875 50  0001 C CNN
+F 2 "Capacitor_SMD:C_0603_1608Metric" H 5713 5875 50  0001 C CNN
 F 3 "" H 5675 6025 50  0001 C CNN
 	1    5675 6025
@@
 F 0 "TH3" H 6273 5921 50  0000 L CNN
 F 1 "Thermistor_NTC" H 6273 5830 50  0000 L CNN
-F 2 "" H 6175 5925 50  0001 C CNN
+F 2 "Resistor_THT:R_Axial_DIN0204_L3.6mm_D1.6mm_P5.08mm_Horizontal" H 6175 5925 50  0001 C CNN
 F 3 "" H 6175 5925 50  0001 C CNN
 	1    6175 5875
@@
 F 0 "D11" V 4804 6529 50  0000 L CNN
 F 1 "D" V 4895 6529 50  0000 L CNN
-F 2 "" H 4850 6450 50  0001 C CNN
+F 2 "Diode_SMD:D_SOD-123" H 4850 6450 50  0001 C CNN
 F 3 "" H 4850 6450 50  0001 C CNN
 	1    4850 6450
 	0    1    1    0
 $EndComp
+$Comp
+L device:R R?
+U 1 1 6073EBF7
+P 5400 4100
+AR Path="/611AF79D/6073EBF7" Ref="R?"  Part="1"
+AR Path="/608F4675/6073EBF7" Ref="R88"  Part="1"
+F 0 "R88" H 5470 4146 50  0000 L CNN
+F 1 "Shunt" H 5470 4055 50  0000 L CNN
+F 2 "Resistor_SMD:R_0805_2012Metric" V 5330 4100 50  0001 C CNN
+F 3 "" H 5400 4100 50  0001 C CNN
+	1    5400 4100
+	1    0    0    -1
+$EndComp
+Wire Wire Line
+	5225 4325 5400 4325
+Connection ~ 5750 4325
+Wire Wire Line
+	5400 4250 5400 4325
+Connection ~ 5400 4325
+Wire Wire Line
+	5400 4325 5750 4325
+Wire Wire Line
+	5400 3950 5400 3900
+Wire Wire Line
+	5750 3900 5400 3900
+Connection ~ 5400 3900
+Text HLabel 5100 4325 0    50   Input ~ 0
+CT-
+Wire Wire Line
+	5225 4325 5100 4325
+$Comp
+L OSM_env01-rescue:C-device-ESP32-EVB_Rev_D-rescue C?
+U 1 1 60B4304E
+P 6175 1125
+AR Path="/608F4675/60959880/60B4304E" Ref="C?"  Part="1"
+AR Path="/608F4675/60B4304E" Ref="C39"  Part="1"
+F 0 "C39" H 6290 1171 50  0000 L CNN
+F 1 "100nF" H 6290 1080 50  0000 L CNN
+F 2 "Capacitor_SMD:C_0603_1608Metric" H 6213 975 50  0001 C CNN
+F 3 "" H 6175 1125 50  0001 C CNN
+	1    6175 1125
+	0    1    -1   0
+$EndComp
+$Comp
+L power:GNDA #PWR?
+U 1 1 60B43055
+P 6525 1125
+AR Path="/608F4675/60959880/60B43055" Ref="#PWR?"  Part="1"
+AR Path="/608F4675/60B43055" Ref="#PWR066"  Part="1"
+F 0 "#PWR066" H 6525 875 50  0001 C CNN
+F 1 "GNDA" H 6530 952 50  0000 C CNN
+F 2 "" H 6525 1125 50  0001 C CNN
+F 3 "" H 6525 1125 50  0001 C CNN
+	1    6525 1125
+	1    0    0    -1
+$EndComp
+Wire Wire Line
+	6025 1125 5850 1125
+Connection ~ 5850 1125
+Wire Wire Line
+	5850 1125 5850 1050
+Wire Wire Line
+	6325 1125 6525 1125
 $EndSCHEMATC

Commit message: Throwdown of parts
Parts:
- C39: footprint Capacitor_SMD:C_0603_1608Metric -> Capacitor_SMD:C_0402_1005Metric
Connections:
- net GND: no longer R99.2
- net GNDA: now also R99.2
Changed lines of the file:
@@
 Wire Wire Line
 	5250 1650 5100 1650
-$Comp
-L OSM_env01:GND #PWR082
-U 1 1 608DAD19
-P 6675 2300
-F 0 "#PWR082" H 6675 2050 50  0001 C CNN
-F 1 "GND" H 6680 2127 50  0000 C CNN
-F 2 "" H 6675 2300 60  0000 C CNN
-F 3 "" H 6675 2300 60  0000 C CNN
-	1    6675 2300
-	1    0    0    -1
-$EndComp
 Wire Wire Line
 	6675 2300 6675 2225
@@
 F 0 "C39" H 6290 1171 50  0000 L CNN
 F 1 "100nF" H 6290 1080 50  0000 L CNN
-F 2 "Capacitor_SMD:C_0603_1608Metric" H 6213 975 50  0001 C CNN
+F 2 "Capacitor_SMD:C_0402_1005Metric" H 6213 975 50  0001 C CNN
 F 3 "" H 6175 1125 50  0001 C CNN
 	1    6175 1125
@@
 Wire Wire Line
 	6325 1125 6525 1125
+$Comp
+L power:GNDA #PWR?
+U 1 1 6075B945
+P 6675 2300
+AR Path="/608F4675/61105411/6075B945" Ref="#PWR?"  Part="1"
+AR Path="/608F4675/6075B945" Ref="#PWR0112"  Part="1"
+F 0 "#PWR0112" H 6675 2050 50  0001 C CNN
+F 1 "GNDA" H 6680 2127 50  0000 C CNN
+F 2 "" H 6675 2300 50  0001 C CNN
+F 3 "" H 6675 2300 50  0001 C CNN
+	1    6675 2300
+	1    0    0    -1
+$EndComp
 $EndSCHEMATC

Commit message: updated 3d step file
Parts:
- added J8: STX-3000, Devtank_PCB_lib:STX-3000, symbol Devtank:STX-3000
- U10: symbol Devtank:ICS-43432 -> OSM_env01-rescue:ICS-43432-Devtank
Changed lines of the file:
@@
 LR
 $Comp
-L Devtank:ICS-43432 U10
+L OSM_env01-rescue:ICS-43432-Devtank U10
 U 1 1 60824917
 P 5850 1975
@@
 $EndComp
 $Comp
-L Devtank:+3V3_A #PWR080
+L OSM_env01-rescue:+3V3_A-Devtank #PWR080
 U 1 1 611A742D
 P 5850 1050
+AR Path="/611A742D" Ref="#PWR080"  Part="1"
+AR Path="/608F4675/611A742D" Ref="#PWR080"  Part="1"
 F 0 "#PWR080" H 5850 900 50  0001 C CNN
 F 1 "+3V3_A" H 5865 1223 50  0000 C CNN
@@
 	1    0    0    -1
 $EndComp
+$Comp
+L Devtank:STX-3000 J8
+U 1 1 6129B739
+P 4575 4050
+F 0 "J8" H 3933 4437 60  0000 C CNN
+F 1 "STX-3000" H 3933 4331 60  0000 C CNN
+F 2 "Devtank_PCB_lib:STX-3000" H 3775 4290 60  0001 C CNN
+F 3 "" H 4575 4050 60  0000 C CNN
+	1    4575 4050
+	1    0    0    -1
+$EndComp
