File: kicad_osm_env01/Sensors_AND_IO.sch (KiCad schematic (older format))
At the start: 49 parts, among them J4 Conn_01x08, J8 STX-3000, U10 ICS-43434, U11 HPP845E131R5, U12 MIC94073YC6, U3 VEML7700-TT

Commit message: schematics and layout submitted for review
Parts:
- TP13, TP14, TP49: footprint TestPoint:TestPoint_Pad_D1.5mm -> TestPoint:TestPoint_THTPad_D1.0mm_Drill0.5mm
- U11: footprint Devtank_PCB_lib:HDC2080D -> Devtank_PCB_lib:HPP845E131R5_temperature_humidity_sensor
Changed lines of the file:
@@
 F 0 "U11" H 8025 5875 60  0000 R CNN
 F 1 "HPP845E131R5" H 8550 5775 60  0000 R CNN
-F 2 "Devtank_PCB_lib:HDC2080D" H 8750 5140 60  0001 C CNN
+F 2 "Devtank_PCB_lib:HPP845E131R5_temperature_humidity_sensor" H 8750 5140 60  0001 C CNN
 F 3 "" H 8750 5200 60  0000 C CNN
 	1    8750 5200
@@
 F 0 "TP14" V 4975 2675 50  0000 C CNN
 F 1 "Test_Point" V 5050 2625 50  0001 C CNN
-F 2 "TestPoint:TestPoint_Pad_D1.5mm" H 5175 2400 50  0001 C CNN
+F 2 "TestPoint:TestPoint_THTPad_D1.0mm_Drill0.5mm" H 5175 2400 50  0001 C CNN
 F 3 "~" H 5175 2400 50  0001 C CNN
 	1    4975 2400
@@
 F 0 "TP13" V 4975 1875 50  0000 C CNN
 F 1 "Test_Point" V 5050 1825 50  0001 C CNN
-F 2 "TestPoint:TestPoint_Pad_D1.5mm" H 5175 1600 50  0001 C CNN
+F 2 "TestPoint:TestPoint_THTPad_D1.0mm_Drill0.5mm" H 5175 1600 50  0001 C CNN
 F 3 "~" H 5175 1600 50  0001 C CNN
 	1    4975 1600
@@
 F 0 "TP49" V 6525 2150 50  0000 C CNN
 F 1 "Test_Point" V 6600 2100 50  0001 C CNN
-F 2 "TestPoint:TestPoint_Pad_D1.5mm" H 6725 1875 50  0001 C CNN
+F 2 "TestPoint:TestPoint_THTPad_D1.0mm_Drill0.5mm" H 6725 1875 50  0001 C CNN
 F 3 "~" H 6725 1875 50  0001 C CNN
 	1    6525 1875

Commit message: Bom and gerbers added
Parts:
- TP48: footprint TestPoint:TestPoint_Pad_D1.5mm -> TestPoint:TestPoint_THTPad_D1.0mm_Drill0.5mm
Other:
- note added: "Note: Can use HDC1080/2080. For HTU21D leave pad 3,4. For all devices leave ep pin 7 unconnected"
- note removed: "Note: Can use HDC1080/2080. For HTU21D leave pad 3,4 and ep unconnected"
Changed lines of the file:
@@
 NoConn ~ 8750 5900
 Text Notes 7775 6450 0    50   ~ 0
-Note: Can use HDC1080/2080. For HTU21D leave pad 3,4 and ep unconnected
+Note: Can use HDC1080/2080. For HTU21D leave pad 3,4. For all devices leave ep pin 7 unconnected
 Text Notes 8700 975  0    118  ~ 24
 Light Sensor\n\n
@@
 F 0 "TP48" H 4325 6250 50  0000 C CNN
 F 1 "Test_Point" V 4400 6250 50  0001 C CNN
-F 2 "TestPoint:TestPoint_Pad_D1.5mm" H 4525 6025 50  0001 C CNN
+F 2 "TestPoint:TestPoint_THTPad_D1.0mm_Drill0.5mm" H 4525 6025 50  0001 C CNN
 F 3 "~" H 4525 6025 50  0001 C CNN
 	1    4325 6025

Commit message: updated folder
Parts:
- added R63, R65: DNF, Resistor_SMD:R_1206_3216Metric, symbol device:R
- R124: value DNF -> 82R
- R88: value 22R -> 30R
Connections:
- net CT+: now also R63.1, R65.1
- net at C71.1, J8.3, R124.2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: now also R63.2, R65.2
Other:
- note added: "22R=30R//82R\n\n22R as suggested on website"
- moved on the sheet: C71, J8, R124, R125, R126, R88, TP56, TP68
