File: kicad_osm_env01/CanTransciever.sch (KiCad schematic (older format))
At the start: 12 parts, among them U8 MCP2551-I-P

Commit message: schematics awaiting review
Parts:
- added TP80, TP81: Test_Point, TestPoint:TestPoint_THTPad_D1.0mm_Drill0.5mm, symbol OSM_env01-rescue:Test_Point-Connector-ESP32-EVB_Rev_D-rescue
Connections:
- wire segments 36 -> 42
Other:
- moved on the sheet: R80, R82
Changed lines of the file:
@@
 $Descr A4 11693 8268
 encoding utf-8
-Sheet 10 11
+Sheet 6 11
 Title ""
 Date ""
@@
 L device:R R82
 U 1 1 6065D32A
-P 4425 3450
-F 0 "R82" H 4495 3496 50  0000 L CNN
-F 1 "DNF" H 4495 3405 50  0000 L CNN
-F 2 "" V 4355 3450 50  0001 C CNN
-F 3 "" H 4425 3450 50  0001 C CNN
-	1    4425 3450
+P 4400 3450
+F 0 "R82" H 4200 3450 50  0000 L CNN
+F 1 "DNF" H 4200 3375 50  0000 L CNN
+F 2 "" V 4330 3450 50  0001 C CNN
+F 3 "" H 4400 3450 50  0001 C CNN
+	1    4400 3450
 	1    0    0    -1
 $EndComp
@@
 L device:R R80
 U 1 1 6065D75A
-P 4275 3800
-F 0 "R80" V 4175 3750 50  0000 L CNN
-F 1 "10k" V 4375 3750 50  0000 L CNN
-F 2 "" V 4205 3800 50  0001 C CNN
-F 3 "" H 4275 3800 50  0001 C CNN
-	1    4275 3800
+P 4250 3800
+F 0 "R80" V 4150 3750 50  0000 L CNN
+F 1 "10k" V 4350 3750 50  0000 L CNN
+F 2 "" V 4180 3800 50  0001 C CNN
+F 3 "" H 4250 3800 50  0001 C CNN
+	1    4250 3800
 	0    1    1    0
 $EndComp
@@
 	6500 3275 6275 3275
 Connection ~ 6275 3275
-Wire Wire Line
-	4825 3950 4925 3950
-Text HLabel 4825 3950 0    50   Input ~ 0
+Text HLabel 4800 3950 0    50   Input ~ 0
 CAN_RX
 Text HLabel 5025 3675 0    50   Input ~ 0
@@
 Wire Wire Line
 	4925 4500 4925 4375
-Text Label 4075 3175 0    50   ~ 0
+Text Label 4050 3175 0    50   ~ 0
 CAN_VDD
 Wire Wire Line
-	4425 3300 4425 3175
-Wire Wire Line
-	4425 3600 4425 3800
-Wire Wire Line
-	4425 3800 5475 3800
-Connection ~ 4425 3800
+	4400 3300 4400 3175
+Wire Wire Line
+	4400 3600 4400 3800
+Connection ~ 4400 3800
 $Comp
 L OSM_env01:GND #PWR060
 U 1 1 6069B827
-P 4000 3800
-F 0 "#PWR060" H 4000 3550 50  0001 C CNN
-F 1 "GND" H 4005 3627 50  0000 C CNN
-F 2 "" H 4000 3800 60  0000 C CNN
-F 3 "" H 4000 3800 60  0000 C CNN
-	1    4000 3800
-	1    0    0    -1
-$EndComp
-Wire Wire Line
-	4000 3800 4125 3800
+P 3975 3800
+F 0 "#PWR060" H 3975 3550 50  0001 C CNN
+F 1 "GND" H 3980 3627 50  0000 C CNN
+F 2 "" H 3975 3800 60  0000 C CNN
+F 3 "" H 3975 3800 60  0000 C CNN
+	1    3975 3800
+	1    0    0    -1
+$EndComp
+Wire Wire Line
+	3975 3800 4100 3800
 $Comp
 L device:Jumper_NC_Dual JP2
@@
 	5925 1400 5925 1550
 Wire Wire Line
-	4425 3175 4075 3175
+	4400 3175 4050 3175
 Text Label 5625 2775 0    50   ~ 0
 CAN_VDD
-Wire Wire Line
-	5975 2775 5625 2775
 Connection ~ 5975 2775
 Wire Wire Line
@@
 Wire Wire Line
 	6275 1550 5925 1550
+$Comp
+L OSM_env01-rescue:Test_Point-Connector-ESP32-EVB_Rev_D-rescue TP?
+U 1 1 608A88D0
+P 4850 3550
+AR Path="/60688D25/608A88D0" Ref="TP?"  Part="1"
+AR Path="/6064BC1D/608A88D0" Ref="TP81"  Part="1"
+F 0 "TP81" V 4850 3825 50  0000 C CNN
+F 1 "Test_Point" V 4954 3622 50  0001 C CNN
+F 2 "TestPoint:TestPoint_THTPad_D1.0mm_Drill0.5mm" H 5050 3550 50  0001 C CNN
+F 3 "~" H 5050 3550 50  0001 C CNN
+	1    4850 3550
+	0    -1   1    0
+$EndComp
+Wire Wire Line
+	4400 3800 5475 3800
+$Comp
+L OSM_env01-rescue:Test_Point-Connector-ESP32-EVB_Rev_D-rescue TP?
+U 1 1 608AF678
+P 4625 4075
+AR Path="/60688D25/608AF678" Ref="TP?"  Part="1"
+AR Path="/6064BC1D/608AF678" Ref="TP80"  Part="1"
+F 0 "TP80" V 4625 4350 50  0000 C CNN
+F 1 "Test_Point" V 4729 4147 50  0001 C CNN
+F 2 "TestPoint:TestPoint_THTPad_D1.0mm_Drill0.5mm" H 4825 4075 50  0001 C CNN
+F 3 "~" H 4825 4075 50  0001 C CNN
+	1    4625 4075
+	0    -1   1    0
+$EndComp
+Wire Wire Line
+	4800 3950 4825 3950
+Wire Wire Line
+	4625 4075 4825 4075
+Wire Wire Line
+	4825 4075 4825 3950
+Connection ~ 4825 3950
+Wire Wire Line
+	4825 3950 4925 3950
+Wire Wire Line
+	4850 3550 5025 3550
+Wire Wire Line
+	5025 3550 5025 3675
+$Comp
+L OSM_env01:PWR_FLAG #FLG0105
+U 1 1 60701638
+P 5475 2625
+F 0 "#FLG0105" H 5475 2720 50  0001 C CNN
+F 1 "PWR_FLAG" H 5475 2848 50  0000 C CNN
+F 2 "" H 5475 2625 60  0000 C CNN
+F 3 "" H 5475 2625 60  0000 C CNN
+	1    5475 2625
+	1    0    0    -1
+$EndComp
+Wire Wire Line
+	5475 2775 5475 2625
+Wire Wire Line
+	5475 2775 5975 2775
 $EndSCHEMATC

Commit message: updated schematics
Parts:
- C37: footprint (none) -> Capacitor_SMD:C_0805_2012Metric
- C38: value 100uF -> 100nF; footprint (none) -> Capacitor_SMD:C_0603_1608Metric
- JP2, JP3: footprint (none) -> Connector_PinHeader_1.27mm:PinHeader_1x03_P1.27mm_Horizontal
- R80, R82, R83, R84, R85, R86, R87: footprint (none) -> Resistor_SMD:R_0603_1608Metric
Changed lines of the file:
@@
 $Descr A4 11693 8268
 encoding utf-8
-Sheet 6 11
+Sheet 6 12
 Title ""
 Date ""
@@
 F 0 "R84" V 5375 3675 50  0000 L CNN
 F 1 "330R" V 5275 3575 50  0000 L CNN
-F 2 "" V 5105 3675 50  0001 C CNN
+F 2 "Resistor_SMD:R_0603_1608Metric" V 5105 3675 50  0001 C CNN
 F 3 "" H 5175 3675 50  0001 C CNN
 	1    5175 3675
@@
 F 0 "R85" V 5075 3950 50  0000 L CNN
 F 1 "330R" V 4975 3850 50  0000 L CNN
-F 2 "" V 5105 3950 50  0001 C CNN
+F 2 "Resistor_SMD:R_0603_1608Metric" V 5105 3950 50  0001 C CNN
 F 3 "" H 5175 3950 50  0001 C CNN
 	1    5175 3950
@@
 F 0 "R83" H 4675 4275 50  0000 L CNN
 F 1 "680R" H 4675 4175 50  0000 L CNN
-F 2 "" V 4855 4225 50  0001 C CNN
+F 2 "Resistor_SMD:R_0603_1608Metric" V 4855 4225 50  0001 C CNN
 F 3 "" H 4925 4225 50  0001 C CNN
 	1    4925 4225
@@
 F 0 "R87" H 7145 4096 50  0000 L CNN
 F 1 "120R" H 7145 4005 50  0000 L CNN
-F 2 "" V 7005 4050 50  0001 C CNN
+F 2 "Resistor_SMD:R_0603_1608Metric" V 7005 4050 50  0001 C CNN
 F 3 "" H 7075 4050 50  0001 C CNN
 	1    7075 4050
@@
 F 0 "R86" H 5370 4546 50  0000 L CNN
 F 1 "DNF" H 5370 4455 50  0000 L CNN
-F 2 "" V 5230 4500 50  0001 C CNN
+F 2 "Resistor_SMD:R_0603_1608Metric" V 5230 4500 50  0001 C CNN
 F 3 "" H 5300 4500 50  0001 C CNN
 	1    5300 4500
@@
 F 0 "R82" H 4200 3450 50  0000 L CNN
 F 1 "DNF" H 4200 3375 50  0000 L CNN
-F 2 "" V 4330 3450 50  0001 C CNN
+F 2 "Resistor_SMD:R_0603_1608Metric" V 4330 3450 50  0001 C CNN
 F 3 "" H 4400 3450 50  0001 C CNN
 	1    4400 3450
@@
 F 0 "R80" V 4150 3750 50  0000 L CNN
 F 1 "10k" V 4350 3750 50  0000 L CNN
-F 2 "" V 4180 3800 50  0001 C CNN
+F 2 "Resistor_SMD:R_0603_1608Metric" V 4180 3800 50  0001 C CNN
 F 3 "" H 4250 3800 50  0001 C CNN
 	1    4250 3800
@@
 F 0 "C37" V 6275 2775 50  0000 L CNN
 F 1 "10uF" V 5975 2675 50  0000 L CNN
-F 2 "" H 6163 2625 50  0001 C CNN
+F 2 "Capacitor_SMD:C_0805_2012Metric" H 6163 2625 50  0001 C CNN
 F 3 "" H 6125 2775 50  0001 C CNN
 	1    6125 2775
@@
 P 6125 3275
 F 0 "C38" V 6275 3300 50  0000 L CNN
-F 1 "100uF" V 5975 3150 50  0000 L CNN
-F 2 "" H 6163 3125 50  0001 C CNN
+F 1 "100nF" V 5975 3150 50  0000 L CNN
+F 2 "Capacitor_SMD:C_0603_1608Metric" H 6163 3125 50  0001 C CNN
 F 3 "" H 6125 3275 50  0001 C CNN
 	1    6125 3275
@@
 F 0 "JP3" V 6825 3375 50  0000 C CNN
 F 1 "Jumper_NC_Small" V 6900 3625 50  0000 C CNN
-F 2 "" H 7075 3625 50  0001 C CNN
+F 2 "Connector_PinHeader_1.27mm:PinHeader_1x03_P1.27mm_Horizontal" H 7075 3625 50  0001 C CNN
 F 3 "" H 7075 3625 50  0001 C CNN
 	1    7075 3625
@@
 F 0 "JP2" H 5925 1539 50  0000 C CNN
 F 1 "Jumper_NC_Dual" H 5925 1448 50  0000 C CNN
-F 2 "" H 5925 1300 50  0001 C CNN
+F 2 "Connector_PinHeader_1.27mm:PinHeader_1x03_P1.27mm_Horizontal" H 5925 1300 50  0001 C CNN
 F 3 "" H 5925 1300 50  0001 C CNN
 	1    5925 1300

Commit message: started layout
Parts:
- JP2: footprint Connector_PinHeader_1.27mm:PinHeader_1x03_P1.27mm_Horizontal -> Connector_PinHeader_1.27mm:PinHeader_1x03_P1.27mm_Vertical
- JP3: footprint Connector_PinHeader_1.27mm:PinHeader_1x03_P1.27mm_Horizontal -> Connector_PinHeader_1.27mm:PinHeader_1x02_P1.27mm_Vertical
- U8: value MCP2551-I-P -> MCP2551-I/SN; footprint Housings_DIP:DIP-8_W7.62mm -> Package_SO:SOIC-8_3.9x4.9mm_P1.27mm
Changed lines of the file:
@@
 $Descr A4 11693 8268
 encoding utf-8
-Sheet 6 12
+Sheet 6 11
 Title ""
 Date ""
@@
 F 0 "JP3" V 6825 3375 50  0000 C CNN
 F 1 "Jumper_NC_Small" V 6900 3625 50  0000 C CNN
-F 2 "Connector_PinHeader_1.27mm:PinHeader_1x03_P1.27mm_Horizontal" H 7075 3625 50  0001 C CNN
+F 2 "Connector_PinHeader_1.27mm:PinHeader_1x02_P1.27mm_Vertical" H 7075 3625 50  0001 C CNN
 F 3 "" H 7075 3625 50  0001 C CNN
 	1    7075 3625
@@
 F 0 "JP2" H 5925 1539 50  0000 C CNN
 F 1 "Jumper_NC_Dual" H 5925 1448 50  0000 C CNN
-F 2 "Connector_PinHeader_1.27mm:PinHeader_1x03_P1.27mm_Horizontal" H 5925 1300 50  0001 C CNN
+F 2 "Connector_PinHeader_1.27mm:PinHeader_1x03_P1.27mm_Vertical" H 5925 1300 50  0001 C CNN
 F 3 "" H 5925 1300 50  0001 C CNN
 	1    5925 1300
@@
 P 5975 3875
 F 0 "U8" H 6225 3450 50  0000 C CNN
-F 1 "MCP2551-I-P" H 6450 3350 50  0000 C CNN
-F 2 "Housings_DIP:DIP-8_W7.62mm" H 5975 3375 50  0001 C CIN
+F 1 "MCP2551-I/SN " H 6450 3350 50  0000 C CNN
+F 2 "Package_SO:SOIC-8_3.9x4.9mm_P1.27mm" H 5975 3375 50  0001 C CIN
 F 3 "http://ww1.microchip.com/downloads/en/devicedoc/21667d.pdf" H 5975 3875 50  0001 C CNN
 	1    5975 3875

Commit message: Throwdown of parts
Parts:
- C38: footprint Capacitor_SMD:C_0603_1608Metric -> Capacitor_SMD:C_0402_1005Metric
Changed lines of the file:
@@
 F 0 "C38" V 6275 3300 50  0000 L CNN
 F 1 "100nF" V 5975 3150 50  0000 L CNN
-F 2 "Capacitor_SMD:C_0603_1608Metric" H 6163 3125 50  0001 C CNN
+F 2 "Capacitor_SMD:C_0402_1005Metric" H 6163 3125 50  0001 C CNN
 F 3 "" H 6125 3275 50  0001 C CNN
 	1    6125 3275

Commit message: updated 3d step file
Parts:
- U8: symbol Devtank:MCP2551-I-P -> OSM_env01-rescue:MCP2551-I-P-Devtank
Changed lines of the file:
@@
 CAN_H
 $Comp
-L Devtank:MCP2551-I-P U8
+L OSM_env01-rescue:MCP2551-I-P-Devtank U8
 U 1 1 6066DC31
 P 5975 3875

Commit message: schematics awaiting review
Parts:
- removed JP2: Jumper_NC_Dual, Connector_PinHeader_1.27mm:PinHeader_1x03_P1.27mm_Vertical, symbol device:Jumper_NC_Dual
- removed JP3: Jumper_NC_Small, Connector_PinHeader_1.27mm:PinHeader_1x02_P1.27mm_Vertical, symbol device:Jumper_NC_Small
- added R23, R25: 0R, symbol device:R
- added R24: DNF, symbol device:R
- added TP22, TP23, TP41: Test_Point, TestPoint:TestPoint_THTPad_D1.0mm_Drill0.5mm, symbol OSM_env01-rescue:Test_Point-Connector-ESP32-EVB_Rev_D-rescue
- R80: value 10k -> DNF
- U8: value MCP2551-I/SN -> SN65HVD230D
Connections:
- net labels added: CAN_RS
- wire segments 42 -> 52
Changed lines of the file:
@@
 $Descr A4 11693 8268
 encoding utf-8
-Sheet 6 11
+Sheet 11 11
 Title ""
 Date ""
@@
 U 1 1 6065BE4A
 P 5175 3675
-F 0 "R84" V 5375 3675 50  0000 L CNN
+F 0 "R84" V 5375 3625 50  0000 L CNN
 F 1 "330R" V 5275 3575 50  0000 L CNN
 F 2 "Resistor_SMD:R_0603_1608Metric" V 5105 3675 50  0001 C CNN
@@
 U 1 1 6065C39F
 P 5175 3950
-F 0 "R85" V 5075 3950 50  0000 L CNN
+F 0 "R85" V 5075 3900 50  0000 L CNN
 F 1 "330R" V 4975 3850 50  0000 L CNN
 F 2 "Resistor_SMD:R_0603_1608Metric" V 5105 3950 50  0001 C CNN
@@
 U 1 1 6065D32A
 P 4400 3450
-F 0 "R82" H 4200 3450 50  0000 L CNN
-F 1 "DNF" H 4200 3375 50  0000 L CNN
+F 0 "R82" H 4200 3475 50  0000 L CNN
+F 1 "DNF" H 4200 3400 50  0000 L CNN
 F 2 "Resistor_SMD:R_0603_1608Metric" V 4330 3450 50  0001 C CNN
 F 3 "" H 4400 3450 50  0001 C CNN
@@
 U 1 1 6065D75A
 P 4250 3800
-F 0 "R80" V 4150 3750 50  0000 L CNN
-F 1 "10k" V 4350 3750 50  0000 L CNN
+F 0 "R80" V 4150 3725 50  0000 L CNN
+F 1 "DNF" V 4350 3725 50  0000 L CNN
 F 2 "Resistor_SMD:R_0603_1608Metric" V 4180 3800 50  0001 C CNN
 F 3 "" H 4250 3800 50  0001 C CNN
@@
 U 1 1 6065DC74
 P 6125 2775
-F 0 "C37" V 6275 2775 50  0000 L CNN
+F 0 "C37" V 6275 2700 50  0000 L CNN
 F 1 "10uF" V 5975 2675 50  0000 L CNN
 F 2 "Capacitor_SMD:C_0805_2012Metric" H 6163 2625 50  0001 C CNN
@@
 U 1 1 6065E430
 P 6125 3275
-F 0 "C38" V 6275 3300 50  0000 L CNN
+F 0 "C38" V 6275 3200 50  0000 L CNN
 F 1 "100nF" V 5975 3150 50  0000 L CNN
 F 2 "Capacitor_SMD:C_0402_1005Metric" H 6163 3125 50  0001 C CNN
@@
 	1    6125 3275
 	0    -1   -1   0
-$EndComp
-$Comp
-L device:Jumper_NC_Small JP3
-U 1 1 60660D81
-P 7075 3625
-F 0 "JP3" V 6825 3375 50  0000 C CNN
-F 1 "Jumper_NC_Small" V 6900 3625 50  0000 C CNN
-F 2 "Connector_PinHeader_1.27mm:PinHeader_1x02_P1.27mm_Vertical" H 7075 3625 50  0001 C CNN
-F 3 "" H 7075 3625 50  0001 C CNN
-	1    7075 3625
-	0    1    1    0
 $EndComp
 Wire Wire Line
@@
 L power:+5V #PWR064
 U 1 1 60688778
-P 6400 1125
-F 0 "#PWR064" H 6400 975 50  0001 C CNN
-F 1 "+5V" H 6415 1298 50  0000 C CNN
-F 2 "" H 6400 1125 50  0001 C CNN
-F 3 "" H 6400 1125 50  0001 C CNN
-	1    6400 1125
+P 5775 1125
+F 0 "#PWR064" H 5775 975 50  0001 C CNN
+F 1 "+5V" H 5790 1298 50  0000 C CNN
+F 2 "" H 5775 1125 50  0001 C CNN
+F 3 "" H 5775 1125 50  0001 C CNN
+	1    5775 1125
 	1    0    0    -1
 $EndComp
@@
 	5475 1125 5475 1300
 Wire Wire Line
-	5475 1300 5675 1300
-Wire Wire Line
-	6175 1300 6400 1300
-Wire Wire Line
-	6400 1300 6400 1125
+	5775 1300 5775 1125
 Wire Wire Line
 	4925 4075 4925 3950
@@
 	4400 3300 4400 3175
 Wire Wire Line
-	4400 3600 4400 3800
+	4400 3600 4400 3625
 Connection ~ 4400 3800
 $Comp
@@
 Wire Wire Line
 	3975 3800 4100 3800
-$Comp
-L device:Jumper_NC_Dual JP2
-U 1 1 60661918
-P 5925 1300
-F 0 "JP2" H 5925 1539 50  0000 C CNN
-F 1 "Jumper_NC_Dual" H 5925 1448 50  0000 C CNN
-F 2 "Connector_PinHeader_1.27mm:PinHeader_1x03_P1.27mm_Vertical" H 5925 1300 50  0001 C CNN
-F 3 "" H 5925 1300 50  0001 C CNN
-	1    5925 1300
-	1    0    0    -1
-$EndComp
-Wire Wire Line
-	5925 1400 5925 1550
 Wire Wire Line
 	4400 3175 4050 3175
@@
 	5975 2775 5975 3275
 Wire Wire Line
-	7075 3900 7075 3725
-Wire Wire Line
 	6475 3775 6800 3775
 Wire Wire Line
 	6800 3775 6800 3525
-Wire Wire Line
-	6800 3525 7075 3525
 Wire Wire Line
 	6475 3975 6800 3975
@@
 	5975 4375 5975 4275
 Wire Wire Line
-	7075 3525 7475 3525
-Connection ~ 7075 3525
-Wire Wire Line
-	7075 4200 7475 4200
+	7075 4200 7375 4200
 Connection ~ 7075 4200
 Text HLabel 7475 4200 2    50   Input ~ 0
@@
 U 1 1 6066DC31
 P 5975 3875
-F 0 "U8" H 6225 3450 50  0000 C CNN
-F 1 "MCP2551-I/SN " H 6450 3350 50  0000 C CNN
+F 0 "U8" H 6250 3500 50  0000 C CNN
+F 1 "SN65HVD230D" H 6525 3400 50  0000 C CNN
 F 2 "Package_SO:SOIC-8_3.9x4.9mm_P1.27mm" H 5975 3375 50  0001 C CIN
 F 3 "http://ww1.microchip.com/downloads/en/devicedoc/21667d.pdf" H 5975 3875 50  0001 C CNN
@@
 	1    0    0    -1
 $EndComp
-Text Label 6275 1550 2    50   ~ 0
+Text Label 6125 1800 2    50   ~ 0
 CAN_VDD
 Wire Wire Line
-	6275 1550 5925 1550
+	6125 1800 5775 1800
 $Comp
 L OSM_env01-rescue:Test_Point-Connector-ESP32-EVB_Rev_D-rescue TP?
@@
 Wire Wire Line
 	5475 2775 5975 2775
+$Comp
+L device:R R23
+U 1 1 6218B593
+P 5475 1450
+F 0 "R23" H 5545 1496 50  0000 L CNN
+F 1 "0R" H 5545 1405 50  0000 L CNN
+F 2 "" V 5405 1450 50  0001 C CNN
+F 3 "" H 5475 1450 50  0001 C CNN
+	1    5475 1450
+	1    0    0    -1
+$EndComp
+$Comp
+L device:R R24
+U 1 1 6218E5ED
+P 5775 1450
+F 0 "R24" H 5845 1496 50  0000 L CNN
+F 1 "DNF" H 5845 1405 50  0000 L CNN
+F 2 "" V 5705 1450 50  0001 C CNN
+F 3 "" H 5775 1450 50  0001 C CNN
+	1    5775 1450
+	1    0    0    -1
+$EndComp
+Wire Wire Line
+	5775 1800 5775 1625
+Wire Wire Line
+	5475 1600 5475 1625
+Wire Wire Line
+	5475 1625 5775 1625
+Connection ~ 5775 1625
+Wire Wire Line
+	5775 1625 5775 1600
+Wire Wire Line
+	6800 3525 7075 3525
+$Comp
+L device:R R25
+U 1 1 621A1F2E
+P 7075 3675
+F 0 "R25" H 7145 3721 50  0000 L CNN
+F 1 "0R" H 7145 3630 50  0000 L CNN
+F 2 "" V 7005 3675 50  0001 C CNN
+F 3 "" H 7075 3675 50  0001 C CNN
+	1    7075 3675
+	1    0    0    -1
+$EndComp
+Connection ~ 7075 3525
+Wire Wire Line
+	7075 3525 7375 3525
+Wire Wire Line
+	7075 3900 7075 3825
+Connection ~ 4400 3625
+Wire Wire Line
+	4400 3625 4400 3800
+Text HLabel 3875 3625 0    50   Input ~ 0
+CAN_RS
+$Comp
+L OSM_env01-rescue:Test_Point-Connector-ESP32-EVB_Rev_D-rescue TP?
+U 1 1 61C968D6
+P 3900 3525
+AR Path="/60688D25/61C968D6" Ref="TP?"  Part="1"
+AR Path="/6064BC1D/61C968D6" Ref="TP22"  Part="1"
+F 0 "TP22" V 3900 3800 50  0000 C CNN
+F 1 "Test_Point" V 4004 3597 50  0001 C CNN
+F 2 "TestPoint:TestPoint_THTPad_D1.0mm_Drill0.5mm" H 4100 3525 50  0001 C CNN
+F 3 "~" H 4100 3525 50  0001 C CNN
+	1    3900 3525
+	0    -1   1    0
+$EndComp
+Wire Wire Line
+	3900 3525 4075 3525
+Wire Wire Line
+	3875 3625 4075 3625
+Wire Wire Line
+	4075 3525 4075 3625
+Connection ~ 4075 3625
+Wire Wire Line
+	4075 3625 4400 3625
+$Comp
+L OSM_env01-rescue:Test_Point-Connector-ESP32-EVB_Rev_D-rescue TP?
+U 1 1 61C9CD32
+P 7375 3400
+AR Path="/60688D25/61C9CD32" Ref="TP?"  Part="1"
+AR Path="/6064BC1D/61C9CD32" Ref="TP23"  Part="1"
+F 0 "TP23" V 7375 3675 50  0000 C CNN
+F 1 "Test_Point" V 7479 3472 50  0001 C CNN
+F 2 "TestPoint:TestPoint_THTPad_D1.0mm_Drill0.5mm" H 7575 3400 50  0001 C CNN
+F 3 "~" H 7575 3400 50  0001 C CNN
+	1    7375 3400
+	0    1    1    0
+$EndComp
+$Comp
+L OSM_env01-rescue:Test_Point-Connector-ESP32-EVB_Rev_D-rescue TP?
+U 1 1 61C9FDCC
+P 7375 4325
+AR Path="/60688D25/61C9FDCC" Ref="TP?"  Part="1"
+AR Path="/6064BC1D/61C9FDCC" Ref="TP41"  Part="1"
+F 0 "TP41" V 7375 4600 50  0000 C CNN
+F 1 "Test_Point" V 7479 4397 50  0001 C CNN
+F 2 "TestPoint:TestPoint_THTPad_D1.0mm_Drill0.5mm" H 7575 4325 50  0001 C CNN
+F 3 "~" H 7575 4325 50  0001 C CNN
+	1    7375 4325
+	0    1    1    0
+$EndComp
+Wire Wire Line
+	7375 4325 7375 4200
+Connection ~ 7375 4200
+Wire Wire Line
+	7375 4200 7475 4200
+Wire Wire Line
+	7375 3400 7375 3525
+Connection ~ 7375 3525
+Wire Wire Line
+	7375 3525 7475 3525
 $EndSCHEMATC

Commit message: rough layout with throwdown of parts
Parts:
- removed R86: DNF, Resistor_SMD:R_0603_1608Metric, symbol device:R
- removed U8: SN65HVD230D, Package_SO:SOIC-8_3.9x4.9mm_P1.27mm, symbol OSM_env01-rescue:MCP2551-I-P-Devtank
- added C58, C75, C77: DNF, Capacitor_SMD:C_0603_1608Metric, symbol device:C
- added C79: C, Capacitor_SMD:C_0603_1608Metric, symbol device:C
- added D12: D_TVS_x2_AAC, Package_TO_SOT_SMD:SOT-23, symbol device:D_TVS_x2_AAC
- added R31: DNF, Resistor_SMD:R_0603_1608Metric, symbol device:R
- added U8: SN65HVD230, Package_SO:SOIC-8_3.9x4.9mm_P1.27mm, symbol interface:SN65HVD230
- R23, R24, R25: footprint (none) -> Resistor_SMD:R_0603_1608Metric
- TP22, TP23, TP41, TP80, TP81: footprint TestPoint:TestPoint_THTPad_D1.0mm_Drill0.5mm -> TestPoint:TestPoint_Pad_D1.5mm
Connections:
- net CAN_H: now also C77.2, D12.2 (A2), U8.7 (CANH)
- net CAN_L: now also C79.2, D12.1 (A1), U8.6 (CANL)
- net CAN_RS: now also C75.2, U8.8 (Rs)
- net CAN_VDD: now also C37.2, C38.2, R31.2, U8.3 (VCC); no longer C37.1, C38.1
- net GND: now also C37.1, C38.1, C58.2, C75.1, C77.1, C79.1, D12.3 (common), U8.2 (GND); no longer C37.2, C38.2
- net at R84.2: now also C58.1, U8.1 (D)
- net at R85.2: now also U8.4 (R)
- new net: R31.1, U8.5 (Vref)
Other:
- note added: "Note: C58 and 75 are filtering caps"
- moved on the sheet: C37, C38, R23, R24, R25, R80, R82, R83, R84, R85, R87, TP22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
