File: kicad_osm_env01/RS485_Comms.sch (KiCad schematic (older format))
At the start: 12 parts

Commit message: kicad review sch initial
Connections:
- net Electric_RX renamed RS485_RX
- net Electric_TX renamed RS485_TX
Changed lines of the file:
@@
 $Descr A4 11693 8268
 encoding utf-8
-Sheet 8 9
+Sheet 7 9
 Title ""
 Date ""
@@
 	6500 3650 6500 3600
 Wire Wire Line
-	6500 4100 7025 4100
+	6500 4100 6950 4100
 Connection ~ 6500 4100
 Wire Wire Line
 	6500 4100 6500 4050
-Text Notes 6750 3775 0    50   ~ 0
+Text Notes 7650 3700 0    50   ~ 0
 black wire
-Text Notes 6775 4200 0    50   ~ 0
+Text Notes 7675 4125 0    50   ~ 0
 red wire
 Wire Wire Line
 	6250 2825 6500 2825
 Connection ~ 6250 2825
-Text Label 7025 4100 2    50   ~ 0
-RS485+
-Wire Wire Line
-	6500 3650 7025 3650
-Text Label 7025 3650 2    50   ~ 0
-RS485-
+Wire Wire Line
+	6500 3650 6950 3650
 Wire Wire Line
 	4425 3825 5025 3825
@@
 $EndComp
 Wire Wire Line
-	4750 3925 5025 3925
-Text Label 4750 3925 0    50   ~ 0
-DE_485
+	4750 3925 4975 3925
 $Comp
 L OSM_env01-rescue:Test_Point-Connector-ESP32-EVB_Rev_D-rescue TP?
@@
 $EndComp
 Wire Wire Line
-	4550 4175 5025 4175
-Text Label 4550 4175 0    50   ~ 0
-Electric_TX
+	4550 4175 4875 4175
 Connection ~ 4900 3625
 $Comp
@@
 $EndComp
 Wire Wire Line
-	4450 3625 4900 3625
-Text Label 4450 3625 0    50   ~ 0
-Electric_RX
+	4450 3625 4775 3625
+Text HLabel 7125 3750 2    50   Input ~ 0
+RS485-
+Text HLabel 7125 4200 2    50   Input ~ 0
+RS485+
+Wire Wire Line
+	7125 3750 6950 3750
+Wire Wire Line
+	6950 3750 6950 3650
+Connection ~ 6950 3650
+Wire Wire Line
+	6950 3650 7025 3650
+Wire Wire Line
+	7125 4200 6950 4200
+Wire Wire Line
+	6950 4200 6950 4100
+Connection ~ 6950 4100
+Wire Wire Line
+	6950 4100 7025 4100
+Text HLabel 4925 4025 0    50   Input ~ 0
+DE_485
+Wire Wire Line
+	4925 4025 4975 4025
+Wire Wire Line
+	4975 4025 4975 3925
+Connection ~ 4975 3925
+Wire Wire Line
+	4975 3925 5025 3925
+Text HLabel 4825 4275 0    50   Input ~ 0
+RS485_TX
+Text HLabel 4725 3525 0    50   Input ~ 0
+RS485_RX
+Wire Wire Line
+	4725 3525 4775 3525
+Wire Wire Line
+	4775 3525 4775 3625
+Connection ~ 4775 3625
+Wire Wire Line
+	4775 3625 4900 3625
+Wire Wire Line
+	4825 4275 4875 4275
+Wire Wire Line
+	4875 4275 4875 4175
+Connection ~ 4875 4175
+Wire Wire Line
+	4875 4175 5025 4175
 $EndSCHEMATC

Commit message: updated schematics
Parts:
- gave numbers to parts that had none: 12
Changed lines of the file:
@@
 $Descr A4 11693 8268
 encoding utf-8
-Sheet 7 9
+Sheet 7 11
 Title ""
 Date ""
@@
 P 5650 3925
 AR Path="/609E7D18" Ref="U?"  Part="1"
-AR Path="/609D4B87/609E7D18" Ref="U?"  Part="1"
-F 0 "U?" H 5225 4775 50  0000 C CNN
+AR Path="/609D4B87/609E7D18" Ref="U7"  Part="1"
+F 0 "U7" H 5225 4775 50  0000 C CNN
 F 1 "ISL83485" H 5350 4675 50  0000 C CNN
 F 2 "Package_SO:SOIC-8_3.9x4.9mm_P1.27mm" H 5525 3925 50  0001 C CIN
@@
 P 4275 3825
 AR Path="/609E7D1E" Ref="R?"  Part="1"
-AR Path="/609D4B87/609E7D1E" Ref="R?"  Part="1"
-F 0 "R?" V 4175 3825 50  0000 C CNN
+AR Path="/609D4B87/609E7D1E" Ref="R70"  Part="1"
+F 0 "R70" V 4175 3825 50  0000 C CNN
 F 1 "10K" V 4100 3825 50  0000 C CNN
 F 2 "Resistor_SMD:R_0603_1608Metric" V 4205 3825 50  0001 C CNN
@@
 P 6250 3075
 AR Path="/609E7D24" Ref="C?"  Part="1"
-AR Path="/609D4B87/609E7D24" Ref="C?"  Part="1"
-F 0 "C?" H 5900 3125 50  0000 L CNN
+AR Path="/609D4B87/609E7D24" Ref="C36"  Part="1"
+F 0 "C36" H 5900 3125 50  0000 L CNN
 F 1 "100nF" H 5900 3050 50  0000 L CNN
 F 2 "Capacitor_SMD:C_0402_1005Metric" H 6288 2925 50  0001 C CNN
@@
 P 4900 3375
 AR Path="/609E7D2A" Ref="R?"  Part="1"
-AR Path="/609D4B87/609E7D2A" Ref="R?"  Part="1"
-F 0 "R?" H 4970 3421 50  0000 L CNN
+AR Path="/609D4B87/609E7D2A" Ref="R72"  Part="1"
+F 0 "R72" H 4970 3421 50  0000 L CNN
 F 1 "10K" H 4970 3330 50  0000 L CNN
 F 2 "Resistor_SMD:R_0603_1608Metric" V 4830 3375 50  0001 C CNN
@@
 P 6500 3450
 AR Path="/609E7D30" Ref="R?"  Part="1"
-AR Path="/609D4B87/609E7D30" Ref="R?"  Part="1"
-F 0 "R?" H 6570 3496 50  0000 L CNN
+AR Path="/609D4B87/609E7D30" Ref="R73"  Part="1"
+F 0 "R73" H 6570 3496 50  0000 L CNN
 F 1 "470R" H 6570 3405 50  0000 L CNN
 F 2 "Resistor_SMD:R_0603_1608Metric" V 6430 3450 50  0001 C CNN
@@
 P 6500 3875
 AR Path="/609E7D36" Ref="R?"  Part="1"
-AR Path="/609D4B87/609E7D36" Ref="R?"  Part="1"
-F 0 "R?" H 6570 3921 50  0000 L CNN
+AR Path="/609D4B87/609E7D36" Ref="R74"  Part="1"
+F 0 "R74" H 6570 3921 50  0000 L CNN
 F 1 "120R" H 6570 3830 50  0000 L CNN
 F 2 "Resistor_SMD:R_0603_1608Metric" V 6430 3875 50  0001 C CNN
@@
 P 6500 4325
 AR Path="/609E7D3C" Ref="R?"  Part="1"
-AR Path="/609D4B87/609E7D3C" Ref="R?"  Part="1"
-F 0 "R?" H 6570 4371 50  0000 L CNN
+AR Path="/609D4B87/609E7D3C" Ref="R75"  Part="1"
+F 0 "R75" H 6570 4371 50  0000 L CNN
 F 1 "470R" H 6570 4280 50  0000 L CNN
 F 2 "Resistor_SMD:R_0603_1608Metric" V 6430 4325 50  0001 C CNN
@@
 P 5650 4775
 AR Path="/609E7D49" Ref="#PWR?"  Part="1"
-AR Path="/609D4B87/609E7D49" Ref="#PWR?"  Part="1"
-F 0 "#PWR?" H 5650 4525 50  0001 C CNN
+AR Path="/609D4B87/609E7D49" Ref="#PWR056"  Part="1"
+F 0 "#PWR056" H 5650 4525 50  0001 C CNN
 F 1 "GND" H 5655 4602 50  0000 C CNN
 F 2 "" H 5650 4775 60  0000 C CNN
@@
 P 5650 2700
 AR Path="/609E7D4F" Ref="#PWR?"  Part="1"
-AR Path="/609D4B87/609E7D4F" Ref="#PWR?"  Part="1"
-F 0 "#PWR?" H 5650 2550 50  0001 C CNN
+AR Path="/609D4B87/609E7D4F" Ref="#PWR055"  Part="1"
+F 0 "#PWR055" H 5650 2550 50  0001 C CNN
 F 1 "+3V3" H 5665 2873 50  0000 C CNN
 F 2 "" H 5650 2700 50  0001 C CNN
@@
 P 6250 3300
 AR Path="/609E7D60" Ref="#PWR?"  Part="1"
-AR Path="/609D4B87/609E7D60" Ref="#PWR?"  Part="1"
-F 0 "#PWR?" H 6250 3050 50  0001 C CNN
+AR Path="/609D4B87/609E7D60" Ref="#PWR057"  Part="1"
+F 0 "#PWR057" H 6250 3050 50  0001 C CNN
 F 1 "GND" H 6255 3127 50  0000 C CNN
 F 2 "" H 6250 3300 60  0000 C CNN
@@
 P 4050 3850
 AR Path="/609E7D6C" Ref="#PWR?"  Part="1"
-AR Path="/609D4B87/609E7D6C" Ref="#PWR?"  Part="1"
-F 0 "#PWR?" H 4050 3600 50  0001 C CNN
+AR Path="/609D4B87/609E7D6C" Ref="#PWR054"  Part="1"
+F 0 "#PWR054" H 4050 3600 50  0001 C CNN
 F 1 "GND" H 3900 3775 50  0000 C CNN
 F 2 "" H 4050 3850 60  0000 C CNN
@@
 P 7025 3650
 AR Path="/609E7D86" Ref="TP?"  Part="1"
-AR Path="/609D4B87/609E7D86" Ref="TP?"  Part="1"
-F 0 "TP?" V 6950 3925 50  0000 C CNN
+AR Path="/609D4B87/609E7D86" Ref="TP39"  Part="1"
+F 0 "TP39" V 6950 3925 50  0000 C CNN
 F 1 "Test_Point" V 7025 4025 50  0000 C CNN
 F 2 "TestPoint:TestPoint_THTPad_D1.0mm_Drill0.5mm" H 7225 3650 50  0001 C CNN
@@
 P 7025 4100
 AR Path="/609E7D8C" Ref="TP?"  Part="1"
-AR Path="/609D4B87/609E7D8C" Ref="TP?"  Part="1"
-F 0 "TP?" V 6950 4375 50  0000 C CNN
+AR Path="/609D4B87/609E7D8C" Ref="TP40"  Part="1"
+F 0 "TP40" V 6950 4375 50  0000 C CNN
 F 1 "Test_Point" V 7025 4475 50  0000 C CNN
 F 2 "TestPoint:TestPoint_THTPad_D1.0mm_Drill0.5mm" H 7225 4100 50  0001 C CNN
@@
 P 4750 3925
 AR Path="/609E7D92" Ref="TP?"  Part="1"
-AR Path="/609D4B87/609E7D92" Ref="TP?"  Part="1"
-F 0 "TP?" V 4700 3925 50  0000 C CNN
+AR Path="/609D4B87/609E7D92" Ref="TP38"  Part="1"
+F 0 "TP38" V 4700 3925 50  0000 C CNN
 F 1 "Test_Point" V 4625 4025 50  0000 C CNN
 F 2 "TestPoint:TestPoint_THTPad_D1.0mm_Drill0.5mm" H 4950 3925 50  0001 C CNN
@@
 P 4550 4175
 AR Path="/609E7D9A" Ref="TP?"  Part="1"
-AR Path="/609D4B87/609E7D9A" Ref="TP?"  Part="1"
-F 0 "TP?" V 4575 4650 50  0000 C CNN
+AR Path="/609D4B87/609E7D9A" Ref="TP37"  Part="1"
+F 0 "TP37" V 4575 4650 50  0000 C CNN
 F 1 "Test_Point" V 4475 4550 50  0000 C CNN
 F 2 "TestPoint:TestPoint_THTPad_D1.0mm_Drill0.5mm" H 4750 4175 50  0001 C CNN
@@
 P 4450 3625
 AR Path="/609E7DA3" Ref="TP?"  Part="1"
-AR Path="/609D4B87/609E7DA3" Ref="TP?"  Part="1"
-F 0 "TP?" V 4645 3697 50  0000 C CNN
+AR Path="/609D4B87/609E7DA3" Ref="TP36"  Part="1"
+F 0 "TP36" V 4645 3697 50  0000 C CNN
 F 1 "Test_Point" V 4554 3697 50  0000 C CNN
 F 2 "TestPoint:TestPoint_THTPad_D1.0mm_Drill0.5mm" H 4650 3625 50  0001 C CNN

Commit message: schematics awaiting review
Other:
- moved on the sheet: R70, TP36, TP37
Changed lines of the file:
@@
 $Descr A4 11693 8268
 encoding utf-8
-Sheet 7 11
+Sheet 4 11
 Title ""
 Date ""
@@
 L OSM_env01-rescue:R-device-ESP32-EVB_Rev_D-rescue R?
 U 1 1 609E7D1E
-P 4275 3825
+P 4150 3825
 AR Path="/609E7D1E" Ref="R?"  Part="1"
 AR Path="/609D4B87/609E7D1E" Ref="R70"  Part="1"
-F 0 "R70" V 4175 3825 50  0000 C CNN
-F 1 "10K" V 4100 3825 50  0000 C CNN
-F 2 "Resistor_SMD:R_0603_1608Metric" V 4205 3825 50  0001 C CNN
-F 3 "" H 4275 3825 50  0001 C CNN
-	1    4275 3825
+F 0 "R70" V 4050 3825 50  0000 C CNN
+F 1 "10K" V 3975 3825 50  0000 C CNN
+F 2 "Resistor_SMD:R_0603_1608Metric" V 4080 3825 50  0001 C CNN
+F 3 "" H 4150 3825 50  0001 C CNN
+	1    4150 3825
 	0    -1   -1   0
 $EndComp
@@
 L OSM_env01-rescue:GND-ESP32-EVB_Rev_D #PWR?
 U 1 1 609E7D6C
-P 4050 3850
+P 3925 3850
 AR Path="/609E7D6C" Ref="#PWR?"  Part="1"
 AR Path="/609D4B87/609E7D6C" Ref="#PWR054"  Part="1"
-F 0 "#PWR054" H 4050 3600 50  0001 C CNN
-F 1 "GND" H 3900 3775 50  0000 C CNN
-F 2 "" H 4050 3850 60  0000 C CNN
-F 3 "" H 4050 3850 60  0000 C CNN
-	1    4050 3850
-	1    0    0    -1
-$EndComp
-Wire Wire Line
-	4050 3850 4050 3825
-Wire Wire Line
-	4050 3825 4125 3825
+F 0 "#PWR054" H 3925 3600 50  0001 C CNN
+F 1 "GND" H 3775 3775 50  0000 C CNN
+F 2 "" H 3925 3850 60  0000 C CNN
+F 3 "" H 3925 3850 60  0000 C CNN
+	1    3925 3850
+	1    0    0    -1
+$EndComp
+Wire Wire Line
+	3925 3850 3925 3825
+Wire Wire Line
+	3925 3825 4000 3825
 Wire Wire Line
 	4900 3025 5650 3025
@@
 	6500 3650 6950 3650
 Wire Wire Line
-	4425 3825 5025 3825
-Wire Wire Line
 	6250 3975 6300 3975
 Wire Wire Line
@@
 AR Path="/609E7D86" Ref="TP?"  Part="1"
 AR Path="/609D4B87/609E7D86" Ref="TP39"  Part="1"
-F 0 "TP39" V 6950 3925 50  0000 C CNN
-F 1 "Test_Point" V 7025 4025 50  0000 C CNN
+F 0 "TP39" V 7025 3925 50  0000 C CNN
+F 1 "Test_Point" V 7025 4025 50  0001 C CNN
 F 2 "TestPoint:TestPoint_THTPad_D1.0mm_Drill0.5mm" H 7225 3650 50  0001 C CNN
 F 3 "~" H 7225 3650 50  0001 C CNN
@@
 AR Path="/609E7D8C" Ref="TP?"  Part="1"
 AR Path="/609D4B87/609E7D8C" Ref="TP40"  Part="1"
-F 0 "TP40" V 6950 4375 50  0000 C CNN
-F 1 "Test_Point" V 7025 4475 50  0000 C CNN
+F 0 "TP40" V 7025 4375 50  0000 C CNN
+F 1 "Test_Point" V 7025 4475 50  0001 C CNN
 F 2 "TestPoint:TestPoint_THTPad_D1.0mm_Drill0.5mm" H 7225 4100 50  0001 C CNN
 F 3 "~" H 7225 4100 50  0001 C CNN
@@
 AR Path="/609E7D92" Ref="TP?"  Part="1"
 AR Path="/609D4B87/609E7D92" Ref="TP38"  Part="1"
-F 0 "TP38" V 4700 3925 50  0000 C CNN
-F 1 "Test_Point" V 4625 4025 50  0000 C CNN
+F 0 "TP38" V 4750 4200 50  0000 C CNN
+F 1 "Test_Point" V 4675 4300 50  0001 C CNN
 F 2 "TestPoint:TestPoint_THTPad_D1.0mm_Drill0.5mm" H 4950 3925 50  0001 C CNN
 F 3 "~" H 4950 3925 50  0001 C CNN
@@
 	0    -1   -1   0
 $EndComp
-Wire Wire Line
-	4750 3925 4975 3925
-$Comp
-L OSM_env01-rescue:Test_Point-Connector-ESP32-EVB_Rev_D-rescue TP?
-U 1 1 609E7D9A
-P 4550 4175
-AR Path="/609E7D9A" Ref="TP?"  Part="1"
-AR Path="/609D4B87/609E7D9A" Ref="TP37"  Part="1"
-F 0 "TP37" V 4575 4650 50  0000 C CNN
-F 1 "Test_Point" V 4475 4550 50  0000 C CNN
-F 2 "TestPoint:TestPoint_THTPad_D1.0mm_Drill0.5mm" H 4750 4175 50  0001 C CNN
-F 3 "~" H 4750 4175 50  0001 C CNN
-	1    4550 4175
-	0    -1   -1   0
-$EndComp
-Wire Wire Line
-	4550 4175 4875 4175
 Connection ~ 4900 3625
 $Comp
 L OSM_env01-rescue:Test_Point-Connector-ESP32-EVB_Rev_D-rescue TP?
 U 1 1 609E7DA3
-P 4450 3625
+P 4650 3525
 AR Path="/609E7DA3" Ref="TP?"  Part="1"
 AR Path="/609D4B87/609E7DA3" Ref="TP36"  Part="1"
-F 0 "TP36" V 4645 3697 50  0000 C CNN
-F 1 "Test_Point" V 4554 3697 50  0000 C CNN
-F 2 "TestPoint:TestPoint_THTPad_D1.0mm_Drill0.5mm" H 4650 3625 50  0001 C CNN
-F 3 "~" H 4650 3625 50  0001 C CNN
-	1    4450 3625
+F 0 "TP36" V 4650 3800 50  0000 C CNN
+F 1 "Test_Point" V 4775 3900 50  0001 C CNN
+F 2 "TestPoint:TestPoint_THTPad_D1.0mm_Drill0.5mm" H 4850 3525 50  0001 C CNN
+F 3 "~" H 4850 3525 50  0001 C CNN
+	1    4650 3525
 	0    -1   -1   0
 $EndComp
-Wire Wire Line
-	4450 3625 4775 3625
 Text HLabel 7125 3750 2    50   Input ~ 0
 RS485-
@@
 Wire Wire Line
 	6950 4100 7025 4100
-Text HLabel 4925 4025 0    50   Input ~ 0
+Text HLabel 4725 4025 0    50   Input ~ 0
 DE_485
-Wire Wire Line
-	4925 4025 4975 4025
-Wire Wire Line
-	4975 4025 4975 3925
-Connection ~ 4975 3925
-Wire Wire Line
-	4975 3925 5025 3925
+Text HLabel 4725 3625 0    50   Input ~ 0
+RS485_RX
+Wire Wire Line
+	4825 4275 4875 4275
+Wire Wire Line
+	4875 4275 4875 4175
+Wire Wire Line
+	4875 4175 5025 4175
+Wire Wire Line
+	4300 3825 5025 3825
+Wire Wire Line
+	4750 3925 4875 3925
+Wire Wire Line
+	4875 3925 4875 4025
+Wire Wire Line
+	4875 4025 4725 4025
+Connection ~ 4875 3925
+Wire Wire Line
+	4875 3925 5025 3925
 Text HLabel 4825 4275 0    50   Input ~ 0
 RS485_TX
-Text HLabel 4725 3525 0    50   Input ~ 0
-RS485_RX
-Wire Wire Line
-	4725 3525 4775 3525
+$Comp
+L OSM_env01-rescue:Test_Point-Connector-ESP32-EVB_Rev_D-rescue TP?
+U 1 1 609E7D9A
+P 4750 4175
+AR Path="/609E7D9A" Ref="TP?"  Part="1"
+AR Path="/609D4B87/609E7D9A" Ref="TP37"  Part="1"
+F 0 "TP37" V 4750 4450 50  0000 C CNN
+F 1 "Test_Point" V 4675 4550 50  0001 C CNN
+F 2 "TestPoint:TestPoint_THTPad_D1.0mm_Drill0.5mm" H 4950 4175 50  0001 C CNN
+F 3 "~" H 4950 4175 50  0001 C CNN
+	1    4750 4175
+	0    -1   -1   0
+$EndComp
+Wire Wire Line
+	4750 4175 4875 4175
+Connection ~ 4875 4175
+Wire Wire Line
+	4725 3625 4775 3625
+Wire Wire Line
+	4650 3525 4775 3525
 Wire Wire Line
 	4775 3525 4775 3625
@@
 Wire Wire Line
 	4775 3625 4900 3625
-Wire Wire Line
-	4825 4275 4875 4275
-Wire Wire Line
-	4875 4275 4875 4175
-Connection ~ 4875 4175
-Wire Wire Line
-	4875 4175 5025 4175
 $EndSCHEMATC

Commit message: schematics awaiting review
Parts:
- added TP20: Test_Point, TestPoint:TestPoint_THTPad_D1.0mm_Drill0.5mm, symbol OSM_env01-rescue:Test_Point-Connector-ESP32-EVB_Rev_D-rescue
- U7: value ISL83485 -> ST3485EBDR
Connections:
- net at R70.2, U7.2 (~RE): now also TP20.1
Other:
- note removed: "Electricty Meter"
- note removed: "black wire"
- note removed: "red wire"
Changed lines of the file:
@@
 AR Path="/609D4B87/609E7D18" Ref="U7"  Part="1"
 F 0 "U7" H 5225 4775 50  0000 C CNN
-F 1 "ISL83485" H 5350 4675 50  0000 C CNN
+F 1 "ST3485EBDR" H 5350 4675 50  0000 C CNN
 F 2 "Package_SO:SOIC-8_3.9x4.9mm_P1.27mm" H 5525 3925 50  0001 C CIN
 F 3 "http://www.intersil.com/content/dam/Intersil/documents/isl8/isl83483-85-88-90-91.pdf" H 5525 3925 50  0001 C CNN
@@
 Wire Wire Line
 	4900 3025 5650 3025
-Text Notes 4750 5250 0    118  ~ 0
-Electricty Meter
 Connection ~ 6500 3650
 Wire Wire Line
@@
 Wire Wire Line
 	6500 4100 6500 4050
-Text Notes 7650 3700 0    50   ~ 0
-black wire
-Text Notes 7675 4125 0    50   ~ 0
-red wire
 Wire Wire Line
 	6250 2825 6500 2825
@@
 	4875 4175 5025 4175
 Wire Wire Line
-	4300 3825 5025 3825
+	4300 3825 4775 3825
 Wire Wire Line
 	4750 3925 4875 3925
@@
 Wire Wire Line
 	4775 3625 4900 3625
+$Comp
+L OSM_env01-rescue:Test_Point-Connector-ESP32-EVB_Rev_D-rescue TP?
+U 1 1 61C934C6
+P 4650 3750
+AR Path="/61C934C6" Ref="TP?"  Part="1"
+AR Path="/609D4B87/61C934C6" Ref="TP20"  Part="1"
+F 0 "TP20" V 4650 4025 50  0000 C CNN
+F 1 "Test_Point" V 4775 4125 50  0001 C CNN
+F 2 "TestPoint:TestPoint_THTPad_D1.0mm_Drill0.5mm" H 4850 3750 50  0001 C CNN
+F 3 "~" H 4850 3750 50  0001 C CNN
+	1    4650 3750
+	0    -1   -1   0
+$EndComp
+Wire Wire Line
+	4650 3750 4775 3750
+Wire Wire Line
+	4775 3750 4775 3825
+Connection ~ 4775 3825
+Wire Wire Line
+	4775 3825 5025 3825
 $EndSCHEMATC

Commit message: rough layout with throwdown of parts
Parts:
- TP20, TP36, TP37, TP38, TP39, TP40: footprint TestPoint:TestPoint_THTPad_D1.0mm_Drill0.5mm -> TestPoint:TestPoint_Pad_D1.5mm
Changed lines of the file:
@@
 $Descr A4 11693 8268
 encoding utf-8
-Sheet 4 11
+Sheet 4 9
 Title ""
 Date ""
@@
 F 0 "TP39" V 7025 3925 50  0000 C CNN
 F 1 "Test_Point" V 7025 4025 50  0001 C CNN
-F 2 "TestPoint:TestPoint_THTPad_D1.0mm_Drill0.5mm" H 7225 3650 50  0001 C CNN
+F 2 "TestPoint:TestPoint_Pad_D1.5mm" H 7225 3650 50  0001 C CNN
 F 3 "~" H 7225 3650 50  0001 C CNN
 	1    7025 3650
@@
 F 0 "TP40" V 7025 4375 50  0000 C CNN
 F 1 "Test_Point" V 7025 4475 50  0001 C CNN
-F 2 "TestPoint:TestPoint_THTPad_D1.0mm_Drill0.5mm" H 7225 4100 50  0001 C CNN
+F 2 "TestPoint:TestPoint_Pad_D1.5mm" H 7225 4100 50  0001 C CNN
 F 3 "~" H 7225 4100 50  0001 C CNN
 	1    7025 4100
@@
 F 0 "TP38" V 4750 4200 50  0000 C CNN
 F 1 "Test_Point" V 4675 4300 50  0001 C CNN
-F 2 "TestPoint:TestPoint_THTPad_D1.0mm_Drill0.5mm" H 4950 3925 50  0001 C CNN
+F 2 "TestPoint:TestPoint_Pad_D1.5mm" H 4950 3925 50  0001 C CNN
 F 3 "~" H 4950 3925 50  0001 C CNN
 	1    4750 3925
@@
 F 0 "TP36" V 4650 3800 50  0000 C CNN
 F 1 "Test_Point" V 4775 3900 50  0001 C CNN
-F 2 "TestPoint:TestPoint_THTPad_D1.0mm_Drill0.5mm" H 4850 3525 50  0001 C CNN
+F 2 "TestPoint:TestPoint_Pad_D1.5mm" H 4850 3525 50  0001 C CNN
 F 3 "~" H 4850 3525 50  0001 C CNN
 	1    4650 3525
@@
 F 0 "TP37" V 4750 4450 50  0000 C CNN
 F 1 "Test_Point" V 4675 4550 50  0001 C CNN
-F 2 "TestPoint:TestPoint_THTPad_D1.0mm_Drill0.5mm" H 4950 4175 50  0001 C CNN
+F 2 "TestPoint:TestPoint_Pad_D1.5mm" H 4950 4175 50  0001 C CNN
 F 3 "~" H 4950 4175 50  0001 C CNN
 	1    4750 4175
@@
 F 0 "TP20" V 4650 4025 50  0000 C CNN
 F 1 "Test_Point" V 4775 4125 50  0001 C CNN
-F 2 "TestPoint:TestPoint_THTPad_D1.0mm_Drill0.5mm" H 4850 3750 50  0001 C CNN
+F 2 "TestPoint:TestPoint_Pad_D1.5mm" H 4850 3750 50  0001 C CNN
 F 3 "~" H 4850 3750 50  0001 C CNN
 	1    4650 3750
