File: kicad_osm_env01/RS485_Comms.sch (KiCad schematic (older format))
At the start: 15 parts, among them U7 ST3485EBDR

Commit message: Updated schematics
Parts:
- removed R70: DNF, Resistor_SMD:R_0603_1608Metric, symbol OSM_env01-rescue:R-device-ESP32-EVB_Rev_D-rescue
- added L5: 2A/0.05DCR, Inductor_SMD:L_0402_1005Metric, symbol device:Ferrite_Bead
Connections:
- net +3V3: now also L5.1; no longer C36.1, R72.1, R73.1, U7.8 (Vcc)
- new net: C36.1, L5.2, R72.1, R73.1, U7.8 (Vcc)
Other:
- moved on the sheet: R33, TP20, TP37
Changed lines of the file:
@@
 encoding utf-8
 Sheet 4 9
-Title ""
-Date ""
-Rev ""
-Comp ""
-Comment1 ""
+Title "Open Smart Monitor"
+Date "2021-09-22"
+Rev "B"
+Comp "Devtank LTD"
+Comment1 "AB"
 Comment2 ""
 Comment3 ""
@@
 AR Path="/609E7D18" Ref="U?"  Part="1"
 AR Path="/609D4B87/609E7D18" Ref="U7"  Part="1"
-F 0 "U7" H 5225 4775 50  0000 C CNN
-F 1 "ST3485EBDR" H 5350 4675 50  0000 C CNN
+F 0 "U7" H 5100 4725 50  0000 C CNN
+F 1 "ST3485EBDR" H 5300 4650 50  0000 C CNN
 F 2 "Package_SO:SOIC-8_3.9x4.9mm_P1.27mm" H 5525 3925 50  0001 C CIN
 F 3 "http://www.intersil.com/content/dam/Intersil/documents/isl8/isl83483-85-88-90-91.pdf" H 5525 3925 50  0001 C CNN
 	1    5650 3925
 	1    0    0    -1
-$EndComp
-$Comp
-L OSM_env01-rescue:R-device-ESP32-EVB_Rev_D-rescue R?
-U 1 1 609E7D1E
-P 3925 3575
-AR Path="/609E7D1E" Ref="R?"  Part="1"
-AR Path="/609D4B87/609E7D1E" Ref="R70"  Part="1"
-F 0 "R70" V 3825 3575 50  0000 C CNN
-F 1 "DNF" V 3750 3575 50  0000 C CNN
-F 2 "Resistor_SMD:R_0603_1608Metric" V 3855 3575 50  0001 C CNN
-F 3 "" H 3925 3575 50  0001 C CNN
-	1    3925 3575
-	0    -1   -1   0
 $EndComp
 $Comp
@@
 $Comp
 L OSM_env01-rescue:R-device-ESP32-EVB_Rev_D-rescue R?
-U 1 1 609E7D2A
-P 4900 3375
-AR Path="/609E7D2A" Ref="R?"  Part="1"
-AR Path="/609D4B87/609E7D2A" Ref="R72"  Part="1"
-F 0 "R72" H 4970 3421 50  0000 L CNN
-F 1 "10K" H 4970 3330 50  0000 L CNN
-F 2 "Resistor_SMD:R_0603_1608Metric" V 4830 3375 50  0001 C CNN
-F 3 "" H 4900 3375 50  0001 C CNN
-	1    4900 3375
-	1    0    0    -1
-$EndComp
-$Comp
-L OSM_env01-rescue:R-device-ESP32-EVB_Rev_D-rescue R?
 U 1 1 609E7D30
 P 6500 3450
@@
 	1    0    0    -1
 $EndComp
-$Comp
-L power:+3V3 #PWR?
-U 1 1 609E7D4F
-P 5650 2700
-AR Path="/609E7D4F" Ref="#PWR?"  Part="1"
-AR Path="/609D4B87/609E7D4F" Ref="#PWR055"  Part="1"
-F 0 "#PWR055" H 5650 2550 50  0001 C CNN
-F 1 "+3V3" H 5665 2873 50  0000 C CNN
-F 2 "" H 5650 2700 50  0001 C CNN
-F 3 "" H 5650 2700 50  0001 C CNN
-	1    5650 2700
-	1    0    0    -1
-$EndComp
 Wire Wire Line
 	5650 4625 5650 4700
@@
 	5025 3625 4900 3625
 Wire Wire Line
-	4900 3625 4900 3525
-Wire Wire Line
-	4900 3225 4900 3025
-Wire Wire Line
 	5650 3025 5650 3100
 Connection ~ 5650 3025
-Wire Wire Line
-	5650 2700 5650 2825
 $Comp
 L OSM_env01-rescue:GND-ESP32-EVB_Rev_D #PWR?
@@
 	6250 2925 6250 2825
 Wire Wire Line
-	6250 2825 5650 2825
-Connection ~ 5650 2825
-Wire Wire Line
 	5650 2825 5650 3025
 Wire Wire Line
@@
 Wire Wire Line
 	6250 3300 6250 3225
-$Comp
-L OSM_env01-rescue:GND-ESP32-EVB_Rev_D #PWR?
-U 1 1 609E7D6C
-P 3700 3600
-AR Path="/609E7D6C" Ref="#PWR?"  Part="1"
-AR Path="/609D4B87/609E7D6C" Ref="#PWR054"  Part="1"
-F 0 "#PWR054" H 3700 3350 50  0001 C CNN
-F 1 "GND" H 3550 3525 50  0000 C CNN
-F 2 "" H 3700 3600 60  0000 C CNN
-F 3 "" H 3700 3600 60  0000 C CNN
-	1    3700 3600
-	1    0    0    -1
-$EndComp
-Wire Wire Line
-	3700 3600 3700 3575
-Wire Wire Line
-	3700 3575 3775 3575
 Wire Wire Line
 	4900 3025 5650 3025
@@
 RS485_RX
 Wire Wire Line
-	4825 4275 4875 4275
+	4700 4275 4875 4275
 Wire Wire Line
 	4875 4275 4875 4175
@@
 Wire Wire Line
 	4375 3925 4525 3925
-Text HLabel 4825 4275 0    50   Input ~ 0
+Text HLabel 4700 4275 0    50   Input ~ 0
 RS485_TX
 $Comp
 L OSM_env01-rescue:Test_Point-Connector-ESP32-EVB_Rev_D-rescue TP?
 U 1 1 609E7D9A
-P 4750 4175
+P 4650 4175
 AR Path="/609E7D9A" Ref="TP?"  Part="1"
 AR Path="/609D4B87/609E7D9A" Ref="TP37"  Part="1"
-F 0 "TP37" V 4750 4450 50  0000 C CNN
-F 1 "Test_Point" V 4675 4550 50  0001 C CNN
-F 2 "TestPoint:TestPoint_Pad_D1.5mm" H 4950 4175 50  0001 C CNN
-F 3 "~" H 4950 4175 50  0001 C CNN
-	1    4750 4175
+F 0 "TP37" V 4650 4450 50  0000 C CNN
+F 1 "Test_Point" V 4575 4550 50  0001 C CNN
+F 2 "TestPoint:TestPoint_Pad_D1.5mm" H 4850 4175 50  0001 C CNN
+F 3 "~" H 4850 4175 50  0001 C CNN
+	1    4650 4175
 	0    -1   -1   0
 $EndComp
 Wire Wire Line
-	4750 4175 4875 4175
+	4650 4175 4875 4175
 Connection ~ 4875 4175
 Wire Wire Line
@@
 L OSM_env01-rescue:Test_Point-Connector-ESP32-EVB_Rev_D-rescue TP?
 U 1 1 61C934C6
-P 3850 3475
+P 3625 3525
 AR Path="/61C934C6" Ref="TP?"  Part="1"
 AR Path="/609D4B87/61C934C6" Ref="TP20"  Part="1"
-F 0 "TP20" V 3850 3750 50  0000 C CNN
-F 1 "Test_Point" V 3975 3850 50  0001 C CNN
-F 2 "TestPoint:TestPoint_Pad_D1.5mm" H 4050 3475 50  0001 C CNN
-F 3 "~" H 4050 3475 50  0001 C CNN
-	1    3850 3475
+F 0 "TP20" V 3625 3800 50  0000 C CNN
+F 1 "Test_Point" V 3750 3900 50  0001 C CNN
+F 2 "TestPoint:TestPoint_Pad_D1.5mm" H 3825 3525 50  0001 C CNN
+F 3 "~" H 3825 3525 50  0001 C CNN
+	1    3625 3525
 	0    -1   -1   0
 $EndComp
-Text HLabel 3625 3300 0    50   Input ~ 0
+Text HLabel 3525 3725 0    50   Input ~ 0
 RS485_RE
 Wire Wire Line
-	3775 3300 3625 3300
-Wire Wire Line
-	3850 3475 4075 3475
-Connection ~ 4075 3475
+	3675 3725 3525 3725
 $Comp
 L device:R R?
@@
 L device:R R?
 U 1 1 614D39E0
-P 3925 3300
+P 3825 3725
 AR Path="/6064BC1D/614D39E0" Ref="R?"  Part="1"
 AR Path="/609D4B87/614D39E0" Ref="R33"  Part="1"
-F 0 "R33" V 3825 3250 50  0000 C CNN
-F 1 "0R" V 4025 3225 50  0000 C CNN
-F 2 "" V 3855 3300 50  0001 C CNN
-F 3 "" H 3925 3300 50  0001 C CNN
-	1    3925 3300
-	0    1    1    0
-$EndComp
-Wire Wire Line
-	4075 3475 4075 3575
-Wire Wire Line
-	4075 3300 4075 3475
+F 0 "R33" V 3750 3725 50  0000 C CNN
+F 1 "0R" V 3900 3725 50  0000 C CNN
+F 2 "" V 3755 3725 50  0001 C CNN
+F 3 "" H 3825 3725 50  0001 C CNN
+	1    3825 3725
+	0    1    1    0
+$EndComp
 Wire Wire Line
 	5025 3925 4825 3925
@@
 	4875 3825 4875 3725
 Wire Wire Line
-	4075 3725 4075 3575
-Wire Wire Line
-	4075 3725 4875 3725
-Connection ~ 4075 3575
+	3625 3525 4125 3525
+Wire Wire Line
+	3975 3725 4125 3725
+Wire Wire Line
+	4900 3625 4900 3525
+Wire Wire Line
+	4900 3225 4900 3025
+$Comp
+L OSM_env01-rescue:R-device-ESP32-EVB_Rev_D-rescue R?
+U 1 1 609E7D2A
+P 4900 3375
+AR Path="/609E7D2A" Ref="R?"  Part="1"
+AR Path="/609D4B87/609E7D2A" Ref="R72"  Part="1"
+F 0 "R72" H 4970 3421 50  0000 L CNN
+F 1 "10K" H 4970 3330 50  0000 L CNN
+F 2 "Resistor_SMD:R_0603_1608Metric" V 4830 3375 50  0001 C CNN
+F 3 "" H 4900 3375 50  0001 C CNN
+	1    4900 3375
+	1    0    0    -1
+$EndComp
+Wire Wire Line
+	4125 3725 4875 3725
+Wire Wire Line
+	4125 3525 4125 3725
+Connection ~ 4125 3725
+$Comp
+L power:+3V3 #PWR?
+U 1 1 61A8701B
+P 6950 2575
+AR Path="/6064BC1D/61A8701B" Ref="#PWR?"  Part="1"
+AR Path="/609D4B87/61A8701B" Ref="#PWR0150"  Part="1"
+F 0 "#PWR0150" H 6950 2425 50  0001 C CNN
+F 1 "+3V3" H 6965 2748 50  0000 C CNN
+F 2 "" H 6950 2575 50  0001 C CNN
+F 3 "" H 6950 2575 50  0001 C CNN
+	1    6950 2575
+	1    0    0    -1
+$EndComp
+Wire Wire Line
+	5650 2825 6050 2825
+$Comp
+L device:Ferrite_Bead L?
+U 1 1 61AB23F3
+P 6650 2825
+AR Path="/61AB23F3" Ref="L?"  Part="1"
+AR Path="/60917DD5/61AB23F3" Ref="L?"  Part="1"
+AR Path="/608F4675/61AB23F3" Ref="L?"  Part="1"
+AR Path="/609D4B87/61AB23F3" Ref="L5"  Part="1"
+F 0 "L5" V 6376 2825 50  0000 C CNN
+F 1 "2A/0.05DCR" V 6467 2825 50  0000 C CNN
+F 2 "Inductor_SMD:L_0402_1005Metric" V 6580 2825 50  0001 C CNN
+F 3 "" H 6650 2825 50  0001 C CNN
+	1    6650 2825
+	0    1    1    0
+$EndComp
+Connection ~ 6500 2825
+Wire Wire Line
+	6800 2825 6950 2825
+Wire Wire Line
+	6950 2575 6950 2825
+$Comp
+L OSM_env01:PWR_FLAG #FLG0107
+U 1 1 61ADD768
+P 6050 2825
+F 0 "#FLG0107" H 6050 2920 50  0001 C CNN
+F 1 "PWR_FLAG" H 6050 3048 50  0000 C CNN
+F 2 "" H 6050 2825 60  0000 C CNN
+F 3 "" H 6050 2825 60  0000 C CNN
+	1    6050 2825
+	1    0    0    -1
+$EndComp
+Connection ~ 6050 2825
+Wire Wire Line
+	6050 2825 6250 2825
 $EndSCHEMATC

Commit message: rough throwdown of all parts
Parts:
- R33, R34: footprint (none) -> Resistor_SMD:R_0603_1608Metric
- R72: value 10K -> 10k
Changed lines of the file:
@@
 F 0 "R34" V 4575 3875 50  0000 C CNN
 F 1 "0R" V 4775 3850 50  0000 C CNN
-F 2 "" V 4605 3925 50  0001 C CNN
+F 2 "Resistor_SMD:R_0603_1608Metric" V 4605 3925 50  0001 C CNN
 F 3 "" H 4675 3925 50  0001 C CNN
 	1    4675 3925
@@
 F 0 "R33" V 3750 3725 50  0000 C CNN
 F 1 "0R" V 3900 3725 50  0000 C CNN
-F 2 "" V 3755 3725 50  0001 C CNN
+F 2 "Resistor_SMD:R_0603_1608Metric" V 3755 3725 50  0001 C CNN
 F 3 "" H 3825 3725 50  0001 C CNN
 	1    3825 3725
@@
 AR Path="/609D4B87/609E7D2A" Ref="R72"  Part="1"
 F 0 "R72" H 4970 3421 50  0000 L CNN
-F 1 "10K" H 4970 3330 50  0000 L CNN
+F 1 "10k" H 4970 3330 50  0000 L CNN
 F 2 "Resistor_SMD:R_0603_1608Metric" V 4830 3375 50  0001 C CNN
 F 3 "" H 4900 3375 50  0001 C CNN
