File: kicad_osm_env01/STM32L4.sch (KiCad schematic (older format))
At the start: 27 parts, among them J5 Conn_01x06, U14 STM32L451RCTx, Y1 8MHZ, Y2 DNF

Commit message: Updated schematics
Parts:
- removed J5: Conn_01x06, Connector:Tag-Connect_TC2030-IDC-NL_2x03_P1.27mm_Vertical, symbol Connector:Conn_01x06
- added J5: Conn_02x03_Odd_Even, symbol Connector:Conn_02x03_Odd_Even
Connections:
- net +3V3: now also J5.1 (Pin_1)
- net GND: now also J5.2 (Pin_2)
- net STM_NRST: now also J5.5 (Pin_5)
- net SWCLK: now also J5.4 (Pin_4)
- net SWD_IO: now also J5.6 (Pin_6)
Changed lines of the file:
@@
 encoding utf-8
 Sheet 6 9
-Title ""
-Date ""
-Rev ""
-Comp ""
-Comment1 ""
+Title "Open Smart Monitor"
+Date "2021-09-22"
+Rev "B"
+Comp "Devtank LTD"
+Comment1 "AB"
 Comment2 ""
 Comment3 ""
@@
 Text Label 7125 1325 2    50   ~ 0
 STM_NRST
-Text Label 9750 10650 0    50   ~ 0
+Text Label 9750 10450 0    50   ~ 0
 STM_NRST
-Text Label 9750 10750 0    50   ~ 0
+Text Label 11250 10450 2    50   ~ 0
 SWD_IO
 Wire Wire Line
-	10250 10650 9750 10650
-Text Label 9750 10550 0    50   ~ 0
+	10250 10450 9750 10450
+Text Label 11250 10350 2    50   ~ 0
 SWCLK
 Wire Wire Line
-	10250 10550 9750 10550
-Wire Wire Line
-	10250 10750 9750 10750
-Text Notes 9825 9875 0    50   ~ 0
+	10750 10350 11250 10350
+Wire Wire Line
+	10750 10450 11250 10450
+Text Notes 9950 9850 0    50   ~ 0
 SWD Programming Header
 $Comp
@@
 F 3 "" H 8000 1125 50  0001 C CNN
 	1    8000 1125
-	0    -1   -1   0
-$EndComp
-$Comp
-L device:R R16
-U 1 1 6142BFB9
-P 8000 1375
-F 0 "R16" V 7900 1300 50  0000 L CNN
-F 1 "10k" V 7800 1300 50  0000 L CNN
-F 2 "Resistor_SMD:R_0402_1005Metric" V 7930 1375 50  0001 C CNN
-F 3 "" H 8000 1375 50  0001 C CNN
-	1    8000 1375
 	0    -1   -1   0
 $EndComp
@@
 GPIO15
 $Comp
-L Connector:Conn_01x06 J5
-U 1 1 61452AC8
-P 10450 10450
-F 0 "J5" H 10530 10442 50  0000 L CNN
-F 1 "Conn_01x06" H 10530 10351 50  0000 L CNN
-F 2 "Connector:Tag-Connect_TC2030-IDC-NL_2x03_P1.27mm_Vertical" H 10450 10450 50  0001 C CNN
-F 3 "~" H 10450 10450 50  0001 C CNN
-	1    10450 10450
-	1    0    0    -1
-$EndComp
-NoConn ~ 10250 10450
-$Comp
 L power:+3V3 #PWR0120
 U 1 1 6147BC6E
@@
 L OSM_env01:GND #PWR0121
 U 1 1 6147C064
-P 10150 10875
-F 0 "#PWR0121" H 10150 10625 50  0001 C CNN
-F 1 "GND" H 10155 10702 50  0000 C CNN
-F 2 "" H 10150 10875 60  0000 C CNN
-F 3 "" H 10150 10875 60  0000 C CNN
-	1    10150 10875
+P 10850 10550
+F 0 "#PWR0121" H 10850 10300 50  0001 C CNN
+F 1 "GND" H 10855 10377 50  0000 C CNN
+F 2 "" H 10850 10550 60  0000 C CNN
+F 3 "" H 10850 10550 60  0000 C CNN
+	1    10850 10550
 	1    0    0    -1
 $EndComp
@@
 Wire Wire Line
 	9975 10200 9975 10250
-Wire Wire Line
-	10150 10875 10150 10350
-Wire Wire Line
-	10150 10350 10250 10350
 Text HLabel 1675 4400 0    50   Input ~ 0
 BOOT0
@@
 Wire Wire Line
 	675  1000 1150 1000
+$Comp
+L Connector:Conn_02x03_Odd_Even J5
+U 1 1 6187503F
+P 10450 10350
+F 0 "J5" H 10500 10575 50  0000 C CNN
+F 1 "Conn_02x03_Odd_Even" H 10500 10576 50  0001 C CNN
+F 2 "" H 10450 10350 50  0001 C CNN
+F 3 "~" H 10450 10350 50  0001 C CNN
+	1    10450 10350
+	1    0    0    -1
+$EndComp
+Wire Wire Line
+	10750 10250 10850 10250
+Wire Wire Line
+	10850 10250 10850 10550
+NoConn ~ 10250 10350
+$Comp
+L device:R R16
+U 1 1 6142BFB9
+P 8000 1375
+F 0 "R16" V 7900 1300 50  0000 L CNN
+F 1 "10k" V 7800 1300 50  0000 L CNN
+F 2 "Resistor_SMD:R_0402_1005Metric" V 7930 1375 50  0001 C CNN
+F 3 "" H 8000 1375 50  0001 C CNN
+	1    8000 1375
+	0    -1   -1   0
+$EndComp
 $EndSCHEMATC

Commit message: rough throwdown of all parts
Parts:
- C59: footprint Capacitor_SMD:C_0402_1005Metric -> Capacitor_SMD:C_0603_1608Metric
- D8: value GRN -> RED
- J5: footprint (none) -> Connector:Tag-Connect_TC2030-IDC-NL_2x03_P1.27mm_Vertical
- R119, R15, R16, R30: footprint Resistor_SMD:R_0402_1005Metric -> Resistor_SMD:R_0603_1608Metric
- R37: footprint (none) -> Resistor_SMD:R_0603_1608Metric
Changed lines of the file:
@@
 F 0 "R119" H 6370 1171 50  0000 L CNN
 F 1 "DNF" H 6370 1080 50  0000 L CNN
-F 2 "Resistor_SMD:R_0402_1005Metric" V 6230 1125 50  0001 C CNN
+F 2 "Resistor_SMD:R_0603_1608Metric" V 6230 1125 50  0001 C CNN
 F 3 "" H 6300 1125 50  0001 C CNN
 	1    6300 1125
@@
 F 0 "R15" V 8200 1050 50  0000 L CNN
 F 1 "DNF" V 8100 1050 50  0000 L CNN
-F 2 "Resistor_SMD:R_0402_1005Metric" V 7930 1125 50  0001 C CNN
+F 2 "Resistor_SMD:R_0603_1608Metric" V 7930 1125 50  0001 C CNN
 F 3 "" H 8000 1125 50  0001 C CNN
 	1    8000 1125
@@
 P 9675 1425
 F 0 "D8" V 9714 1308 50  0000 R CNN
-F 1 "GRN" V 9623 1308 50  0000 R CNN
+F 1 "RED" V 9623 1308 50  0000 R CNN
 F 2 "Devtank_PCB_lib:LED_Rectangular_W4.5mm_H7.3mm_Horizontal_2.54mm_Z3.0mm" H 9675 1425 50  0001 C CNN
 F 3 "~" H 9675 1425 50  0001 C CNN
@@
 F 0 "R30" H 5120 2146 50  0000 L CNN
 F 1 "0R" H 5120 2055 50  0000 L CNN
-F 2 "Resistor_SMD:R_0402_1005Metric" V 4980 2100 50  0001 C CNN
+F 2 "Resistor_SMD:R_0603_1608Metric" V 4980 2100 50  0001 C CNN
 F 3 "" H 5050 2100 50  0001 C CNN
 	1    5050 2100
@@
 F 0 "C59" H 790 1196 50  0000 L CNN
 F 1 "4.7uF" H 790 1105 50  0000 L CNN
-F 2 "Capacitor_SMD:C_0402_1005Metric" H 713 1000 50  0001 C CNN
+F 2 "Capacitor_SMD:C_0603_1608Metric" H 713 1000 50  0001 C CNN
 F 3 "" H 675 1150 50  0001 C CNN
 	1    675  1150
@@
 F 0 "R37" V 1493 4900 50  0000 C CNN
 F 1 "0R" V 1584 4900 50  0000 C CNN
-F 2 "" V 1630 4900 50  0001 C CNN
+F 2 "Resistor_SMD:R_0603_1608Metric" V 1630 4900 50  0001 C CNN
 F 3 "" H 1700 4900 50  0001 C CNN
 	1    1700 4900
@@
 F 0 "J5" H 10500 10575 50  0000 C CNN
 F 1 "Conn_02x03_Odd_Even" H 10500 10576 50  0001 C CNN
-F 2 "" H 10450 10350 50  0001 C CNN
+F 2 "Connector:Tag-Connect_TC2030-IDC-NL_2x03_P1.27mm_Vertical" H 10450 10350 50  0001 C CNN
 F 3 "~" H 10450 10350 50  0001 C CNN
 	1    10450 10350
@@
 F 0 "R16" V 7900 1300 50  0000 L CNN
 F 1 "10k" V 7800 1300 50  0000 L CNN
-F 2 "Resistor_SMD:R_0402_1005Metric" V 7930 1375 50  0001 C CNN
+F 2 "Resistor_SMD:R_0603_1608Metric" V 7930 1375 50  0001 C CNN
 F 3 "" H 8000 1375 50  0001 C CNN
 	1    8000 1375

Commit message: schematics and layout submitted for review
Connections:
- net GPIO11: now also U14.38 (PC7/DFSDM_DATIN3/LCD_SEG25/SAI2_MCLK_B/SDMMC1_D7/TIM3_CH2/TIM8_CH2/TSC_G4_IO2); no longer U14.28 (COMP1_INP/DFSDM_CKIN0/I2C3_SMBA/LPTIM1_OUT/RTC_OUT_ALARM/RTC_OUT_CALIB/PB2)
- net GPIO2: now also U14.39 (PC8/LCD_SEG26/SDMMC1_D0/TIM3_CH3/TIM8_CH3/TSC_G4_IO3); no longer U14.38 (PC7/DFSDM_DATIN3/LCD_SEG25/SAI2_MCLK_B/SDMMC1_D7/TIM3_CH2/TIM8_CH2/TSC_G4_IO2)
- net GPIO3: now also U14.28 (COMP1_INP/DFSDM_CKIN0/I2C3_SMBA/LPTIM1_OUT/RTC_OUT_ALARM/RTC_OUT_CALIB/PB2); no longer U14.39 (PC8/LCD_SEG26/SDMMC1_D0/TIM3_CH3/TIM8_CH3/TSC_G4_IO3)
- net GPIO5 renamed ADC8
Changed lines of the file:
@@
 Wire Wire Line
 	2150 6600 1675 6600
-Text HLabel 1675 6600 0    50   Input ~ 0
+Text HLabel 1675 6700 0    50   Input ~ 0
 GPIO2
 Wire Wire Line
 	2150 6700 1675 6700
-Text HLabel 1675 6700 0    50   Input ~ 0
+Text HLabel 14825 6100 2    50   Input ~ 0
 GPIO3
 Wire Wire Line
@@
 	2150 6000 1675 6000
 Text HLabel 1675 6000 0    50   Input ~ 0
-GPIO5
+ADC8
 Wire Wire Line
 	14350 6200 14825 6200
@@
 Wire Wire Line
 	14350 6100 14825 6100
-Text HLabel 14825 6100 2    50   Input ~ 0
+Text HLabel 1675 6600 0    50   Input ~ 0
 GPIO11
 Wire Wire Line
