File: kicad_osm_env01/STM32L4.sch (KiCad schematic (older format))
At the start: 27 parts, among them J5 Conn_02x03_Odd_Even, U14 STM32L451RCTx, Y1 8MHZ, Y2 DNF

Commit message: osm env-01 revB finished
Connections:
- net ADC1 renamed GPIO16
Changed lines of the file:
@@
 Sheet 6 9
 Title "Open Smart Monitor"
-Date "2021-09-22"
+Date "2021-09-29"
 Rev "B"
 Comp "Devtank LTD"
-Comment1 "AB"
+Comment1 "Part No: 304-010"
 Comment2 ""
 Comment3 ""
@@
 	2150 5700 1675 5700
 Text HLabel 1675 5700 0    50   Input ~ 0
-ADC1
+GPIO16
 Wire Wire Line
 	14350 5000 14825 5000

Commit message: updated folder
Parts:
- C1, C12: value 18pF -> 10pF
Changed lines of the file:
@@
 P 11475 1675
 F 0 "C12" V 11325 1650 50  0000 L CNN
-F 1 "18pF" V 11250 1550 50  0000 L CNN
+F 1 "10pF" V 11250 1550 50  0000 L CNN
 F 2 "Capacitor_SMD:C_0402_1005Metric" H 11513 1525 50  0001 C CNN
 F 3 "" H 11475 1675 50  0001 C CNN
@@
 P 11475 1000
 F 0 "C1" V 11700 1000 50  0000 L CNN
-F 1 "18pF" V 11625 900 50  0000 L CNN
+F 1 "10pF" V 11625 900 50  0000 L CNN
 F 2 "Capacitor_SMD:C_0402_1005Metric" H 11513 850 50  0001 C CNN
 F 3 "" H 11475 1000 50  0001 C CNN
