File: kicad_osm_env01/USB_debug.sch (KiCad schematic (older format))
At the start: 26 parts, among them J3 USB_B_Micro, J7 632723100011, Q2 S8050, Q3 S8050, U13 CP2102N-A01-GQFN24

Commit message: schematics awaiting review
Parts:
- removed J7: 632723100011, Devtank_PCB_lib:WURTH_632723100011_USB_C, symbol Devtank:632723100011
- removed Q2, Q3: S8050, Package_TO_SOT_SMD:SOT-23, symbol OSM_env01-rescue:Q_NPN_BEC-device-ESP32-EVB_Rev_D-rescue
- removed R11, R12, R23: 0R, Resistor_SMD:R_0603_1608Metric, symbol OSM_env01-rescue:R-device-ESP32-EVB_Rev_D-rescue
- removed R21, R29: 12K, Resistor_SMD:R_0603_1608Metric, symbol OSM_env01-rescue:R-device-ESP32-EVB_Rev_D-rescue
- removed TP41: Test_Point, TestPoint:TestPoint_THTPad_D1.0mm_Drill0.5mm, symbol OSM_env01-rescue:Test_Point-Connector-ESP32-EVB_Rev_D-rescue
- added C54: 100nF, Capacitor_SMD:C_0402_1005Metric, symbol OSM_env01-rescue:C-device-ESP32-EVB_Rev_D-rescue
- added TP1, TP21: Test_Point, symbol Connector:Test_Point
- added U15: M74VHC1GT14DFT2G, Package_TO_SOT_SMD:SOT-353_SC-70-5, symbol OSM_env01-rescue:NL17SZ14-Devtank-ESP32-EVB_Rev_D-rescue
Connections:
- net labels added: RS232_GPIO0, RS232_GPIO1, RS232_GPIO2, RS232_GPIO3
- net labels removed: EN, ESP_BOOT, ESP_RES1, ESP_RES2, ESP_RESET, IO0, RS232_CTS, RS232_DTR, RS232_RTS
- wire segments 80 -> 67
- no-connect marks 6 -> 9
Other:
- moved on the sheet: C15, C16, C17, C31, C32, D5, J3, R20, R48, R49, R50, R51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

Commit message: rough layout with throwdown of parts
Parts:
- removed D5: SP0503BAHT, Package_TO_SOT_SMD:SOT-143, symbol OSM_env01-rescue:SP0503BAHT-ESD_Protection-ESP32-EVB_Rev_D-rescue
- removed TP21: Test_Point, symbol Connector:Test_Point
- added D5: SP0504BAHT, Package_TO_SOT_SMD:SOT-23-5, symbol ESD_Protection:SP0504BAHT
- J3: footprint Devtank_PCB_lib:MOLEX_105017-0001_Micro_USB_b -> Devtank_PCB_lib:MOLEX_105017-0001_USB_B
- TP1: footprint (none) -> TestPoint:TestPoint_Pad_D1.5mm
- U13: footprint Devtank_PCB_lib:CP2102n_qfn-24_ep-2.6x2.6_thermalvias-0.3 -> Devtank_PCB_lib:CP2102_QFN-24-1EP_4x4mm_P0.5mm_EP2.6x2.6mm_ThermalVias_0.3mmdrill
Connections:
- wire segments 67 -> 65
- no-connect marks 9 -> 10
Other:
- note added: "notes: use SP0504BAHTG, and SP0504BAJTG instead"
Changed lines of the file:
@@
 $Descr A4 11693 8268
 encoding utf-8
-Sheet 5 11
+Sheet 5 9
 Title "Open Smart Monitor"
 Date ""
@@
 F 0 "U13" H 5200 2650 50  0000 C CNN
 F 1 "CP2102N-A01-GQFN24" H 5575 2550 50  0000 C CNN
-F 2 "Devtank_PCB_lib:CP2102n_qfn-24_ep-2.6x2.6_thermalvias-0.3" H 5375 2675 50  0001 L CNN
+F 2 "Devtank_PCB_lib:CP2102_QFN-24-1EP_4x4mm_P0.5mm_EP2.6x2.6mm_ThermalVias_0.3mmdrill" H 5375 2675 50  0001 L CNN
 F 3 "http://www.silabs.com/support%20documents/technicaldocs/cp2102n-datasheet.pdf" H 4975 2425 50  0001 C CNN
 F 4 "118-007" H 4925 3475 50  0001 C CNN "Devtank"
@@
 	6825 4075 7225 4075
 Wire Wire Line
-	8875 3775 9150 3775
-Wire Wire Line
 	6825 3875 7225 3875
 $Comp
@@
 F 0 "J3" H 1082 7167 50  0000 C CNN
 F 1 "USB_B_Micro" H 1082 7076 50  0000 C CNN
-F 2 "Devtank_PCB_lib:MOLEX_105017-0001_Micro_USB_b" H 1175 6650 50  0001 C CNN
+F 2 "Devtank_PCB_lib:MOLEX_105017-0001_USB_B" H 1175 6650 50  0001 C CNN
 F 3 "~" H 1175 6650 50  0001 C CNN
 	1    1025 6700
@@
 USB_D-
 NoConn ~ 1325 6900
-$Comp
-L OSM_env01-rescue:SP0503BAHT-ESD_Protection-ESP32-EVB_Rev_D-rescue D?
-U 1 1 6097E558
-P 2050 7150
-AR Path="/6097E558" Ref="D?"  Part="1"
-AR Path="/5F4610BE/6097E558" Ref="D5"  Part="1"
-F 0 "D5" H 2255 7196 50  0000 L CNN
-F 1 "SP0503BAHT" H 2255 7105 50  0000 L CNN
-F 2 "Package_TO_SOT_SMD:SOT-143" H 2275 7100 50  0001 L CNN
-F 3 "http://www.littelfuse.com/~/media/files/littelfuse/technical%20resources/documents/data%20sheets/sp05xxba.pdf" H 2175 7275 50  0001 C CNN
-	1    2050 7150
-	1    0    0    -1
-$EndComp
 Wire Wire Line
 	1950 6500 1950 6950
@@
 F 0 "TP1" H 7750 3725 50  0000 L CNN
 F 1 "Test_Point" H 7758 3627 50  0001 L CNN
-F 2 "" H 7900 3600 50  0001 C CNN
+F 2 "TestPoint:TestPoint_Pad_D1.5mm" H 7900 3600 50  0001 C CNN
 F 3 "~" H 7900 3600 50  0001 C CNN
 	1    7700 3600
@@
 Wire Wire Line
 	7700 3775 7975 3775
-$Comp
-L Connector:Test_Point TP21
-U 1 1 61BAD885
-P 9150 3600
-F 0 "TP21" H 9225 3725 50  0000 L CNN
-F 1 "Test_Point" H 9208 3627 50  0001 L CNN
-F 2 "" H 9350 3600 50  0001 C CNN
-F 3 "~" H 9350 3600 50  0001 C CNN
-	1    9150 3600
-	1    0    0    -1
-$EndComp
-Wire Wire Line
-	9150 3600 9150 3775
-Connection ~ 9150 3775
-Wire Wire Line
-	9150 3775 9275 3775
+Text Notes 1225 7725 0    50   ~ 0
+notes: use SP0504BAHTG, and SP0504BAJTG instead
+$Comp
+L ESD_Protection:SP0504BAHT D5
+U 1 1 6158731D
+P 2050 7150
+F 0 "D5" H 2355 7196 50  0000 L CNN
+F 1 "SP0504BAHT" H 2355 7105 50  0000 L CNN
+F 2 "Package_TO_SOT_SMD:SOT-23-5" H 2350 7100 50  0001 L CNN
+F 3 "http://www.littelfuse.com/~/media/files/littelfuse/technical%20resources/documents/data%20sheets/sp05xxba.pdf" H 2175 7275 50  0001 C CNN
+	1    2050 7150
+	1    0    0    -1
+$EndComp
+NoConn ~ 2250 6950
+Wire Wire Line
+	8875 3775 9275 3775
 $EndSCHEMATC

Commit message: updated schematics
Parts:
- removed C31: 10uF, Capacitor_SMD:C_0805_2012Metric, symbol OSM_env01-rescue:C-device-ESP32-EVB_Rev_D-rescue
- removed C32: 100nF, Capacitor_SMD:C_0402_1005Metric, symbol OSM_env01-rescue:C-device-ESP32-EVB_Rev_D-rescue
- removed D5: SP0504BAHT, Package_TO_SOT_SMD:SOT-23-5, symbol ESD_Protection:SP0504BAHT
- removed R20: 47K, Resistor_SMD:R_0603_1608Metric, symbol OSM_env01-rescue:R-device-ESP32-EVB_Rev_D-rescue
- removed R49: 24K, Resistor_SMD:R_0603_1608Metric, symbol OSM_env01-rescue:R-device-ESP32-EVB_Rev_D-rescue
- added C47: 4.7uF, symbol device:C
- added C48: 100nF, symbol device:C
- added R35: 0R, symbol device:R
- added R36: DNF, symbol device:R
- added U5: SP3003-02JTG, Package_TO_SOT_SMD:SOT-353_SC-70-5, symbol Devtank:SP3003-02XJ
Connections:
- net labels added: VDD
- net labels removed: 5V_IN
- wire segments 65 -> 67
Other:
- note removed: "notes: use SP0504BAHTG, and SP0504BAJTG instead"

Commit message: Updated schematics
Parts:
- added R23: DNF, symbol device:R
- added R24: 0R, symbol device:R
Connections:
- net +3V3: now also R23.1; no longer C54.2, U15.5 (VCC)
- net VDD: now also R24.1
- new net: C54.2, R23.2, R24.2, U15.5 (VCC)
Changed lines of the file:
@@
 Sheet 5 9
 Title "Open Smart Monitor"
-Date ""
-Rev "A"
-Comp "Devtank Ltd"
-Comment1 "www.devtank.co.uk"
+Date "2021-09-22"
+Rev "B"
+Comp "Devtank LTD"
+Comment1 "AB"
 Comment2 ""
 Comment3 ""
@@
 L power:GND #PWR0131
 U 1 1 5CA85BC8
-P 2375 2875
-F 0 "#PWR0131" H 2375 2625 50  0001 C CNN
-F 1 "GND" H 2375 2725 50  0000 C CNN
-F 2 "" H 2375 2875 50  0001 C CNN
-F 3 "" H 2375 2875 50  0001 C CNN
-	1    2375 2875
-	0    1    1    0
-$EndComp
-Wire Wire Line
-	2450 2875 2375 2875
+P 2300 2875
+F 0 "#PWR0131" H 2300 2625 50  0001 C CNN
+F 1 "GND" H 2300 2725 50  0000 C CNN
+F 2 "" H 2300 2875 50  0001 C CNN
+F 3 "" H 2300 2875 50  0001 C CNN
+	1    2300 2875
+	1    0    0    -1
+$EndComp
 $Comp
 L OSM_env01-rescue:C-device-ESP32-EVB_Rev_D-rescue C16
@@
 L power:+3V3 #PWR?
 U 1 1 61E4E6DF
-P 8375 3425
+P 8100 2800
 AR Path="/61E4E6DF" Ref="#PWR?"  Part="1"
 AR Path="/608F4675/61E4E6DF" Ref="#PWR?"  Part="1"
 AR Path="/5F4610BE/61E4E6DF" Ref="#PWR0113"  Part="1"
-F 0 "#PWR0113" H 8375 3275 50  0001 C CNN
-F 1 "+3V3" H 8250 3550 50  0000 C CNN
-F 2 "" H 8375 3425 50  0001 C CNN
-F 3 "" H 8375 3425 50  0001 C CNN
-	1    8375 3425
+F 0 "#PWR0113" H 8100 2650 50  0001 C CNN
+F 1 "+3V3" H 8075 2950 50  0000 C CNN
+F 2 "" H 8100 2800 50  0001 C CNN
+F 3 "" H 8100 2800 50  0001 C CNN
+	1    8100 2800
 	1    0    0    -1
 $EndComp
@@
 $EndComp
 Connection ~ 8375 3525
-Wire Wire Line
-	8375 3525 8375 3425
 $Comp
 L OSM_env01-rescue:GND-ESP32-EVB_Rev_D #PWR?
@@
 $EndComp
 Connection ~ 5625 1925
+$Comp
+L power:VDD #PWR0148
+U 1 1 618E8D17
+P 8375 2800
+F 0 "#PWR0148" H 8375 2650 50  0001 C CNN
+F 1 "VDD" H 8375 2950 50  0000 C CNN
+F 2 "" H 8375 2800 50  0001 C CNN
+F 3 "" H 8375 2800 50  0001 C CNN
+	1    8375 2800
+	1    0    0    -1
+$EndComp
+$Comp
+L device:R R23
+U 1 1 618EA583
+P 8100 3000
+F 0 "R23" H 8170 3046 50  0000 L CNN
+F 1 "DNF" H 8170 2955 50  0000 L CNN
+F 2 "" V 8030 3000 50  0001 C CNN
+F 3 "" H 8100 3000 50  0001 C CNN
+	1    8100 3000
+	1    0    0    -1
+$EndComp
+$Comp
+L device:R R24
+U 1 1 618EB471
+P 8375 3000
+F 0 "R24" H 8445 3046 50  0000 L CNN
+F 1 "0R" H 8445 2955 50  0000 L CNN
+F 2 "" V 8305 3000 50  0001 C CNN
+F 3 "" H 8375 3000 50  0001 C CNN
+	1    8375 3000
+	1    0    0    -1
+$EndComp
+Wire Wire Line
+	8100 2850 8100 2800
+Wire Wire Line
+	8375 2850 8375 2800
+Wire Wire Line
+	8375 3150 8375 3200
+Wire Wire Line
+	8100 3150 8100 3200
+Wire Wire Line
+	8100 3200 8375 3200
+Connection ~ 8375 3200
+Wire Wire Line
+	8375 3200 8375 3525
+Wire Wire Line
+	2300 2875 2450 2875
+$Comp
+L OSM_env01:PWR_FLAG #FLG0108
+U 1 1 61AE1271
+P 8825 3050
+F 0 "#FLG0108" H 8825 3145 50  0001 C CNN
+F 1 "PWR_FLAG" H 8825 3273 50  0000 C CNN
+F 2 "" H 8825 3050 60  0000 C CNN
+F 3 "" H 8825 3050 60  0000 C CNN
+	1    8825 3050
+	1    0    0    -1
+$EndComp
+Wire Wire Line
+	8375 3200 8825 3200
+Wire Wire Line
+	8825 3200 8825 3050
 $EndSCHEMATC

Commit message: rough throwdown of all parts
Parts:
- C47: footprint (none) -> Capacitor_SMD:C_0603_1608Metric
- C48: footprint (none) -> Capacitor_SMD:C_0402_1005Metric
- R23, R24, R35, R36: footprint (none) -> Resistor_SMD:R_0603_1608Metric
- R48: value 10K -> 10k
Changed lines of the file:
@@
 P 3225 2625
 F 0 "R48" H 3155 2579 50  0000 R CNN
-F 1 "10K" H 3155 2670 50  0000 R CNN
+F 1 "10k" H 3155 2670 50  0000 R CNN
 F 2 "Resistor_SMD:R_0603_1608Metric" V 3155 2625 50  0001 C CNN
 F 3 "" H 3225 2625 50  0001 C CNN
@@
 F 0 "C48" H 3790 3246 50  0000 L CNN
 F 1 "100nF" H 3790 3155 50  0000 L CNN
-F 2 "" H 3713 3050 50  0001 C CNN
+F 2 "Capacitor_SMD:C_0402_1005Metric" H 3713 3050 50  0001 C CNN
 F 3 "" H 3675 3200 50  0001 C CNN
 	1    3675 3200
@@
 F 0 "C47" H 3340 3246 50  0000 L CNN
 F 1 "4.7uF" H 3340 3155 50  0000 L CNN
-F 2 "" H 3263 3050 50  0001 C CNN
+F 2 "Capacitor_SMD:C_0603_1608Metric" H 3263 3050 50  0001 C CNN
 F 3 "" H 3225 3200 50  0001 C CNN
 	1    3225 3200
@@
 F 0 "R36" H 4195 4371 50  0000 L CNN
 F 1 "DNF" H 4195 4280 50  0000 L CNN
-F 2 "" V 4055 4325 50  0001 C CNN
+F 2 "Resistor_SMD:R_0603_1608Metric" V 4055 4325 50  0001 C CNN
 F 3 "" H 4125 4325 50  0001 C CNN
 	1    4125 4325
@@
 F 0 "R35" V 3550 3975 50  0000 L CNN
 F 1 "0R" V 3550 3500 50  0000 L CNN
-F 2 "" V 3430 3775 50  0001 C CNN
+F 2 "Resistor_SMD:R_0603_1608Metric" V 3430 3775 50  0001 C CNN
 F 3 "" H 3500 3775 50  0001 C CNN
 	1    3500 3775
@@
 F 0 "R23" H 8170 3046 50  0000 L CNN
 F 1 "DNF" H 8170 2955 50  0000 L CNN
-F 2 "" V 8030 3000 50  0001 C CNN
+F 2 "Resistor_SMD:R_0603_1608Metric" V 8030 3000 50  0001 C CNN
 F 3 "" H 8100 3000 50  0001 C CNN
 	1    8100 3000
@@
 F 0 "R24" H 8445 3046 50  0000 L CNN
 F 1 "0R" H 8445 2955 50  0000 L CNN
-F 2 "" V 8305 3000 50  0001 C CNN
+F 2 "Resistor_SMD:R_0603_1608Metric" V 8305 3000 50  0001 C CNN
 F 3 "" H 8375 3000 50  0001 C CNN
 	1    8375 3000
