File: kicad_osm_env01/PowerSupply.sch (KiCad schematic (older format))
At the start: 66 parts, among them Q1 SI2301BDS-T1-E3, Q4 IRF7319TRPBF, SW3 SW_Push, U1 MIC2288YD5-TR, U2 MCP73833(MSOP10), U4 NCP1117ST33T3G

Commit message: rough layout with throwdown of parts
Parts:
- C2: footprint Capacitor_SMD:C_0805_2012Metric -> Capacitor_SMD:C_0603_1608Metric
- C22: footprint Capacitor_SMD:C_0603_1608Metric -> Capacitor_SMD:C_0402_1005Metric
- C5, C6: footprint Capacitor_SMD:C_1206_3216Metric -> Capacitor_SMD:C_0805_2012Metric
- CHARGING1, COMPLETE1: footprint Devtank_PCB_lib:LED_Rectangular_W4.5mm_H7.3mm_Horizontal_2.54mm_Z5.0mm -> Devtank_PCB_lib:LED_Rectangular_W4.5mm_H7.3mm_Horizontal_2.54mm_Z3.0mm
- D10: value D -> DNF
- R18, R19, R21, R22, R27, R28: footprint (none) -> Resistor_SMD:R_0603_1608Metric
- TP18, TP27, TP28, TP29, TP79: footprint TestPoint:TestPoint_THTPad_D1.0mm_Drill0.5mm -> TestPoint:TestPoint_Pad_D1.5mm
- U2: footprint Devtank_PCB_lib:MCP73833-AMI_UN_buck_converter -> Package_SO:MSOP-10_3x3mm_P0.5mm
Changed lines of the file:
@@
 $Descr A3 16535 11693
 encoding utf-8
-Sheet 2 11
+Sheet 2 9
 Title ""
 Date ""
@@
 F 0 "C5" H 3815 5871 50  0000 L CNN
 F 1 "22uF" H 3815 5780 50  0000 L CNN
-F 2 "Capacitor_SMD:C_1206_3216Metric" H 3738 5675 50  0001 C CNN
+F 2 "Capacitor_SMD:C_0805_2012Metric" H 3738 5675 50  0001 C CNN
 F 3 "" H 3700 5825 50  0001 C CNN
 F 4 "X5R/X7R" H 3900 5650 50  0000 C CNN "Dielectric"
@@
 F 0 "C2" H 1225 5825 50  0000 L CNN
 F 1 "4.7uF" H 1225 5750 50  0000 L CNN
-F 2 "Capacitor_SMD:C_0805_2012Metric" H 1588 5650 50  0001 C CNN
+F 2 "Capacitor_SMD:C_0603_1608Metric" H 1588 5650 50  0001 C CNN
 F 3 "" H 1550 5800 50  0001 C CNN
 F 4 "10V" H 1550 5800 50  0001 C CNN "Voltage"
@@
 F 0 "C6" H 4240 5871 50  0000 L CNN
 F 1 "DNF" H 4240 5780 50  0000 L CNN
-F 2 "Capacitor_SMD:C_1206_3216Metric" H 4163 5675 50  0001 C CNN
+F 2 "Capacitor_SMD:C_0805_2012Metric" H 4163 5675 50  0001 C CNN
 F 3 "" H 4125 5825 50  0001 C CNN
 	1    4125 5825
@@
 F 0 "C22" V 10552 2425 50  0000 C CNN
 F 1 "0.1uF" V 10461 2425 50  0000 C CNN
-F 2 "Capacitor_SMD:C_0603_1608Metric" H 10338 2275 50  0001 C CNN
+F 2 "Capacitor_SMD:C_0402_1005Metric" H 10338 2275 50  0001 C CNN
 F 3 "" H 10300 2425 50  0001 C CNN
 	1    10300 2425
@@
 F 0 "TP27" V 7975 4775 50  0000 C CNN
 F 1 "Test_Point" V 8050 4800 50  0001 C CNN
-F 2 "TestPoint:TestPoint_THTPad_D1.0mm_Drill0.5mm" H 8175 4500 50  0001 C CNN
+F 2 "TestPoint:TestPoint_Pad_D1.5mm" H 8175 4500 50  0001 C CNN
 F 3 "~" H 8175 4500 50  0001 C CNN
 	1    7975 4500
@@
 F 0 "TP29" V 12850 1950 50  0000 C CNN
 F 1 "Test_Point" V 12954 1747 50  0001 C CNN
-F 2 "TestPoint:TestPoint_THTPad_D1.0mm_Drill0.5mm" H 13050 1675 50  0001 C CNN
+F 2 "TestPoint:TestPoint_Pad_D1.5mm" H 13050 1675 50  0001 C CNN
 F 3 "~" H 13050 1675 50  0001 C CNN
 	1    12850 1675
@@
 F 0 "TP28" V 9250 4775 50  0000 C CNN
 F 1 "Test_Point" V 9325 4725 50  0001 C CNN
-F 2 "TestPoint:TestPoint_THTPad_D1.0mm_Drill0.5mm" H 9450 4500 50  0001 C CNN
+F 2 "TestPoint:TestPoint_Pad_D1.5mm" H 9450 4500 50  0001 C CNN
 F 3 "~" H 9450 4500 50  0001 C CNN
 	1    9250 4500
@@
 P 10700 2175
 F 0 "D10" V 10654 2254 50  0000 L CNN
-F 1 "D" V 10745 2254 50  0000 L CNN
+F 1 "DNF" V 10745 2254 50  0000 L CNN
 F 2 "Diode_SMD:D_SOD-123" H 10700 2175 50  0001 C CNN
 F 3 "" H 10700 2175 50  0001 C CNN
@@
 F 0 "R18" H 10770 4846 50  0000 L CNN
 F 1 "100K" H 10770 4755 50  0000 L CNN
-F 2 "" V 10630 4800 50  0001 C CNN
+F 2 "Resistor_SMD:R_0603_1608Metric" V 10630 4800 50  0001 C CNN
 F 3 "" H 10700 4800 50  0001 C CNN
 	1    10700 4800
@@
 F 0 "R19" H 10770 5321 50  0000 L CNN
 F 1 "47K" H 10770 5230 50  0000 L CNN
-F 2 "" V 10630 5275 50  0001 C CNN
+F 2 "Resistor_SMD:R_0603_1608Metric" V 10630 5275 50  0001 C CNN
 F 3 "" H 10700 5275 50  0001 C CNN
 	1    10700 5275
@@
 F 0 "R21" H 11895 4821 50  0000 L CNN
 F 1 "100K" H 11895 4730 50  0000 L CNN
-F 2 "" V 11755 4775 50  0001 C CNN
+F 2 "Resistor_SMD:R_0603_1608Metric" V 11755 4775 50  0001 C CNN
 F 3 "" H 11825 4775 50  0001 C CNN
 	1    11825 4775
@@
 F 0 "R22" H 11895 5296 50  0000 L CNN
 F 1 "47K" H 11895 5205 50  0000 L CNN
-F 2 "" V 11755 5250 50  0001 C CNN
+F 2 "Resistor_SMD:R_0603_1608Metric" V 11755 5250 50  0001 C CNN
 F 3 "" H 11825 5250 50  0001 C CNN
 	1    11825 5250
@@
 F 0 "R27" H 9820 1946 50  0000 L CNN
 F 1 "0R" H 9820 1855 50  0000 L CNN
-F 2 "" V 9680 1900 50  0001 C CNN
+F 2 "Resistor_SMD:R_0603_1608Metric" V 9680 1900 50  0001 C CNN
 F 3 "" H 9750 1900 50  0001 C CNN
 	1    9750 1900
@@
 F 0 "R28" H 9820 2346 50  0000 L CNN
 F 1 "DNF" H 9820 2255 50  0000 L CNN
-F 2 "" V 9680 2300 50  0001 C CNN
+F 2 "Resistor_SMD:R_0603_1608Metric" V 9680 2300 50  0001 C CNN
 F 3 "" H 9750 2300 50  0001 C CNN
 	1    9750 2300
@@
 F 0 "TP79" V 6825 3025 50  0000 C CNN
 F 1 "Test_Point" V 6929 2822 50  0001 C CNN
-F 2 "TestPoint:TestPoint_THTPad_D1.0mm_Drill0.5mm" H 7025 2750 50  0001 C CNN
+F 2 "TestPoint:TestPoint_Pad_D1.5mm" H 7025 2750 50  0001 C CNN
 F 3 "~" H 7025 2750 50  0001 C CNN
 	1    6825 2750
@@
 F 0 "COMPLETE1" V 2981 1872 50  0000 R CNN
 F 1 "GRN" V 2904 1872 35  0000 R CNN
-F 2 "Devtank_PCB_lib:LED_Rectangular_W4.5mm_H7.3mm_Horizontal_2.54mm_Z5.0mm" H 2950 1950 60  0001 C CNN
+F 2 "Devtank_PCB_lib:LED_Rectangular_W4.5mm_H7.3mm_Horizontal_2.54mm_Z3.0mm" H 2950 1950 60  0001 C CNN
 F 3 "" H 2950 1950 60  0000 C CNN
 F 4 "Value 1" H 2950 1950 60  0001 C CNN "Fieldname 1"
@@
 F 0 "CHARGING1" V 3596 1872 50  0000 R CNN
 F 1 "YLW" V 3505 1872 35  0000 R CNN
-F 2 "Devtank_PCB_lib:LED_Rectangular_W4.5mm_H7.3mm_Horizontal_2.54mm_Z5.0mm" H 3550 1950 60  0001 C CNN
+F 2 "Devtank_PCB_lib:LED_Rectangular_W4.5mm_H7.3mm_Horizontal_2.54mm_Z3.0mm" H 3550 1950 60  0001 C CNN
 F 3 "" H 3550 1950 60  0000 C CNN
 F 4 "Value 1" H 3550 1950 60  0001 C CNN "Fieldname 1"
@@
 F 0 "U2" H 4370 3110 60  0000 C CNN
 F 1 "MCP73833(MSOP10)" H 4610 2290 43  0000 C CNN
-F 2 "Devtank_PCB_lib:MCP73833-AMI_UN_buck_converter" H 4650 2650 60  0001 C CNN
+F 2 "Package_SO:MSOP-10_3x3mm_P0.5mm" H 4650 2650 60  0001 C CNN
 F 3 "" H 4650 2650 60  0001 C CNN
 F 4 "Value 1" H 4550 2650 60  0001 C CNN "Fieldname 1"
@@
 F 0 "TP18" V 5625 3325 50  0000 C CNN
 F 1 "Test_Point" V 5729 3122 50  0001 C CNN
-F 2 "TestPoint:TestPoint_THTPad_D1.0mm_Drill0.5mm" H 5825 3050 50  0001 C CNN
+F 2 "TestPoint:TestPoint_Pad_D1.5mm" H 5825 3050 50  0001 C CNN
 F 3 "~" H 5825 3050 50  0001 C CNN
 	1    5625 3050

Commit message: updated schematics
Parts:
- removed C10, C7: 10uF, Capacitor_SMD:C_Elec_4x5.4, symbol OSM_env01-rescue:CP-device-ESP32-EVB_Rev_D-rescue
- removed U4: NCP1117ST33T3G, Package_TO_SOT_SMD:SOT-223, symbol OSM_env01-rescue:NCP1117-3.3_SOT223-regul-ESP32-EVB_Rev_D-rescue
- added C?: 4.7nF, symbol device:C
- added C? (x2): DNF, symbol device:C
- added C?: 10uF, symbol device:CP
- added C?: 100pF, symbol device:C
- added C?: 1uF, symbol device:C
- added D?: D_TVS, symbol device:D_TVS
- added D?: RB160M-40TR, Diode_SMD:D_SMA, symbol OSM_env01-rescue:D_Schottky-device-ESP32-EVB_Rev_D-rescue
- added R? (x2): 0R, symbol device:R
- added U?: MIC5219-3.3, TO_SOT_Packages_SMD:SOT-23-5, symbol regul:MIC5219-3.3
- C2: value 4.7uF -> 10uF
- C5: value 22uF -> 10uF
- D2: value SK24A -> RB160M-40TR
- D3: value SS34 -> RB160M-40TR
- R18, R21, R58: value 100K -> 1M
- R19, R22: value 47K -> 470K
- R46: value 15K -> 110k
- R47: value 4.87K -> 36k
- R64: value 47K -> 470k
- U1: value MIC2288YD5-TR -> MIC2250-1YD5
Connections:
- wire segments 200 -> 226
Other:
- note added: "100pf used elweher\n"
- note added: "The diode must be rated for the peak inductor current, \nand its reverse voltage rating must be greater than the \noutput voltage.\n"
- note removed: "Note: If MIC2250 used R1 should be as large as poosible ideally around 100k\n"
- moved on the sheet: C2, C23, C5, C6, D2, L1, R18, R19, R21, R22, R46, R47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

Commit message: updated schematics
Parts:
- removed D1: SMBJ6.0A, Diode_SMD:D_SMB, symbol device:D_Zener
- removed D?: D_TVS, symbol device:D_TVS
- removed TH1: DNF, Resistor_THT:R_Axial_DIN0204_L3.6mm_D1.6mm_P2.54mm_Vertical, symbol OSM_env01-rescue:Thermistor_NTC-device-ESP32-EVB_Rev_D-rescue
- added D1: RB160M-40TR, Diode_SMD:D_SOD-123, symbol device:D_Schottky
- added D5: SMFE5-0A, Diode_SMD:D_SOD-123, symbol device:D_TVS
- D2, D3: footprint Diode_SMD:D_SMA -> Diode_SMD:D_SOD-123
- D4: value SK24A -> RB160M-40TR
- D9: renamed from D?; footprint Diode_SMD:D_SMA -> Diode_SMD:D_SOD-123
- Q4: value IRF7319TRPBF -> IRF7509TRPBF
- gave numbers to parts that had none: 9
Connections:
- wire segments 226 -> 220
Other:
- note added: "100pf used elsewhere\n"
- note removed: "100pf used elweher\n"
- moved on the sheet: C23, R18, R19, R21, R22, R58, R64, TP27, TP28

Commit message: Updated schematics
Parts:
- added C63: 1uF, symbol device:C
- C32: value 100pF -> DNF
- C46: value 10uF -> DNF
- D1: Current (none) -> 1A
- D2, D4, D9: Current 2A -> 1A
- U2: value MCP73833(MSOP10) -> MCP73833
Connections:
- net +3V3: now also C63.1
- net GND: now also C63.2
Other:
- moved on the sheet: C46, TP25, TP26
Changed lines of the file:
@@
 encoding utf-8
 Sheet 2 9
-Title ""
-Date ""
-Rev ""
-Comp ""
-Comment1 ""
+Title "Open Smart Monitor"
+Date "2021-09-22"
+Rev "B"
+Comp "Devtank LTD"
+Comment1 "AB"
 Comment2 ""
 Comment3 ""
@@
 U 1 1 607F8C4F
 P 3150 6225
-F 0 "R47" H 2875 6275 50  0000 L CNN
-F 1 "36k" H 2875 6200 50  0000 L CNN
+F 0 "R47" H 2925 6275 50  0000 L CNN
+F 1 "36k" H 2925 6200 50  0000 L CNN
 F 2 "Resistor_SMD:R_0603_1608Metric" V 3080 6225 50  0001 C CNN
 F 3 "" H 3150 6225 50  0001 C CNN
@@
 U 1 1 607F8C65
 P 2800 5475
-F 0 "D2" H 2800 5691 50  0000 C CNN
-F 1 "RB160M-40TR" H 2800 5600 50  0000 C CNN
+F 0 "D2" H 3000 5300 50  0000 C CNN
+F 1 "RB160M-40TR" H 2775 5375 50  0000 C CNN
 F 2 "Diode_SMD:D_SOD-123" H 2800 5475 50  0001 C CNN
 F 3 "" H 2800 5475 50  0001 C CNN
-F 4 "2A" H 2825 5350 50  0000 C CNN "Current"
+F 4 "1A" H 2800 5600 50  0000 C CNN "Current"
 	1    2800 5475
 	-1   0    0    1
@@
 $EndComp
 Wire Wire Line
-	4000 5475 4425 5475
+	4000 5475 4125 5475
 $Comp
 L OSM_env01-rescue:C-device-ESP32-EVB_Rev_D-rescue C6
@@
 L OSM_env01-rescue:Test_Point-Connector-ESP32-EVB_Rev_D-rescue TP25
 U 1 1 607F8D09
-P 4700 5475
-F 0 "TP25" V 4700 5750 50  0000 C CNN
-F 1 "Test_Point" H 4725 5325 50  0001 C CNN
-F 2 "TestPoint:TestPoint_THTPad_D1.0mm_Drill0.5mm" H 4900 5475 50  0001 C CNN
-F 3 "~" H 4900 5475 50  0001 C CNN
-	1    4700 5475
-	1    0    0    -1
-$EndComp
-Wire Wire Line
-	4425 5475 4525 5475
-Wire Wire Line
-	4525 5425 4525 5475
-Connection ~ 4525 5475
-Wire Wire Line
-	4525 5475 4700 5475
+P 4125 5250
+F 0 "TP25" V 4125 5525 50  0000 C CNN
+F 1 "Test_Point" H 4150 5100 50  0001 C CNN
+F 2 "TestPoint:TestPoint_THTPad_D1.0mm_Drill0.5mm" H 4325 5250 50  0001 C CNN
+F 3 "~" H 4325 5250 50  0001 C CNN
+	1    4125 5250
+	0    1    1    0
+$EndComp
+Wire Wire Line
+	4825 5425 4825 5475
 $Comp
 L power:+3V3 #PWR041
 U 1 1 607F8D3D
-P 7300 5475
-F 0 "#PWR041" H 7300 5325 50  0001 C CNN
-F 1 "+3V3" H 7315 5648 50  0000 C CNN
-F 2 "" H 7300 5475 50  0001 C CNN
-F 3 "" H 7300 5475 50  0001 C CNN
-	1    7300 5475
-	1    0    0    -1
-$EndComp
-Connection ~ 7300 5475
-Wire Wire Line
-	7300 5475 7525 5475
+P 7500 5475
+F 0 "#PWR041" H 7500 5325 50  0001 C CNN
+F 1 "+3V3" H 7515 5648 50  0000 C CNN
+F 2 "" H 7500 5475 50  0001 C CNN
+F 3 "" H 7500 5475 50  0001 C CNN
+	1    7500 5475
+	1    0    0    -1
+$EndComp
+Connection ~ 7500 5475
 $Comp
 L power:+5V #PWR030
 U 1 1 607F8D54
-P 4525 5425
-F 0 "#PWR030" H 4525 5275 50  0001 C CNN
-F 1 "+5V" H 4540 5598 50  0000 C CNN
-F 2 "" H 4525 5425 50  0001 C CNN
-F 3 "" H 4525 5425 50  0001 C CNN
-	1    4525 5425
+P 4825 5425
+F 0 "#PWR030" H 4825 5275 50  0001 C CNN
+F 1 "+5V" H 4840 5598 50  0000 C CNN
+F 2 "" H 4825 5425 50  0001 C CNN
+F 3 "" H 4825 5425 50  0001 C CNN
+	1    4825 5425
 	1    0    0    -1
 $EndComp
@@
 U 1 1 607F8E1E
 P 8775 3175
-F 0 "D4" H 8775 3391 50  0000 C CNN
-F 1 "RB160M-40TR" H 8775 3300 50  0000 C CNN
+F 0 "D4" H 8775 3100 50  0000 C CNN
+F 1 "RB160M-40TR" H 8900 3300 50  0000 C CNN
 F 2 "Diode_SMD:D_SOD-123" H 8775 3175 50  0001 C CNN
 F 3 "" H 8775 3175 50  0001 C CNN
-F 4 "2A" H 8800 3050 50  0000 C CNN "Current"
+F 4 "1A" H 8800 3050 50  0001 C CNN "Current"
 	1    8775 3175
 	0    1    1    0
@@
 	525  4550 7425 4525
 Wire Notes Line
-	7425 3825 11200 3825
-Wire Notes Line
 	7425 4525 7450 550
-Text HLabel 4375 5250 0    50   Input ~ 0
+Text HLabel 4225 5150 2    50   Input ~ 0
 5Vout
-Text HLabel 7575 5475 2    50   Input ~ 0
+Text HLabel 7775 5475 2    50   Input ~ 0
 3.3Vout
-Wire Wire Line
-	4375 5250 4425 5250
-Wire Wire Line
-	4425 5250 4425 5475
 Text HLabel 10075 4600 2    50   Input ~ 0
 BatMon
@@
 L OSM_env01-rescue:Test_Point-Connector-ESP32-EVB_Rev_D-rescue TP?
 U 1 1 60A59EE0
-P 7525 5475
+P 7675 5575
 AR Path="/5F6F7717/60A59EE0" Ref="TP?"  Part="1"
 AR Path="/60A59EE0" Ref="TP?"  Part="1"
 AR Path="/608F4675/60A59EE0" Ref="TP?"  Part="1"
 AR Path="/60688D25/60A59EE0" Ref="TP26"  Part="1"
-F 0 "TP26" V 7525 5750 50  0000 C CNN
-F 1 "Test_Point" V 7600 5700 50  0001 C CNN
-F 2 "TestPoint:TestPoint_THTPad_D1.0mm_Drill0.5mm" H 7725 5475 50  0001 C CNN
-F 3 "~" H 7725 5475 50  0001 C CNN
-	1    7525 5475
-	1    0    0    -1
-$EndComp
-Connection ~ 7525 5475
-Wire Wire Line
-	7525 5475 7575 5475
+F 0 "TP26" V 7675 5850 50  0000 C CNN
+F 1 "Test_Point" V 7750 5800 50  0001 C CNN
+F 2 "TestPoint:TestPoint_THTPad_D1.0mm_Drill0.5mm" H 7875 5575 50  0001 C CNN
+F 3 "~" H 7875 5575 50  0001 C CNN
+	1    7675 5575
+	0    1    1    0
+$EndComp
 $Comp
 L OSM_env01-rescue:Test_Point-Connector-ESP32-EVB_Rev_D-rescue TP?
@@
 P 6350 1900
 F 0 "D3" H 6400 2000 50  0000 R CNN
-F 1 "RB160M-40TR" H 6450 1800 50  0000 R CNN
+F 1 "RB160M-40TR" H 6625 1775 50  0000 R CNN
 F 2 "Diode_SMD:D_SOD-123" H 6350 1900 60  0001 C CNN
 F 3 "" H 6350 1900 60  0000 C CNN
@@
 U 1 1 607F8B9E
 P 4550 2650
-F 0 "U2" H 4370 3110 60  0000 C CNN
-F 1 "MCP73833(MSOP10)" H 4610 2290 43  0000 C CNN
+F 0 "U2" H 4300 3225 60  0000 C CNN
+F 1 "MCP73833" H 4400 3125 43  0000 C CNN
 F 2 "Package_SO:MSOP-10_3x3mm_P0.5mm" H 4650 2650 60  0001 C CNN
 F 3 "" H 4650 2650 60  0001 C CNN
@@
 Voltage Rail Monitor\n\n\n
 Wire Notes Line
-	11100 4075 11100 6750
+	11075 3850 11075 6525
 $Comp
 L OSM_env01-rescue:Test_Point-Connector-ESP32-EVB_Rev_D-rescue TP18
@@
 	3550 5850 3550 5475
 Connection ~ 3550 5475
-Wire Wire Line
-	3550 5475 3875 5475
 $Comp
 L device:R R20
@@
 L device:CP C46
 U 1 1 61638EE1
-P 6900 5625
-F 0 "C46" H 7018 5671 50  0000 L CNN
-F 1 "10uF" H 7018 5580 50  0000 L CNN
-F 2 "" H 6938 5475 50  0001 C CNN
-F 3 "" H 6900 5625 50  0001 C CNN
-	1    6900 5625
+P 7300 5625
+F 0 "C46" H 7418 5671 50  0000 L CNN
+F 1 "DNF" H 7418 5580 50  0000 L CNN
+F 2 "" H 7338 5475 50  0001 C CNN
+F 3 "" H 7300 5625 50  0001 C CNN
+	1    7300 5625
 	1    0    0    -1
 $EndComp
@@
 P 6525 5725
 F 0 "C32" H 6640 5771 50  0000 L CNN
-F 1 "100pF" H 6640 5680 50  0000 L CNN
+F 1 "DNF" H 6640 5680 50  0000 L CNN
 F 2 "" H 6563 5575 50  0001 C CNN
 F 3 "" H 6525 5725 50  0001 C CNN
@@
 Text Notes 5875 6225 0    50   ~ 0
 100pf used elsewhere\n
-Text Notes 3100 5200 0    118  ~ 24
+Text Notes 3050 4850 0    118  ~ 24
 5V and 3V3 Power Supplies\n\n\n
 Wire Wire Line
-	4925 5475 4700 5475
+	4925 5475 4825 5475
 Connection ~ 4925 5475
-Connection ~ 4700 5475
-Connection ~ 6900 5475
 $Comp
 L OSM_env01-rescue:D_Schottky-device-ESP32-EVB_Rev_D-rescue D9
 U 1 1 61835A37
 P 6025 4900
-F 0 "D9" H 6025 5116 50  0000 C CNN
+F 0 "D9" H 6025 4800 50  0000 C CNN
 F 1 "RB160M-40TR" H 6025 5025 50  0000 C CNN
 F 2 "Diode_SMD:D_SOD-123" H 6025 4900 50  0001 C CNN
 F 3 "" H 6025 4900 50  0001 C CNN
-F 4 "2A" H 6050 4775 50  0000 C CNN "Current"
+F 4 "1A" H 6050 4775 50  0001 C CNN "Current"
 	1    6025 4900
 	1    0    0    1
@@
 U 1 1 614EE47C
 P 1300 1650
-F 0 "D1" H 1350 1750 50  0000 R CNN
-F 1 "RB160M-40TR" H 1400 1550 50  0000 R CNN
+F 0 "D1" H 1550 1475 50  0000 R CNN
+F 1 "RB160M-40TR" H 1550 1550 50  0000 R CNN
 F 2 "Diode_SMD:D_SOD-123" H 1300 1650 60  0001 C CNN
 F 3 "" H 1300 1650 60  0000 C CNN
@@
 F 5 "Value2" H 1300 1650 60  0001 C CNN "Fieldname2"
 F 6 "Value3" H 1300 1650 60  0001 C CNN "Fieldname3"
+F 7 "1A" H 1300 1775 50  0000 C CNN "Current"
 	1    1300 1650
 	-1   0    0    1
@@
 	0    1    1    0
 $EndComp
+Wire Notes Line
+	8225 3875 8225 6550
+Wire Wire Line
+	5150 3750 5150 3850
+Wire Wire Line
+	5150 3250 5150 3450
+Wire Wire Line
+	7500 5475 7675 5475
+Wire Wire Line
+	7675 5575 7675 5475
+Connection ~ 7675 5475
+Wire Wire Line
+	7675 5475 7775 5475
+Connection ~ 4825 5475
+Wire Wire Line
+	3550 5475 4000 5475
+Wire Wire Line
+	4425 5475 4825 5475
+Wire Wire Line
+	4225 5150 4125 5150
+Wire Wire Line
+	4125 5150 4125 5250
+Wire Wire Line
+	4125 5250 4125 5475
+Connection ~ 4125 5250
+Connection ~ 4125 5475
+Wire Wire Line
+	4125 5475 4425 5475
+$Comp
+L device:C C63
+U 1 1 615DB725
+P 6900 5625
+F 0 "C63" H 7015 5671 50  0000 L CNN
+F 1 "1uF" H 7015 5580 50  0000 L CNN
+F 2 "" H 6938 5475 50  0001 C CNN
+F 3 "" H 6900 5625 50  0001 C CNN
+	1    6900 5625
+	1    0    0    -1
+$EndComp
+Connection ~ 7300 5475
+Wire Wire Line
+	7300 5475 7500 5475
 Wire Wire Line
 	6900 5475 7300 5475
-Wire Wire Line
-	3875 5475 3875 5325
-$Comp
-L OSM_env01:PWR_FLAG #FLG0106
-U 1 1 61839B40
-P 3875 5325
-F 0 "#FLG0106" H 3875 5420 50  0001 C CNN
-F 1 "PWR_FLAG" H 3875 5548 50  0000 C CNN
-F 2 "" H 3875 5325 60  0000 C CNN
-F 3 "" H 3875 5325 60  0000 C CNN
-	1    3875 5325
-	1    0    0    -1
-$EndComp
-Connection ~ 3875 5475
-Wire Wire Line
-	3875 5475 4000 5475
+Connection ~ 6900 5475
+Wire Wire Line
+	7300 5775 7300 5875
+Wire Wire Line
+	7300 5875 6900 5875
 Wire Notes Line
-	8050 3975 8050 6650
-Wire Wire Line
-	5150 3750 5150 3850
-Wire Wire Line
-	5150 3250 5150 3450
+	7425 3825 16000 3825
 $EndSCHEMATC

Commit message: rough throwdown of all parts
Parts:
- C10, C25, C32, C63: footprint (none) -> Capacitor_SMD:C_0402_1005Metric
- C11, C3, C4, C9: Dielectric X5R -> (none); Tolerance 20% -> (none); Voltage 6.3V -> (none)
- C14, C23, C72, C8: footprint Capacitor_SMD:C_0603_1608Metric -> Capacitor_SMD:C_0402_1005Metric
- C22: value 0.1uF -> 100nF
- C24, C6: footprint Capacitor_SMD:C_0805_2012Metric -> Capacitor_SMD:C_0603_1608Metric
- C31, C7: footprint (none) -> Capacitor_SMD:C_0603_1608Metric
- C46: footprint (none) -> Capacitor_SMD:CP_Elec_4x5.4
- C5: footprint Capacitor_SMD:C_0805_2012Metric -> Capacitor_SMD:C_0603_1608Metric; Dielectric X5R/X7R -> (none); Voltage  16V -> (none)
- D1: Current 1A -> (none); Fieldname2 Value2 -> (none); Fieldname3 Value3 -> (none); Package SMA -> (none)
- D2, D4, D9: Current 1A -> (none)
- D3: Fieldname2 Value2 -> (none); Fieldname3 Value3 -> (none); Package SMA -> (none)
- R19, R22: value 470K -> 470k
- R20, R32: footprint (none) -> Resistor_SMD:R_0603_1608Metric
- R41, R53: value 2.2K -> 2.2k
- R43, R45: value 4.99K -> 4.99k
- R46, R47, R52: Tolerance 1% -> (none)
- R56: value 10K -> 10k
- R57, R68, R69: value 100K -> 100k
- R67: value 300K -> 300k
- TH2: Tolerance 0.1% -> (none)
- U4: footprint TO_SOT_Packages_SMD:SOT-23-5 -> Package_TO_SOT_SMD:SOT-23-5

Commit message: schematics and layout submitted for review
Parts:
- added R59, R60, R61, R62: 0R, Resistor_SMD:R_0805_2012Metric, symbol device:R
- added TP19: Test_Point, TestPoint:TestPoint_THTPad_D1.0mm_Drill0.5mm, symbol OSM_env01-rescue:Test_Point-Connector-ESP32-EVB_Rev_D-rescue
Connections:
- net +3V3: now also R60.1; no longer C46.1, C63.1, D9.2 (A), U4.5 (OUT)
- net +5V: now also R59.1; no longer C10.1, C5.1, C6.1, D2.1 (K), R46.1
- net BAT_OP: now also R61.1; no longer Q4.3 (S), R127.1, R27.1, R56.1, R57.1
- net BOOST_EN: now also R62.1; no longer C24.1, C72.1, Q4.5 (D), Q4.6 (D), R68.1, R69.1
- net GND: now also TP19.1
- new net: C10.1, C5.1, C6.1, D2.1 (K), R46.1, R59.2
- new net: Q4.3 (S), R127.1, R27.1, R56.1, R57.1, R61.2
- new net: C24.1, C72.1, Q4.5 (D), Q4.6 (D), R62.2, R68.1, R69.1
- new net: C46.1, C63.1, D9.2 (A), R60.2, U4.5 (OUT)
Other:
- moved on the sheet: C10, C2, C23, C25, C31, C32, C46, C5, C6, C63, C7, D2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

Commit message: osm env-01 revB finished
Parts:
- BAT1: footprint Battery:BatteryHolder_Keystone_1042_1x18650 -> Devtank_PCB_lib:BatteryHolder_Keystone_1042_1x18650
Changed lines of the file:
@@
 Sheet 2 9
 Title "Open Smart Monitor"
-Date "2021-09-22"
+Date "2021-09-29"
 Rev "B"
 Comp "Devtank LTD"
-Comment1 "AB"
+Comment1 "Part No: 304-010"
 Comment2 ""
 Comment3 ""
@@
 F 0 "BAT1" V 5575 3175 60  0000 L CNN
 F 1 "18650" V 5575 3625 51  0000 L CNN
-F 2 "Battery:BatteryHolder_Keystone_1042_1x18650" H 5625 3525 60  0001 C CNN
+F 2 "Devtank_PCB_lib:BatteryHolder_Keystone_1042_1x18650" H 5625 3525 60  0001 C CNN
 F 3 "" H 5625 3525 60  0000 C CNN
 F 4 "Value 1" H 5625 3525 60  0001 C CNN "Fieldname 1"
