File: kicad_osm_env01/Digital_IO.sch (KiCad schematic (older format))
At the start: 4 parts

Commit message: rough throwdown of all parts
Parts:
- R104, R105: value 1K -> 1k
Changed lines of the file:
@@
 P 3500 3675
 F 0 "R104" V 3293 3675 50  0000 C CNN
-F 1 "1K" V 3384 3675 50  0000 C CNN
+F 1 "1k" V 3384 3675 50  0000 C CNN
 F 2 "Resistor_SMD:R_0603_1608Metric" V 3430 3675 50  0001 C CNN
 F 3 "" H 3500 3675 50  0001 C CNN
@@
 P 3500 3875
 F 0 "R105" V 3600 3875 50  0000 C CNN
-F 1 "1K" V 3675 3850 50  0000 C CNN
+F 1 "1k" V 3675 3850 50  0000 C CNN
 F 2 "Resistor_SMD:R_0603_1608Metric" V 3430 3875 50  0001 C CNN
 F 3 "" H 3500 3875 50  0001 C CNN

Commit message: updated folder
Parts:
- D14, D16: Devtank 134-001 -> (none)
Changed lines of the file:
@@
 F 2 "Package_TO_SOT_SMD:SOT-23" H 4050 4925 50  0001 C CNN
 F 3 "www.nxp.com/documents/data_sheet/BAV99_SER.pdf" H 4050 5175 50  0001 C CNN
-F 4 "134-001" H 4050 5075 50  0001 C CNN "Devtank"
+F 4 "" H 4050 5075 50  0001 C CNN "Devtank"
 	1    4050 5075
 	0    1    1    0
@@
 F 2 "Package_TO_SOT_SMD:SOT-23" H 4000 3125 50  0001 C CNN
 F 3 "www.nxp.com/documents/data_sheet/BAV99_SER.pdf" H 4000 3375 50  0001 C CNN
-F 4 "134-001" H 4000 3275 50  0001 C CNN "Devtank"
+F 4 "" H 4000 3275 50  0001 C CNN "Devtank"
 	2    4000 3275
 	0    1    1    0
@@
 F 2 "Package_TO_SOT_SMD:SOT-23" H 3800 3125 50  0001 C CNN
 F 3 "www.nxp.com/documents/data_sheet/BAV99_SER.pdf" H 3800 3375 50  0001 C CNN
-F 4 "134-001" H 3800 3275 50  0001 C CNN "Devtank"
+F 4 "" H 3800 3275 50  0001 C CNN "Devtank"
 	2    3800 3275
 	0    1    1    0
@@
 F 2 "Package_TO_SOT_SMD:SOT-23" H 3850 4925 50  0001 C CNN
 F 3 "www.nxp.com/documents/data_sheet/BAV99_SER.pdf" H 3850 5175 50  0001 C CNN
-F 4 "134-001" H 3850 5075 50  0001 C CNN "Devtank"
+F 4 "" H 3850 5075 50  0001 C CNN "Devtank"
 	1    3850 5075
 	0    1    1    0
