File: kicad_osm_env01/Digital_IO.kicad_sch (KiCad schematic)
At the start: 20 parts, among them U18 MIC94073YC6, U20 MIC94073YC6

Commit message: before fixing devtank symbol issues
Parts:
- added R154, R155: (no value), symbol Device:R
Connections:
- net PULSE1_PULLUP_EN: now also R154.1; no longer R92.1, U18.3 (EN)
- net PULSE2_PULLUP_EN: now also R155.1; no longer R93.1, U20.3 (EN)
- new net: R154.2, R92.1, U18.3 (EN)
- new net: R155.2, R93.1, U20.3 (EN)
Changed lines of the file:
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@@
+    (stroke (width 0) (type default) (color 0 0 0 0))
+  )
+  (wire (pts (xy 81.915 132.08) (xy 84.455 132.08))
     (stroke (width 0) (type default) (color 0 0 0 0))
   )
@@
   )
   (wire (pts (xy 74.295 111.76) (xy 74.295 110.49))
+    (stroke (width 0) (type default) (color 0 0 0 0))
+  )
+  (wire (pts (xy 81.28 85.725) (xy 83.82 85.725))
     (stroke (width 0) (type default) (color 0 0 0 0))
   )
@@
     (effects (font (size 1.27 1.27)) (justify right))
   )
-  (hierarchical_label "PULSE2_PULLUP_EN" (shape input) (at 92.075 132.08 180)
+  (hierarchical_label "PULSE2_PULLUP_EN" (shape input) (at 81.915 132.08 180)
     (effects (font (size 1.27 1.27)) (justify right))
   )
-  (hierarchical_label "PULSE1_PULLUP_EN" (shape input) (at 91.44 85.725 180)
+  (hierarchical_label "PULSE1_PULLUP_EN" (shape input) (at 81.28 85.725 180)
     (effects (font (size 1.27 1.27)) (justify right))
   )
@@
     (pin "2")
   )
+  (symbol (lib_id "Device:R") (at 87.63 85.725 90) (unit 1)
+    (in_bom yes) (on_board yes) (fields_autoplaced)
+    (property "Reference" "R154" (id 0) (at 87.63 81.0092 90))
+    (property "Value" "" (id 1) (at 87.63 83.5461 90))
+    (property "Footprint" "" (id 2) (at 87.63 87.503 90)
+      (effects (font (size 1.27 1.27)) hide)
+    )
+    (property "Datasheet" "~" (id 3) (at 87.63 85.725 0)
+      (effects (font (size 1.27 1.27)) hide)
+    )
+    (pin "1")
+    (pin "2")
+  )
   (symbol (lib_id "power:+3V3") (at 154.94 99.695 0) (unit 1)
     (in_bom yes) (on_board yes)
@@
     (pin "6")
   )
+  (symbol (lib_id "Device:R") (at 88.265 132.08 90) (unit 1)
+    (in_bom yes) (on_board yes) (fields_autoplaced)
+    (property "Reference" "R155" (id 0) (at 88.265 127.3642 90))
+    (property "Value" "" (id 1) (at 88.265 129.9011 90))
+    (property "Footprint" "" (id 2) (at 88.265 133.858 90)
+      (effects (font (size 1.27 1.27)) hide)
+    )
+    (property "Datasheet" "~" (id 3) (at 88.265 132.08 0)
+      (effects (font (size 1.27 1.27)) hide)
+    )
+    (pin "1")
+    (pin "2")
+  )
   (symbol (lib_id "OSM_env01-rescue:R-device-ESP32-EVB_Rev_D-rescue") (at 154.94 115.57 0) (unit 1)

Commit message: started layout with throwdown
Parts:
- C23, C49: value DNF -> (none); footprint Capacitor_SMD:C_0603_1608Metric -> (none); symbol device:C -> Device:C
- C50, C57: value 1nF -> (none); footprint Capacitor_SMD:C_0402_1005Metric -> (none); symbol device:C -> Device:C
- D6, D7: value BAV99 -> (none); footprint Package_TO_SOT_SMD:SOT-23 -> (none)
- R104, R105: value 100R -> (none); footprint Resistor_SMD:R_0603_1608Metric -> (none); symbol OSM_env01-rescue:R-device-ESP32-EVB_Rev_D-rescue -> Device:R
- R130, R94: value 0R -> (none); footprint Resistor_SMD:R_0603_1608Metric -> (none); symbol device:R -> Device:R
- R137, R138, R139, R140: value DNF -> (none); footprint Resistor_SMD:R_0603_1608Metric -> (none); symbol OSM_env01-rescue:R-device-ESP32-EVB_Rev_D-rescue -> Device:R
- R81, R91: value 10k -> (none)
- R92, R93: value 100k -> (none); footprint Resistor_SMD:R_0603_1608Metric -> (none); symbol device:R -> Device:R
- U18, U20: value MIC94073YC6 -> (none); footprint Package_TO_SOT_SMD:SOT-363_SC-70-6 -> (none)
