File: kicad_osm_env01/PowerSupply.kicad_sch (KiCad schematic)
At the start: 73 parts, among them Q1 SI2301BDS-T1-E3, Q7 FDS9926A, SW1 EG1247, U1 MIC2251YML-TR, U14 S-8261ACBMD-G4BT2U, U17 MIC5219-3.3YMM, U2 MCP73832T-2AC, U4 MIC5219-3.3YMM, U9 DNF

Commit message: started layout with throwdown
Parts:
- BAT1: value 18650 -> (none); footprint Devtank_PCB_lib:BatteryHolder_Keystone_1042_1x18650 -> (none); symbol device:Battery -> Device:Battery
- C10: value 4.7nF -> (none); footprint Capacitor_SMD:C_0402_1005Metric -> (none); symbol device:C -> Device:C
- C11, C7: value DNF -> (none); footprint Capacitor_SMD:C_0603_1608Metric -> (none); symbol device:C -> Device:C
- C14, C32: value DNF -> (none); footprint Capacitor_SMD:C_0402_1005Metric -> (none); symbol device:C -> Device:C
- C2, C5: value 10uF -> (none); footprint Capacitor_SMD:C_0603_1608Metric -> (none); symbol OSM_env01-rescue:C-device-ESP32-EVB_Rev_D-rescue -> Device:C
- C22, C25, C63, C9: value 1uF -> (none); footprint Capacitor_SMD:C_0402_1005Metric -> (none); symbol device:C -> Device:C
- C24, C46: value DNF -> (none); footprint Capacitor_SMD:CP_Elec_4x5.4 -> (none); symbol device:C -> Device:C
- C3: value 4.7uF -> (none); footprint Capacitor_SMD:C_0805_2012Metric -> (none); symbol device:C -> Device:C
- C31, C6: value DNF -> (none); footprint Capacitor_SMD:C_0603_1608Metric -> (none); symbol OSM_env01-rescue:C-device-ESP32-EVB_Rev_D-rescue -> Device:C
- C33: value DNF -> (none); footprint Capacitor_SMD:C_0805_2012Metric -> (none); symbol device:C -> Device:C
- C34, R5: value DNF -> (none)
- C65: value 100nF -> (none)
- C74: value 4.7uF -> (none); symbol device:C -> Device:C
- D10, D2, D9: value RB160M-40TR -> (none); footprint Diode_SMD:D_SOD-123 -> (none)
- D14: value YLW -> (none); footprint Devtank_PCB_lib:LED_Rectangular_W4.5mm_H7.3mm_Horizontal_2.54mm_Z3.0mm -> (none); symbol device:LED -> Device:LED
- D3: value RB160M-40TR -> (none); footprint Diode_SMD:D_SOD-123 -> (none); symbol device:D_Schottky -> Device:D_Schottky
- D5: value SMFE5-0A -> (none); footprint Diode_SMD:D_SOD-123 -> (none); symbol device:D_TVS -> Device:D_TVS
- JP19: value Jumper_2_Open -> (none)
- L1: value 10uH -> (none); footprint Inductor_SMD:L_1812_4532Metric -> (none)
- Q1: value SI2301BDS-T1-E3 -> (none); footprint Package_TO_SOT_SMD:SOT-23 -> (none)
- Q7: value FDS9926A -> (none); footprint Package_SO:SOIC-8_3.9x4.9mm_P1.27mm -> (none)
- R102: value 2k -> (none)
- R112, R114, R18: value 1M -> (none); footprint Resistor_SMD:R_0603_1608Metric -> (none); symbol device:R -> Device:R
- R113, R116, R19: value 470k -> (none); footprint Resistor_SMD:R_0603_1608Metric -> (none); symbol device:R -> Device:R
- R115, R20, R68: value 0R -> (none); footprint Resistor_SMD:R_0603_1608Metric -> (none); symbol device:R -> Device:R
- R128: value DNF -> (none); footprint Resistor_SMD:R_0603_1608Metric -> (none); symbol device:R -> Device:R
- R131: value 10k -> (none); footprint Resistor_SMD:R_0603_1608Metric -> (none); symbol device:R -> Device:R
- R44: value 2k -> (none); footprint Resistor_SMD:R_0603_1608Metric -> (none); symbol OSM_env01-rescue:R-ESP32-EVB_Rev_D -> Device:R
- R45, R69: value 0R -> (none)
- R46: value 110k -> (none); footprint Resistor_SMD:R_0603_1608Metric -> (none); symbol OSM_env01-rescue:R-device-ESP32-EVB_Rev_D-rescue -> Device:R
- R47: value 36k -> (none); footprint Resistor_SMD:R_0603_1608Metric -> (none); symbol OSM_env01-rescue:R-device-ESP32-EVB_Rev_D-rescue -> Device:R
- R52: value 5k -> (none); symbol device:R -> Device:R
- R54: value DNF -> (none); footprint Resistor_SMD:R_0603_1608Metric -> (none); symbol OSM_env01-rescue:R-ESP32-EVB_Rev_D -> Device:R
- R58: value 1M -> (none); footprint Resistor_SMD:R_0603_1608Metric -> (none); symbol OSM_env01-rescue:R-device-ESP32-EVB_Rev_D-rescue -> Device:R
- R59, R60, R70: value 0R -> (none); footprint Resistor_SMD:R_0805_2012Metric -> (none); symbol device:R -> Device:R
- R64: value 470k -> (none); footprint Resistor_SMD:R_0603_1608Metric -> (none); symbol OSM_env01-rescue:R-device-ESP32-EVB_Rev_D-rescue -> Device:R
- R98: value 470R -> (none)
- SW1: value EG1247 -> (none)
- TH1: value 10k -> (none); symbol device:Thermistor -> Device:Thermistor
- TP18, TP34, TP77, TP79: value Test_Point -> (none); footprint TestPoint:TestPoint_Pad_D1.5mm -> (none)
- TP25, TP26, TP52: value Test_Point -> (none); footprint TestPoint:TestPoint_THTPad_D1.0mm_Drill0.5mm -> (none)
- TP65: value Test_Point -> (none)
- U1: value MIC2251YML-TR -> (none); footprint MLF-8_ML_MCH -> (none)
- U14: value S-8261ACBMD-G4BT2U -> (none)
- U17: value MIC5219-3.3YMM -> (none); footprint Package_SO:MSOP-8_3x3mm_P0.65mm -> (none)
- U2: value MCP73832T-2AC -> (none); footprint TO_SOT_Packages_SMD:SOT-23-5 -> (none)
- U4: value MIC5219-3.3YMM -> (none)
- U9: value DNF -> (none); footprint Package_TO_SOT_SMD:SOT-23-5 -> (none)
Connections:
- net 5Vin: no longer R45.1
- net GND: no longer C10.2
- net at R46.2, R47.1, U1.1 (FB): now also C10.2
- new net 5V_INPUT: R45.1
Other:
- moved on the sheet: C10, R44, R54
