File: kicad_osm_env01/STM32L4.kicad_sch (KiCad schematic)
At the start: 37 parts, among them J6 Conn_02x03_Odd_Even, U6 STM32L433VCTx, Y1 8MHZ, Y2 DNF

Commit message: Schematics waiting review
Parts:
- removed R13, R14: 0R, symbol device:R
Connections:
- net PB13 is gone; now on net SPI1_CS: U6.52 (DFSDM_CKIN1/I2C2_SCL/LCD_SEG13/LPUART1_CTS/SAI2_SCK_A/SPI2_SCK/SWPMI1_TX/TIM15_CH1N/TIM1_CH1N/TSC_G1_IO2/USART3_CTS/PB13)
- net CAN1_RX: now also U6.70 (ADC1_EXTI11/ADC2_EXTI11/ADC3_EXTI11/CAN1_RX/TIM1_BKIN2/TIM1_BKIN2_COMP1/TIM1_CH4/USART1_CTS/USB_OTG_FS_DM/PA11)
- net CAN1_TX: now also U6.71 (CAN1_TX/TIM1_ETR/USART1_DE/USART1_RTS/USB_OTG_FS_DP/PA12)
- net SPI1_CS: no longer U6.16 (ADC1_IN2/ADC2_IN2/ADC3_IN2/DFSDM_CKIN4/I2C3_SDA/LCD_SEG19/LPTIM1_OUT/LPUART1_TX/PC1)
- net +3V3 renamed +3V3_CORE
- net PB12 renamed GPIO17
- new net ADC1: U6.16 (ADC1_IN2/ADC2_IN2/ADC3_IN2/DFSDM_CKIN4/I2C3_SDA/LCD_SEG19/LPTIM1_OUT/LPUART1_TX/PC1)
Other:
- note added: "Please note: - usb may not be available on all packages - For comfirmation of pin functions refer to datasheet. Symbol may not be correct - The I/Os with wakeup from Standby/Shutdown capability are: PA0, PC13, PE6, PA2, PC5 -I/Os can be configured with internal pull-up, pull-down or floating in Shutdown mode but the configuration is lost when exiting the Shutdown mode. - After reset, these pins a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"
- note removed: "STM32l451 Note: For comfirmation of pin functions refer to datasheet. Symbol may not be correct - wkup pins 2,14,16,25 -pa13, pa15, pb4 avoid as after reset internal pull up and pull down activated"
- note removed: "please not usb may not be available on all packages"
- moved on the sheet: C1, C12, C13, C27, C51, C62, D8, J6, R119, R12, R15, R16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

Commit message: before fixing devtank symbol issues
Parts:
- J6: value Conn_02x03_Odd_Even -> (none); footprint Connector:Tag-Connect_TC2030-IDC-NL_2x03_P1.27mm_Vertical -> (none); symbol Connector:Conn_02x03_Odd_Even -> Connector_Generic:Conn_02x03_Odd_Even
Changed lines of the file:
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@@
     (pin "1")
   )
-  (symbol (lib_name "PWR_FLAG_3") (lib_id "power:PWR_FLAG") (at 38.1 108.585 0) (unit 1)
-    (in_bom yes) (on_board yes)
-    (property "Reference" "#FLG0111" (id 0) (at 38.1 106.68 0)
-      (effects (font (size 1.27 1.27)) hide)
-    )
-    (property "Value" "PWR_FLAG" (id 1) (at 38.1 104.775 0))
+  (symbol (lib_id "power:PWR_FLAG") (at 38.1 108.585 0) (unit 1)
+    (in_bom yes) (on_board yes) (fields_autoplaced)
+    (property "Reference" "#FLG09" (id 0) (at 38.1 106.68 0)
+      (effects (font (size 1.27 1.27)) hide)
+    )
+    (property "Value" "" (id 1) (at 38.1 105.0092 0))
     (property "Footprint" "" (id 2) (at 38.1 108.585 0)
       (effects (font (size 1.27 1.27)) hide)
     )
-    (property "Datasheet" "~" (id 3) (at 38.1 108.585 0)
+    (property "Datasheet" "" (id 3) (at 38.1 108.585 0)
       (effects (font (size 1.27 1.27)) hide)
     )
@@
     (pin "1")
   )
-  (symbol (lib_name "PWR_FLAG_3") (lib_id "power:PWR_FLAG") (at 54.61 125.095 180) (unit 1)
-    (in_bom yes) (on_board yes)
-    (property "Reference" "#FLG0113" (id 0) (at 54.61 127 0)
-      (effects (font (size 1.27 1.27)) hide)
-    )
-    (property "Value" "PWR_FLAG" (id 1) (at 52.705 129.54 0))
-    (property "Footprint" "" (id 2) (at 54.61 125.095 0)
-      (effects (font (size 1.27 1.27)) hide)
-    )
-    (property "Datasheet" "~" (id 3) (at 54.61 125.095 0)
+  (symbol (lib_id "power:PWR_FLAG") (at 236.855 81.28 0) (unit 1)
+    (in_bom yes) (on_board yes) (fields_autoplaced)
+    (property "Reference" "#FLG08" (id 0) (at 236.855 79.375 0)
+      (effects (font (size 1.27 1.27)) hide)
+    )
+    (property "Value" "" (id 1) (at 236.855 77.7042 0))
+    (property "Footprint" "" (id 2) (at 236.855 81.28 0)
+      (effects (font (size 1.27 1.27)) hide)
+    )
+    (property "Datasheet" "" (id 3) (at 236.855 81.28 0)
       (effects (font (size 1.27 1.27)) hide)
     )
@@
     (pin "1")
   )
+  (symbol (lib_id "power:PWR_FLAG") (at 54.61 125.095 180) (unit 1)
+    (in_bom yes) (on_board yes) (fields_autoplaced)
+    (property "Reference" "#FLG010" (id 0) (at 54.61 127 0)
+      (effects (font (size 1.27 1.27)) hide)
+    )
+    (property "Value" "" (id 1) (at 54.61 129.5384 0))
+    (property "Footprint" "" (id 2) (at 54.61 125.095 0)
+      (effects (font (size 1.27 1.27)) hide)
+    )
+    (property "Datasheet" "" (id 3) (at 54.61 125.095 0)
+      (effects (font (size 1.27 1.27)) hide)
+    )
+    (pin "1")
+  )
   (symbol (lib_id "Device:R") (at 27.305 115.57 90) (unit 1)
     (in_bom yes) (on_board yes) (fields_autoplaced)
@@
     (pin "1")
   )
-  (symbol (lib_name "PWR_FLAG_1") (lib_id "power:PWR_FLAG") (at 236.855 81.28 0) (unit 1)
-    (in_bom yes) (on_board yes)
-    (property "Reference" "#FLG0110" (id 0) (at 236.855 79.375 0)
-      (effects (font (size 1.27 1.27)) hide)
-    )
-    (property "Value" "PWR_FLAG" (id 1) (at 243.84 80.01 0))
-    (property "Footprint" "" (id 2) (at 236.855 81.28 0)
-      (effects (font (size 1.27 1.27)) hide)
-    )
-    (property "Datasheet" "~" (id 3) (at 236.855 81.28 0)
-      (effects (font (size 1.27 1.27)) hide)
-    )
-    (pin "1")
-  )
   (symbol (lib_id "device:Ferrite_Bead") (at 89.535 54.61 270) (unit 1)
     (in_bom yes) (on_board yes)
@@
     (pin "1")
   )
-  (symbol (lib_id "Connector:Conn_02x03_Odd_Even") (at 289.56 30.48 0) (unit 1)
+  (symbol (lib_id "Connector_Generic:Conn_02x03_Odd_Even") (at 289.56 30.48 0) (unit 1)
     (in_bom yes) (on_board yes)
     (property "Reference" "J6" (id 0) (at 290.83 24.765 0))
-    (property "Value" "Conn_02x03_Odd_Even" (id 1) (at 290.83 24.7396 0)
-      (effects (font (size 1.27 1.27)) hide)
-    )
-    (property "Footprint" "Connector:Tag-Connect_TC2030-IDC-NL_2x03_P1.27mm_Vertical" (id 2) (at 289.56 30.48 0)
-      (effects (font (size 1.27 1.27)) hide)
-    )
+    (property "Value" "" (id 1) (at 290.83 24.7396 0)
+      (effects (font (size 1.27 1.27)) hide)
+    )
+    (property "Footprint" "" (id 2) (at 289.56 30.48 0)
+      (effects (font (size 1.27 1.27)) hide)
+    )

Commit message: started layout with throwdown
Parts:
- removed Y2: DNF, Crystal:Crystal_SMD_7050-4Pin_7.0x5.0mm, symbol device:Crystal_GND23
- added C68: (no value), symbol Device:C
- added Y2: (no value), symbol Device:Crystal
- C1, C12: value 10pF -> (none); footprint Capacitor_SMD:C_0402_1005Metric -> (none); symbol device:C -> Device:C
- C13, C27: value DNF -> (none); footprint Capacitor_SMD:C_0402_1005Metric -> (none); symbol device:C -> Device:C
- C28, C29, C30, C43, C44, C51, C62, C64: value 100nF -> (none); footprint Capacitor_SMD:C_0402_1005Metric -> (none); symbol device:C -> Device:C
- C52, C53, C60: value 1uF -> (none); footprint Capacitor_SMD:C_0402_1005Metric -> (none); symbol device:C -> Device:C
- C59: value 4.7uF -> (none); footprint Capacitor_SMD:C_0603_1608Metric -> (none); symbol device:C -> Device:C
- C61: value 10nF -> (none); footprint Capacitor_SMD:C_0402_1005Metric -> (none); symbol device:C -> Device:C
- D8: value RED -> (none); footprint Devtank_PCB_lib:LED_Rectangular_W4.5mm_H7.3mm_Horizontal_2.54mm_Z3.0mm -> (none); symbol device:LED -> Device:LED
- L2, L7: value 2A/0.05DCR -> (none); footprint Inductor_SMD:L_0402_1005Metric -> (none); symbol device:Ferrite_Bead -> Device:FerriteBead
- R119, R16: value 10k -> (none); footprint Resistor_SMD:R_0603_1608Metric -> (none); symbol device:R -> Device:R
- R12, R7: value 0R -> (none); symbol device:R -> Device:R
- R15, R30: value DNF -> (none); footprint Resistor_SMD:R_0603_1608Metric -> (none); symbol device:R -> Device:R
- R26: value 390R -> (none); footprint Resistor_SMD:R_0603_1608Metric -> (none); symbol device:R -> Device:R
- R6: value 1.3k -> (none); footprint Resistor_SMD:R_0603_1608Metric -> (none); symbol device:R -> Device:R
- R90, R95: value 0R -> (none)
- S1: value B3U-1100P -> (none); footprint Button_Switch_SMD:SW_SPST_B3U-1100P -> (none)
- U6: value STM32L433VCTx -> (none); footprint LQFP100 -> (none)
- Y1: value 8MHZ -> (none); footprint Crystal:Crystal_SMD_Abracon_ABM3C-4Pin_5.0x3.2mm -> (none); symbol device:Crystal_GND24 -> Device:Crystal_GND24
Connections:
- net +3V3_CORE: now also C68.1
- net 32.768KHZ_crystal_in: now also Y2.2
- net 32.768KHZ_crystal_out: now also Y2.1
- net GND: now also C68.2
- no-connect marks 34 -> 32
Other:
- moved on the sheet: C43, C52, C59
