File: kicad_osm_env01/Sensors_AND_IO.kicad_sch (KiCad schematic)
At the start: 59 parts, among them J4 Conn_01x08, J8 STX-3000, U10 ICS-43434, U11 HPP845E131R5, U12 MIC94073YC6, U3 VEML7700-TT

Commit message: started layout with throwdown
Parts:
- removed J7: (no value), symbol Connector_Generic:Conn_01x05
- removed R61, R62, R63, R65, R66, R67: DNF, Resistor_SMD:R_1206_3216Metric, symbol device:R
- removed TP42, TP43, TP46, TP47, TP75, TP76: Test_Point, TestPoint:TestPoint_Pad_D1.5mm, symbol OSM_env01-rescue:Test_Point-Connector-ESP32-EVB_Rev_D-rescue
- added J7: (no value), symbol Connector_Generic:Conn_01x03
- C39, C41: value 100nF -> (none); footprint Capacitor_SMD:C_0402_1005Metric -> (none); symbol OSM_env01-rescue:C-device-ESP32-EVB_Rev_D-rescue -> Device:C
- C4, C8: value 100nF -> (none); footprint Capacitor_SMD:C_0603_1608Metric -> (none); symbol device:C -> Device:C
- C40: value 22uF -> (none); footprint Capacitor_SMD:C_0805_2012Metric -> (none); symbol OSM_env01-rescue:C-device-ESP32-EVB_Rev_D-rescue -> Device:C
- C42: value 10nF -> (none); footprint Capacitor_SMD:C_0402_1005Metric -> (none); symbol OSM_env01-rescue:C-device-ESP32-EVB_Rev_D-rescue -> Device:C
- C55: value DNF -> (none); footprint Capacitor_SMD:C_0603_1608Metric -> (none); symbol device:C -> Device:C
- C56: value 100nF -> (none); footprint Capacitor_SMD:C_0402_1005Metric -> (none); symbol device:C -> Device:C
- C71: value 10uF -> (none); footprint Capacitor_SMD:CP_Elec_4x5.4 -> (none); symbol device:CP -> Device:C
- D1, D19, D4: value DNF -> (none); footprint Diode_SMD:D_SOD-123 -> (none); symbol device:D_TVS -> Device:D_TVS
- J4: value Conn_01x08 -> (none); footprint Connector_Molex:Molex_PicoBlade_53047-0810_1x08_P1.25mm_Vertical -> (none)
- J8: value STX-3000 -> (none); footprint Devtank_PCB_lib:STX-3000 -> (none)
- L11, L12, L3: value 2A/0.05DCR -> (none); footprint Inductor_SMD:L_0402_1005Metric -> (none); symbol device:Ferrite_Bead -> Device:FerriteBead
- R100, R101: value DNF -> (none); footprint Resistor_SMD:R_0603_1608Metric -> (none); symbol OSM_env01-rescue:R-device-ESP32-EVB_Rev_D-rescue -> Device:R
- R124: value 82R -> (none); footprint Resistor_SMD:R_1206_3216Metric -> (none); symbol device:R -> Device:R
- R125, R126: value 1M -> (none); footprint Resistor_SMD:R_0603_1608Metric -> (none); symbol device:R -> Device:R
- R39: value 0R -> (none); footprint Resistor_SMD:R_0603_1608Metric -> (none); symbol device:R -> Device:R
- R40, R97, R99: value 100k -> (none); footprint Resistor_SMD:R_0603_1608Metric -> (none); symbol device:R -> Device:R
- R41, R53, R56, R57: value DNF -> (none); footprint Resistor_SMD:R_1206_3216Metric -> (none); symbol device:R -> Device:R
- R71: value DNF -> (none); symbol device:R -> Device:R
- R88: value 30R -> (none); footprint Resistor_SMD:R_1206_3216Metric -> (none); symbol device:R -> Device:R
- R96: value DNF -> (none); footprint Resistor_SMD:R_0603_1608Metric -> (none); symbol device:R -> Device:R
- TP13, TP14, TP48, TP49: value Test_Point -> (none); footprint TestPoint:TestPoint_THTPad_D1.0mm_Drill0.5mm -> (none)
- TP44, TP45, TP50, TP51, TP56: value Test_Point -> (none); footprint TestPoint:TestPoint_Pad_D1.5mm -> (none)
- U10: value ICS-43434 -> (none); footprint Devtank_PCB_lib:ICS-43434 -> (none)
- U11: value HPP845E131R5 -> (none); footprint Devtank_PCB_lib:HPP845E131R5_temperature_humidity_sensor -> (none)
- U12: value MIC94073YC6 -> (none); footprint Package_TO_SOT_SMD:SOT-363_SC-70-6 -> (none)
- U3: value VEML7700-TT -> (none); footprint Devtank_PCB_lib:VEML7700-TT -> (none)
Connections:
- net CT2+: now also J7.1 (Pin_1)
- net CT3+: now also J7.2 (Pin_2)
- net CT_REF: now also J7.3 (Pin_3)
