File: kicad_osm_env01/LORA.kicad_sch (KiCad schematic)
At the start: 15 parts, among them U16 RAK3172

Commit message: started layout with throwdown
Parts:
- C26: value DNF -> (none); footprint Capacitor_SMD:C_0402_1005Metric -> (none); symbol device:C -> Device:C
- C35: value 10uF -> (none); footprint Capacitor_SMD:C_0603_1608Metric -> (none); symbol device:C -> Device:C
- C70: value 100nF -> (none); footprint Capacitor_SMD:C_0402_1005Metric -> (none); symbol device:C -> Device:C
- L4: value 2A/0.05DCR -> (none); footprint Inductor_SMD:L_0402_1005Metric -> (none); symbol device:Ferrite_Bead -> Device:FerriteBead
- R103, R121, R132, R133: value 0R -> (none); symbol device:R -> Device:R
- R122, R129: value DNF -> (none); footprint Resistor_SMD:R_0603_1608Metric -> (none); symbol device:R -> Device:R
- R123: value 10k -> (none); footprint Resistor_SMD:R_0603_1608Metric -> (none); symbol device:R -> Device:R
- R134, R135: value DNF -> (none); symbol device:R -> Device:R
- U16: value RAK3172 -> (none)
Changed lines of the file:
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@@
     (effects (font (size 1.27 1.27)) (justify right))
   )
-  (symbol (lib_id "device:R") (at 248.285 27.94 0) (unit 1)
+  (symbol (lib_id "Device:R") (at 248.285 27.94 0) (unit 1)
     (in_bom yes) (on_board yes)
     (property "Reference" "R123" (id 0) (at 250.063 26.7716 0)
       (effects (font (size 1.27 1.27)) (justify left))
     )
-    (property "Value" "10k" (id 1) (at 250.063 29.083 0)
-      (effects (font (size 1.27 1.27)) (justify left))
-    )
-    (property "Footprint" "Resistor_SMD:R_0603_1608Metric" (id 2) (at 246.507 27.94 90)
+    (property "Value" "" (id 1) (at 250.063 29.083 0)
+      (effects (font (size 1.27 1.27)) (justify left))
+    )
+    (property "Footprint" "" (id 2) (at 246.507 27.94 90)
       (effects (font (size 1.27 1.27)) hide)
     )
@@
     (pin "2")
   )
-  (symbol (lib_id "device:C") (at 248.285 38.735 0) (unit 1)
+  (symbol (lib_id "Device:C") (at 248.285 38.735 0) (unit 1)
     (in_bom yes) (on_board yes)
     (property "Reference" "C70" (id 0) (at 251.206 37.5666 0)
       (effects (font (size 1.27 1.27)) (justify left))
     )
-    (property "Value" "100nF" (id 1) (at 251.206 39.878 0)
-      (effects (font (size 1.27 1.27)) (justify left))
-    )
-    (property "Footprint" "Capacitor_SMD:C_0402_1005Metric" (id 2) (at 249.2502 42.545 0)
+    (property "Value" "" (id 1) (at 251.206 39.878 0)
+      (effects (font (size 1.27 1.27)) (justify left))
+    )
+    (property "Footprint" "" (id 2) (at 249.2502 42.545 0)
       (effects (font (size 1.27 1.27)) hide)
     )
@@
     (pin "1")
   )
-  (symbol (lib_id "device:C") (at 81.28 62.865 0) (mirror y) (unit 1)
+  (symbol (lib_id "Device:C") (at 81.28 62.865 0) (mirror y) (unit 1)
     (in_bom yes) (on_board yes)
     (property "Reference" "C26" (id 0) (at 78.359 61.6966 0)
       (effects (font (size 1.27 1.27)) (justify left))
     )
-    (property "Value" "DNF" (id 1) (at 78.359 64.008 0)
-      (effects (font (size 1.27 1.27)) (justify left))
-    )
-    (property "Footprint" "Capacitor_SMD:C_0402_1005Metric" (id 2) (at 80.3148 66.675 0)
+    (property "Value" "" (id 1) (at 78.359 64.008 0)
+      (effects (font (size 1.27 1.27)) (justify left))
+    )
+    (property "Footprint" "" (id 2) (at 80.3148 66.675 0)
       (effects (font (size 1.27 1.27)) hide)
     )
@@
     (pin "2")
   )
-  (symbol (lib_id "device:C") (at 69.215 62.865 0) (mirror y) (unit 1)
+  (symbol (lib_id "Device:C") (at 69.215 62.865 0) (mirror y) (unit 1)
     (in_bom yes) (on_board yes)
     (property "Reference" "C35" (id 0) (at 66.294 61.6966 0)
       (effects (font (size 1.27 1.27)) (justify left))
     )
-    (property "Value" "10uF" (id 1) (at 66.294 64.008 0)
-      (effects (font (size 1.27 1.27)) (justify left))
-    )
-    (property "Footprint" "Capacitor_SMD:C_0603_1608Metric" (id 2) (at 68.2498 66.675 0)
+    (property "Value" "" (id 1) (at 66.294 64.008 0)
+      (effects (font (size 1.27 1.27)) (justify left))
+    )
+    (property "Footprint" "" (id 2) (at 68.2498 66.675 0)
       (effects (font (size 1.27 1.27)) hide)
     )
@@
     (pin "2")
   )
-  (symbol (lib_id "OSM_env01:GND") (at 74.93 69.215 0) (mirror y) (unit 1)
+  (symbol (lib_id "power:GND") (at 74.93 69.215 0) (mirror y) (unit 1)
     (in_bom yes) (on_board yes)
     (property "Reference" "#PWR052" (id 0) (at 74.93 75.565 0)
@@
     (pin "1")
   )
-  (symbol (lib_id "OSM_env01:GND") (at 97.155 125.095 0) (unit 1)
+  (symbol (lib_id "power:GND") (at 97.155 125.095 0) (unit 1)
     (in_bom yes) (on_board yes)
     (property "Reference" "#PWR051" (id 0) (at 97.155 131.445 0)
@@
     (pin "1")
   )
-  (symbol (lib_id "device:Ferrite_Bead") (at 54.61 59.055 270) (unit 1)
+  (symbol (lib_id "Device:FerriteBead") (at 54.61 59.055 270) (unit 1)
     (in_bom yes) (on_board yes)
     (property "Reference" "L4" (id 0) (at 54.61 52.0954 90))
-    (property "Value" "2A/0.05DCR" (id 1) (at 54.61 54.4068 90))
-    (property "Footprint" "Inductor_SMD:L_0402_1005Metric" (id 2) (at 54.61 57.277 90)
+    (property "Value" "" (id 1) (at 54.61 54.4068 90))
+    (property "Footprint" "" (id 2) (at 54.61 57.277 90)
       (effects (font (size 1.27 1.27)) hide)
     )
@@
     (pin "1")
   )
-  (symbol (lib_id "device:R") (at 147.32 82.55 90) (unit 1)
+  (symbol (lib_id "Device:R") (at 147.32 82.55 90) (unit 1)
     (in_bom yes) (on_board yes)
     (property "Reference" "R103" (id 0) (at 141.605 81.28 90))
-    (property "Value" "0R" (id 1) (at 152.4 81.28 90))
+    (property "Value" "" (id 1) (at 152.4 81.28 90))
     (property "Footprint" "" (id 2) (at 147.32 84.328 90)
       (effects (font (size 1.27 1.27)) hide)
@@
     (pin "2")
   )
-  (symbol (lib_id "device:R") (at 71.12 94.615 90) (unit 1)
+  (symbol (lib_id "Device:R") (at 71.12 94.615 90) (unit 1)
     (in_bom yes) (on_board yes)
     (property "Reference" "R135" (id 0) (at 62.865 93.345 90))
-    (property "Value" "DNF" (id 1) (at 76.2 93.345 90))
+    (property "Value" "" (id 1) (at 76.2 93.345 90))
     (property "Footprint" "" (id 2) (at 71.12 96.393 90)
       (effects (font (size 1.27 1.27)) hide)
@@
     (pin "2")
   )
-  (symbol (lib_id "device:R") (at 71.12 81.915 90) (unit 1)
+  (symbol (lib_id "Device:R") (at 71.12 81.915 90) (unit 1)
     (in_bom yes) (on_board yes)
     (property "Reference" "R132" (id 0) (at 62.865 80.645 90))
-    (property "Value" "0R" (id 1) (at 75.565 80.645 90))
+    (property "Value" "" (id 1) (at 75.565 80.645 90))
     (property "Footprint" "" (id 2) (at 71.12 83.693 90)
       (effects (font (size 1.27 1.27)) hide)
@@
     (pin "2")
   )
-  (symbol (lib_id "device:R") (at 270.51 38.735 0) (unit 1)
+  (symbol (lib_id "Device:R") (at 270.51 38.735 0) (unit 1)
     (in_bom yes) (on_board yes)
     (property "Reference" "R129" (id 0) (at 272.288 37.5666 0)
       (effects (font (size 1.27 1.27)) (justify left))
     )
-    (property "Value" "DNF" (id 1) (at 272.288 39.878 0)
-      (effects (font (size 1.27 1.27)) (justify left))
-    )
-    (property "Footprint" "Resistor_SMD:R_0603_1608Metric" (id 2) (at 268.732 38.735 90)
+    (property "Value" "" (id 1) (at 272.288 39.878 0)
+      (effects (font (size 1.27 1.27)) (justify left))
+    )
+    (property "Footprint" "" (id 2) (at 268.732 38.735 90)
       (effects (font (size 1.27 1.27)) hide)
     )
@@
     (in_bom yes) (on_board yes)
     (property "Reference" "U16" (id 0) (at 124.46 72.39 0))
-    (property "Value" "RAK3172" (id 1) (at 127 74.93 0))
+    (property "Value" "" (id 1) (at 127 74.93 0))
     (property "Footprint" "" (id 2) (at 95.885 85.09 0)
       (effects (font (size 1.27 1.27)) hide)
@@
     (pin "9")
   )
-  (symbol (lib_id "device:R") (at 71.12 91.44 90) (unit 1)
+  (symbol (lib_id "Device:R") (at 71.12 91.44 90) (unit 1)
     (in_bom yes) (on_board yes)
     (property "Reference" "R134" (id 0) (at 62.865 90.17 90))
-    (property "Value" "DNF" (id 1) (at 76.2 90.17 90))
+    (property "Value" "" (id 1) (at 76.2 90.17 90))
     (property "Footprint" "" (id 2) (at 71.12 93.218 90)
       (effects (font (size 1.27 1.27)) hide)
@@
     (pin "2")
   )
-  (symbol (lib_id "device:R") (at 270.51 27.94 0) (unit 1)
+  (symbol (lib_id "Device:R") (at 270.51 27.94 0) (unit 1)
     (in_bom yes) (on_board yes)
     (property "Reference" "R122" (id 0) (at 272.288 26.7716 0)
       (effects (font (size 1.27 1.27)) (justify left))
     )
-    (property "Value" "DNF" (id 1) (at 272.288 29.083 0)
-      (effects (font (size 1.27 1.27)) (justify left))
-    )
-    (property "Footprint" "Resistor_SMD:R_0603_1608Metric" (id 2) (at 268.732 27.94 90)
+    (property "Value" "" (id 1) (at 272.288 29.083 0)
+      (effects (font (size 1.27 1.27)) (justify left))
+    )
+    (property "Footprint" "" (id 2) (at 268.732 27.94 90)
       (effects (font (size 1.27 1.27)) hide)
     )
@@
     (pin "1")
   )
-  (symbol (lib_id "OSM_env01:GND") (at 197.485 41.275 0) (mirror y) (unit 1)
+  (symbol (lib_id "power:GND") (at 197.485 41.275 0) (mirror y) (unit 1)
     (in_bom yes) (on_board yes)
     (property "Reference" "#PWR098" (id 0) (at 197.485 47.625 0)
@@
     (pin "1")
   )
-  (symbol (lib_id "device:R") (at 71.12 85.09 90) (unit 1)
+  (symbol (lib_id "Device:R") (at 71.12 85.09 90) (unit 1)
     (in_bom yes) (on_board yes)
     (property "Reference" "R133" (id 0) (at 62.865 83.82 90))
-    (property "Value" "0R" (id 1) (at 75.565 83.82 90))
+    (property "Value" "" (id 1) (at 75.565 83.82 90))
     (property "Footprint" "" (id 2) (at 71.12 86.868 90)
       (effects (font (size 1.27 1.27)) hide)
@@
     (pin "2")
   )
-  (symbol (lib_id "device:R") (at 147.32 85.725 90) (unit 1)
+  (symbol (lib_id "Device:R") (at 147.32 85.725 90) (unit 1)
     (in_bom yes) (on_board yes)
     (property "Reference" "R121" (id 0) (at 141.605 84.455 90))
-    (property "Value" "0R" (id 1) (at 152.4 84.455 90))
+    (property "Value" "" (id 1) (at 152.4 84.455 90))
     (property "Footprint" "" (id 2) (at 147.32 87.503 90)
       (effects (font (size 1.27 1.27)) hide)

Commit message: Complete half pcb layout with routed signals
Parts:
- removed J9: (no value), symbol Connector_Generic:Conn_01x06
Connections:
- net LORA_BOOT0: no longer R121.1, U16.21 (BOOT0)
- net LORA_NRST: no longer R103.1, U16.22 (NRST)
- new net: R103.1, U16.22 (NRST)
- new net: R121.1, U16.21 (BOOT0)
Changed lines of the file:
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@@
-    (stroke (width 0) (type default) (color 0 0 0 0))
-  )
-  (wire (pts (xy 197.485 24.765) (xy 197.485 20.955))
-    (stroke (width 0) (type default) (color 0 0 0 0))
-  )
-  (wire (pts (xy 197.485 37.465) (xy 197.485 41.275))
     (stroke (width 0) (type default) (color 0 0 0 0))
   )
@@
     (stroke (width 0) (type default) (color 0 0 0 0))
   )
-  (wire (pts (xy 207.01 32.385) (xy 194.31 32.385))
-    (stroke (width 0) (type default) (color 0 0 0 0))
-  )
   (wire (pts (xy 74.93 91.44) (xy 80.01 91.44))
     (stroke (width 0) (type default) (color 0 0 0 0))
@@
     (stroke (width 0) (type default) (color 0 0 0 0))
   )
-  (wire (pts (xy 194.31 27.305) (xy 207.01 27.305))
-    (stroke (width 0) (type default) (color 0 0 0 0))
-  )
   (wire (pts (xy 88.9 71.755) (xy 88.9 59.055))
     (stroke (width 0) (type default) (color 0 0 0 0))
@@
     (stroke (width 0) (type default) (color 0 0 0 0))
   )
-  (wire (pts (xy 194.31 24.765) (xy 197.485 24.765))
-    (stroke (width 0) (type default) (color 0 0 0 0))
-  )
   (wire (pts (xy 92.075 122.555) (xy 92.075 123.825))
     (stroke (width 0) (type default) (color 0 0 0 0))
@@
     (stroke (width 0) (type default) (color 0 0 0 0))
   )
-  (wire (pts (xy 194.31 34.925) (xy 207.01 34.925))
-    (stroke (width 0) (type default) (color 0 0 0 0))
-  )
   (wire (pts (xy 236.855 33.02) (xy 248.285 33.02))
     (stroke (width 0) (type default) (color 0 0 0 0))
   )
-  (wire (pts (xy 194.31 29.845) (xy 207.01 29.845))
-    (stroke (width 0) (type default) (color 0 0 0 0))
-  )
   (wire (pts (xy 124.46 85.725) (xy 143.51 85.725))
     (stroke (width 0) (type default) (color 0 0 0 0))
@@
   )
   (wire (pts (xy 89.535 123.825) (xy 86.995 123.825))
-    (stroke (width 0) (type default) (color 0 0 0 0))
-  )
-  (wire (pts (xy 194.31 37.465) (xy 197.485 37.465))
     (stroke (width 0) (type default) (color 0 0 0 0))
   )
@@
     (effects (font (size 1.27 1.27)) (justify left bottom))
   )
-  (label "LORA_TX" (at 207.01 29.845 180)
-    (effects (font (size 1.27 1.27)) (justify right bottom))
-  )
-  (label "LORA_RX" (at 207.01 27.305 180)
-    (effects (font (size 1.27 1.27)) (justify right bottom))
-  )
   (label "LORA_BOOT0" (at 257.81 33.02 0)
     (effects (font (size 1.27 1.27)) (justify left bottom))
   )
-  (label "LORA_BOOT0" (at 207.01 34.925 180)
-    (effects (font (size 1.27 1.27)) (justify right bottom))
-  )
-  (label "LORA_BOOT0" (at 125.095 85.725 0)
-    (effects (font (size 1.27 1.27)) (justify left bottom))
-  )
   (label "LORA_NRST" (at 236.855 33.02 0)
-    (effects (font (size 1.27 1.27)) (justify left bottom))
-  )
-  (label "LORA_NRST" (at 207.01 32.385 180)
-    (effects (font (size 1.27 1.27)) (justify right bottom))
-  )
-  (label "LORA_NRST" (at 125.095 82.55 0)
     (effects (font (size 1.27 1.27)) (justify left bottom))
   )
@@
     (pin "2")
   )
-  (symbol (lib_id "Devtank:+3V3_CORE") (at 197.485 20.955 0) (unit 1)
-    (in_bom yes) (on_board yes) (fields_autoplaced)
-    (property "Reference" "#PWR091" (id 0) (at 197.485 24.765 0)
-      (effects (font (size 1.27 1.27)) hide)
-    )
-    (property "Value" "+3V3_CORE" (id 1) (at 197.485 17.3792 0))
-    (property "Footprint" "" (id 2) (at 197.485 20.955 0))
-    (property "Datasheet" "" (id 3) (at 197.485 20.955 0))
-    (pin "1")
-  )
   (symbol (lib_id "Devtank:+3V3_CORE") (at 43.815 52.705 0) (unit 1)
     (in_bom yes) (on_board yes) (fields_autoplaced)
@@
     (pin "1")
   )
-  (symbol (lib_id "power:GND") (at 197.485 41.275 0) (mirror y) (unit 1)
-    (in_bom yes) (on_board yes)
-    (property "Reference" "#PWR098" (id 0) (at 197.485 47.625 0)
-      (effects (font (size 1.27 1.27)) hide)
-    )
-    (property "Value" "GND" (id 1) (at 197.358 45.6692 0))
-    (property "Footprint" "" (id 2) (at 197.485 41.275 0)
-      (effects (font (size 1.524 1.524)))
-    )
-    (property "Datasheet" "" (id 3) (at 197.485 41.275 0)
-      (effects (font (size 1.524 1.524)))
-    )
-    (pin "1")
-  )
-  (symbol (lib_id "Connector_Generic:Conn_01x06") (at 189.23 29.845 0) (mirror y) (unit 1)
-    (in_bom yes) (on_board yes)
-    (property "Reference" "J9" (id 0) (at 184.785 19.685 0))
-    (property "Value" "" (id 1) (at 189.23 22.3321 0))
-    (property "Footprint" "" (id 2) (at 189.23 29.845 0)
-      (effects (font (size 1.27 1.27)) hide)
-    )
-    (property "Datasheet" "~" (id 3) (at 189.23 29.845 0)
-      (effects (font (size 1.27 1.27)) hide)
-    )
-    (pin "1")
-    (pin "2")
-    (pin "3")
-    (pin "4")
-    (pin "5")
-    (pin "6")
-  )
   (symbol (lib_id "Devtank:+3V3_CORE") (at 270.51 21.59 0) (unit 1)
