File: kicad_osm_env01/ADC_Filtering.kicad_sch (KiCad schematic)
At the start: 14 parts

Commit message: Schematics waiting review
Parts:
- added C45: 100nF, symbol Device:C
- added R136: 100R, symbol Device:R
- C90: value 1M -> 100nF
- R111: value DNF -> 100R
Connections:
- net ADC2_IN: now also R107.1; no longer R106.1
- net ADC2_OUT: now also C86.1, R107.2; no longer C66.1, R106.2
- net ADC3_IN: now also R108.1; no longer R110.1
- net ADC3_OUT: now also C87.1, R108.2; no longer C89.1, R110.2
- net ADC4_IN: now also R109.1; no longer R107.1
- net ADC4_OUT: now also C88.1, R109.2; no longer C86.1, R107.2
- net ADC5_IN: now also R110.1; no longer R111.1
- net ADC5_OUT: now also C89.1, R110.2; no longer C90.1, R111.2
- net ADC6_IN: now also R111.1; no longer R108.1
- net ADC6_OUT: now also C90.1, R111.2; no longer C87.1, R108.2
- net ADC8_IN: now also R136.1; no longer R109.1
- net ADC8_OUT: now also C45.1, R136.2; no longer C88.1, R109.2
- net GND: now also C45.2
- new net ADC1_IN: R106.1
- new net ADC1_OUT: C66.1, R106.2
Other:
- note removed: "ADC5 Unsused"
Changed lines of the file:
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@@
   (junction (at 78.74 43.18) (diameter 0) (color 0 0 0 0)
   )
+  (junction (at 139.065 81.28) (diameter 0) (color 0 0 0 0)
+  )
   (junction (at 78.74 81.28) (diameter 0) (color 0 0 0 0)
   )
@@
     (stroke (width 0) (type default) (color 0 0 0 0))
   )
+  (wire (pts (xy 139.065 91.44) (xy 139.065 88.9))
+    (stroke (width 0) (type default) (color 0 0 0 0))
+  )
   (wire (pts (xy 78.74 62.23) (xy 85.725 62.23))
     (stroke (width 0) (type default) (color 0 0 0 0))
   )
+  (wire (pts (xy 139.065 81.28) (xy 146.05 81.28))
+    (stroke (width 0) (type default) (color 0 0 0 0))
+  )
   (wire (pts (xy 78.74 53.34) (xy 78.74 50.8))
     (stroke (width 0) (type default) (color 0 0 0 0))
@@
     (stroke (width 0) (type default) (color 0 0 0 0))
   )
+  (wire (pts (xy 119.38 81.28) (xy 126.365 81.28))
+    (stroke (width 0) (type default) (color 0 0 0 0))
+  )
   (wire (pts (xy 133.985 24.765) (xy 139.065 24.765))
     (stroke (width 0) (type default) (color 0 0 0 0))
@@
     (stroke (width 0) (type default) (color 0 0 0 0))
   )
+  (wire (pts (xy 133.985 81.28) (xy 139.065 81.28))
+    (stroke (width 0) (type default) (color 0 0 0 0))
+  )
   (wire (pts (xy 78.74 43.18) (xy 85.725 43.18))
     (stroke (width 0) (type default) (color 0 0 0 0))
@@
     (stroke (width 0) (type default) (color 0 0 0 0))
   )
-  (text "ADC5 Unsused" (at 163.195 51.435 0)
-    (effects (font (size 1.27 1.27)) (justify left bottom))
-  )
-  (hierarchical_label "ADC2_IN" (shape input) (at 59.055 24.765 180)
-    (effects (font (size 1.27 1.27)) (justify right))
-  )
-  (hierarchical_label "ADC2_OUT" (shape output) (at 85.725 24.765 0)
-    (effects (font (size 1.27 1.27)) (justify left))
-  )
-  (hierarchical_label "ADC8_IN" (shape input) (at 59.055 81.28 180)
-    (effects (font (size 1.27 1.27)) (justify right))
-  )
-  (hierarchical_label "ADC5_OUT" (shape output) (at 146.05 43.18 0)
+  (hierarchical_label "ADC8_OUT" (shape output) (at 146.05 81.28 0)
+    (effects (font (size 1.27 1.27)) (justify left))
+  )
+  (hierarchical_label "ADC1_IN" (shape input) (at 59.055 24.765 180)
+    (effects (font (size 1.27 1.27)) (justify right))
+  )
+  (hierarchical_label "ADC1_OUT" (shape output) (at 85.725 24.765 0)
+    (effects (font (size 1.27 1.27)) (justify left))
+  )
+  (hierarchical_label "ADC4_IN" (shape input) (at 59.055 81.28 180)
+    (effects (font (size 1.27 1.27)) (justify right))
+  )
+  (hierarchical_label "ADC6_OUT" (shape output) (at 146.05 43.18 0)
     (effects (font (size 1.27 1.27)) (justify left))
   )
@@
     (effects (font (size 1.27 1.27)) (justify right))
   )
-  (hierarchical_label "ADC4_OUT" (shape output) (at 85.725 43.18 0)
-    (effects (font (size 1.27 1.27)) (justify left))
-  )
-  (hierarchical_label "ADC6_OUT" (shape output) (at 85.725 62.23 0)
-    (effects (font (size 1.27 1.27)) (justify left))
-  )
-  (hierarchical_label "ADC6_IN" (shape input) (at 59.055 62.23 180)
+  (hierarchical_label "ADC2_OUT" (shape output) (at 85.725 43.18 0)
+    (effects (font (size 1.27 1.27)) (justify left))
+  )
+  (hierarchical_label "ADC3_OUT" (shape output) (at 85.725 62.23 0)
+    (effects (font (size 1.27 1.27)) (justify left))
+  )
+  (hierarchical_label "ADC8_IN" (shape input) (at 119.38 81.28 180)
+    (effects (font (size 1.27 1.27)) (justify right))
+  )
+  (hierarchical_label "ADC3_IN" (shape input) (at 59.055 62.23 180)
     (effects (font (size 1.27 1.27)) (justify right))
   )
@@
     (effects (font (size 1.27 1.27)) (justify left))
   )
-  (hierarchical_label "ADC3_IN" (shape input) (at 119.38 24.765 180)
-    (effects (font (size 1.27 1.27)) (justify right))
-  )
-  (hierarchical_label "ADC4_IN" (shape input) (at 59.055 43.18 180)
-    (effects (font (size 1.27 1.27)) (justify right))
-  )
-  (hierarchical_label "ADC3_OUT" (shape output) (at 146.05 24.765 0)
-    (effects (font (size 1.27 1.27)) (justify left))
-  )
-  (hierarchical_label "ADC8_OUT" (shape output) (at 85.725 81.28 0)
-    (effects (font (size 1.27 1.27)) (justify left))
-  )
-  (hierarchical_label "ADC5_IN" (shape input) (at 119.38 43.18 180)
+  (hierarchical_label "ADC5_IN" (shape input) (at 119.38 24.765 180)
+    (effects (font (size 1.27 1.27)) (justify right))
+  )
+  (hierarchical_label "ADC2_IN" (shape input) (at 59.055 43.18 180)
+    (effects (font (size 1.27 1.27)) (justify right))
+  )
+  (hierarchical_label "ADC5_OUT" (shape output) (at 146.05 24.765 0)
+    (effects (font (size 1.27 1.27)) (justify left))
+  )
+  (hierarchical_label "ADC4_OUT" (shape output) (at 85.725 81.28 0)
+    (effects (font (size 1.27 1.27)) (justify left))
+  )
+  (hierarchical_label "ADC6_IN" (shape input) (at 119.38 43.18 180)
     (effects (font (size 1.27 1.27)) (justify right))
   )
@@
     (pin "1")
   )
+  (symbol (lib_id "Device:R") (at 130.175 81.28 90) (unit 1)
+    (in_bom yes) (on_board yes) (fields_autoplaced)
+    (property "Reference" "R136" (id 0) (at 130.175 76.5642 90))
+    (property "Value" "100R" (id 1) (at 130.175 79.1011 90))
+    (property "Footprint" "" (id 2) (at 130.175 83.058 90)
+      (effects (font (size 1.27 1.27)) hide)
+    )
+    (property "Datasheet" "~" (id 3) (at 130.175 81.28 0)
+      (effects (font (size 1.27 1.27)) hide)
+    )
+    (pin "1")
+    (pin "2")
+  )
   (symbol (lib_id "Device:R") (at 130.175 24.765 90) (unit 1)
     (in_bom yes) (on_board yes) (fields_autoplaced)
@@
     (pin "1")
   )
+  (symbol (lib_id "Device:C") (at 139.065 85.09 0) (unit 1)
+    (in_bom yes) (on_board yes) (fields_autoplaced)
+    (property "Reference" "C45" (id 0) (at 141.986 84.2553 0)
+      (effects (font (size 1.27 1.27)) (justify left))
+    )
+    (property "Value" "100nF" (id 1) (at 141.986 86.7922 0)
+      (effects (font (size 1.27 1.27)) (justify left))
+    )
+    (property "Footprint" "" (id 2) (at 140.0302 88.9 0)
+      (effects (font (size 1.27 1.27)) hide)
+    )
+    (property "Datasheet" "~" (id 3) (at 139.065 85.09 0)
+      (effects (font (size 1.27 1.27)) hide)
+    )
+    (pin "1")
+    (pin "2")
+  )
+  (symbol (lib_id "OSM_env01:GND") (at 139.065 91.44 0) (unit 1)
+    (in_bom yes) (on_board yes) (fields_autoplaced)
+    (property "Reference" "#PWR095" (id 0) (at 139.065 97.79 0)
+      (effects (font (size 1.27 1.27)) hide)
+    )
+    (property "Value" "~" (id 1) (at 139.065 95.8834 0))
+    (property "Footprint" "" (id 2) (at 139.065 91.44 0)
+      (effects (font (size 1.524 1.524)))
+    )
+    (property "Datasheet" "" (id 3) (at 139.065 91.44 0)
+      (effects (font (size 1.524 1.524)))
+    )
+    (pin "1")
+  )
   (symbol (lib_id "Device:C") (at 139.065 46.99 0) (unit 1)
     (in_bom yes) (on_board yes) (fields_autoplaced)
@@
       (effects (font (size 1.27 1.27)) (justify left))
     )
-    (property "Value" "1M" (id 1) (at 141.986 48.6922 0)
+    (property "Value" "100nF" (id 1) (at 141.986 48.6922 0)
       (effects (font (size 1.27 1.27)) (justify left))
     )
@@
     (in_bom yes) (on_board yes) (fields_autoplaced)
     (property "Reference" "R111" (id 0) (at 130.175 38.4642 90))
-    (property "Value" "DNF" (id 1) (at 130.175 41.0011 90))
+    (property "Value" "100R" (id 1) (at 130.175 41.0011 90))
     (property "Footprint" "" (id 2) (at 130.175 44.958 90)
       (effects (font (size 1.27 1.27)) hide)

Commit message: started layout with throwdown
Parts:
- C45, C66, C86, C87, C88, C89, C90, C91: value 100nF -> (none)
- R106, R107, R108, R109, R110, R111, R136, R142: value 100R -> (none)
Changed lines of the file:
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@@
     (in_bom yes) (on_board yes) (fields_autoplaced)
     (property "Reference" "R106" (id 0) (at 69.85 20.0492 90))
-    (property "Value" "100R" (id 1) (at 69.85 22.5861 90))
+    (property "Value" "" (id 1) (at 69.85 22.5861 90))
     (property "Footprint" "" (id 2) (at 69.85 26.543 90)
       (effects (font (size 1.27 1.27)) hide)
@@
       (effects (font (size 1.27 1.27)) (justify left))
     )
-    (property "Value" "100nF" (id 1) (at 81.661 48.6922 0)
+    (property "Value" "" (id 1) (at 81.661 48.6922 0)
       (effects (font (size 1.27 1.27)) (justify left))
     )
@@
     (in_bom yes) (on_board yes) (fields_autoplaced)
     (property "Reference" "R136" (id 0) (at 130.175 76.5642 90))
-    (property "Value" "100R" (id 1) (at 130.175 79.1011 90))
+    (property "Value" "" (id 1) (at 130.175 79.1011 90))
     (property "Footprint" "" (id 2) (at 130.175 83.058 90)
       (effects (font (size 1.27 1.27)) hide)
@@
     (in_bom yes) (on_board yes) (fields_autoplaced)
     (property "Reference" "R110" (id 0) (at 130.175 20.0492 90))
-    (property "Value" "100R" (id 1) (at 130.175 22.5861 90))
+    (property "Value" "" (id 1) (at 130.175 22.5861 90))
     (property "Footprint" "" (id 2) (at 130.175 26.543 90)
       (effects (font (size 1.27 1.27)) hide)
@@
     (in_bom yes) (on_board yes) (fields_autoplaced)
     (property "Reference" "R108" (id 0) (at 69.85 57.5142 90))
-    (property "Value" "100R" (id 1) (at 69.85 60.0511 90))
+    (property "Value" "" (id 1) (at 69.85 60.0511 90))
     (property "Footprint" "" (id 2) (at 69.85 64.008 90)
       (effects (font (size 1.27 1.27)) hide)
@@
       (effects (font (size 1.27 1.27)) (justify left))
     )
-    (property "Value" "100nF" (id 1) (at 141.986 86.7922 0)
+    (property "Value" "" (id 1) (at 141.986 86.7922 0)
       (effects (font (size 1.27 1.27)) (justify left))
     )
@@
       (effects (font (size 1.27 1.27)) (justify left))
     )
-    (property "Value" "100nF" (id 1) (at 141.986 48.6922 0)
+    (property "Value" "" (id 1) (at 141.986 48.6922 0)
       (effects (font (size 1.27 1.27)) (justify left))
     )
@@
     (in_bom yes) (on_board yes) (fields_autoplaced)
     (property "Reference" "R109" (id 0) (at 69.85 76.5642 90))
-    (property "Value" "100R" (id 1) (at 69.85 79.1011 90))
+    (property "Value" "" (id 1) (at 69.85 79.1011 90))
     (property "Footprint" "" (id 2) (at 69.85 83.058 90)
       (effects (font (size 1.27 1.27)) hide)
@@
       (effects (font (size 1.27 1.27)) (justify left))
     )
-    (property "Value" "100nF" (id 1) (at 81.661 30.2772 0)
+    (property "Value" "" (id 1) (at 81.661 30.2772 0)
       (effects (font (size 1.27 1.27)) (justify left))
     )
@@
       (effects (font (size 1.27 1.27)) (justify left))
     )
-    (property "Value" "100nF" (id 1) (at 81.661 67.7422 0)
+    (property "Value" "" (id 1) (at 81.661 67.7422 0)
       (effects (font (size 1.27 1.27)) (justify left))
     )
@@
       (effects (font (size 1.27 1.27)) (justify left))
     )
-    (property "Value" "100nF" (id 1) (at 81.661 86.7922 0)
+    (property "Value" "" (id 1) (at 81.661 86.7922 0)
       (effects (font (size 1.27 1.27)) (justify left))
     )
@@
     (in_bom yes) (on_board yes) (fields_autoplaced)
     (property "Reference" "R111" (id 0) (at 130.175 38.4642 90))
-    (property "Value" "100R" (id 1) (at 130.175 41.0011 90))
+    (property "Value" "" (id 1) (at 130.175 41.0011 90))
     (property "Footprint" "" (id 2) (at 130.175 44.958 90)
       (effects (font (size 1.27 1.27)) hide)
@@
       (effects (font (size 1.27 1.27)) (justify left))
     )
-    (property "Value" "100nF" (id 1) (at 141.986 67.7422 0)
+    (property "Value" "" (id 1) (at 141.986 67.7422 0)
       (effects (font (size 1.27 1.27)) (justify left))
     )
@@
     (in_bom yes) (on_board yes) (fields_autoplaced)
     (property "Reference" "R142" (id 0) (at 130.175 57.5142 90))
-    (property "Value" "100R" (id 1) (at 130.175 60.0511 90))
+    (property "Value" "" (id 1) (at 130.175 60.0511 90))
     (property "Footprint" "" (id 2) (at 130.175 64.008 90)
       (effects (font (size 1.27 1.27)) hide)
@@
       (effects (font (size 1.27 1.27)) (justify left))
     )
-    (property "Value" "100nF" (id 1) (at 141.986 30.2772 0)
+    (property "Value" "" (id 1) (at 141.986 30.2772 0)
       (effects (font (size 1.27 1.27)) (justify left))
     )
@@
     (in_bom yes) (on_board yes) (fields_autoplaced)
     (property "Reference" "R107" (id 0) (at 69.85 38.4642 90))
-    (property "Value" "100R" (id 1) (at 69.85 41.0011 90))
+    (property "Value" "" (id 1) (at 69.85 41.0011 90))
     (property "Footprint" "" (id 2) (at 69.85 44.958 90)
       (effects (font (size 1.27 1.27)) hide)

Commit message: majority of signals routed on layout
Parts:
- C45, C66, C86, C87, C88, C89, C90, C91: value (none) -> 100nF; footprint (none) -> Capacitor_SMD:C_0402_1005Metric
- R106, R107, R108, R109, R110, R111, R136, R142: value (none) -> 100R; footprint (none) -> Resistor_SMD:R_0603_1608Metric
Changed lines of the file:
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@@
     (in_bom yes) (on_board yes) (fields_autoplaced)
     (property "Reference" "R106" (id 0) (at 69.85 20.0492 90))
-    (property "Value" "" (id 1) (at 69.85 22.5861 90))
-    (property "Footprint" "" (id 2) (at 69.85 26.543 90)
+    (property "Value" "100R" (id 1) (at 69.85 22.5861 90))
+    (property "Footprint" "Resistor_SMD:R_0603_1608Metric" (id 2) (at 69.85 26.543 90)
       (effects (font (size 1.27 1.27)) hide)
     )
@@
       (effects (font (size 1.27 1.27)) (justify left))
     )
-    (property "Value" "" (id 1) (at 81.661 48.6922 0)
-      (effects (font (size 1.27 1.27)) (justify left))
-    )
-    (property "Footprint" "" (id 2) (at 79.7052 50.8 0)
+    (property "Value" "100nF" (id 1) (at 81.661 48.6922 0)
+      (effects (font (size 1.27 1.27)) (justify left))
+    )
+    (property "Footprint" "Capacitor_SMD:C_0402_1005Metric" (id 2) (at 79.7052 50.8 0)
       (effects (font (size 1.27 1.27)) hide)
     )
@@
     (in_bom yes) (on_board yes) (fields_autoplaced)
     (property "Reference" "R136" (id 0) (at 130.175 76.5642 90))
-    (property "Value" "" (id 1) (at 130.175 79.1011 90))
-    (property "Footprint" "" (id 2) (at 130.175 83.058 90)
+    (property "Value" "100R" (id 1) (at 130.175 79.1011 90))
+    (property "Footprint" "Resistor_SMD:R_0603_1608Metric" (id 2) (at 130.175 83.058 90)
       (effects (font (size 1.27 1.27)) hide)
     )
@@
     (in_bom yes) (on_board yes) (fields_autoplaced)
     (property "Reference" "R110" (id 0) (at 130.175 20.0492 90))
-    (property "Value" "" (id 1) (at 130.175 22.5861 90))
-    (property "Footprint" "" (id 2) (at 130.175 26.543 90)
+    (property "Value" "100R" (id 1) (at 130.175 22.5861 90))
+    (property "Footprint" "Resistor_SMD:R_0603_1608Metric" (id 2) (at 130.175 26.543 90)
       (effects (font (size 1.27 1.27)) hide)
     )
@@
     (in_bom yes) (on_board yes) (fields_autoplaced)
     (property "Reference" "R108" (id 0) (at 69.85 57.5142 90))
-    (property "Value" "" (id 1) (at 69.85 60.0511 90))
-    (property "Footprint" "" (id 2) (at 69.85 64.008 90)
+    (property "Value" "100R" (id 1) (at 69.85 60.0511 90))
+    (property "Footprint" "Resistor_SMD:R_0603_1608Metric" (id 2) (at 69.85 64.008 90)
       (effects (font (size 1.27 1.27)) hide)
     )
@@
       (effects (font (size 1.27 1.27)) (justify left))
     )
-    (property "Value" "" (id 1) (at 141.986 86.7922 0)
-      (effects (font (size 1.27 1.27)) (justify left))
-    )
-    (property "Footprint" "" (id 2) (at 140.0302 88.9 0)
+    (property "Value" "100nF" (id 1) (at 141.986 86.7922 0)
+      (effects (font (size 1.27 1.27)) (justify left))
+    )
+    (property "Footprint" "Capacitor_SMD:C_0402_1005Metric" (id 2) (at 140.0302 88.9 0)
       (effects (font (size 1.27 1.27)) hide)
     )
@@
       (effects (font (size 1.27 1.27)) (justify left))
     )
-    (property "Value" "" (id 1) (at 141.986 48.6922 0)
-      (effects (font (size 1.27 1.27)) (justify left))
-    )
-    (property "Footprint" "" (id 2) (at 140.0302 50.8 0)
+    (property "Value" "100nF" (id 1) (at 141.986 48.6922 0)
+      (effects (font (size 1.27 1.27)) (justify left))
+    )
+    (property "Footprint" "Capacitor_SMD:C_0402_1005Metric" (id 2) (at 140.0302 50.8 0)
       (effects (font (size 1.27 1.27)) hide)
     )
@@
     (in_bom yes) (on_board yes) (fields_autoplaced)
     (property "Reference" "R109" (id 0) (at 69.85 76.5642 90))
-    (property "Value" "" (id 1) (at 69.85 79.1011 90))
-    (property "Footprint" "" (id 2) (at 69.85 83.058 90)
+    (property "Value" "100R" (id 1) (at 69.85 79.1011 90))
+    (property "Footprint" "Resistor_SMD:R_0603_1608Metric" (id 2) (at 69.85 83.058 90)
       (effects (font (size 1.27 1.27)) hide)
     )
@@
       (effects (font (size 1.27 1.27)) (justify left))
     )
-    (property "Value" "" (id 1) (at 81.661 30.2772 0)
-      (effects (font (size 1.27 1.27)) (justify left))
-    )
-    (property "Footprint" "" (id 2) (at 79.7052 32.385 0)
+    (property "Value" "100nF" (id 1) (at 81.661 30.2772 0)
+      (effects (font (size 1.27 1.27)) (justify left))
+    )
+    (property "Footprint" "Capacitor_SMD:C_0402_1005Metric" (id 2) (at 79.7052 32.385 0)
       (effects (font (size 1.27 1.27)) hide)
     )
@@
       (effects (font (size 1.27 1.27)) (justify left))
     )
-    (property "Value" "" (id 1) (at 81.661 67.7422 0)
-      (effects (font (size 1.27 1.27)) (justify left))
-    )
-    (property "Footprint" "" (id 2) (at 79.7052 69.85 0)
+    (property "Value" "100nF" (id 1) (at 81.661 67.7422 0)
+      (effects (font (size 1.27 1.27)) (justify left))
+    )
+    (property "Footprint" "Capacitor_SMD:C_0402_1005Metric" (id 2) (at 79.7052 69.85 0)
       (effects (font (size 1.27 1.27)) hide)
     )
@@
       (effects (font (size 1.27 1.27)) (justify left))
     )
-    (property "Value" "" (id 1) (at 81.661 86.7922 0)
-      (effects (font (size 1.27 1.27)) (justify left))
-    )
-    (property "Footprint" "" (id 2) (at 79.7052 88.9 0)
+    (property "Value" "100nF" (id 1) (at 81.661 86.7922 0)
+      (effects (font (size 1.27 1.27)) (justify left))
+    )
+    (property "Footprint" "Capacitor_SMD:C_0402_1005Metric" (id 2) (at 79.7052 88.9 0)
       (effects (font (size 1.27 1.27)) hide)
     )
@@
     (in_bom yes) (on_board yes) (fields_autoplaced)
     (property "Reference" "R111" (id 0) (at 130.175 38.4642 90))
-    (property "Value" "" (id 1) (at 130.175 41.0011 90))
-    (property "Footprint" "" (id 2) (at 130.175 44.958 90)
+    (property "Value" "100R" (id 1) (at 130.175 41.0011 90))
+    (property "Footprint" "Resistor_SMD:R_0603_1608Metric" (id 2) (at 130.175 44.958 90)
       (effects (font (size 1.27 1.27)) hide)
     )
@@
       (effects (font (size 1.27 1.27)) (justify left))
     )
-    (property "Value" "" (id 1) (at 141.986 67.7422 0)
-      (effects (font (size 1.27 1.27)) (justify left))
-    )
-    (property "Footprint" "" (id 2) (at 140.0302 69.85 0)
+    (property "Value" "100nF" (id 1) (at 141.986 67.7422 0)
+      (effects (font (size 1.27 1.27)) (justify left))
+    )
+    (property "Footprint" "Capacitor_SMD:C_0402_1005Metric" (id 2) (at 140.0302 69.85 0)
       (effects (font (size 1.27 1.27)) hide)
     )
@@
     (in_bom yes) (on_board yes) (fields_autoplaced)
     (property "Reference" "R142" (id 0) (at 130.175 57.5142 90))
-    (property "Value" "" (id 1) (at 130.175 60.0511 90))
-    (property "Footprint" "" (id 2) (at 130.175 64.008 90)
+    (property "Value" "100R" (id 1) (at 130.175 60.0511 90))
+    (property "Footprint" "Resistor_SMD:R_0603_1608Metric" (id 2) (at 130.175 64.008 90)
       (effects (font (size 1.27 1.27)) hide)
     )
@@
       (effects (font (size 1.27 1.27)) (justify left))
     )
-    (property "Value" "" (id 1) (at 141.986 30.2772 0)
-      (effects (font (size 1.27 1.27)) (justify left))
-    )
-    (property "Footprint" "" (id 2) (at 140.0302 32.385 0)
+    (property "Value" "100nF" (id 1) (at 141.986 30.2772 0)
+      (effects (font (size 1.27 1.27)) (justify left))
+    )
+    (property "Footprint" "Capacitor_SMD:C_0402_1005Metric" (id 2) (at 140.0302 32.385 0)
       (effects (font (size 1.27 1.27)) hide)
     )
@@
     (in_bom yes) (on_board yes) (fields_autoplaced)
     (property "Reference" "R107" (id 0) (at 69.85 38.4642 90))
-    (property "Value" "" (id 1) (at 69.85 41.0011 90))
-    (property "Footprint" "" (id 2) (at 69.85 44.958 90)
-      (effects (font (size 1.27 1.27)) hide)
-    )
+    (property "Value" "100R" (id 1) (at 69.85 41.0011 90))
+    (property "Footprint" "Resistor_SMD:R_0603_1608Metric" (id 2) (at 69.85 44.958 90)
+      (effects (font (size 1.27 1.27)) hide)
+    )
