File: kicad_osm_env01/RS232_comms.kicad_sch (KiCad schematic)
At the start: 11 parts, among them U23 MAX3232

Commit message: added information to symbol entries table, added jumper settings table, minor single track update on layout
Parts:
- C24, C26, C27, C43, C96: Characteristics (none) -> X5R; Other (none) -> Can use own part, but needs to meet the specs
- L8: Manufacturer (none) -> TDK; Manufacturer Part Number (none) -> MPZ1005S121HT000; Other (none) -> Can use own part, but needs to meet the specs
- R117, R127, R17, R21: Tolerance (none) -> 1%
Changed lines of the file:
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@@
+      (effects (font (size 1.27 1.27)) hide)
+    )
+    (property "Manufacturer" "TDK" (at 123.19 56.515 0)
+      (effects (font (size 1.27 1.27)) hide)
+    )
+    (property "Manufacturer Part Number" "MPZ1005S121HT000 " (at 123.19 56.515 0)
+      (effects (font (size 1.27 1.27)) hide)
+    )
+    (property "Power Rating" "" (at 123.19 56.515 0)
+      (effects (font (size 1.27 1.27)) hide)
+    )
+    (property "Current Rating" "" (at 123.19 56.515 0)
+      (effects (font (size 1.27 1.27)) hide)
+    )
+    (property "Other" "Can use own part, but needs to meet the specs" (at 123.19 56.515 0)
       (effects (font (size 1.27 1.27)) hide)
     )
@@
     )
     (property "Datasheet" "" (at 106.68 52.07 0)
+      (effects (font (size 1.27 1.27)) hide)
+    )
+    (property "Tolerance" "1%" (at 106.68 52.07 0)
+      (effects (font (size 1.27 1.27)) hide)
+    )
+    (property "Power Rating" "" (at 106.68 52.07 0)
+      (effects (font (size 1.27 1.27)) hide)
+    )
+    (property "Current Rating" "" (at 106.68 52.07 0)
       (effects (font (size 1.27 1.27)) hide)
     )
@@
     )
     (property "Voltage" "50V" (at 135.89 60.325 0)
+      (effects (font (size 1.27 1.27)) hide)
+    )
+    (property "Power Rating" "" (at 135.89 60.325 0)
+      (effects (font (size 1.27 1.27)) hide)
+    )
+    (property "Characteristics" "X5R" (at 135.89 60.325 0)
+      (effects (font (size 1.27 1.27)) hide)
+    )
+    (property "Current Rating" "" (at 135.89 60.325 0)
+      (effects (font (size 1.27 1.27)) hide)
+    )
+    (property "Other" "Can use own part, but needs to meet the specs" (at 135.89 60.325 0)
       (effects (font (size 1.27 1.27)) hide)
     )
@@
       (effects (font (size 1.27 1.27)) hide)
     )
-    (property "Characteristics" "" (at 177.165 81.915 0)
+    (property "Characteristics" "X5R" (at 177.165 81.915 0)
+      (effects (font (size 1.27 1.27)) hide)
+    )
+    (property "Power Rating" "" (at 177.165 81.915 0)
+      (effects (font (size 1.27 1.27)) hide)
+    )
+    (property "Current Rating" "" (at 177.165 81.915 0)
+      (effects (font (size 1.27 1.27)) hide)
+    )
+    (property "Other" "Can use own part, but needs to meet the specs" (at 177.165 81.915 0)
       (effects (font (size 1.27 1.27)) hide)
     )
@@
       (effects (font (size 1.27 1.27)) hide)
     )
+    (property "Tolerance" "1%" (at 106.68 56.515 0)
+      (effects (font (size 1.27 1.27)) hide)
+    )
+    (property "Power Rating" "" (at 106.68 56.515 0)
+      (effects (font (size 1.27 1.27)) hide)
+    )
+    (property "Current Rating" "" (at 106.68 56.515 0)
+      (effects (font (size 1.27 1.27)) hide)
+    )
     (pin "1")
     (pin "2")
@@
       (effects (font (size 1.27 1.27)) hide)
     )
-    (property "Characteristics" "" (at 180.975 98.425 0)
+    (property "Characteristics" "X5R" (at 180.975 98.425 0)
+      (effects (font (size 1.27 1.27)) hide)
+    )
+    (property "Power Rating" "" (at 180.975 98.425 0)
+      (effects (font (size 1.27 1.27)) hide)
+    )
+    (property "Current Rating" "" (at 180.975 98.425 0)
+      (effects (font (size 1.27 1.27)) hide)
+    )
+    (property "Other" "Can use own part, but needs to meet the specs" (at 180.975 98.425 0)
       (effects (font (size 1.27 1.27)) hide)
     )
@@
       (effects (font (size 1.27 1.27)) hide)
     )
-    (property "Characteristics" "" (at 180.975 90.805 0)
+    (property "Characteristics" "X5R" (at 180.975 90.805 0)
+      (effects (font (size 1.27 1.27)) hide)
+    )
+    (property "Power Rating" "" (at 180.975 90.805 0)
+      (effects (font (size 1.27 1.27)) hide)
+    )
+    (property "Current Rating" "" (at 180.975 90.805 0)
+      (effects (font (size 1.27 1.27)) hide)
+    )
+    (property "Other" "Can use own part, but needs to meet the specs" (at 180.975 90.805 0)
       (effects (font (size 1.27 1.27)) hide)
     )
@@
       (effects (font (size 1.27 1.27)) hide)
     )
-    (property "Characteristics" "" (at 122.555 81.915 0)
+    (property "Characteristics" "X5R" (at 122.555 81.915 0)
+      (effects (font (size 1.27 1.27)) hide)
+    )
+    (property "Power Rating" "" (at 122.555 81.915 0)
+      (effects (font (size 1.27 1.27)) hide)
+    )
+    (property "Current Rating" "" (at 122.555 81.915 0)
+      (effects (font (size 1.27 1.27)) hide)
+    )
+    (property "Other" "Can use own part, but needs to meet the specs" (at 122.555 81.915 0)
       (effects (font (size 1.27 1.27)) hide)
     )
@@
     )
     (property "Manufacturer Part Number" "MAX3232IPWR" (at 149.225 100.965 0)
+      (effects (font (size 1.27 1.27)) hide)
+    )
+    (property "Power Rating" "" (at 149.225 100.965 0)
+      (effects (font (size 1.27 1.27)) hide)
+    )
+    (property "Current Rating" "" (at 149.225 100.965 0)
       (effects (font (size 1.27 1.27)) hide)
     )
@@
       (effects (font (size 1.27 1.27)) hide)
     )
+    (property "Tolerance" "1%" (at 113.03 95.885 0)
+      (effects (font (size 1.27 1.27)) hide)
+    )
+    (property "Power Rating" "" (at 113.03 95.885 0)
+      (effects (font (size 1.27 1.27)) hide)
+    )
+    (property "Current Rating" "" (at 113.03 95.885 0)
+      (effects (font (size 1.27 1.27)) hide)
+    )
     (pin "1")
     (pin "2")
@@
       (effects (font (size 1.27 1.27)) hide)
     )
+    (property "Tolerance" "1%" (at 106.045 95.885 0)
+      (effects (font (size 1.27 1.27)) hide)
+    )
+    (property "Power Rating" "" (at 106.045 95.885 0)
+      (effects (font (size 1.27 1.27)) hide)
+    )
+    (property "Current Rating" "" (at 106.045 95.885 0)
+      (effects (font (size 1.27 1.27)) hide)
+    )
