File: kicad_osm_env01/RS232_comms.kicad_sch (KiCad schematic)
At the start: 11 parts, among them U23 MAX3232

Commit message: removed 0R links and DNF parts on schematics
Parts:
- removed R117: 0R, Resistor_SMD:R_0402_1005Metric, symbol Device:R
- removed R127: DNF, Resistor_SMD:R_0402_1005Metric, symbol Device:R
Connections:
- net +3V3: now also L8.2
Changed lines of the file:
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@@
     (comment 1 "Part No: 304-010")
   )
-  (junction (at 113.665 56.515) (diameter 0) (color 0 0 0 0)
-  )
   (junction (at 149.225 56.515) (diameter 0) (color 0 0 0 0)
   )
@@
   (junction (at 113.03 108.585) (diameter 0) (color 0 0 0 0)
   )
-  (wire (pts (xy 113.665 52.07) (xy 113.665 56.515))
-    (stroke (width 0) (type default))
-  )
   (wire (pts (xy 149.225 56.515) (xy 135.89 56.515))
     (stroke (width 0) (type default))
@@
     (stroke (width 0) (type default))
   )
-  (wire (pts (xy 102.87 56.515) (xy 92.71 56.515))
+  (wire (pts (xy 109.22 56.515) (xy 119.38 56.515))
     (stroke (width 0) (type default))
   )
@@
     (stroke (width 0) (type default))
   )
-  (wire (pts (xy 113.665 52.07) (xy 110.49 52.07))
-    (stroke (width 0) (type default))
-  )
-  (wire (pts (xy 110.49 56.515) (xy 113.665 56.515))
-    (stroke (width 0) (type default))
-  )
   (wire (pts (xy 189.865 90.805) (xy 195.58 90.805))
     (stroke (width 0) (type default))
@@
     (stroke (width 0) (type default))
   )
-  (wire (pts (xy 92.71 45.72) (xy 92.71 56.515))
+  (wire (pts (xy 109.22 45.72) (xy 109.22 56.515))
     (stroke (width 0) (type default))
   )
@@
     (stroke (width 0) (type default))
   )
-  (wire (pts (xy 102.87 52.07) (xy 99.06 52.07))
-    (stroke (width 0) (type default))
-  )
   (wire (pts (xy 149.225 56.515) (xy 161.29 56.515))
     (stroke (width 0) (type default))
@@
     (stroke (width 0) (type default))
   )
-  (wire (pts (xy 99.06 45.72) (xy 99.06 52.07))
-    (stroke (width 0) (type default))
-  )
   (wire (pts (xy 184.785 98.425) (xy 189.865 98.425))
     (stroke (width 0) (type default))
@@
   )
   (wire (pts (xy 149.225 133.985) (xy 149.225 131.445))
-    (stroke (width 0) (type default))
-  )
-  (wire (pts (xy 119.38 56.515) (xy 113.665 56.515))
     (stroke (width 0) (type default))
   )
@@
         (path "/ab8b0540-9c9f-4195-88f5-7bed0b0a8ed6/b9a077bb-8b65-41fb-9650-f17f6dddad7c"
           (reference "L8") (unit 1)
-        )
-      )
-    )
-  )
-  (symbol (lib_id "Device:R") (at 106.68 52.07 270) (mirror x) (unit 1)
-    (in_bom yes) (on_board yes) (dnp no)
-    (property "Reference" "R117" (at 106.68 47.3542 90)
-      (effects (font (size 1.27 1.27)))
-    )
-    (property "Value" "0R" (at 106.68 49.53 90)
-      (effects (font (size 1.27 1.27)))
-    )
-    (property "Footprint" "Resistor_SMD:R_0402_1005Metric" (at 106.68 53.848 90)
-      (effects (font (size 1.27 1.27)) hide)
-    )
-    (property "Datasheet" "" (at 106.68 52.07 0)
-      (effects (font (size 1.27 1.27)) hide)
-    )
-    (property "Tolerance" "1%" (at 106.68 52.07 0)
-      (effects (font (size 1.27 1.27)) hide)
-    )
-    (property "Power Rating" "" (at 106.68 52.07 0)
-      (effects (font (size 1.27 1.27)) hide)
-    )
-    (property "Current Rating" "" (at 106.68 52.07 0)
-      (effects (font (size 1.27 1.27)) hide)
-    )
-    (pin "1")
-    (pin "2")
-    (instances
-      (project "OSM_env01"
-        (path "/ab8b0540-9c9f-4195-88f5-7bed0b0a8ed6/b9a077bb-8b65-41fb-9650-f17f6dddad7c"
-          (reference "R117") (unit 1)
         )
       )
@@
     )
   )
-  (symbol (lib_id "OSM_env01:+5V") (at 92.71 45.72 0) (mirror y) (unit 1)
-    (in_bom yes) (on_board yes) (dnp no) (fields_autoplaced)
-    (property "Reference" "#PWR062" (at 92.71 49.53 0)
-      (effects (font (size 1.27 1.27)) hide)
-    )
-    (property "Value" "+5V" (at 92.71 42.1442 0)
-      (effects (font (size 1.27 1.27)))
-    )
-    (property "Footprint" "" (at 92.71 45.72 0)
-      (effects (font (size 1.524 1.524)))
-    )
-    (property "Datasheet" "" (at 92.71 45.72 0)
-      (effects (font (size 1.524 1.524)))
-    )
-    (pin "1")
-    (instances
-      (project "OSM_env01"
-        (path "/ab8b0540-9c9f-4195-88f5-7bed0b0a8ed6/b9a077bb-8b65-41fb-9650-f17f6dddad7c"
-          (reference "#PWR062") (unit 1)
-        )
-      )
-    )
-  )
-  (symbol (lib_id "power:+3V3") (at 99.06 45.72 0) (mirror y) (unit 1)
+  (symbol (lib_id "power:+3V3") (at 109.22 45.72 0) (mirror y) (unit 1)
     (in_bom yes) (on_board yes) (dnp no)
-    (property "Reference" "#PWR071" (at 99.06 49.53 0)
-      (effects (font (size 1.27 1.27)) hide)
-    )
-    (property "Value" "+3V3" (at 98.679 41.3258 0)
-      (effects (font (size 1.27 1.27)))
-    )
-    (property "Footprint" "" (at 99.06 45.72 0)
-      (effects (font (size 1.27 1.27)) hide)
-    )
-    (property "Datasheet" "" (at 99.06 45.72 0)
+    (property "Reference" "#PWR071" (at 109.22 49.53 0)
+      (effects (font (size 1.27 1.27)) hide)
+    )
+    (property "Value" "+3V3" (at 108.839 41.3258 0)
+      (effects (font (size 1.27 1.27)))
+    )
+    (property "Footprint" "" (at 109.22 45.72 0)
+      (effects (font (size 1.27 1.27)) hide)
+    )
+    (property "Datasheet" "" (at 109.22 45.72 0)
       (effects (font (size 1.27 1.27)) hide)
     )
@@
         )
       )
-    )
-  )
-  (symbol (lib_id "Device:R") (at 106.68 56.515 270) (mirror x) (unit 1)
-    (in_bom yes) (on_board yes) (dnp no)
-    (property "Reference" "R127" (at 106.68 59.055 90)
-      (effects (font (size 1.27 1.27)))
-    )
-    (property "Value" "DNF" (at 106.68 61.595 90)
-      (effects (font (size 1.27 1.27)))
-    )
-    (property "Footprint" "Resistor_SMD:R_0402_1005Metric" (at 106.68 58.293 90)
-      (effects (font (size 1.27 1.27)) hide)
-    )
-    (property "Datasheet" "" (at 106.68 56.515 0)
-      (effects (font (size 1.27 1.27)) hide)
-    )
-    (property "Tolerance" "1%" (at 106.68 56.515 0)
-      (effects (font (size 1.27 1.27)) hide)
-    )
-    (property "Power Rating" "" (at 106.68 56.515 0)
-      (effects (font (size 1.27 1.27)) hide)
-    )
-    (property "Current Rating" "" (at 106.68 56.515 0)
-      (effects (font (size 1.27 1.27)) hide)
-    )
-    (pin "1")
-    (pin "2")
-    (instances
-      (project "OSM_env01"
-        (path "/ab8b0540-9c9f-4195-88f5-7bed0b0a8ed6/b9a077bb-8b65-41fb-9650-f17f6dddad7c"
-          (reference "R127") (unit 1)
-        )
-      )

Commit message: minor update to layout
Parts:
- R17, R21: Other (none) -> Can use own part, but needs to meet the specs
Changed lines of the file:
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@@
+      (effects (font (size 1.27 1.27)) hide)
+    )
+    (property "Other" "Can use own part, but needs to meet the specs" (at 113.03 95.885 0)
       (effects (font (size 1.27 1.27)) hide)
     )
@@
       (effects (font (size 1.27 1.27)) hide)
     )
+    (property "Other" "Can use own part, but needs to meet the specs" (at 106.045 95.885 0)
+      (effects (font (size 1.27 1.27)) hide)
+    )
