File: kicad_osm_env01/USB_debug.kicad_sch (KiCad schematic)
At the start: 30 parts, among them U13 CP2102N-A02-GQFN24, U15 M74VHC1GT14DFT2G, U21 74AUP1T87GWH, U5 SP3003-02JTG

Commit message: layout updated with a few ic packages due to errors, silk screen tidy up, logos added, minor update to rs232 schematics and pinmap to stm
Parts:
- U15: value M74VHC1GT14DFT2G -> M74VHC1GT14DTT1G; footprint Package_TO_SOT_SMD:SOT-353_SC-70-5 -> Package_TO_SOT_SMD:SOT-23-5
- U21: footprint Devtank_PCB_lib:tssop-5 -> Package_TO_SOT_SMD:SOT-353_SC-70-5
Changed lines of the file:
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@@
       (effects (font (size 1.27 1.27)))
     )
-    (property "Value" "M74VHC1GT14DFT2G" (at 255.27 62.23 0)
-      (effects (font (size 1.27 1.27)))
-    )
-    (property "Footprint" "Package_TO_SOT_SMD:SOT-353_SC-70-5" (at 233.045 57.785 0)
+    (property "Value" "M74VHC1GT14DTT1G" (at 255.27 62.23 0)
+      (effects (font (size 1.27 1.27)))
+    )
+    (property "Footprint" "Package_TO_SOT_SMD:SOT-23-5" (at 233.045 57.785 0)
       (effects (font (size 1.524 1.524)) hide)
     )
@@
       (effects (font (size 1.524 1.524)))
     )
-    (property "Footprint" "Devtank_PCB_lib:tssop-5" (at 206.375 110.49 0)
+    (property "Footprint" "Package_TO_SOT_SMD:SOT-353_SC-70-5" (at 206.375 110.49 0)
       (effects (font (size 1.27 1.27) italic) hide)
     )

Commit message: added information to symbol entries table, added jumper settings table, minor single track update on layout
Parts:
- C16: Characteristics (none) -> X5R; Other (none) -> Can use own part, but needs to meet the specs; Voltage (none) -> 6.3V
- C17, C54, C601, C72: Characteristics (none) -> X5R; Other (none) -> Can use own part, but needs to meet the specs
- L9: Manufacturer (none) -> TDK; Manufacturer Part Number (none) -> MPZ1005S121HT000; Other (none) -> Can use own part, but needs to meet the specs
- R49, R50, R51, R602, R603, R604, R62, R76, R77, R78, R79, R80, R82: Tolerance (none) -> 1%
- U13: value CP2102N-A02-GQFN24 -> CP2102N-A02-GQFN24R; Manufacturer (none) -> Silicon Labs; Manufacturer Part Number (none) -> CP2102N-A02-GQFN24R
- U15: Manufacturer (none) -> ONSEMI; Manufacturer Part Number (none) -> M74VHC1GT14DTT1G
- U21: Manufacturer (none) -> Nexperia; Manufacturer Part Number (none) -> 74AUP1T87GWH
- U5: Manufacturer (none) -> Littelfuse; Manufacturer Part Number (none) -> SP3003-02JTG

Commit message: removed 0R links and DNF parts on schematics
Parts:
- removed R49, R50, R51, R62, R76, R77, R80, R82: 0R, Resistor_SMD:R_0402_1005Metric, symbol Device:R
- removed R78, R79: 330R, Resistor_SMD:R_0603_1608Metric, symbol Device:R
- removed TP1, TP71, TP73, TP74, TP78: Test_Point, TestPoint:TestPoint_Pad_D1.5mm, symbol Connector:TestPoint
Connections:
- net BOOT0: now also U15.4
- net NRST: now also U21.4 (Y)
- net USB_DEBUG_DTR: now also U13.23 (DTR)
- net USB_DEBUG_GPIO0: now also U13.14 (GPIO.0)
- net USB_DEBUG_GPIO1: now also U13.13 (GPIO.1)
- net USB_DEBUG_GPIO2: now also U13.12 (GPIO.2)
- net USB_DEBUG_GPIO3: now also U13.11 (GPIO.3)
- net USB_DEBUG_RTS: now also U13.19 (RTS)
- net USB_DEBUG_RX: now also U13.20 (RXD)
- net USB_DEBUG_TX: now also U13.21 (TXD)
- no-connect marks 4 -> 6

Commit message: minor update to layout
Parts:
- R602, R603, R604: Other (none) -> Can use own part, but needs to meet the specs
- TP62, TP63: footprint TestPoint:TestPoint_Pad_D1.5mm -> Devtank_PCB_lib:TestPoint_Pad_D1.5mm
Connections:
- no-connect marks 6 -> 7
Changed lines of the file:
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@@
   (no_connect (at 94.615 118.745))
   (no_connect (at 115.57 77.47))
+  (no_connect (at 115.57 62.23))
   (no_connect (at 115.57 59.69))
   (no_connect (at 115.57 72.39))
@@
       (effects (font (size 1.27 1.27)) hide)
     )
-    (property "Other" "" (at 69.215 76.835 0)
+    (property "Other" "Can use own part, but needs to meet the specs" (at 69.215 76.835 0)
       (effects (font (size 1.27 1.27)) hide)
     )
@@
       (effects (font (size 1.27 1.27)) (justify left) hide)
     )
-    (property "Footprint" "TestPoint:TestPoint_Pad_D1.5mm" (at 165.735 69.85 0)
+    (property "Footprint" "Devtank_PCB_lib:TestPoint_Pad_D1.5mm" (at 165.735 69.85 0)
       (effects (font (size 1.27 1.27)) hide)
     )
@@
       (effects (font (size 1.27 1.27)) hide)
     )
-    (property "Other" "" (at 62.865 82.55 0)
+    (property "Other" "Can use own part, but needs to meet the specs" (at 62.865 82.55 0)
       (effects (font (size 1.27 1.27)) hide)
     )
@@
       (effects (font (size 1.27 1.27)) hide)
     )
-    (property "Other" "" (at 48.26 53.34 0)
+    (property "Other" "Can use own part, but needs to meet the specs" (at 48.26 53.34 0)
       (effects (font (size 1.27 1.27)) hide)
     )
@@
       (effects (font (size 1.27 1.27)) (justify left) hide)
     )
-    (property "Footprint" "TestPoint:TestPoint_Pad_D1.5mm" (at 165.735 80.01 0)
-      (effects (font (size 1.27 1.27)) hide)
-    )
+    (property "Footprint" "Devtank_PCB_lib:TestPoint_Pad_D1.5mm" (at 165.735 80.01 0)
+      (effects (font (size 1.27 1.27)) hide)
+    )
