File: kicad_osm_env01/CanTransciever.kicad_sch (KiCad schematic)
At the start: 19 parts, among them U8 SN65HVD230DR

Commit message: minor update to layout
Parts:
- removed R84, R85: 330R, Resistor_SMD:R_0603_1608Metric, symbol Device:R
- C67: value DNF -> 4.7nF
- R25: value 0R -> 60.4R; footprint Resistor_SMD:R_0402_1005Metric -> Resistor_SMD:R_0603_1608Metric; Other (none) -> Can use own part, but needs to meet the specs
- R31: Other (none) -> Can use own part, but needs to meet the specs
- R87: value 120R -> 60.4R; Other (none) -> Can use own part, but needs to meet the specs
- TP22, TP23, TP41, TP80, TP81: footprint TestPoint:TestPoint_Pad_D1.5mm -> Devtank_PCB_lib:TestPoint_Pad_D1.5mm
Connections:
- net CAN_RX: now also U8.4 (R)
- net CAN_TX: now also C58.1, U8.1 (D)
Changed lines of the file:
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@@
     (stroke (width 0) (type default))
   )
-  (wire (pts (xy 121.285 86.36) (xy 126.365 86.36))
+  (wire (pts (xy 111.76 86.36) (xy 126.365 86.36))
     (stroke (width 0) (type default))
   )
@@
     (stroke (width 0) (type default))
   )
-  (wire (pts (xy 113.665 86.36) (xy 111.76 86.36))
-    (stroke (width 0) (type default))
-  )
   (wire (pts (xy 175.26 92.075) (xy 175.26 92.71))
     (stroke (width 0) (type default))
@@
     (stroke (width 0) (type default))
   )
-  (wire (pts (xy 131.445 119.38) (xy 133.35 119.38))
-    (stroke (width 0) (type default))
-  )
-  (wire (pts (xy 117.475 119.38) (xy 123.825 119.38))
+  (wire (pts (xy 117.475 119.38) (xy 133.35 119.38))
     (stroke (width 0) (type default))
   )
@@
     (effects (font (size 1.27 1.27)) (justify right))
   )
-  (symbol (lib_id "Device:R") (at 117.475 86.36 90) (unit 1)
-    (in_bom yes) (on_board yes) (dnp no)
-    (property "Reference" "R84" (at 118.745 84.455 90)
-      (effects (font (size 1.27 1.27)) (justify left))
-    )
-    (property "Value" "330R" (at 120.015 88.9 90)
-      (effects (font (size 1.27 1.27)) (justify left))
-    )
-    (property "Footprint" "Resistor_SMD:R_0603_1608Metric" (at 117.475 88.138 90)
-      (effects (font (size 1.27 1.27)) hide)
-    )
-    (property "Datasheet" "" (at 117.475 86.36 0)
-      (effects (font (size 1.27 1.27)) hide)
-    )
-    (property "Tolerance" "1%" (at 117.475 86.36 0)
-      (effects (font (size 1.27 1.27)) hide)
-    )
-    (property "Power Rating" "" (at 117.475 86.36 0)
-      (effects (font (size 1.27 1.27)) hide)
-    )
-    (property "Current Rating" "" (at 117.475 86.36 0)
-      (effects (font (size 1.27 1.27)) hide)
-    )
-    (pin "1")
-    (pin "2")
-    (instances
-      (project "OSM_env01"
-        (path "/ab8b0540-9c9f-4195-88f5-7bed0b0a8ed6/00000000-0000-0000-0000-00006064bc1d"
-          (reference "R84") (unit 1)
-        )
-      )
-    )
-  )
-  (symbol (lib_id "Device:R") (at 127.635 119.38 90) (unit 1)
-    (in_bom yes) (on_board yes) (dnp no)
-    (property "Reference" "R85" (at 129.54 117.475 90)
-      (effects (font (size 1.27 1.27)) (justify left))
-    )
-    (property "Value" "330R" (at 130.175 121.92 90)
-      (effects (font (size 1.27 1.27)) (justify left))
-    )
-    (property "Footprint" "Resistor_SMD:R_0603_1608Metric" (at 127.635 121.158 90)
-      (effects (font (size 1.27 1.27)) hide)
-    )
-    (property "Datasheet" "" (at 127.635 119.38 0)
-      (effects (font (size 1.27 1.27)) hide)
-    )
-    (property "Tolerance" "1%" (at 127.635 119.38 0)
-      (effects (font (size 1.27 1.27)) hide)
-    )
-    (property "Power Rating" "" (at 127.635 119.38 0)
-      (effects (font (size 1.27 1.27)) hide)
-    )
-    (property "Current Rating" "" (at 127.635 119.38 0)
-      (effects (font (size 1.27 1.27)) hide)
-    )
-    (pin "1")
-    (pin "2")
-    (instances
-      (project "OSM_env01"
-        (path "/ab8b0540-9c9f-4195-88f5-7bed0b0a8ed6/00000000-0000-0000-0000-00006064bc1d"
-          (reference "R85") (unit 1)
-        )
-      )
-    )
-  )
   (symbol (lib_id "Device:R") (at 175.26 106.045 0) (mirror y) (unit 1)
     (in_bom yes) (on_board yes) (dnp no)
@@
       (effects (font (size 1.27 1.27)) (justify left))
     )
-    (property "Value" "120R" (at 173.482 107.188 0)
+    (property "Value" "60.4R" (at 173.482 107.188 0)
       (effects (font (size 1.27 1.27)) (justify left))
     )
@@
       (effects (font (size 1.27 1.27)) hide)
     )
+    (property "Other" "Can use own part, but needs to meet the specs" (at 175.26 106.045 0)
+      (effects (font (size 1.27 1.27)) hide)
+    )
     (pin "1")
     (pin "2")
@@
       (effects (font (size 1.27 1.27)) hide)
     )
-    (property "Footprint" "TestPoint:TestPoint_Pad_D1.5mm" (at 111.76 88.265 0)
+    (property "Footprint" "Devtank_PCB_lib:TestPoint_Pad_D1.5mm" (at 111.76 88.265 0)
       (effects (font (size 1.27 1.27)) hide)
     )
@@
       (effects (font (size 1.27 1.27)) hide)
     )
-    (property "Footprint" "TestPoint:TestPoint_Pad_D1.5mm" (at 117.475 122.555 0)
+    (property "Footprint" "Devtank_PCB_lib:TestPoint_Pad_D1.5mm" (at 117.475 122.555 0)
       (effects (font (size 1.27 1.27)) hide)
     )
@@
       (effects (font (size 1.27 1.27)) hide)
     )
+    (property "Other" "Can use own part, but needs to meet the specs" (at 154.94 76.2 0)
+      (effects (font (size 1.27 1.27)) hide)
+    )
     (pin "1")
     (pin "2")
@@
       (effects (font (size 1.27 1.27)) hide)
     )
-    (property "Footprint" "TestPoint:TestPoint_Pad_D1.5mm" (at 109.22 100.965 0)
+    (property "Footprint" "Devtank_PCB_lib:TestPoint_Pad_D1.5mm" (at 109.22 100.965 0)
       (effects (font (size 1.27 1.27)) hide)
     )
@@
       (effects (font (size 1.27 1.27)) hide)
     )
-    (property "Footprint" "TestPoint:TestPoint_Pad_D1.5mm" (at 206.375 93.98 0)
+    (property "Footprint" "Devtank_PCB_lib:TestPoint_Pad_D1.5mm" (at 206.375 93.98 0)
       (effects (font (size 1.27 1.27)) hide)
     )
@@
       (effects (font (size 1.27 1.27)) hide)
     )
-    (property "Footprint" "TestPoint:TestPoint_Pad_D1.5mm" (at 206.375 118.11 0)
+    (property "Footprint" "Devtank_PCB_lib:TestPoint_Pad_D1.5mm" (at 206.375 118.11 0)
       (effects (font (size 1.27 1.27)) hide)
     )
@@
       (effects (font (size 1.27 1.27)) (justify left))
     )
-    (property "Value" "0R" (at 177.038 97.663 0)
-      (effects (font (size 1.27 1.27)) (justify left))
-    )
-    (property "Footprint" "Resistor_SMD:R_0402_1005Metric" (at 173.482 96.52 90)
+    (property "Value" "60.4R" (at 177.038 97.663 0)
+      (effects (font (size 1.27 1.27)) (justify left))
+    )
+    (property "Footprint" "Resistor_SMD:R_0603_1608Metric" (at 173.482 96.52 90)
       (effects (font (size 1.27 1.27)) hide)
     )
@@
       (effects (font (size 1.27 1.27)) hide)
     )
+    (property "Other" "Can use own part, but needs to meet the specs" (at 175.26 96.52 0)
+      (effects (font (size 1.27 1.27)) hide)
+    )
     (pin "1")
     (pin "2")
@@
   (symbol (lib_id "Device:C") (at 185.42 101.6 270) (mirror x) (unit 1)
     (in_bom yes) (on_board yes) (dnp no)
-    (property "Reference" "C67" (at 184.15 98.425 0)
-      (effects (font (size 1.27 1.27)) (justify left))
-    )
-    (property "Value" "DNF" (at 186.055 98.425 0)
-      (effects (font (size 1.27 1.27)) (justify left))
-    )
+    (property "Reference" "C67" (at 183.515 97.79 90)
+      (effects (font (size 1.27 1.27)) (justify left))
+    )
+    (property "Value" "4.7nF" (at 182.245 105.41 90)
+      (effects (font (size 1.27 1.27)) (justify left))
+    )

Commit message: Rev D finished, minor update to bom, schematic exported and folder structure updated
Parts:
- C67: Characteristics X5R -> C0G/NP0
Changed lines of the file:
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@@
   (title_block
     (title "Open Smart Monitor")
-    (date "2023-12-08")
+    (date "2023-12-19")
     (rev "D")
     (company "Devtank LTD")
@@
       (effects (font (size 1.27 1.27)) hide)
     )
-    (property "Characteristics" "X5R" (at 185.42 101.6 0)
-      (effects (font (size 1.27 1.27)) hide)
-    )
+    (property "Characteristics" "C0G/NP0" (at 185.42 101.6 0)
+      (effects (font (size 1.27 1.27)) hide)
+    )
