File: kicad_osm_env01/RS485_Comms.kicad_sch (KiCad schematic)
At the start: 13 parts, among them U7 ST3485EBDR

Commit message: minor update to layout
Parts:
- R72, R73, R74, R75: Other (none) -> Can use own part, but needs to meet the specs
- TP20, TP36, TP37, TP38, TP39, TP40: footprint TestPoint:TestPoint_Pad_D1.5mm -> Devtank_PCB_lib:TestPoint_Pad_D1.5mm
Changed lines of the file:
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@@
+      (effects (font (size 1.27 1.27)) hide)
+    )
+    (property "Other" "Can use own part, but needs to meet the specs" (at 124.46 85.725 0)
       (effects (font (size 1.27 1.27)) hide)
     )
@@
       (effects (font (size 1.27 1.27)) hide)
     )
+    (property "Other" "Can use own part, but needs to meet the specs" (at 165.1 87.63 0)
+      (effects (font (size 1.27 1.27)) hide)
+    )
     (pin "1")
     (pin "2")
@@
       (effects (font (size 1.27 1.27)) hide)
     )
+    (property "Other" "Can use own part, but needs to meet the specs" (at 165.1 98.425 0)
+      (effects (font (size 1.27 1.27)) hide)
+    )
     (pin "1")
     (pin "2")
@@
       (effects (font (size 1.27 1.27)) hide)
     )
+    (property "Other" "Can use own part, but needs to meet the specs" (at 165.1 109.855 0)
+      (effects (font (size 1.27 1.27)) hide)
+    )
     (pin "1")
     (pin "2")
@@
       (effects (font (size 1.27 1.27)) hide)
     )
-    (property "Footprint" "TestPoint:TestPoint_Pad_D1.5mm" (at 178.435 97.79 0)
+    (property "Footprint" "Devtank_PCB_lib:TestPoint_Pad_D1.5mm" (at 178.435 97.79 0)
       (effects (font (size 1.27 1.27)) hide)
     )
@@
       (effects (font (size 1.27 1.27)) hide)
     )
-    (property "Footprint" "TestPoint:TestPoint_Pad_D1.5mm" (at 178.435 109.22 0)
+    (property "Footprint" "Devtank_PCB_lib:TestPoint_Pad_D1.5mm" (at 178.435 109.22 0)
       (effects (font (size 1.27 1.27)) hide)
     )
@@
       (effects (font (size 1.27 1.27)) hide)
     )
-    (property "Footprint" "TestPoint:TestPoint_Pad_D1.5mm" (at 107.95 94.615 0)
+    (property "Footprint" "Devtank_PCB_lib:TestPoint_Pad_D1.5mm" (at 107.95 94.615 0)
       (effects (font (size 1.27 1.27)) hide)
     )
@@
       (effects (font (size 1.27 1.27)) hide)
     )
-    (property "Footprint" "TestPoint:TestPoint_Pad_D1.5mm" (at 118.11 100.965 0)
+    (property "Footprint" "Devtank_PCB_lib:TestPoint_Pad_D1.5mm" (at 118.11 100.965 0)
       (effects (font (size 1.27 1.27)) hide)
     )
@@
       (effects (font (size 1.27 1.27)) hide)
     )
-    (property "Footprint" "TestPoint:TestPoint_Pad_D1.5mm" (at 118.11 84.455 0)
+    (property "Footprint" "Devtank_PCB_lib:TestPoint_Pad_D1.5mm" (at 118.11 84.455 0)
       (effects (font (size 1.27 1.27)) hide)
     )
@@
       (effects (font (size 1.27 1.27)) hide)
     )
-    (property "Footprint" "TestPoint:TestPoint_Pad_D1.5mm" (at 92.075 84.455 0)
-      (effects (font (size 1.27 1.27)) hide)
-    )
+    (property "Footprint" "Devtank_PCB_lib:TestPoint_Pad_D1.5mm" (at 92.075 84.455 0)
+      (effects (font (size 1.27 1.27)) hide)
+    )
